Commit message: ergoCubSN001: simplify collision of feet

File: urdf/ergoCub/robots/ergoCubSN001/model.urdf (robot description, URDF)
Before this commit: robot ergoCub, 204 links, 203 joints
Links:
- link l_foot_front: geometry collision box size=0.117 0.1 0.006; visual mesh filename=package://ergoCub/meshes/simmechanics/sim_ecub_1-1_l_foot_f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 scale=0.001 0.001 0.001
- link l_foot_rear: geometry collision box size=0.117 0.1 0.006; visual mesh filename=package://ergoCub/meshes/simmechanics/sim_ecub_1-1_l_foot_r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 scale=0.001 0.001 0.001
- link r_foot_front: geometry collision box size=0.117 0.1 0.006; visual mesh filename=package://ergoCub/meshes/simmechanics/sim_ecub_1-1_r_foot_f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 scale=0.001 0.001 0.001
- link r_foot_rear: geometry collision box size=0.117 0.1 0.006; visual mesh filename=package://ergoCub/meshes/simmechanics/sim_ecub_1-1_r_foot_r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 scale=0.001 0.001 0.001
Joints:
- joint l_index_add: axis 1.5978340464762954e-11 0.9999999999999999 -3.7677226824487294e-11 -> 1.5978451487065422e-11 1.0000000000000002 -3.767719906891169e-11; origin xyz=0.022500000000000023 -0.0015000000000006952 -0.0685999999999996 rpy=-8.416895217637947e-16 -0.29670597224465534 5.804755322508926e-17 -> xyz=0.022500000000000034 -0.0015000000000006397 -0.06859999999999966 rpy=-8.126657451512497e-16 -0.2967059722446555 1.7414265967526777e-16
- joint l_index_dist: axis -0.9781476007113552 -1.553317034713362e-8 0.20791169092337955 -> -0.9781476007113552 -1.5533170287064815e-8 0.2079116909233797; origin xyz=-1.3877787807814457e-17 -0.001500000000000029 -0.03999999999999987 rpy=-7.482326172536535e-8 1.8041124150158794e-16 -6.106226635438361e-16 -> xyz=-2.7755575615628914e-17 -0.0014999999999999736 -0.039999999999999925 rpy=-7.482326169760975e-8 1.734723475976807e-16 -6.106226635438361e-16
- joint l_index_prox: axis -0.9781476007113543 2.3461557522424743e-11 0.2079116909233844 -> -0.9781476007113546 2.346155062839741e-11 0.20791169092338443; origin xyz=0.00919253334679343 0 -0.030713451309624218 rpy=-3.0531133177191815e-16 -7.023611484080483e-10 -7.771561172376096e-16 -> xyz=0.009192533346793416 -2.7755575615628914e-17 -0.030713451309624162 rpy=-2.7755575615628914e-16 -7.023611553469422e-10 -7.771561172376094e-16

Commit message: fixup

File: urdf/ergoCub/robots/ergoCubSN001/model.urdf (robot description, URDF)
Before this commit: robot ergoCub, 204 links, 203 joints
Links:
- link chest: geometry collision mesh filename=package://ergoCub/meshes/simmechanics/sim_ecub_1-1_chest.obj scale=0.001 0.001 0.001; visual mesh filename=package://ergoCub/meshes/simmechanics/sim_ecub_1-1_chest.obj scale=0.001 0.001 0.001
- link head: geometry collision mesh filename=package://ergoCub/meshes/simmechanics/sim_ecub_1-1_head.obj scale=0.001 0.001 0.001; visual mesh filename=package://ergoCub/meshes/simmechanics/sim_ecub_1-1_head.obj scale=0.001 0.001 0.001
