Commit message: Sixth mode

File: urdf/ergoCub/robots/ergoCubGazeboV1/model.urdf (robot description, URDF)
Before this commit: robot ergoCub, 71 links, 70 joints
Joints:
- removed joint SIM_ECUB_CHEST--SIM_ECUB_HEAD_NECK_2
- added joint neck_pitch: type revolute, parent chest, child neck_2, origin xyz=0.00486151 0 0.22529999999999997 rpy=0 0 0, axis 0.0 -1.0 0.0, limit lower=-0.5235987755982988 upper=0.3839724354387525 effort=50000 velocity=120.0

File: urdf/ergoCub/robots/ergoCubSN000/model.urdf (robot description, URDF)
Before this commit: robot ergoCub, 71 links, 70 joints
Joints:
- removed joint SIM_ECUB_CHEST--SIM_ECUB_HEAD_NECK_2
- added joint neck_pitch: type revolute, parent chest, child neck_2, origin xyz=0.00486151 0 0.22529999999999997 rpy=0 0 0, axis 0.0 -1.0 0.0, limit lower=-0.5235987755982988 upper=0.3839724354387525 effort=50000 velocity=120.0

Commit message: Seventh urdf

File: urdf/ergoCub/robots/ergoCubGazeboV1/model.urdf (robot description, URDF)
Before this commit: robot ergoCub, 71 links, 70 joints
Joints:
- removed joint SIM_ECUB_HEAD_NECK_3--SIM_ECUB_HEAD
- added joint neck_yaw: type revolute, parent neck_3, child head, origin xyz=0 0 0.06915000000000004 rpy=0 0 0, axis 0.0 0.0 1.0, limit lower=-0.7853981633974483 upper=0.7853981633974483 effort=50000 velocity=120.0

File: urdf/ergoCub/robots/ergoCubSN000/model.urdf (robot description, URDF)
Before this commit: robot ergoCub, 71 links, 70 joints
Joints:
- removed joint SIM_ECUB_HEAD_NECK_3--SIM_ECUB_HEAD
- added joint neck_yaw: type revolute, parent neck_3, child head, origin xyz=0 0 0.06915000000000004 rpy=0 0 0, axis 0.0 0.0 -1.0, limit lower=-0.7853981633974483 upper=0.7853981633974483 effort=50000 velocity=120.0

Commit message: Eighth urdf

File: urdf/ergoCub/robots/ergoCubGazeboV1/model.urdf (robot description, URDF)
Before this commit: robot ergoCub, 71 links, 70 joints
Joints:
- removed joint camera-tilt
- added joint camera_tilt: type continuous, parent head, child realsense, origin xyz=0.06250999 -3e-05 0.07639299999999999 rpy=0 0.0002595819985423862 0, axis -2.220446049250313e-16 1.0000000000000002 0.0

File: urdf/ergoCub/robots/ergoCubSN000/model.urdf (robot description, URDF)
Before this commit: robot ergoCub, 71 links, 70 joints
Joints:
- removed joint camera-tilt
- added joint camera_tilt: type continuous, parent head, child realsense, origin xyz=0.06250999 -3e-05 0.07639299999999999 rpy=0 0.0002595819985423862 0, axis -2.220446049250313e-16 1.0000000000000002 0.0

Commit message: Eleventh urdf

File: urdf/ergoCub/robots/ergoCubGazeboV1/model.urdf (robot description, URDF)
Before this commit: robot ergoCub, 71 links, 70 joints
Links:
- link chest: mass 7.5231 -> 8.06547
- link head: mass 1.8728 -> 2.31933
- link l_ankle_1: mass 0.36569 -> 0.348128
- link l_ankle_2: mass 1.377 -> 1.54182
- link l_foot_front: mass 0.17896 -> 0.221105
- link l_foot_rear: mass 0.17851 -> 0.221105
- link l_forearm: mass 0.87311 -> 1.46045
- link l_hip_1: mass 2.1611 -> 2.22805
- link l_hip_2: mass 1.7731 -> 1.83384
- link l_hip_3: mass 2.1622 -> 2.14752
- link l_lower_leg: mass 5.0486 -> 3.74161
- link l_shoulder_1: mass 0.78644 -> 0.792333
- link l_shoulder_2: mass 0.42492 -> 0.440933
- link l_shoulder_3: mass 0.2625 -> 0.271466
- link l_upper_leg: mass 0.90926 -> 2.78492
- link l_wrist_1: mass 0.033183 -> 0.0565425
- link neck_2: mass 0.1214 -> 0.121003
- link neck_3: mass 0.18386 -> 0.178114
- link r_ankle_1: mass 0.36569 -> 0.348128
- link r_ankle_2: mass 1.3771 -> 1.54182
- link r_foot_front: mass 0.17964 -> 0.221105
- link r_foot_rear: mass 0.17874 -> 0.221105
- link r_forearm: mass 0.8686 -> 1.47607
- link r_hip_1: mass 2.1623 -> 2.22779
- link r_hip_2: mass 1.7731 -> 1.8336
- link r_hip_3: mass 2.1635 -> 2.1479
- link r_lower_leg: mass 5.0761 -> 3.74161
- link r_shoulder_1: mass 0.78697 -> 0.792333
- link r_shoulder_2: mass 0.42492 -> 0.439227
- link r_shoulder_3: mass 0.2625 -> 0.271466
- link r_upper_leg: mass 0.90926 -> 2.78492
- link r_wrist_1: mass 0.033183 -> 0.0565425
- link root_link: mass 2.5751 -> 2.82266
- link torso_1: mass 1.6998 -> 2.01154
- link torso_2: mass 0.77098 -> 0.705163

Commit message: Automatic update of urdf

File: urdf/ergoCub/robots/ergoCubGazeboV1/model.urdf (robot description, URDF)
Before this commit: robot ergoCub, 167 links, 166 joints
Joints:
- joint l_ankle_pitch: axis 0.0 1.0 0.0 -> 0.0 -1.0 0.0
- joint l_shoulder_yaw: axis 3.936910710766739e-07 -1.8507626386998766e-07 -0.9999995705743131 -> -3.936910710766739e-07 1.8507626386998766e-07 0.9999995705743131
- joint l_wrist_pitch: axis -1.4958988243767013e-07 -0.9999999783534517 -2.7220291587415346e-07 -> 1.4958988243767013e-07 0.9999999783534517 2.7220291587415346e-07
- joint l_wrist_yaw: axis -3.936910710766739e-07 1.8507626386998766e-07 0.9999995705743131 -> 3.936910710766739e-07 -1.8507626386998766e-07 -0.9999995705743131
- joint neck_yaw: axis 0.0 0.0 1.0 -> 0.0 0.0 -1.0
- joint r_ankle_roll: axis -1.0 0.0 0.0 -> 1.0 0.0 0.0
- joint r_hip_roll: axis -1.0 0.0 0.0 -> 1.0 0.0 0.0
- joint r_hip_yaw: axis 0.0 0.0 -1.0 -> 0.0 0.0 1.0
- joint r_knee: axis 0.0 -1.0 0.0 -> 0.0 1.0 0.0
- joint torso_pitch: axis 0.0 1.0 0.0 -> 0.0 -1.0 0.0
- joint torso_roll: axis -1.0 0.0 0.0 -> 1.0 0.0 0.0
- joint torso_yaw: axis 0.0 0.0 -1.0 -> 0.0 0.0 1.0

File: urdf/ergoCub/robots/ergoCubSN000/model.urdf (robot description, URDF)
Before this commit: robot ergoCub, 167 links, 166 joints
Joints:
- joint l_shoulder_pitch: axis -4.453300185801312e-07 -0.9999999783533606 -2.834495320125363e-07 -> 4.453300185801312e-07 0.9999999783533606 2.834495320125363e-07
- joint l_shoulder_roll: axis -0.9999998262416893 -3.56920377206707e-07 -2.721582535170075e-07 -> 0.9999998262416893 3.56920377206707e-07 2.721582535170075e-07
- joint r_elbow: axis -3.352246002574083e-07 0.9999999783534191 -2.2068612626213735e-07 -> 3.352246002574083e-07 -0.9999999783534191 2.2068612626213735e-07

Commit message: Automatic update of urdf

File: urdf/ergoCub/robots/ergoCubGazeboV1/model.urdf (robot description, URDF)
Before this commit: robot ergoCub, 167 links, 166 joints
Joints:
- joint l_wrist_pitch: limit lower=-1.2217304763960306 upper=0.4363323129985824 effort=50000 velocity=120.0 -> lower=-0.5585053606381855 upper=0.5585053606381855 effort=50000 velocity=120.0
- joint l_wrist_roll: limit lower=-1.53588974175501 upper=1.53588974175501 effort=50000 velocity=120.0 -> lower=-1.0821041362364843 upper=0.9075712110370514 effort=50000 velocity=120.0
- joint l_wrist_yaw: limit lower=-0.2617993877991494 upper=0.6108652381980153 effort=50000 velocity=120.0 -> lower=-1.6057029118347832 upper=1.6057029118347832 effort=50000 velocity=120.0
- joint r_wrist_pitch: limit lower=-1.2217304763960306 upper=0.4363323129985824 effort=50000 velocity=120.0 -> lower=-0.5585053606381855 upper=0.5585053606381855 effort=50000 velocity=120.0
- joint r_wrist_roll: limit lower=-1.53588974175501 upper=1.53588974175501 effort=50000 velocity=120.0 -> lower=-1.0821041362364843 upper=0.9075712110370514 effort=50000 velocity=120.0
- joint r_wrist_yaw: limit lower=-0.2617993877991494 upper=0.6108652381980153 effort=50000 velocity=120.0 -> lower=-1.6057029118347832 upper=1.6057029118347832 effort=50000 velocity=120.0

File: urdf/ergoCub/robots/ergoCubSN000/model.urdf (robot description, URDF)
Before this commit: robot ergoCub, 167 links, 166 joints
Joints:
- joint l_wrist_pitch: limit lower=-1.2217304763960306 upper=0.4363323129985824 effort=50000 velocity=120.0 -> lower=-0.5585053606381855 upper=0.5585053606381855 effort=50000 velocity=120.0
- joint l_wrist_roll: limit lower=-1.53588974175501 upper=1.53588974175501 effort=50000 velocity=120.0 -> lower=-1.0821041362364843 upper=0.9075712110370514 effort=50000 velocity=120.0
- joint l_wrist_yaw: limit lower=-0.2617993877991494 upper=0.6108652381980153 effort=50000 velocity=120.0 -> lower=-1.6057029118347832 upper=1.6057029118347832 effort=50000 velocity=120.0
- joint r_wrist_pitch: limit lower=-1.2217304763960306 upper=0.4363323129985824 effort=50000 velocity=120.0 -> lower=-0.5585053606381855 upper=0.5585053606381855 effort=50000 velocity=120.0
- joint r_wrist_roll: limit lower=-1.53588974175501 upper=1.53588974175501 effort=50000 velocity=120.0 -> lower=-1.0821041362364843 upper=0.9075712110370514 effort=50000 velocity=120.0
- joint r_wrist_yaw: limit lower=-0.2617993877991494 upper=0.6108652381980153 effort=50000 velocity=120.0 -> lower=-1.6057029118347832 upper=1.6057029118347832 effort=50000 velocity=120.0

Commit message: Automatic update of urdf

File: urdf/ergoCub/robots/ergoCubGazeboV1/model.urdf (robot description, URDF)
Before this commit: robot ergoCub, 167 links, 166 joints
Links:
- added link l_sole
- added link r_sole
- link l_wrist_1: geometry 
Joints:
- added joint l_sole_fixed_joint: type fixed, parent l_foot_rear, child l_sole, origin xyz=0.05963 0 0 rpy=0 0 0
- added joint r_sole_fixed_joint: type fixed, parent r_foot_rear, child r_sole, origin xyz=0.05963 0 0 rpy=0 0 0
- joint l_wrist_pitch: axis 1.4958988243767013e-07 0.9999999783534517 2.7220291587415346e-07 -> -1.4958988243767013e-07 -0.9999999783534517 -2.7220291587415346e-07
- joint r_wrist_pitch: axis -3.352246002574083e-07 0.9999999783534191 -2.2068612626213735e-07 -> 3.352246002574083e-07 -0.9999999783534191 2.2068612626213735e-07
- joint r_wrist_roll: axis -0.9999998262417322 1.7128582631247002e-07 2.9287109011566503e-07 -> 0.9999998262417322 -1.7128582631247002e-07 -2.9287109011566503e-07
- joint r_wrist_yaw: axis -1.7133815359560156e-07 2.3659291614741562e-07 -0.999999570574365 -> 1.7133815359560156e-07 -2.3659291614741562e-07 0.999999570574365

File: urdf/ergoCub/robots/ergoCubSN000/model.urdf (robot description, URDF)
Before this commit: robot ergoCub, 167 links, 166 joints
Links:
- added link l_sole
- added link r_sole
- link l_wrist_1: geometry 
Joints:
- added joint l_sole_fixed_joint: type fixed, parent l_foot_rear, child l_sole, origin xyz=0.05963 0 0 rpy=0 0 0
- added joint r_sole_fixed_joint: type fixed, parent r_foot_rear, child r_sole, origin xyz=0.05963 0 0 rpy=0 0 0
- joint l_wrist_pitch: axis 1.4958988243767013e-07 0.9999999783534517 2.7220291587415346e-07 -> -1.4958988243767013e-07 -0.9999999783534517 -2.7220291587415346e-07
- joint r_wrist_pitch: axis -3.352246002574083e-07 0.9999999783534191 -2.2068612626213735e-07 -> 3.352246002574083e-07 -0.9999999783534191 2.2068612626213735e-07
- joint r_wrist_roll: axis -0.9999998262417322 1.7128582631247002e-07 2.9287109011566503e-07 -> 0.9999998262417322 -1.7128582631247002e-07 -2.9287109011566503e-07
- joint r_wrist_yaw: axis -1.7133815359560156e-07 2.3659291614741562e-07 -0.999999570574365 -> 1.7133815359560156e-07 -2.3659291614741562e-07 0.999999570574365

Commit message: Automatic update of urdf

File: urdf/ergoCub/robots/ergoCubGazeboV1/model.urdf (robot description, URDF)
Before this commit: robot ergoCub, 169 links, 168 joints
Joints:
- joint l_ankle_pitch: axis 0.0 -1.0 0.0 -> 0.0 1.0 0.0
- joint l_knee: axis 0.0 -1.0 0.0 -> 0.0 1.0 0.0
- joint neck_yaw: axis 0.0 0.0 -1.0 -> 0.0 0.0 1.0
- joint r_ankle_roll: axis 1.0 0.0 0.0 -> -1.0 0.0 0.0
- joint r_hip_roll: axis 1.0 0.0 0.0 -> -1.0 0.0 0.0
- joint r_hip_yaw: axis 0.0 0.0 1.0 -> 0.0 0.0 -1.0
- joint torso_pitch: axis 0.0 -1.0 0.0 -> 0.0 1.0 0.0
- joint torso_roll: axis 1.0 0.0 0.0 -> -1.0 0.0 0.0
- joint torso_yaw: axis 0.0 0.0 1.0 -> 0.0 0.0 -1.0

File: urdf/ergoCub/robots/ergoCubSN000/model.urdf (robot description, URDF)
Before this commit: robot ergoCub, 169 links, 168 joints
Joints:
- joint l_ankle_pitch: axis 0.0 -1.0 0.0 -> 0.0 1.0 0.0
- joint l_knee: axis 0.0 -1.0 0.0 -> 0.0 1.0 0.0
- joint neck_yaw: axis 0.0 0.0 -1.0 -> 0.0 0.0 1.0
- joint r_ankle_roll: axis 1.0 0.0 0.0 -> -1.0 0.0 0.0
- joint r_hip_roll: axis 1.0 0.0 0.0 -> -1.0 0.0 0.0
- joint r_hip_yaw: axis 0.0 0.0 1.0 -> 0.0 0.0 -1.0
- joint torso_pitch: axis 0.0 -1.0 0.0 -> 0.0 1.0 0.0
- joint torso_roll: axis 1.0 0.0 0.0 -> -1.0 0.0 0.0
- joint torso_yaw: axis 0.0 0.0 1.0 -> 0.0 0.0 -1.0

Commit message: Automatic update of urdf

File: urdf/ergoCub/robots/ergoCubGazeboV1/model.urdf (robot description, URDF)
Before this commit: robot ergoCub, 169 links, 168 joints
Joints:
- joint l_index_add: axis 3.992524267790176e-07 0.999999978353397 2.1441989261905547e-07 -> -3.992524267790176e-07 -0.999999978353397 -2.1441989261905547e-07; limit lower=0.0 upper=1.7453292519943295 effort=50000 velocity=120.0 -> lower=0.0 upper=0.3490658503988659 effort=50000 velocity=120.0
- joint l_index_dist: limit lower=0.0 upper=1.7453292519943295 effort=50000 velocity=120.0 -> lower=0.0 upper=2.792526803190927 effort=50000 velocity=120.0
- joint l_index_prox: limit lower=0.0 upper=1.7453292519943295 effort=50000 velocity=120.0 -> lower=0.0 upper=2.792526803190927 effort=50000 velocity=120.0
- joint l_middle_dist: limit lower=0.0 upper=1.7453292519943295 effort=50000 velocity=120.0 -> lower=0.0 upper=2.792526803190927 effort=50000 velocity=120.0
- joint l_middle_prox: limit lower=0.0 upper=1.7453292519943295 effort=50000 velocity=120.0 -> lower=0.0 upper=2.792526803190927 effort=50000 velocity=120.0
- joint l_pinkie_dist: limit lower=0.0 upper=1.7453292519943295 effort=50000 velocity=120.0 -> lower=0.0 upper=2.792526803190927 effort=50000 velocity=120.0
- joint l_pinkie_prox: limit lower=0.0 upper=1.7453292519943295 effort=50000 velocity=120.0 -> lower=0.0 upper=2.792526803190927 effort=50000 velocity=120.0
- joint l_ring_dist: limit lower=0.0 upper=1.7453292519943295 effort=50000 velocity=120.0 -> lower=0.0 upper=2.792526803190927 effort=50000 velocity=120.0
- joint l_ring_prox: axis 1.0000005135466863 1.979209419246744e-07 4.060128685548503e-07 -> -1.0000005135466863 -1.979209419246744e-07 -4.060128685548503e-07; limit lower=0.0 upper=1.7453292519943295 effort=50000 velocity=120.0 -> lower=0.0 upper=2.792526803190927 effort=50000 velocity=120.0
- joint l_thumb_add: limit lower=0.0 upper=1.7453292519943295 effort=50000 velocity=120.0 -> lower=0.0 upper=1.0471975511965976 effort=50000 velocity=120.0
- joint l_thumb_dist: axis -6.65068723482154e-07 2.7824760159833595e-07 1.0000002266902146 -> 6.65068723482154e-07 -2.7824760159833595e-07 -1.0000002266902146; limit lower=0.0 upper=1.7453292519943295 effort=50000 velocity=120.0 -> lower=0.0 upper=2.792526803190927 effort=50000 velocity=120.0
- joint l_thumb_prox: axis -6.65068723482154e-07 2.7824760159833595e-07 1.0000002266902146 -> 6.65068723482154e-07 -2.7824760159833595e-07 -1.0000002266902146; limit lower=0.0 upper=1.7453292519943295 effort=50000 velocity=120.0 -> lower=0.0 upper=2.792526803190927 effort=50000 velocity=120.0
- joint r_index_add: limit lower=0.0 upper=1.7453292519943295 effort=50000 velocity=120.0 -> lower=0.0 upper=0.3490658503988659 effort=50000 velocity=120.0
- joint r_index_dist: limit lower=0.0 upper=1.7453292519943295 effort=50000 velocity=120.0 -> lower=0.0 upper=2.792526803190927 effort=50000 velocity=120.0
- joint r_index_prox: limit lower=0.0 upper=1.7453292519943295 effort=50000 velocity=120.0 -> lower=0.0 upper=2.792526803190927 effort=50000 velocity=120.0
- joint r_middle_dist: limit lower=0.0 upper=1.7453292519943295 effort=50000 velocity=120.0 -> lower=0.0 upper=2.792526803190927 effort=50000 velocity=120.0
- joint r_middle_prox: limit lower=0.0 upper=1.7453292519943295 effort=50000 velocity=120.0 -> lower=0.0 upper=2.792526803190927 effort=50000 velocity=120.0
- joint r_pinkie_dist: limit lower=0.0 upper=1.7453292519943295 effort=50000 velocity=120.0 -> lower=0.0 upper=2.792526803190927 effort=50000 velocity=120.0
- joint r_pinkie_prox: limit lower=0.0 upper=1.7453292519943295 effort=50000 velocity=120.0 -> lower=0.0 upper=2.792526803190927 effort=50000 velocity=120.0
- joint r_ring_dist: limit lower=0.0 upper=1.7453292519943295 effort=50000 velocity=120.0 -> lower=0.0 upper=2.792526803190927 effort=50000 velocity=120.0
- joint r_ring_prox: limit lower=0.0 upper=1.7453292519943295 effort=50000 velocity=120.0 -> lower=0.0 upper=2.792526803190927 effort=50000 velocity=120.0
- joint r_thumb_add: limit lower=0.0 upper=1.7453292519943295 effort=50000 velocity=120.0 -> lower=0.0 upper=1.0471975511965976 effort=50000 velocity=120.0
- joint r_thumb_dist: axis -2.036798052024169e-07 -1.5008516943137984e-07 1.000000226690442 -> 2.036798052024169e-07 1.5008516943137984e-07 -1.000000226690442; limit lower=0.0 upper=1.7453292519943295 effort=50000 velocity=120.0 -> lower=0.0 upper=2.792526803190927 effort=50000 velocity=120.0
- joint r_thumb_prox: axis -2.036798052024169e-07 -1.5008516943137984e-07 1.000000226690442 -> 2.036798052024169e-07 1.5008516943137984e-07 -1.000000226690442; limit lower=0.0 upper=1.7453292519943295 effort=50000 velocity=120.0 -> lower=0.0 upper=2.792526803190927 effort=50000 velocity=120.0

File: urdf/ergoCub/robots/ergoCubSN000/model.urdf (robot description, URDF)
Before this commit: robot ergoCub, 169 links, 168 joints
Joints:
- joint l_index_add: axis 3.992524267790176e-07 0.999999978353397 2.1441989261905547e-07 -> -3.992524267790176e-07 -0.999999978353397 -2.1441989261905547e-07; limit lower=0.0 upper=1.7453292519943295 effort=50000 velocity=120.0 -> lower=0.0 upper=0.3490658503988659 effort=50000 velocity=120.0
- joint l_index_dist: limit lower=0.0 upper=1.7453292519943295 effort=50000 velocity=120.0 -> lower=0.0 upper=2.792526803190927 effort=50000 velocity=120.0
- joint l_index_prox: limit lower=0.0 upper=1.7453292519943295 effort=50000 velocity=120.0 -> lower=0.0 upper=2.792526803190927 effort=50000 velocity=120.0
- joint l_middle_dist: limit lower=0.0 upper=1.7453292519943295 effort=50000 velocity=120.0 -> lower=0.0 upper=2.792526803190927 effort=50000 velocity=120.0
- joint l_middle_prox: limit lower=0.0 upper=1.7453292519943295 effort=50000 velocity=120.0 -> lower=0.0 upper=2.792526803190927 effort=50000 velocity=120.0
- joint l_pinkie_dist: limit lower=0.0 upper=1.7453292519943295 effort=50000 velocity=120.0 -> lower=0.0 upper=2.792526803190927 effort=50000 velocity=120.0
- joint l_pinkie_prox: limit lower=0.0 upper=1.7453292519943295 effort=50000 velocity=120.0 -> lower=0.0 upper=2.792526803190927 effort=50000 velocity=120.0
- joint l_ring_dist: limit lower=0.0 upper=1.7453292519943295 effort=50000 velocity=120.0 -> lower=0.0 upper=2.792526803190927 effort=50000 velocity=120.0
- joint l_ring_prox: axis 1.0000005135466863 1.979209419246744e-07 4.060128685548503e-07 -> -1.0000005135466863 -1.979209419246744e-07 -4.060128685548503e-07; limit lower=0.0 upper=1.7453292519943295 effort=50000 velocity=120.0 -> lower=0.0 upper=2.792526803190927 effort=50000 velocity=120.0
- joint l_thumb_add: limit lower=0.0 upper=1.7453292519943295 effort=50000 velocity=120.0 -> lower=0.0 upper=1.0471975511965976 effort=50000 velocity=120.0
- joint l_thumb_dist: axis -6.65068723482154e-07 2.7824760159833595e-07 1.0000002266902146 -> 6.65068723482154e-07 -2.7824760159833595e-07 -1.0000002266902146; limit lower=0.0 upper=1.7453292519943295 effort=50000 velocity=120.0 -> lower=0.0 upper=2.792526803190927 effort=50000 velocity=120.0
- joint l_thumb_prox: axis -6.65068723482154e-07 2.7824760159833595e-07 1.0000002266902146 -> 6.65068723482154e-07 -2.7824760159833595e-07 -1.0000002266902146; limit lower=0.0 upper=1.7453292519943295 effort=50000 velocity=120.0 -> lower=0.0 upper=2.792526803190927 effort=50000 velocity=120.0
- joint r_index_add: limit lower=0.0 upper=1.7453292519943295 effort=50000 velocity=120.0 -> lower=0.0 upper=0.3490658503988659 effort=50000 velocity=120.0
- joint r_index_dist: limit lower=0.0 upper=1.7453292519943295 effort=50000 velocity=120.0 -> lower=0.0 upper=2.792526803190927 effort=50000 velocity=120.0
- joint r_index_prox: limit lower=0.0 upper=1.7453292519943295 effort=50000 velocity=120.0 -> lower=0.0 upper=2.792526803190927 effort=50000 velocity=120.0
- joint r_middle_dist: limit lower=0.0 upper=1.7453292519943295 effort=50000 velocity=120.0 -> lower=0.0 upper=2.792526803190927 effort=50000 velocity=120.0
- joint r_middle_prox: limit lower=0.0 upper=1.7453292519943295 effort=50000 velocity=120.0 -> lower=0.0 upper=2.792526803190927 effort=50000 velocity=120.0
- joint r_pinkie_dist: limit lower=0.0 upper=1.7453292519943295 effort=50000 velocity=120.0 -> lower=0.0 upper=2.792526803190927 effort=50000 velocity=120.0
- joint r_pinkie_prox: limit lower=0.0 upper=1.7453292519943295 effort=50000 velocity=120.0 -> lower=0.0 upper=2.792526803190927 effort=50000 velocity=120.0
- joint r_ring_dist: limit lower=0.0 upper=1.7453292519943295 effort=50000 velocity=120.0 -> lower=0.0 upper=2.792526803190927 effort=50000 velocity=120.0
- joint r_ring_prox: limit lower=0.0 upper=1.7453292519943295 effort=50000 velocity=120.0 -> lower=0.0 upper=2.792526803190927 effort=50000 velocity=120.0
- joint r_thumb_add: limit lower=0.0 upper=1.7453292519943295 effort=50000 velocity=120.0 -> lower=0.0 upper=1.0471975511965976 effort=50000 velocity=120.0
- joint r_thumb_dist: axis -2.036798052024169e-07 -1.5008516943137984e-07 1.000000226690442 -> 2.036798052024169e-07 1.5008516943137984e-07 -1.000000226690442; limit lower=0.0 upper=1.7453292519943295 effort=50000 velocity=120.0 -> lower=0.0 upper=2.792526803190927 effort=50000 velocity=120.0
- joint r_thumb_prox: axis -2.036798052024169e-07 -1.5008516943137984e-07 1.000000226690442 -> 2.036798052024169e-07 1.5008516943137984e-07 -1.000000226690442; limit lower=0.0 upper=1.7453292519943295 effort=50000 velocity=120.0 -> lower=0.0 upper=2.792526803190927 effort=50000 velocity=120.0

Commit message: Automatic update of urdf

File: urdf/ergoCub/robots/ergoCubGazeboV1/model.urdf (robot description, URDF)
Before this commit: robot ergoCub, 169 links, 168 joints
Links:
- removed link imu_frame
- removed link realsense_depth_frame
- added link head_imu_0
- added link realsense_imu_0
Joints:
- removed joint imu_frame_fixed_joint
- removed joint realsense_depth_frame_fixed_joint
- added joint head_imu_0_fixed_joint: type fixed, parent head, child head_imu_0, origin xyz=-0.004299998 -0.0055 0.03823499999999996 rpy=3.141592653589793 0 1.5707963267948966
- added joint realsense_imu_0_fixed_joint: type fixed, parent realsense, child realsense_imu_0, origin xyz=0.00751550026595621 0.010000000000000005 0 rpy=-1.5707962931078618 0 -1.5707963267948968

File: urdf/ergoCub/robots/ergoCubSN000/model.urdf (robot description, URDF)
Before this commit: robot ergoCub, 169 links, 168 joints
Links:
- removed link imu_frame
- removed link realsense_depth_frame
- added link head_imu_0
- added link realsense_imu_0
Joints:
- removed joint imu_frame_fixed_joint
- removed joint realsense_depth_frame_fixed_joint
- added joint head_imu_0_fixed_joint: type fixed, parent head, child head_imu_0, origin xyz=-0.004299998 -0.0055 0.03823499999999996 rpy=3.141592653589793 0 1.5707963267948966
- added joint realsense_imu_0_fixed_joint: type fixed, parent realsense, child realsense_imu_0, origin xyz=0.00751550026595621 0.010000000000000005 0 rpy=-1.5707962931078618 0 -1.5707963267948968
