Commit message: Automatic update of urdf

File: urdf/ergoCub/robots/ergoCubGazeboV1/model.urdf (robot description, URDF)
Before this commit: robot ergoCub, 169 links, 168 joints
Joints:
- joint camera_tilt: axis -2.220446049250313e-16 1.0000000000000002 0.0 -> 2.220446049250313e-16 -1.0000000000000002 0.0
- joint l_shoulder_yaw: axis -3.936910710766739e-07 1.8507626386998766e-07 0.9999995705743131 -> 3.936910710766739e-07 -1.8507626386998766e-07 -0.9999995705743131

File: urdf/ergoCub/robots/ergoCubSN000/model.urdf (robot description, URDF)
Before this commit: robot ergoCub, 169 links, 168 joints
Joints:
- joint camera_tilt: axis -2.220446049250313e-16 1.0000000000000002 0.0 -> 2.220446049250313e-16 -1.0000000000000002 0.0
- joint l_shoulder_yaw: axis -3.936910710766739e-07 1.8507626386998766e-07 0.9999995705743131 -> 3.936910710766739e-07 -1.8507626386998766e-07 -0.9999995705743131

Commit message: added lidar frame and joint. Fixed sensor parameters.

File: urdf/ergoCub/robots/ergoCubGazeboV1/model.urdf (robot description, URDF)
Before this commit: robot ergoCub, 169 links, 168 joints
Links:
- added link lidar, mass 0.2; visual cylinder length=0.04 radius=0.04
Joints:
- added joint lidar_joint: type fixed, parent head, child lidar, origin xyz=0.00117 0.00115 0.1348 rpy=0.0 0.0 0.0, axis 0. 0. 1., limit lower=-0.7853981633974483 upper=0.7853981633974483 effort=50000.0 velocity=120.0

Commit message: aligned hip_roll joints lower limit to -35 deg

File: urdf/ergoCub/robots/ergoCubGazeboV1/model.urdf (robot description, URDF)
Before this commit: robot ergoCub, 170 links, 169 joints
Joints:
- joint l_hip_roll: limit lower=-0.17453292519943295 upper=1.9547687622336491 effort=50000 velocity=120.0 -> lower=-0.610865 upper=1.9547687622336491 effort=50000 velocity=120.0
- joint r_hip_roll: limit lower=-0.17453292519943295 upper=1.9547687622336491 effort=50000 velocity=120.0 -> lower=-0.610865 upper=1.9547687622336491 effort=50000 velocity=120.0

Commit message: added remappers for all the fingers (with placeholder config values). Commented out some URDF parts (skin) to reduce the number of frames

File: urdf/ergoCub/robots/ergoCubGazeboV1/model.urdf (robot description, URDF)
Before this commit: robot ergoCub, 170 links, 169 joints
Links:
- removed link l_hand_index_skin_0
- removed link l_hand_index_skin_1
- removed link l_hand_index_skin_10
- removed link l_hand_index_skin_11
- removed link l_hand_index_skin_2
- removed link l_hand_index_skin_3
- removed link l_hand_index_skin_4
- removed link l_hand_index_skin_5
- removed link l_hand_index_skin_6
- removed link l_hand_index_skin_7
- removed link l_hand_index_skin_8
- removed link l_hand_index_skin_9
- removed link l_hand_middle_skin_0
- removed link l_hand_middle_skin_1
- removed link l_hand_middle_skin_10
- removed link l_hand_middle_skin_11
- removed link l_hand_middle_skin_2
- removed link l_hand_middle_skin_3
- removed link l_hand_middle_skin_4
- removed link l_hand_middle_skin_5
- removed link l_hand_middle_skin_6
- removed link l_hand_middle_skin_7
- removed link l_hand_middle_skin_8
- removed link l_hand_middle_skin_9
- removed link l_hand_ring_skin_0
- removed link l_hand_ring_skin_1
- removed link l_hand_ring_skin_10
- removed link l_hand_ring_skin_11
- removed link l_hand_ring_skin_2
- removed link l_hand_ring_skin_3
- removed link l_hand_ring_skin_4
- removed link l_hand_ring_skin_5
- removed link l_hand_ring_skin_6
- removed link l_hand_ring_skin_7
- removed link l_hand_ring_skin_8
- removed link l_hand_ring_skin_9
- removed link l_hand_thumb_skin_0
- removed link l_hand_thumb_skin_1
- removed link l_hand_thumb_skin_10
- removed link l_hand_thumb_skin_11
- removed link l_hand_thumb_skin_2
- removed link l_hand_thumb_skin_3
- removed link l_hand_thumb_skin_4
- removed link l_hand_thumb_skin_5
- removed link l_hand_thumb_skin_6
- removed link l_hand_thumb_skin_7
- removed link l_hand_thumb_skin_8
- removed link l_hand_thumb_skin_9
- removed link lidar
- removed link r_hand_index_skin_0
- removed link r_hand_index_skin_1
- removed link r_hand_index_skin_10
- removed link r_hand_index_skin_11
- removed link r_hand_index_skin_2
- removed link r_hand_index_skin_3
- removed link r_hand_index_skin_4
- removed link r_hand_index_skin_5
- removed link r_hand_index_skin_6
- removed link r_hand_index_skin_7
- removed link r_hand_index_skin_8
- removed link r_hand_index_skin_9
- removed link r_hand_middle_skin_0
- removed link r_hand_middle_skin_1
- removed link r_hand_middle_skin_10
- removed link r_hand_middle_skin_11
- removed link r_hand_middle_skin_2
- removed link r_hand_middle_skin_3
- removed link r_hand_middle_skin_4
- removed link r_hand_middle_skin_5
- removed link r_hand_middle_skin_6
- removed link r_hand_middle_skin_7
- removed link r_hand_middle_skin_8
- removed link r_hand_middle_skin_9
- removed link r_hand_ring_skin_0
- removed link r_hand_ring_skin_1
- removed link r_hand_ring_skin_10
- removed link r_hand_ring_skin_11
- removed link r_hand_ring_skin_2
- removed link r_hand_ring_skin_3
- removed link r_hand_ring_skin_4
- removed link r_hand_ring_skin_5
- removed link r_hand_ring_skin_6
- removed link r_hand_ring_skin_7
- removed link r_hand_ring_skin_8
- removed link r_hand_ring_skin_9
- removed link r_hand_thumb_skin_0
- removed link r_hand_thumb_skin_1
- removed link r_hand_thumb_skin_10
- removed link r_hand_thumb_skin_11
- removed link r_hand_thumb_skin_2
- removed link r_hand_thumb_skin_3
- removed link r_hand_thumb_skin_4
- removed link r_hand_thumb_skin_5
- removed link r_hand_thumb_skin_6
- removed link r_hand_thumb_skin_7
- removed link r_hand_thumb_skin_8
- removed link r_hand_thumb_skin_9
Joints:
- removed joint l_hand_index_skin_0_fixed_joint
- removed joint l_hand_index_skin_10_fixed_joint
- removed joint l_hand_index_skin_11_fixed_joint
- removed joint l_hand_index_skin_1_fixed_joint
- removed joint l_hand_index_skin_2_fixed_joint
- removed joint l_hand_index_skin_3_fixed_joint
- removed joint l_hand_index_skin_4_fixed_joint
- removed joint l_hand_index_skin_5_fixed_joint
- removed joint l_hand_index_skin_6_fixed_joint
- removed joint l_hand_index_skin_7_fixed_joint
- removed joint l_hand_index_skin_8_fixed_joint
- removed joint l_hand_index_skin_9_fixed_joint
- removed joint l_hand_middle_skin_0_fixed_joint
- removed joint l_hand_middle_skin_10_fixed_joint
- removed joint l_hand_middle_skin_11_fixed_joint
- removed joint l_hand_middle_skin_1_fixed_joint
- removed joint l_hand_middle_skin_2_fixed_joint
- removed joint l_hand_middle_skin_3_fixed_joint
- removed joint l_hand_middle_skin_4_fixed_joint
- removed joint l_hand_middle_skin_5_fixed_joint
- removed joint l_hand_middle_skin_6_fixed_joint
- removed joint l_hand_middle_skin_7_fixed_joint
- removed joint l_hand_middle_skin_8_fixed_joint
- removed joint l_hand_middle_skin_9_fixed_joint
- removed joint l_hand_ring_skin_0_fixed_joint
- removed joint l_hand_ring_skin_10_fixed_joint
- removed joint l_hand_ring_skin_11_fixed_joint
- removed joint l_hand_ring_skin_1_fixed_joint
- removed joint l_hand_ring_skin_2_fixed_joint
- removed joint l_hand_ring_skin_3_fixed_joint
- removed joint l_hand_ring_skin_4_fixed_joint
- removed joint l_hand_ring_skin_5_fixed_joint
- removed joint l_hand_ring_skin_6_fixed_joint
- removed joint l_hand_ring_skin_7_fixed_joint
- removed joint l_hand_ring_skin_8_fixed_joint
- removed joint l_hand_ring_skin_9_fixed_joint
- removed joint l_hand_thumb_skin_0_fixed_joint
- removed joint l_hand_thumb_skin_10_fixed_joint
- removed joint l_hand_thumb_skin_11_fixed_joint
- removed joint l_hand_thumb_skin_1_fixed_joint
- removed joint l_hand_thumb_skin_2_fixed_joint
- removed joint l_hand_thumb_skin_3_fixed_joint
- removed joint l_hand_thumb_skin_4_fixed_joint
- removed joint l_hand_thumb_skin_5_fixed_joint
- removed joint l_hand_thumb_skin_6_fixed_joint
- removed joint l_hand_thumb_skin_7_fixed_joint
- removed joint l_hand_thumb_skin_8_fixed_joint
- removed joint l_hand_thumb_skin_9_fixed_joint
- removed joint lidar_joint
- removed joint r_hand_index_skin_0_fixed_joint
- removed joint r_hand_index_skin_10_fixed_joint
- removed joint r_hand_index_skin_11_fixed_joint
- removed joint r_hand_index_skin_1_fixed_joint
- removed joint r_hand_index_skin_2_fixed_joint
- removed joint r_hand_index_skin_3_fixed_joint
- removed joint r_hand_index_skin_4_fixed_joint
- removed joint r_hand_index_skin_5_fixed_joint
- removed joint r_hand_index_skin_6_fixed_joint
- removed joint r_hand_index_skin_7_fixed_joint
- removed joint r_hand_index_skin_8_fixed_joint
- removed joint r_hand_index_skin_9_fixed_joint
- removed joint r_hand_middle_skin_0_fixed_joint
- removed joint r_hand_middle_skin_10_fixed_joint
- removed joint r_hand_middle_skin_11_fixed_joint
- removed joint r_hand_middle_skin_1_fixed_joint
- removed joint r_hand_middle_skin_2_fixed_joint
- removed joint r_hand_middle_skin_3_fixed_joint
- removed joint r_hand_middle_skin_4_fixed_joint
- removed joint r_hand_middle_skin_5_fixed_joint
- removed joint r_hand_middle_skin_6_fixed_joint
- removed joint r_hand_middle_skin_7_fixed_joint
- removed joint r_hand_middle_skin_8_fixed_joint
- removed joint r_hand_middle_skin_9_fixed_joint
- removed joint r_hand_ring_skin_0_fixed_joint
- removed joint r_hand_ring_skin_10_fixed_joint
- removed joint r_hand_ring_skin_11_fixed_joint
- removed joint r_hand_ring_skin_1_fixed_joint
- removed joint r_hand_ring_skin_2_fixed_joint
- removed joint r_hand_ring_skin_3_fixed_joint
- removed joint r_hand_ring_skin_4_fixed_joint
- removed joint r_hand_ring_skin_5_fixed_joint
- removed joint r_hand_ring_skin_6_fixed_joint
- removed joint r_hand_ring_skin_7_fixed_joint
- removed joint r_hand_ring_skin_8_fixed_joint
- removed joint r_hand_ring_skin_9_fixed_joint
- removed joint r_hand_thumb_skin_0_fixed_joint
- removed joint r_hand_thumb_skin_10_fixed_joint
- removed joint r_hand_thumb_skin_11_fixed_joint
- removed joint r_hand_thumb_skin_1_fixed_joint
- removed joint r_hand_thumb_skin_2_fixed_joint
- removed joint r_hand_thumb_skin_3_fixed_joint
- removed joint r_hand_thumb_skin_4_fixed_joint
- removed joint r_hand_thumb_skin_5_fixed_joint
- removed joint r_hand_thumb_skin_6_fixed_joint
- removed joint r_hand_thumb_skin_7_fixed_joint
- removed joint r_hand_thumb_skin_8_fixed_joint
- removed joint r_hand_thumb_skin_9_fixed_joint

Commit message: removed collisions meshes from every link except feet soles

File: urdf/ergoCub/robots/ergoCubGazeboV1/model.urdf (robot description, URDF)
Before this commit: robot ergoCub, 73 links, 72 joints
Links:
- link chest: geometry visual mesh filename=package://ergoCub/meshes/simmechanics/sim_ecub_chest_prt.stl scale=0.001 0.001 0.001
- link head: geometry visual mesh filename=package://ergoCub/meshes/simmechanics/sim_ecub_head_prt.stl scale=0.001 0.001 0.001
- link l_ankle_1: geometry visual mesh filename=package://ergoCub/meshes/simmechanics/sim_ecub_l_ankle_1_pr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 scale=0.001 0.001 0.001
- link l_ankle_2: geometry visual mesh filename=package://ergoCub/meshes/simmechanics/sim_ecub_l_ankle_2_pr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 scale=0.001 0.001 0.001
- link l_forearm: geometry visual mesh filename=package://ergoCub/meshes/simmechanics/sim_ecub_l_forearm_pr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 scale=0.001 0.001 0.001
- link l_hand_index_1: geometry visual mesh filename=package://ergoCub/meshes/simmechanics/sim_ecub_l_hand_index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 scale=0.001 0.001 0.001
- link l_hand_index_2: geometry visual mesh filename=package://ergoCub/meshes/simmechanics/sim_ecub_l_hand_index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 scale=0.001 0.001 0.001
- link l_hand_index_3: geometry visual mesh filename=package://ergoCub/meshes/simmechanics/sim_ecub_l_hand_index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 scale=0.001 0.001 0.001
- link l_hand_middle_1: geometry visual mesh filename=package://ergoCub/meshes/simmechanics/sim_ecub_l_hand_middl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 scale=0.001 0.001 0.001
- link l_hand_middle_2: geometry visual mesh filename=package://ergoCub/meshes/simmechanics/sim_ecub_l_hand_middl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 scale=0.001 0.001 0.001
- link l_hand_palm: geometry visual mesh filename=package://ergoCub/meshes/simmechanics/sim_ecub_l_hand_palm_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 scale=0.001 0.001 0.001
- link l_hand_pinkie_1: geometry visual mesh filename=package://ergoCub/meshes/simmechanics/sim_ecub_l_hand_pinki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 scale=0.001 0.001 0.001
- link l_hand_pinkie_2: geometry visual mesh filename=package://ergoCub/meshes/simmechanics/sim_ecub_l_hand_pinki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 scale=0.001 0.001 0.001
- link l_hand_ring_1: geometry visual mesh filename=package://ergoCub/meshes/simmechanics/sim_ecub_l_hand_ring_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 scale=0.001 0.001 0.001
- link l_hand_ring_2: geometry visual mesh filename=package://ergoCub/meshes/simmechanics/sim_ecub_l_hand_ring_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 scale=0.001 0.001 0.001
- link l_hand_thumb_1: geometry visual mesh filename=package://ergoCub/meshes/simmechanics/sim_ecub_l_hand_thumb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 scale=0.001 0.001 0.001
- link l_hand_thumb_2: geometry visual mesh filename=package://ergoCub/meshes/simmechanics/sim_ecub_l_hand_thumb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 scale=0.001 0.001 0.001
- link l_hand_thumb_3: geometry visual mesh filename=package://ergoCub/meshes/simmechanics/sim_ecub_l_hand_thumb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 scale=0.001 0.001 0.001
- link l_hip_1: geometry visual mesh filename=package://ergoCub/meshes/simmechanics/sim_ecub_l_hip_1_prt.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 scale=0.001 0.001 0.001
- link l_hip_2: geometry visual mesh filename=package://ergoCub/meshes/simmechanics/sim_ecub_l_hip_2_prt.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 scale=0.001 0.001 0.001
- link l_hip_3: geometry visual mesh filename=package://ergoCub/meshes/simmechanics/sim_ecub_l_hip_3_prt.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 scale=0.001 0.001 0.001
- link l_lower_leg: geometry visual mesh filename=package://ergoCub/meshes/simmechanics/sim_ecub_l_lower_leg_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 scale=0.001 0.001 0.001
- link l_shoulder_1: geometry visual mesh filename=package://ergoCub/meshes/simmechanics/sim_ecub_l_shoulder_1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 scale=0.001 0.001 0.001
- link l_shoulder_2: geometry visual mesh filename=package://ergoCub/meshes/simmechanics/sim_ecub_l_shoulder_2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 scale=0.001 0.001 0.001
- link l_shoulder_3: geometry visual mesh filename=package://ergoCub/meshes/simmechanics/sim_ecub_l_shoulder_3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 scale=0.001 0.001 0.001
- link l_upper_leg: geometry visual mesh filename=package://ergoCub/meshes/simmechanics/sim_ecub_l_upper_leg_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 scale=0.001 0.001 0.001
- link l_upperarm: geometry visual mesh filename=package://ergoCub/meshes/simmechanics/sim_ecub_l_upperarm_p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 scale=0.001 0.001 0.001
- link l_wrist_1: geometry visual mesh filename=package://ergoCub/meshes/simmechanics/sim_ecub_l_wrist_1_pr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 scale=0.001 0.001 0.001
- link l_wrist_2: geometry visual mesh filename=package://ergoCub/meshes/simmechanics/sim_ecub_l_wrist_2_pr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 scale=0.001 0.001 0.001
- link neck_2: geometry visual mesh filename=package://ergoCub/meshes/simmechanics/sim_ecub_head_neck_2_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 scale=0.001 0.001 0.001
- link neck_3: geometry visual mesh filename=package://ergoCub/meshes/simmechanics/sim_ecub_head_neck_3_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 scale=0.001 0.001 0.001
- link r_ankle_1: geometry visual mesh filename=package://ergoCub/meshes/simmechanics/sim_ecub_r_ankle_1_pr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 scale=0.001 0.001 0.001
- link r_ankle_2: geometry visual mesh filename=package://ergoCub/meshes/simmechanics/sim_ecub_r_ankle_2_pr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 scale=0.001 0.001 0.001
- link r_forearm: geometry visual mesh filename=package://ergoCub/meshes/simmechanics/sim_ecub_r_forearm_pr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 scale=0.001 0.001 0.001
- link r_hand_index_1: geometry visual mesh filename=package://ergoCub/meshes/simmechanics/sim_ecub_r_hand_index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 scale=0.001 0.001 0.001
- link r_hand_index_2: geometry visual mesh filename=package://ergoCub/meshes/simmechanics/sim_ecub_r_hand_index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 scale=0.001 0.001 0.001
- link r_hand_index_3: geometry visual mesh filename=package://ergoCub/meshes/simmechanics/sim_ecub_r_hand_index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 scale=0.001 0.001 0.001
- link r_hand_middle_1: geometry visual mesh filename=package://ergoCub/meshes/simmechanics/sim_ecub_r_hand_middl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 scale=0.001 0.001 0.001
- link r_hand_middle_2: geometry visual mesh filename=package://ergoCub/meshes/simmechanics/sim_ecub_r_hand_middl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 scale=0.001 0.001 0.001
- link r_hand_palm: geometry visual mesh filename=package://ergoCub/meshes/simmechanics/sim_ecub_r_hand_palm_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 scale=0.001 0.001 0.001
- link r_hand_pinkie_1: geometry visual mesh filename=package://ergoCub/meshes/simmechanics/sim_ecub_r_hand_pinki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 scale=0.001 0.001 0.001
- link r_hand_pinkie_2: geometry visual mesh filename=package://ergoCub/meshes/simmechanics/sim_ecub_r_hand_pinki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 scale=0.001 0.001 0.001
- link r_hand_ring_1: geometry visual mesh filename=package://ergoCub/meshes/simmechanics/sim_ecub_r_hand_ring_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 scale=0.001 0.001 0.001
- link r_hand_ring_2: geometry visual mesh filename=package://ergoCub/meshes/simmechanics/sim_ecub_r_hand_ring_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 scale=0.001 0.001 0.001
- link r_hand_thumb_1: geometry visual mesh filename=package://ergoCub/meshes/simmechanics/sim_ecub_r_hand_thumb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 scale=0.001 0.001 0.001
- link r_hand_thumb_2: geometry visual mesh filename=package://ergoCub/meshes/simmechanics/sim_ecub_r_hand_thumb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 scale=0.001 0.001 0.001
- link r_hand_thumb_3: geometry visual mesh filename=package://ergoCub/meshes/simmechanics/sim_ecub_r_hand_thumb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 scale=0.001 0.001 0.001
- link r_hip_1: geometry visual mesh filename=package://ergoCub/meshes/simmechanics/sim_ecub_r_hip_1_prt.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 scale=0.001 0.001 0.001
- link r_hip_2: geometry visual mesh filename=package://ergoCub/meshes/simmechanics/sim_ecub_r_hip_2_prt.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 scale=0.001 0.001 0.001
- link r_hip_3: geometry visual mesh filename=package://ergoCub/meshes/simmechanics/sim_ecub_r_hip_3_prt.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 scale=0.001 0.001 0.001
- link r_lower_leg: geometry visual mesh filename=package://ergoCub/meshes/simmechanics/sim_ecub_r_lower_leg_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 scale=0.001 0.001 0.001
- link r_shoulder_1: geometry visual mesh filename=package://ergoCub/meshes/simmechanics/sim_ecub_r_shoulder_1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 scale=0.001 0.001 0.001
- link r_shoulder_2: geometry visual mesh filename=package://ergoCub/meshes/simmechanics/sim_ecub_r_shoulder_2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 scale=0.001 0.001 0.001
- link r_shoulder_3: geometry visual mesh filename=package://ergoCub/meshes/simmechanics/sim_ecub_r_shoulder_3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 scale=0.001 0.001 0.001
- link r_upper_leg: geometry visual mesh filename=package://ergoCub/meshes/simmechanics/sim_ecub_r_upper_leg_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 scale=0.001 0.001 0.001
- link r_upperarm: geometry visual mesh filename=package://ergoCub/meshes/simmechanics/sim_ecub_r_upperarm_p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 scale=0.001 0.001 0.001
- link r_wrist_1: geometry visual mesh filename=package://ergoCub/meshes/simmechanics/sim_ecub_r_wrist_1_pr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 scale=0.001 0.001 0.001
- link r_wrist_2: geometry visual mesh filename=package://ergoCub/meshes/simmechanics/sim_ecub_r_wrist_2_pr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 scale=0.001 0.001 0.001
- link realsense: geometry visual mesh filename=package://ergoCub/meshes/simmechanics/sim_ecub_realsense_pr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 scale=0.001 0.001 0.001
- link root_link: geometry visual mesh filename=package://ergoCub/meshes/simmechanics/sim_ecub_root_link_pr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 scale=0.001 0.001 0.001
- link torso_1: geometry visual mesh filename=package://ergoCub/meshes/simmechanics/sim_ecub_torso_1_prt.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 scale=0.001 0.001 0.001
- link torso_2: geometry visual mesh filename=package://ergoCub/meshes/simmechanics/sim_ecub_torso_2_prt.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 scale=0.001 0.001 0.001

Commit message: Automatic update of urdf

File: urdf/ergoCub/robots/ergoCubGazeboV1/model.urdf (robot description, URDF)
Before this commit: robot ergoCub, 169 links, 168 joints
Joints:
- joint l_hip_roll: limit lower=-0.17453292519943295 upper=1.9547687622336491 effort=50000 velocity=120.0 -> lower=-0.6108652381980153 upper=1.9547687622336491 effort=50000 velocity=120.0
- joint r_hip_roll: limit lower=-0.17453292519943295 upper=1.9547687622336491 effort=50000 velocity=120.0 -> lower=-0.6108652381980153 upper=1.9547687622336491 effort=50000 velocity=120.0

File: urdf/ergoCub/robots/ergoCubSN000/model.urdf (robot description, URDF)
Before this commit: robot ergoCub, 169 links, 168 joints
Joints:
- joint l_hip_roll: limit lower=-0.17453292519943295 upper=1.9547687622336491 effort=50000 velocity=120.0 -> lower=-0.6108652381980153 upper=1.9547687622336491 effort=50000 velocity=120.0
- joint r_hip_roll: limit lower=-0.17453292519943295 upper=1.9547687622336491 effort=50000 velocity=120.0 -> lower=-0.6108652381980153 upper=1.9547687622336491 effort=50000 velocity=120.0

Commit message: Automatic update of urdf

File: urdf/ergoCub/robots/ergoCubGazeboV1/model.urdf (robot description, URDF)
Before this commit: robot ergoCub, 169 links, 168 joints
Joints:
- joint l_shoulder_pitch: limit lower=-3.0543261909900767 upper=0.3490658503988659 effort=50000 velocity=120.0 -> lower=-2.9670597283903604 upper=0.6108652381980153 effort=50000 velocity=120.0
- joint l_shoulder_roll: limit lower=0.20943951023931956 upper=2.8448866807507573 effort=50000 velocity=120.0 -> lower=-0.2617993877991494 upper=2.6179938779914944 effort=50000 velocity=120.0
- joint r_shoulder_pitch: limit lower=-3.0543261909900767 upper=0.3490658503988659 effort=50000 velocity=120.0 -> lower=-2.9670597283903604 upper=0.6108652381980153 effort=50000 velocity=120.0
- joint r_shoulder_roll: limit lower=0.20943951023931956 upper=2.8448866807507573 effort=50000 velocity=120.0 -> lower=-0.2617993877991494 upper=2.6179938779914944 effort=50000 velocity=120.0

File: urdf/ergoCub/robots/ergoCubSN000/model.urdf (robot description, URDF)
Before this commit: robot ergoCub, 169 links, 168 joints
Joints:
- joint l_shoulder_pitch: limit lower=-3.0543261909900767 upper=0.3490658503988659 effort=50000 velocity=120.0 -> lower=-2.9670597283903604 upper=0.6108652381980153 effort=50000 velocity=120.0
- joint l_shoulder_roll: limit lower=0.20943951023931956 upper=2.8448866807507573 effort=50000 velocity=120.0 -> lower=-0.2617993877991494 upper=2.6179938779914944 effort=50000 velocity=120.0
- joint r_shoulder_pitch: limit lower=-3.0543261909900767 upper=0.3490658503988659 effort=50000 velocity=120.0 -> lower=-2.9670597283903604 upper=0.6108652381980153 effort=50000 velocity=120.0
- joint r_shoulder_roll: limit lower=0.20943951023931956 upper=2.8448866807507573 effort=50000 velocity=120.0 -> lower=-0.2617993877991494 upper=2.6179938779914944 effort=50000 velocity=120.0
