Commit message: Aligned ergoCubGazeboV1 urdf with master removing experimental stuff and comments

File: urdf/ergoCub/robots/ergoCubGazeboV1/model.urdf (robot description, URDF)
Before this commit: robot ergoCub, 73 links, 72 joints
Links:
- added link l_hand_index_skin_0
- added link l_hand_index_skin_1
- added link l_hand_index_skin_10
- added link l_hand_index_skin_11
- added link l_hand_index_skin_2
- added link l_hand_index_skin_3
- added link l_hand_index_skin_4
- added link l_hand_index_skin_5
- added link l_hand_index_skin_6
- added link l_hand_index_skin_7
- added link l_hand_index_skin_8
- added link l_hand_index_skin_9
- added link l_hand_middle_skin_0
- added link l_hand_middle_skin_1
- added link l_hand_middle_skin_10
- added link l_hand_middle_skin_11
- added link l_hand_middle_skin_2
- added link l_hand_middle_skin_3
- added link l_hand_middle_skin_4
- added link l_hand_middle_skin_5
- added link l_hand_middle_skin_6
- added link l_hand_middle_skin_7
- added link l_hand_middle_skin_8
- added link l_hand_middle_skin_9
- added link l_hand_ring_skin_0
- added link l_hand_ring_skin_1
- added link l_hand_ring_skin_10
- added link l_hand_ring_skin_11
- added link l_hand_ring_skin_2
- added link l_hand_ring_skin_3
- added link l_hand_ring_skin_4
- added link l_hand_ring_skin_5
- added link l_hand_ring_skin_6
- added link l_hand_ring_skin_7
- added link l_hand_ring_skin_8
- added link l_hand_ring_skin_9
- added link l_hand_thumb_skin_0
- added link l_hand_thumb_skin_1
- added link l_hand_thumb_skin_10
- added link l_hand_thumb_skin_11
- added link l_hand_thumb_skin_2
- added link l_hand_thumb_skin_3
- added link l_hand_thumb_skin_4
- added link l_hand_thumb_skin_5
- added link l_hand_thumb_skin_6
- added link l_hand_thumb_skin_7
- added link l_hand_thumb_skin_8
- added link l_hand_thumb_skin_9
- added link r_hand_index_skin_0
- added link r_hand_index_skin_1
- added link r_hand_index_skin_10
- added link r_hand_index_skin_11
- added link r_hand_index_skin_2
- added link r_hand_index_skin_3
- added link r_hand_index_skin_4
- added link r_hand_index_skin_5
- added link r_hand_index_skin_6
- added link r_hand_index_skin_7
- added link r_hand_index_skin_8
- added link r_hand_index_skin_9
- added link r_hand_middle_skin_0
- added link r_hand_middle_skin_1
- added link r_hand_middle_skin_10
- added link r_hand_middle_skin_11
- added link r_hand_middle_skin_2
- added link r_hand_middle_skin_3
- added link r_hand_middle_skin_4
- added link r_hand_middle_skin_5
- added link r_hand_middle_skin_6
- added link r_hand_middle_skin_7
- added link r_hand_middle_skin_8
- added link r_hand_middle_skin_9
- added link r_hand_ring_skin_0
- added link r_hand_ring_skin_1
- added link r_hand_ring_skin_10
- added link r_hand_ring_skin_11
- added link r_hand_ring_skin_2
- added link r_hand_ring_skin_3
- added link r_hand_ring_skin_4
- added link r_hand_ring_skin_5
- added link r_hand_ring_skin_6
- added link r_hand_ring_skin_7
- added link r_hand_ring_skin_8
- added link r_hand_ring_skin_9
- added link r_hand_thumb_skin_0
- added link r_hand_thumb_skin_1
- added link r_hand_thumb_skin_10
- added link r_hand_thumb_skin_11
- added link r_hand_thumb_skin_2
- added link r_hand_thumb_skin_3
- added link r_hand_thumb_skin_4
- added link r_hand_thumb_skin_5
- added link r_hand_thumb_skin_6
- added link r_hand_thumb_skin_7
- added link r_hand_thumb_skin_8
- added link r_hand_thumb_skin_9
Joints:
- added joint l_hand_index_skin_0_fixed_joint: type fixed, parent l_hand_index_3, child l_hand_index_skin_0, origin xyz=2.02830541008725e-07 -0.0024337142787178856 -0.0214068046370407 rpy=1.3589739287870087e-06 1.222488567730119 -1.5707956227077366
- added joint l_hand_index_skin_10_fixed_joint: type fixed, parent l_hand_index_3, child l_hand_index_skin_10, origin xyz=-0.0033001087817297603 -0.004081475640777432 -0.027767928417915755 rpy=3.1415923305252225 1.5047762567210512 1.5707960116499358
- added joint l_hand_index_skin_11_fixed_joint: type fixed, parent l_hand_index_3, child l_hand_index_skin_11, origin xyz=-0.003300196027624047 -0.0031310503040746507 -0.02328184486187923 rpy=1.0045087854148686e-06 1.2201097511639785 -1.5707952579461582
- added joint l_hand_index_skin_1_fixed_joint: type fixed, parent l_hand_index_3, child l_hand_index_skin_1, origin xyz=0.00330018002039012 -0.0031312039972868355 -0.023281879205948874 rpy=1.0045087854148686e-06 1.2201097511639785 -1.5707952579461582
- added joint l_hand_index_skin_2_fixed_joint: type fixed, parent l_hand_index_3, child l_hand_index_skin_2, origin xyz=0 -0.0037582722604465324 -0.025193049887115737 rpy=2.019258946672971e-07 1.305739917586136 -1.5707964798904088
- added joint l_hand_index_skin_3_fixed_joint: type fixed, parent l_hand_index_3, child l_hand_index_skin_3, origin xyz=0.003300267266284379 -0.004081629333989534 -0.027767962761985454 rpy=3.1415923305252225 1.5047762567210512 1.5707960116499358
- added joint l_hand_index_skin_4_fixed_joint: type fixed, parent l_hand_index_3, child l_hand_index_skin_4, origin xyz=0.005929574139393212 -0.0011921762933711222 -0.02800035143013324 rpy=-3.141592000798577 1.2994444690524731 2.7771560098086976
- added joint l_hand_index_skin_5_fixed_joint: type fixed, parent l_hand_index_3, child l_hand_index_skin_5, origin xyz=0 -0.0034767433707287576 -0.029836323676495524 rpy=3.1415916993735475 1.0862258770767357 1.570795618249084
- added joint l_hand_index_skin_6_fixed_joint: type fixed, parent l_hand_index_3, child l_hand_index_skin_6, origin xyz=0.0032998108383007554 -0.0018242465422362297 -0.03177275148589709 rpy=3.1415920569068843 0.7785360318433139 2.532384926237606
- added joint l_hand_index_skin_7_fixed_joint: type fixed, parent l_hand_index_3, child l_hand_index_skin_7, origin xyz=-1.7765327827573563e-07 -0.000272313592458967 -0.03327286783966488 rpy=3.141592488071993 0.6184189897566703 1.5713167119394844
- added joint l_hand_index_skin_8_fixed_joint: type fixed, parent l_hand_index_3, child l_hand_index_skin_8, origin xyz=-0.003299617986161782 -0.001823842286354016 -0.03177291710655328 rpy=3.1415926400948937 0.7785356574796937 0.6092071825770647
- added joint l_hand_index_skin_9_fixed_joint: type fixed, parent l_hand_index_3, child l_hand_index_skin_9, origin xyz=-0.005929289581785957 -0.0011924954736174942 -0.0280007264298755 rpy=-3.141591222167342 1.2994438865660223 0.36443832683545135
- added joint l_hand_middle_skin_0_fixed_joint: type fixed, parent l_hand_middle_2, child l_hand_middle_skin_0, origin xyz=0 -0.0024341633880323454 -0.02140626784029226 rpy=2.8880021565356356e-07 1.2224888157071614 -1.5707959092703505
- added joint l_hand_middle_skin_10_fixed_joint: type fixed, parent l_hand_middle_2, child l_hand_middle_skin_10, origin xyz=-0.0032999688028366864 -0.004081937549531761 -0.027767599906222185 rpy=3.14159206598453 1.504776403539619 1.5707957068952807
- added joint l_hand_middle_skin_11_fixed_joint: type fixed, parent l_hand_middle_2, child l_hand_middle_skin_11, origin xyz=-0.0032999302761450126 -0.0031315344195035066 -0.023280711530192733 rpy=1.4298532751994242e-06 1.2201100060845365 -1.5707950386454854
- added joint l_hand_middle_skin_1_fixed_joint: type fixed, parent l_hand_middle_2, child l_hand_middle_skin_1, origin xyz=0.0032999923469937895 -0.0031310595632358384 -0.023281089805274435 rpy=1.4298532751994242e-06 1.2201100060845365 -1.5707950386454854
- added joint l_hand_middle_skin_2_fixed_joint: type fixed, parent l_hand_middle_2, child l_hand_middle_skin_2, origin xyz=0 -0.0037584600637464993 -0.025193167911877645 rpy=2.67805384222918e-06 1.3057397262072086 -1.5707938810851714
- added joint l_hand_middle_skin_3_fixed_joint: type fixed, parent l_hand_middle_2, child l_hand_middle_skin_3, origin xyz=0.003300181170510192 -0.004082174556855278 -0.027766773373389564 rpy=3.14159206598453 1.504776403539619 1.5707957068952807
- added joint l_hand_middle_skin_4_fixed_joint: type fixed, parent l_hand_middle_2, child l_hand_middle_skin_4, origin xyz=0.005929732632988013 -0.001192832553830403 -0.027999915681298115 rpy=3.141592336413363 1.299444945688194 2.7771552495198835
- added joint l_hand_middle_skin_5_fixed_joint: type fixed, parent l_hand_middle_2, child l_hand_middle_skin_5, origin xyz=0 -0.0034765832806818997 -0.02983570347842418 rpy=3.1415923106025314 1.086225709334958 1.5707962889575584
- added joint l_hand_middle_skin_6_fixed_joint: type fixed, parent l_hand_middle_2, child l_hand_middle_skin_6, origin xyz=0.0033001032954547184 -0.0018248945553451246 -0.031771757727755756 rpy=-3.1415924841511433 0.7785357399039169 2.532385692627037
- added joint l_hand_middle_skin_7_fixed_joint: type fixed, parent l_hand_middle_2, child l_hand_middle_skin_7, origin xyz=0 -0.0002725978091493997 -0.033271502713935364 rpy=3.141592263055179 0.6184187545317414 1.5713165725114155
- added joint l_hand_middle_skin_8_fixed_joint: type fixed, parent l_hand_middle_2, child l_hand_middle_skin_8, origin xyz=-0.0032999946700499154 -0.0018244087955724964 -0.0317716170907979 rpy=-3.141592114011197 0.7785357191047289 0.60920707683613
- added joint l_hand_middle_skin_9_fixed_joint: type fixed, parent l_hand_middle_2, child l_hand_middle_skin_9, origin xyz=-0.005929566529031996 -0.0011920519924579764 -0.028000347463470243 rpy=-3.141592260042174 1.299444239340149 0.3644371706703166
- added joint l_hand_ring_skin_0_fixed_joint: type fixed, parent l_hand_ring_2, child l_hand_ring_skin_0, origin xyz=0 -0.002434109766516368 -0.021405903344744404 rpy=3.19241308601029e-07 1.2224879756285634 -1.5707957505342052
- added joint l_hand_ring_skin_10_fixed_joint: type fixed, parent l_hand_ring_2, child l_hand_ring_skin_10, origin xyz=-0.0032999678913585937 -0.00408208342496913 -0.027766666771285198 rpy=3.141583892131502 1.5047765106577695 1.5707878943439342
- added joint l_hand_ring_skin_11_fixed_joint: type fixed, parent l_hand_ring_2, child l_hand_ring_skin_11, origin xyz=-0.003299969312657214 -0.003131389602053558 -0.023280510569694823 rpy=7.841409816247398e-07 1.220109279873348 -1.5707953766916674
- added joint l_hand_ring_skin_1_fixed_joint: type fixed, parent l_hand_ring_2, child l_hand_ring_skin_1, origin xyz=0.003299959717504228 -0.0031312149423083635 -0.02328043103333599 rpy=7.841409816247398e-07 1.220109279873348 -1.5707953766916674
- added joint l_hand_ring_skin_2_fixed_joint: type fixed, parent l_hand_ring_2, child l_hand_ring_skin_2, origin xyz=0 -0.003758755164085026 -0.02519260657118344 rpy=2.109983659924688e-06 1.3057391422971405 -1.57079420774816
- added joint l_hand_ring_skin_3_fixed_joint: type fixed, parent l_hand_ring_2, child l_hand_ring_skin_3, origin xyz=0.0032999611388028777 -0.004081908765223963 -0.02776658723492642 rpy=3.141583892131502 1.5047765106577695 1.5707878943439342
- added joint l_hand_ring_skin_4_fixed_joint: type fixed, parent l_hand_ring_2, child l_hand_ring_skin_4, origin xyz=0.005929559072218151 -0.0011924106023348813 -0.02799965564814172 rpy=3.1415923272373556 1.299444799530583 2.7771553646234826
- added joint l_hand_ring_skin_5_fixed_joint: type fixed, parent l_hand_ring_2, child l_hand_ring_skin_5, origin xyz=0 -0.0034766110824936136 -0.02983485885572207 rpy=3.141592267163769 1.086225807890324 1.570796144313782
- added joint l_hand_ring_skin_6_fixed_joint: type fixed, parent l_hand_ring_2, child l_hand_ring_skin_6, origin xyz=0.0033000024742935834 -0.0018246687466073053 -0.03177155146156402 rpy=3.1415925874639985 0.7785363357981874 2.5323859043537085
- added joint l_hand_ring_skin_7_fixed_joint: type fixed, parent l_hand_ring_2, child l_hand_ring_skin_7, origin xyz=0 -0.000273182602237132 -0.03327141530303279 rpy=3.141592083365392 0.6184190542087526 1.5713170178340956
- added joint l_hand_ring_skin_8_fixed_joint: type fixed, parent l_hand_ring_2, child l_hand_ring_skin_8, origin xyz=-0.003299926555867876 -0.001824843406352472 -0.03177163099792274 rpy=-3.141592630967883 0.7785355069422046 0.6092077934143093
- added joint l_hand_ring_skin_9_fixed_joint: type fixed, parent l_hand_ring_2, child l_hand_ring_skin_9, origin xyz=-0.005929446120504852 -0.0011926740085302368 -0.02800007942441246 rpy=-3.1415921627311505 1.2994436529688218 0.36443765521426325
- added joint l_hand_thumb_skin_0_fixed_joint: type fixed, parent l_hand_thumb_3, child l_hand_thumb_skin_0, origin xyz=0.020306533379063282 -0.0024343101858567417 -1.02177518712665e-06 rpy=1.5707963529634608 -7.763677284389983e-07 -0.348308299608484
- added joint l_hand_thumb_skin_10_fixed_joint: type fixed, parent l_hand_thumb_3, child l_hand_thumb_skin_10, origin xyz=0.026667719682656202 -0.00408229584322653 -0.003299911601186978 rpy=1.5707965227938288 -9.019462447191873e-07 0.06601977594073062
- added joint l_hand_thumb_skin_11_fixed_joint: type fixed, parent l_hand_thumb_3, child l_hand_thumb_skin_11, origin xyz=0.022181516794865866 -0.00313158061241825 -0.00330035824525321 rpy=1.5707968798775 -6.358788514904552e-07 -0.3506868205285684
- added joint l_hand_thumb_skin_1_fixed_joint: type fixed, parent l_hand_thumb_3, child l_hand_thumb_skin_1, origin xyz=0.02218144130259432 -0.003131520277003974 0.0033000550744306523 rpy=1.5707968798775 -6.358788514904552e-07 -0.3506868205285684
- added joint l_hand_thumb_skin_2_fixed_joint: type fixed, parent l_hand_thumb_3, child l_hand_thumb_skin_2, origin xyz=0.024092765288315235 -0.0037586699455105788 0 rpy=1.5707966249662435 -6.175239036510354e-07 -0.26505736279648673
- added joint l_hand_thumb_skin_3_fixed_joint: type fixed, parent l_hand_thumb_3, child l_hand_thumb_skin_3, origin xyz=0.02666722402677603 -0.004082581893144865 0.0032996629815040257 rpy=1.5707965227938288 -9.019462447191873e-07 0.06601977594073062
- added joint l_hand_thumb_skin_4_fixed_joint: type fixed, parent l_hand_thumb_3, child l_hand_thumb_skin_4, origin xyz=0.02690021104599309 -0.0011927877443135282 0.0059287648863864395 rpy=0.37702429099789225 0.2531248955594458 0.09883894762271977
- added joint l_hand_thumb_skin_5_fixed_joint: type fixed, parent l_hand_thumb_3, child l_hand_thumb_skin_5, origin xyz=0.028735478235047893 -0.00347687151090062 -3.1587642940200666e-07 rpy=1.5707957126757448 -5.513795408585156e-07 0.4845703956395784
- added joint l_hand_thumb_skin_6_fixed_joint: type fixed, parent l_hand_thumb_3, child l_hand_thumb_skin_6, origin xyz=0.030672478717119214 -0.0018246658485785439 0.0032996972420061 rpy=0.7821843436480906 0.6234816082641762 0.5256769446782557
- added joint l_hand_thumb_skin_7_fixed_joint: type fixed, parent l_hand_thumb_3, child l_hand_thumb_skin_7, origin xyz=0.03217216332171892 -0.0002731248779968831 0 rpy=1.5704939137056884 0.00042393168110662526 0.9523772903877968
- added joint l_hand_thumb_skin_8_fixed_joint: type fixed, parent l_hand_thumb_3, child l_hand_thumb_skin_8, origin xyz=0.030671762678273276 -0.0018250383011248483 -0.0033001906622364408 rpy=2.3594071882842584 -0.6234824919681496 0.5256776375213161
- added joint l_hand_thumb_skin_9_fixed_joint: type fixed, parent l_hand_thumb_3, child l_hand_thumb_skin_9, origin xyz=0.026900642650424703 -0.0011927733091181558 -0.005929763387118231 rpy=2.764568857310248 -0.253126241141505 0.09883859873338112
- added joint r_hand_index_skin_0_fixed_joint: type fixed, parent r_hand_index_3, child r_hand_index_skin_0, origin xyz=6.083293345379714e-07 -0.0024337142786424737 -0.02140564618132018 rpy=-1.358973927973795e-06 1.2224885677301185 -1.5707970308820571
- added joint r_hand_index_skin_10_fixed_joint: type fixed, parent r_hand_index_3, child r_hand_index_skin_10, origin xyz=-0.0032994561064087977 -0.004081629333914094 -0.027766804306264936 rpy=-3.141590806265971 1.5047757593824544 1.570798933120569
- added joint r_hand_index_skin_11_fixed_joint: type fixed, parent r_hand_index_3, child r_hand_index_skin_11, origin xyz=-0.0032993688605145247 -0.003131203997211396 -0.023280720750228412 rpy=-1.004508784930116e-06 1.2201097511639787 -1.5707973956436345
- added joint r_hand_index_skin_1_fixed_joint: type fixed, parent r_hand_index_3, child r_hand_index_skin_1, origin xyz=0.0033010071874996078 -0.0031310503039992388 -0.023280686406158713 rpy=-1.004508784930116e-06 1.2201097511639787 -1.5707973956436345
- added joint r_hand_index_skin_2_fixed_joint: type fixed, parent r_hand_index_3, child r_hand_index_skin_2, origin xyz=9.879565030165849e-07 -0.003758522823116728 -0.025192849922389737 rpy=-2.0192589424348972e-07 1.3057399175861366 -1.5707961736993847
- added joint r_hand_index_skin_3_fixed_joint: type fixed, parent r_hand_index_3, child r_hand_index_skin_3, origin xyz=0.0033009199416053556 -0.0040814756407019925 -0.027766769962195237 rpy=-3.141590806265971 1.5047757593824544 1.570798933120569
- added joint r_hand_index_skin_4_fixed_joint: type fixed, parent r_hand_index_3, child r_hand_index_skin_4, origin xyz=0.005930100741661552 -0.001192495473541999 -0.027999567974154982 rpy=3.1415912221673423 1.2994438865660232 2.777154326754342
- added joint r_hand_index_skin_5_fixed_joint: type fixed, parent r_hand_index_3, child r_hand_index_skin_5, origin xyz=8.852545381604626e-07 -0.0034767433706533735 -0.029835165220775006 rpy=-3.1415916993735475 1.0862258770767357 1.5707970353407095
- added joint r_hand_index_skin_6_fixed_joint: type fixed, parent r_hand_index_3, child r_hand_index_skin_6, origin xyz=0.003300138880263745 -0.001824777399458355 -0.03177155540437698 rpy=-3.1415926400948937 0.7785356574796939 2.532385471012728
- added joint r_hand_index_skin_7_fixed_joint: type fixed, parent r_hand_index_3, child r_hand_index_skin_7, origin xyz=9.888131538363099e-07 -0.0002723135923835829 -0.03327170938394436 rpy=-3.1415924489774776 0.6184188472429561 1.5713175931002388
- added joint r_hand_index_skin_8_fixed_joint: type fixed, parent r_hand_index_3, child r_hand_index_skin_8, origin xyz=-0.003298999678425174 -0.0018242465421608456 -0.031771593030176515 rpy=-3.1415920569068843 0.7785360318433138 0.6092077273521872
- added joint r_hand_index_skin_9_fixed_joint: type fixed, parent r_hand_index_3, child r_hand_index_skin_9, origin xyz=-0.0059286269158415825 -0.0011924268560412343 -0.028000151465407297 rpy=3.1415920007985783 1.2994444690524727 0.3644366437810966
- added joint r_hand_middle_skin_0_fixed_joint: type fixed, parent r_hand_middle_2, child r_hand_middle_skin_0, origin xyz=0 -0.0024341633880323454 -0.02140626784029226 rpy=-2.888002141897799e-07 1.2224888157071614 -1.5707967443194422
- added joint r_hand_middle_skin_10_fixed_joint: type fixed, parent r_hand_middle_2, child r_hand_middle_skin_10, origin xyz=-0.003300181170510192 -0.004082174556855278 -0.027766773373389564 rpy=-3.1415858006046733 1.5047760963753847 1.5708033199852864
- added joint r_hand_middle_skin_11_fixed_joint: type fixed, parent r_hand_middle_2, child r_hand_middle_skin_11, origin xyz=-0.0032999923469937895 -0.0031310595632358384 -0.023281089805274435 rpy=-1.4298532745530854e-06 1.2201100060845362 -1.5707976149443068
- added joint r_hand_middle_skin_1_fixed_joint: type fixed, parent r_hand_middle_2, child r_hand_middle_skin_1, origin xyz=0.0032999302761450126 -0.0031315344195035066 -0.023280711530192733 rpy=-1.4298532745530854e-06 1.2201100060845362 -1.5707976149443068
- added joint r_hand_middle_skin_2_fixed_joint: type fixed, parent r_hand_middle_2, child r_hand_middle_skin_2, origin xyz=0 -0.0037584600637464993 -0.025193167911877645 rpy=-2.6780538415934596e-06 1.305739726207208 -1.5707987725046209
- added joint r_hand_middle_skin_3_fixed_joint: type fixed, parent r_hand_middle_2, child r_hand_middle_skin_3, origin xyz=0.0032999688028366864 -0.004081937549531761 -0.027767599906222185 rpy=-3.1415858006046733 1.5047760963753847 1.5708033199852864
- added joint r_hand_middle_skin_4_fixed_joint: type fixed, parent r_hand_middle_2, child r_hand_middle_skin_4, origin xyz=0.005929566529031996 -0.0011920519924579764 -0.028000347463470243 rpy=3.141592260042173 1.2994442393401489 2.777155482919476
- added joint r_hand_middle_skin_5_fixed_joint: type fixed, parent r_hand_middle_2, child r_hand_middle_skin_5, origin xyz=0 -0.0034765832806818997 -0.02983570347842418 rpy=-3.1415923106025314 1.086225709334958 1.570796364632236
- added joint r_hand_middle_skin_6_fixed_joint: type fixed, parent r_hand_middle_2, child r_hand_middle_skin_6, origin xyz=0.0032999946700499154 -0.0018244087955724964 -0.0317716170907979 rpy=3.141592114011197 0.778535719104729 2.532385576753663
- added joint r_hand_middle_skin_7_fixed_joint: type fixed, parent r_hand_middle_2, child r_hand_middle_skin_7, origin xyz=0 -0.0002725978091493997 -0.033271502713935364 rpy=-3.1415924148088807 0.618418747537505 1.5713170250376087
- added joint r_hand_middle_skin_8_fixed_joint: type fixed, parent r_hand_middle_2, child r_hand_middle_skin_8, origin xyz=-0.0033001032954547184 -0.0018248945553451246 -0.031771757727755756 rpy=3.1415924841511433 0.7785357399039171 0.6092069609627565
- added joint r_hand_middle_skin_9_fixed_joint: type fixed, parent r_hand_middle_2, child r_hand_middle_skin_9, origin xyz=-0.005929732632988013 -0.001192832553830403 -0.027999915681298115 rpy=-3.1415923364133644 1.2994449456881931 0.36443740406990854
- added joint r_hand_ring_skin_0_fixed_joint: type fixed, parent r_hand_ring_2, child r_hand_ring_skin_0, origin xyz=6.369438959753088e-07 -0.0024437159778973594 -0.021405514485143107 rpy=-1.8198440874177978e-06 1.222171074662119 -1.570798078779304
- added joint r_hand_ring_skin_10_fixed_joint: type fixed, parent r_hand_ring_2, child r_hand_ring_skin_10, origin xyz=-0.0032993838888264685 -0.00409348890113434 -0.02776568877248392 rpy=-3.1415881649812016 1.5050938361710562 1.5708006164943
- added joint r_hand_ring_skin_11_fixed_joint: type fixed, parent r_hand_ring_2, child r_hand_ring_skin_11, origin xyz=-0.0032994485112988765 -0.0031417855839680486 -0.02327979056232371 rpy=-8.828925104148836e-07 1.2197920927650072 -1.5707973488537736
- added joint r_hand_ring_skin_1_fixed_joint: type fixed, parent r_hand_ring_2, child r_hand_ring_skin_1, origin xyz=0.003300577895109416 -0.0031419827756992147 -0.023279866908672953 rpy=-8.828925104148836e-07 1.2197920927650072 -1.5707973488537736
- added joint r_hand_ring_skin_2_fixed_joint: type fixed, parent r_hand_ring_2, child r_hand_ring_skin_2, origin xyz=6.542383091199394e-07 -0.003769121754147453 -0.02519099159351179 rpy=-2.1979342417368875e-06 1.3054216764415913 -1.5707985350956188
- added joint r_hand_ring_skin_3_fixed_joint: type fixed, parent r_hand_ring_2, child r_hand_ring_skin_3, origin xyz=0.0033005451413349873 -0.00409366356087959 -0.027765768308842753 rpy=-3.1415881649812016 1.5050938361710562 1.5708006164943
- added joint r_hand_ring_skin_4_fixed_joint: type fixed, parent r_hand_ring_2, child r_hand_ring_skin_4, origin xyz=0.005930120746728084 -0.0012042766764265855 -0.02799917777196037 rpy=-3.1404875010050004 1.2995572108592925 2.778219856114847
- added joint r_hand_ring_skin_5_fixed_joint: type fixed, parent r_hand_ring_2, child r_hand_ring_skin_5, origin xyz=5.308718775357685e-07 -0.0034891781806687394 -0.02983370559185905 rpy=-3.141591609794059 1.0865431510862156 1.5707972515436073
- added joint r_hand_ring_skin_6_fixed_joint: type fixed, parent r_hand_ring_2, child r_hand_ring_skin_6, origin xyz=0.0033005698496152962 -0.0018374330365136249 -0.03177047454405013 rpy=-3.1412265136676125 0.7787173410213876 2.5326427664034585
- added joint r_hand_ring_skin_7_fixed_joint: type fixed, parent r_hand_ring_2, child r_hand_ring_skin_7, origin xyz=6.201472224371535e-07 -0.0002860438799534015 -0.03327122378579056 rpy=-3.1415918554197564 0.6187360445083335 1.5713172257908574
- added joint r_hand_ring_skin_8_fixed_joint: type fixed, parent r_hand_ring_2, child r_hand_ring_skin_8, origin xyz=-0.0032993851081752224 -0.0018375074923376311 -0.03177136313433143 rpy=3.1412269734474307 0.7787178284081474 0.608949710350258
- added joint r_hand_ring_skin_9_fixed_joint: type fixed, parent r_hand_ring_2, child r_hand_ring_skin_9, origin xyz=-0.0059288844459949135 -0.00120401327023123 -0.02799875399568963 rpy=3.140488583833023 1.2995578078276662 0.3633736430221612
- added joint r_hand_thumb_skin_0_fixed_joint: type fixed, parent r_hand_thumb_3, child r_hand_thumb_skin_0, origin xyz=0.020306533907145166 -0.0024343057730962236 1.0397284419816355e-06 rpy=1.5707964766707783 0 -0.3483080823075038
- added joint r_hand_thumb_skin_10_fixed_joint: type fixed, parent r_hand_thumb_3, child r_hand_thumb_skin_10, origin xyz=0.026667227780490785 -0.004082576521223208 -0.0032996392911617267 rpy=1.5707959455998035 0 0.06601999324156192
- added joint r_hand_thumb_skin_11_fixed_joint: type fixed, parent r_hand_thumb_3, child r_hand_thumb_skin_11, origin xyz=0.022181444849985063 -0.003131515879897573 -0.0033000354029952272 rpy=1.5707959518025376 -2.240241662176975e-07 -0.35068660322761297
- added joint r_hand_thumb_skin_1_fixed_joint: type fixed, parent r_hand_thumb_3, child r_hand_thumb_skin_1, origin xyz=0.022181514608171235 -0.0031315753693715864 0.0033003779167594116 rpy=1.5707959518025376 -2.240241662176975e-07 -0.35068660322761297
- added joint r_hand_thumb_skin_2_fixed_joint: type fixed, parent r_hand_thumb_3, child r_hand_thumb_skin_2, origin xyz=0.024092766105114335 -0.003758664710135945 0 rpy=1.5707964275257265 -1.835551116380351e-07 -0.2650566454956479
- added joint r_hand_thumb_skin_3_fixed_joint: type fixed, parent r_hand_thumb_3, child r_hand_thumb_skin_3, origin xyz=0.026667717702939006 -0.004082289625380764 0.0032999352919206304 rpy=1.5707959455998035 0 0.06601999324156192
- added joint r_hand_thumb_skin_4_fixed_joint: type fixed, parent r_hand_thumb_3, child r_hand_thumb_skin_4, origin xyz=0.02690063775813216 -0.001192766703610404 0.00592978690987403 rpy=0.3770235759970468 0.2531253892798945 0.09883876086864818
- added joint r_hand_thumb_skin_5_fixed_joint: type fixed, parent r_hand_thumb_3, child r_hand_thumb_skin_5, origin xyz=0.02873547899028915 -0.0034768652666125888 3.412859334861462e-07 rpy=1.5707964228187474 -1.5765261132672026e-07 0.48457061294039566
- added joint r_hand_thumb_skin_6_fixed_joint: type fixed, parent r_hand_thumb_3, child r_hand_thumb_skin_6, origin xyz=0.030671760207808 -0.0018250312131609936 0.0033002175421802393 rpy=0.7821848393014904 0.6234818225335702 0.5256775270061106
- added joint r_hand_thumb_skin_7_fixed_joint: type fixed, parent r_hand_thumb_3, child r_hand_thumb_skin_7, origin xyz=0.03217216338109173 -0.000273117886959634 0 rpy=1.5704937922637117 0.00042413338882563444 0.952377708566445
- added joint r_hand_thumb_skin_8_fixed_joint: type fixed, parent r_hand_thumb_3, child r_hand_thumb_skin_8, origin xyz=0.030672481980215036 -0.0018246596063155873 -0.003299670361485485 rpy=2.359407636424222 -0.6234822954061497 0.5256775552228076
- added joint r_hand_thumb_skin_9_fixed_joint: type fixed, parent r_hand_thumb_3, child r_hand_thumb_skin_9, origin xyz=0.026900216455781042 -0.0011927826587152801 -0.005928741363999179 rpy=2.764568142309075 -0.25312574742097016 0.09883922008926718
- joint r_hip_roll: limit lower=-0.610865 upper=1.9547687622336491 effort=50000 velocity=120.0 -> lower=-0.6108652381980153 upper=1.9547687622336491 effort=50000 velocity=120.0
