Commit message: Reverted content of file

File: urdf/ergoCub/robots/ergoCubGazeboV1/model.urdf (robot description, URDF)
Before this commit: robot ergoCub, 193 links, 192 joints
Links:
- link chest: geometry collision mesh filename=package://ergoCub/meshes/simmechanics/sim_ecub_chest_prt.stl scale=0.001 0.001 0.001; visual mesh filename=package://ergoCub/meshes/simmechanics/sim_ecub_chest_prt.stl scale=0.001 0.001 0.001
- link head: geometry collision mesh filename=package://ergoCub/meshes/simmechanics/sim_ecub_head_prt.stl scale=0.001 0.001 0.001; visual mesh filename=package://ergoCub/meshes/simmechanics/sim_ecub_head_prt.stl scale=0.001 0.001 0.001
- link l_ankle_1: geometry collision mesh filename=package://ergoCub/meshes/simmechanics/sim_ecub_l_ankle_1_pr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 scale=0.001 0.001 0.001; visual mesh filename=package://ergoCub/meshes/simmechanics/sim_ecub_l_ankle_1_pr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 scale=0.001 0.001 0.001
- link l_ankle_2: geometry collision mesh filename=package://ergoCub/meshes/simmechanics/sim_ecub_l_ankle_2_pr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 scale=0.001 0.001 0.001; visual mesh filename=package://ergoCub/meshes/simmechanics/sim_ecub_l_ankle_2_pr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 scale=0.001 0.001 0.001
- link l_forearm: geometry collision mesh filename=package://ergoCub/meshes/simmechanics/sim_ecub_l_forearm_pr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 scale=0.001 0.001 0.001; visual mesh filename=package://ergoCub/meshes/simmechanics/sim_ecub_l_forearm_pr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 scale=0.001 0.001 0.001
- link l_hand_index_1: geometry collision mesh filename=package://ergoCub/meshes/simmechanics/sim_ecub_l_hand_index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 scale=0.001 0.001 0.001; visual mesh filename=package://ergoCub/meshes/simmechanics/sim_ecub_l_hand_index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 scale=0.001 0.001 0.001
- link l_hand_index_2: geometry collision mesh filename=package://ergoCub/meshes/simmechanics/sim_ecub_l_hand_index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 scale=0.001 0.001 0.001; visual mesh filename=package://ergoCub/meshes/simmechanics/sim_ecub_l_hand_index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 scale=0.001 0.001 0.001
- link l_hand_index_3: geometry collision mesh filename=package://ergoCub/meshes/simmechanics/sim_ecub_l_hand_index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 scale=0.001 0.001 0.001; visual mesh filename=package://ergoCub/meshes/simmechanics/sim_ecub_l_hand_index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 scale=0.001 0.001 0.001
- link l_hand_middle_1: geometry collision mesh filename=package://ergoCub/meshes/simmechanics/sim_ecub_l_hand_middl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 scale=0.001 0.001 0.001; visual mesh filename=package://ergoCub/meshes/simmechanics/sim_ecub_l_hand_middl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 scale=0.001 0.001 0.001
- link l_hand_middle_2: geometry collision mesh filename=package://ergoCub/meshes/simmechanics/sim_ecub_l_hand_middl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 scale=0.001 0.001 0.001; visual mesh filename=package://ergoCub/meshes/simmechanics/sim_ecub_l_hand_middl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 scale=0.001 0.001 0.001
- link l_hand_palm: geometry collision mesh filename=package://ergoCub/meshes/simmechanics/sim_ecub_l_hand_palm_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 scale=0.001 0.001 0.001; visual mesh filename=package://ergoCub/meshes/simmechanics/sim_ecub_l_hand_palm_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 scale=0.001 0.001 0.001
- link l_hand_pinkie_1: geometry collision mesh filename=package://ergoCub/meshes/simmechanics/sim_ecub_l_hand_pinki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 scale=0.001 0.001 0.001; visual mesh filename=package://ergoCub/meshes/simmechanics/sim_ecub_l_hand_pinki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 scale=0.001 0.001 0.001
- link l_hand_pinkie_2: geometry collision mesh filename=package://ergoCub/meshes/simmechanics/sim_ecub_l_hand_pinki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 scale=0.001 0.001 0.001; visual mesh filename=package://ergoCub/meshes/simmechanics/sim_ecub_l_hand_pinki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 scale=0.001 0.001 0.001
- link l_hand_ring_1: geometry collision mesh filename=package://ergoCub/meshes/simmechanics/sim_ecub_l_hand_ring_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 scale=0.001 0.001 0.001; visual mesh filename=package://ergoCub/meshes/simmechanics/sim_ecub_l_hand_ring_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 scale=0.001 0.001 0.001
- link l_hand_ring_2: geometry collision mesh filename=package://ergoCub/meshes/simmechanics/sim_ecub_l_hand_ring_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 scale=0.001 0.001 0.001; visual mesh filename=package://ergoCub/meshes/simmechanics/sim_ecub_l_hand_ring_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 scale=0.001 0.001 0.001
- link l_hand_thumb_1: geometry collision mesh filename=package://ergoCub/meshes/simmechanics/sim_ecub_l_hand_thumb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 scale=0.001 0.001 0.001; visual mesh filename=package://ergoCub/meshes/simmechanics/sim_ecub_l_hand_thumb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 scale=0.001 0.001 0.001
- link l_hand_thumb_2: geometry collision mesh filename=package://ergoCub/meshes/simmechanics/sim_ecub_l_hand_thumb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 scale=0.001 0.001 0.001; visual mesh filename=package://ergoCub/meshes/simmechanics/sim_ecub_l_hand_thumb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 scale=0.001 0.001 0.001
- link l_hand_thumb_3: geometry collision mesh filename=package://ergoCub/meshes/simmechanics/sim_ecub_l_hand_thumb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 scale=0.001 0.001 0.001; visual mesh filename=package://ergoCub/meshes/simmechanics/sim_ecub_l_hand_thumb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 scale=0.001 0.001 0.001
- link l_hip_1: geometry collision mesh filename=package://ergoCub/meshes/simmechanics/sim_ecub_l_hip_1_prt.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 scale=0.001 0.001 0.001; visual mesh filename=package://ergoCub/meshes/simmechanics/sim_ecub_l_hip_1_prt.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 scale=0.001 0.001 0.001
- link l_hip_2: geometry collision mesh filename=package://ergoCub/meshes/simmechanics/sim_ecub_l_hip_2_prt.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 scale=0.001 0.001 0.001; visual mesh filename=package://ergoCub/meshes/simmechanics/sim_ecub_l_hip_2_prt.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 scale=0.001 0.001 0.001
- link l_hip_3: geometry collision mesh filename=package://ergoCub/meshes/simmechanics/sim_ecub_l_hip_3_prt.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 scale=0.001 0.001 0.001; visual mesh filename=package://ergoCub/meshes/simmechanics/sim_ecub_l_hip_3_prt.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 scale=0.001 0.001 0.001
- link l_lower_leg: geometry collision mesh filename=package://ergoCub/meshes/simmechanics/sim_ecub_l_lower_leg_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 scale=0.001 0.001 0.001; visual mesh filename=package://ergoCub/meshes/simmechanics/sim_ecub_l_lower_leg_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 scale=0.001 0.001 0.001
- link l_shoulder_1: geometry collision mesh filename=package://ergoCub/meshes/simmechanics/sim_ecub_l_shoulder_1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 scale=0.001 0.001 0.001; visual mesh filename=package://ergoCub/meshes/simmechanics/sim_ecub_l_shoulder_1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 scale=0.001 0.001 0.001
- link l_shoulder_2: geometry collision mesh filename=package://ergoCub/meshes/simmechanics/sim_ecub_l_shoulder_2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 scale=0.001 0.001 0.001; visual mesh filename=package://ergoCub/meshes/simmechanics/sim_ecub_l_shoulder_2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 scale=0.001 0.001 0.001
- link l_shoulder_3: geometry collision mesh filename=package://ergoCub/meshes/simmechanics/sim_ecub_l_shoulder_3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 scale=0.001 0.001 0.001; visual mesh filename=package://ergoCub/meshes/simmechanics/sim_ecub_l_shoulder_3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 scale=0.001 0.001 0.001
- link l_upper_leg: geometry collision mesh filename=package://ergoCub/meshes/simmechanics/sim_ecub_l_upper_leg_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 scale=0.001 0.001 0.001; visual mesh filename=package://ergoCub/meshes/simmechanics/sim_ecub_l_upper_leg_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 scale=0.001 0.001 0.001
- link l_upperarm: geometry collision mesh filename=package://ergoCub/meshes/simmechanics/sim_ecub_l_upperarm_p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 scale=0.001 0.001 0.001; visual mesh filename=package://ergoCub/meshes/simmechanics/sim_ecub_l_upperarm_p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 scale=0.001 0.001 0.001
- link l_wrist_1: geometry collision mesh filename=package://ergoCub/meshes/simmechanics/sim_ecub_l_wrist_1_pr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 scale=0.001 0.001 0.001; visual mesh filename=package://ergoCub/meshes/simmechanics/sim_ecub_l_wrist_1_pr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 scale=0.001 0.001 0.001
- link l_wrist_2: geometry collision mesh filename=package://ergoCub/meshes/simmechanics/sim_ecub_l_wrist_2_pr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 scale=0.001 0.001 0.001; visual mesh filename=package://ergoCub/meshes/simmechanics/sim_ecub_l_wrist_2_pr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 scale=0.001 0.001 0.001
- link neck_2: geometry collision mesh filename=package://ergoCub/meshes/simmechanics/sim_ecub_head_neck_2_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 scale=0.001 0.001 0.001; visual mesh filename=package://ergoCub/meshes/simmechanics/sim_ecub_head_neck_2_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 scale=0.001 0.001 0.001
- link neck_3: geometry collision mesh filename=package://ergoCub/meshes/simmechanics/sim_ecub_head_neck_3_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 scale=0.001 0.001 0.001; visual mesh filename=package://ergoCub/meshes/simmechanics/sim_ecub_head_neck_3_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 scale=0.001 0.001 0.001
- link r_ankle_1: geometry collision mesh filename=package://ergoCub/meshes/simmechanics/sim_ecub_r_ankle_1_pr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 scale=0.001 0.001 0.001; visual mesh filename=package://ergoCub/meshes/simmechanics/sim_ecub_r_ankle_1_pr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 scale=0.001 0.001 0.001
- link r_ankle_2: geometry collision mesh filename=package://ergoCub/meshes/simmechanics/sim_ecub_r_ankle_2_pr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 scale=0.001 0.001 0.001; visual mesh filename=package://ergoCub/meshes/simmechanics/sim_ecub_r_ankle_2_pr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 scale=0.001 0.001 0.001
- link r_forearm: geometry collision mesh filename=package://ergoCub/meshes/simmechanics/sim_ecub_r_forearm_pr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 scale=0.001 0.001 0.001; visual mesh filename=package://ergoCub/meshes/simmechanics/sim_ecub_r_forearm_pr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 scale=0.001 0.001 0.001
- link r_hand_index_1: geometry collision mesh filename=package://ergoCub/meshes/simmechanics/sim_ecub_r_hand_index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 scale=0.001 0.001 0.001; visual mesh filename=package://ergoCub/meshes/simmechanics/sim_ecub_r_hand_index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 scale=0.001 0.001 0.001
- link r_hand_index_2: geometry collision mesh filename=package://ergoCub/meshes/simmechanics/sim_ecub_r_hand_index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 scale=0.001 0.001 0.001; visual mesh filename=package://ergoCub/meshes/simmechanics/sim_ecub_r_hand_index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 scale=0.001 0.001 0.001
- link r_hand_index_3: geometry collision mesh filename=package://ergoCub/meshes/simmechanics/sim_ecub_r_hand_index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 scale=0.001 0.001 0.001; visual mesh filename=package://ergoCub/meshes/simmechanics/sim_ecub_r_hand_index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 scale=0.001 0.001 0.001
- link r_hand_middle_1: geometry collision mesh filename=package://ergoCub/meshes/simmechanics/sim_ecub_r_hand_middl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 scale=0.001 0.001 0.001; visual mesh filename=package://ergoCub/meshes/simmechanics/sim_ecub_r_hand_middl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 scale=0.001 0.001 0.001
- link r_hand_middle_2: geometry collision mesh filename=package://ergoCub/meshes/simmechanics/sim_ecub_r_hand_middl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 scale=0.001 0.001 0.001; visual mesh filename=package://ergoCub/meshes/simmechanics/sim_ecub_r_hand_middl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 scale=0.001 0.001 0.001
- link r_hand_palm: geometry collision mesh filename=package://ergoCub/meshes/simmechanics/sim_ecub_r_hand_palm_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 scale=0.001 0.001 0.001; visual mesh filename=package://ergoCub/meshes/simmechanics/sim_ecub_r_hand_palm_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 scale=0.001 0.001 0.001
- link r_hand_pinkie_1: geometry collision mesh filename=package://ergoCub/meshes/simmechanics/sim_ecub_r_hand_pinki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 scale=0.001 0.001 0.001; visual mesh filename=package://ergoCub/meshes/simmechanics/sim_ecub_r_hand_pinki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 scale=0.001 0.001 0.001
- link r_hand_pinkie_2: geometry collision mesh filename=package://ergoCub/meshes/simmechanics/sim_ecub_r_hand_pinki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 scale=0.001 0.001 0.001; visual mesh filename=package://ergoCub/meshes/simmechanics/sim_ecub_r_hand_pinki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 scale=0.001 0.001 0.001
- link r_hand_ring_1: geometry collision mesh filename=package://ergoCub/meshes/simmechanics/sim_ecub_r_hand_ring_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 scale=0.001 0.001 0.001; visual mesh filename=package://ergoCub/meshes/simmechanics/sim_ecub_r_hand_ring_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 scale=0.001 0.001 0.001
- link r_hand_ring_2: geometry collision mesh filename=package://ergoCub/meshes/simmechanics/sim_ecub_r_hand_ring_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 scale=0.001 0.001 0.001; visual mesh filename=package://ergoCub/meshes/simmechanics/sim_ecub_r_hand_ring_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 scale=0.001 0.001 0.001
- link r_hand_thumb_1: geometry collision mesh filename=package://ergoCub/meshes/simmechanics/sim_ecub_r_hand_thumb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 scale=0.001 0.001 0.001; visual mesh filename=package://ergoCub/meshes/simmechanics/sim_ecub_r_hand_thumb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 scale=0.001 0.001 0.001
- link r_hand_thumb_2: geometry collision mesh filename=package://ergoCub/meshes/simmechanics/sim_ecub_r_hand_thumb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 scale=0.001 0.001 0.001; visual mesh filename=package://ergoCub/meshes/simmechanics/sim_ecub_r_hand_thumb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 scale=0.001 0.001 0.001
- link r_hand_thumb_3: geometry collision mesh filename=package://ergoCub/meshes/simmechanics/sim_ecub_r_hand_thumb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 scale=0.001 0.001 0.001; visual mesh filename=package://ergoCub/meshes/simmechanics/sim_ecub_r_hand_thumb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 scale=0.001 0.001 0.001
- link r_hip_1: geometry collision mesh filename=package://ergoCub/meshes/simmechanics/sim_ecub_r_hip_1_prt.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 scale=0.001 0.001 0.001; visual mesh filename=package://ergoCub/meshes/simmechanics/sim_ecub_r_hip_1_prt.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 scale=0.001 0.001 0.001
- link r_hip_2: geometry collision mesh filename=package://ergoCub/meshes/simmechanics/sim_ecub_r_hip_2_prt.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 scale=0.001 0.001 0.001; visual mesh filename=package://ergoCub/meshes/simmechanics/sim_ecub_r_hip_2_prt.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 scale=0.001 0.001 0.001
- link r_hip_3: geometry collision mesh filename=package://ergoCub/meshes/simmechanics/sim_ecub_r_hip_3_prt.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 scale=0.001 0.001 0.001; visual mesh filename=package://ergoCub/meshes/simmechanics/sim_ecub_r_hip_3_prt.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 scale=0.001 0.001 0.001
- link r_lower_leg: geometry collision mesh filename=package://ergoCub/meshes/simmechanics/sim_ecub_r_lower_leg_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 scale=0.001 0.001 0.001; visual mesh filename=package://ergoCub/meshes/simmechanics/sim_ecub_r_lower_leg_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 scale=0.001 0.001 0.001
- link r_shoulder_1: geometry collision mesh filename=package://ergoCub/meshes/simmechanics/sim_ecub_r_shoulder_1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 scale=0.001 0.001 0.001; visual mesh filename=package://ergoCub/meshes/simmechanics/sim_ecub_r_shoulder_1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 scale=0.001 0.001 0.001
- link r_shoulder_2: geometry collision mesh filename=package://ergoCub/meshes/simmechanics/sim_ecub_r_shoulder_2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 scale=0.001 0.001 0.001; visual mesh filename=package://ergoCub/meshes/simmechanics/sim_ecub_r_shoulder_2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 scale=0.001 0.001 0.001
- link r_shoulder_3: geometry collision mesh filename=package://ergoCub/meshes/simmechanics/sim_ecub_r_shoulder_3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 scale=0.001 0.001 0.001; visual mesh filename=package://ergoCub/meshes/simmechanics/sim_ecub_r_shoulder_3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 scale=0.001 0.001 0.001
- link r_upper_leg: geometry collision mesh filename=package://ergoCub/meshes/simmechanics/sim_ecub_r_upper_leg_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 scale=0.001 0.001 0.001; visual mesh filename=package://ergoCub/meshes/simmechanics/sim_ecub_r_upper_leg_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 scale=0.001 0.001 0.001
- link r_upperarm: geometry collision mesh filename=package://ergoCub/meshes/simmechanics/sim_ecub_r_upperarm_p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 scale=0.001 0.001 0.001; visual mesh filename=package://ergoCub/meshes/simmechanics/sim_ecub_r_upperarm_p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 scale=0.001 0.001 0.001
- link r_wrist_1: geometry collision mesh filename=package://ergoCub/meshes/simmechanics/sim_ecub_r_wrist_1_pr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 scale=0.001 0.001 0.001; visual mesh filename=package://ergoCub/meshes/simmechanics/sim_ecub_r_wrist_1_pr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 scale=0.001 0.001 0.001
- link r_wrist_2: geometry collision mesh filename=package://ergoCub/meshes/simmechanics/sim_ecub_r_wrist_2_pr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 scale=0.001 0.001 0.001; visual mesh filename=package://ergoCub/meshes/simmechanics/sim_ecub_r_wrist_2_pr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 scale=0.001 0.001 0.001
- link realsense: geometry collision mesh filename=package://ergoCub/meshes/simmechanics/sim_ecub_realsense_pr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 scale=0.001 0.001 0.001; visual mesh filename=package://ergoCub/meshes/simmechanics/sim_ecub_realsense_pr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 scale=0.001 0.001 0.001
- link root_link: geometry collision mesh filename=package://ergoCub/meshes/simmechanics/sim_ecub_root_link_pr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 scale=0.001 0.001 0.001; visual mesh filename=package://ergoCub/meshes/simmechanics/sim_ecub_root_link_pr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 scale=0.001 0.001 0.001
- link torso_1: geometry collision mesh filename=package://ergoCub/meshes/simmechanics/sim_ecub_torso_1_prt.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 scale=0.001 0.001 0.001; visual mesh filename=package://ergoCub/meshes/simmechanics/sim_ecub_torso_1_prt.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 scale=0.001 0.001 0.001
- link torso_2: geometry collision mesh filename=package://ergoCub/meshes/simmechanics/sim_ecub_torso_2_prt.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 scale=0.001 0.001 0.001; visual mesh filename=package://ergoCub/meshes/simmechanics/sim_ecub_torso_2_prt.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 scale=0.001 0.001 0.001

Commit message: Add waist_imu in urdf file

File: urdf/ergoCub/robots/ergoCubGazeboV1/model.urdf (robot description, URDF)
Before this commit: robot ergoCub, 193 links, 192 joints
Links:
- added link waist_imu_0
- link torso_1: mass 2.01685 -> 2.0645667
Joints:
- added joint waist_imu_0_fixed_joint: type fixed, parent torso_1, child waist_imu_0, origin xyz=0.0354497 0.00639688 0.060600 rpy=-1.5707322 1.5707963 0

File: urdf/ergoCub/robots/ergoCubGazeboV1_minContacts/model.urdf (robot description, URDF)
Before this commit: robot ergoCub, 193 links, 192 joints
Links:
- added link waist_imu_0
- link torso_1: mass 2.01685 -> 2.0645667
Joints:
- added joint waist_imu_0_fixed_joint: type fixed, parent torso_1, child waist_imu_0, origin xyz=0.0354497 0.00639688 0.060600 rpy=-1.5707322 1.5707963 0

File: urdf/ergoCub/robots/ergoCubSN000/model.urdf (robot description, URDF)
Before this commit: robot ergoCub, 193 links, 192 joints
Links:
- added link waist_imu_0
- link torso_1: mass 2.01685 -> 2.0645667
Joints:
- added joint waist_imu_0_fixed_joint: type fixed, parent torso_1, child waist_imu_0, origin xyz=0.0354497 0.00639688 0.060600 rpy=-1.5707322 1.5707963 0

Commit message: Add the XMLBlobs, the assigned mass and inertia for waist_imu

File: urdf/ergoCub/robots/ergoCubGazeboV1/model.urdf (robot description, URDF)
Before this commit: robot ergoCub, 194 links, 193 joints
Links:
- removed link waist_imu_0
Joints:
- removed joint waist_imu_0_fixed_joint

File: urdf/ergoCub/robots/ergoCubGazeboV1_minContacts/model.urdf (robot description, URDF)
Before this commit: robot ergoCub, 194 links, 193 joints
Links:
- removed link waist_imu_0
Joints:
- removed joint waist_imu_0_fixed_joint

File: urdf/ergoCub/robots/ergoCubSN000/model.urdf (robot description, URDF)
Before this commit: robot ergoCub, 194 links, 193 joints
Links:
- removed link waist_imu_0
Joints:
- removed joint waist_imu_0_fixed_joint

Commit message: Remove changes made by hand from model.urdf

File: urdf/ergoCub/robots/ergoCubGazeboV1/model.urdf (robot description, URDF)
Before this commit: robot ergoCub, 193 links, 192 joints
Links:
- link torso_1: mass 2.0645667 -> 2.01685

File: urdf/ergoCub/robots/ergoCubGazeboV1_minContacts/model.urdf (robot description, URDF)
Before this commit: robot ergoCub, 193 links, 192 joints
Links:
- link torso_1: mass 2.0645667 -> 2.01685

File: urdf/ergoCub/robots/ergoCubSN000/model.urdf (robot description, URDF)
Before this commit: robot ergoCub, 193 links, 192 joints
Links:
- link torso_1: mass 2.0645667 -> 2.01685

Commit message: Automatic update of urdf

File: urdf/ergoCub/robots/ergoCubGazeboV1/model.urdf (robot description, URDF)
Before this commit: robot ergoCub, 194 links, 193 joints
Joints:
- joint torso_pitch: origin xyz=0 0 0.11800000000000005 rpy=0 0 0 -> xyz=0 0 0.11800000000000005 rpy=0 0.174533 0; type revolute -> fixed

File: urdf/ergoCub/robots/ergoCubGazeboV1_minContacts/model.urdf (robot description, URDF)
Before this commit: robot ergoCub, 194 links, 193 joints
Joints:
- joint torso_pitch: origin xyz=0 0 0.11800000000000005 rpy=0 0 0 -> xyz=0 0 0.11800000000000005 rpy=0 0.174533 0; type revolute -> fixed

File: urdf/ergoCub/robots/ergoCubSN000/model.urdf (robot description, URDF)
Before this commit: robot ergoCub, 194 links, 193 joints
Joints:
- joint torso_pitch: origin xyz=0 0 0.11800000000000005 rpy=0 0 0 -> xyz=0 0 0.11800000000000005 rpy=0 0.174533 0; type revolute -> fixed

Commit message: Automatic update of urdf

File: urdf/ergoCub/robots/ergoCubGazeboV1/model.urdf (robot description, URDF)
Before this commit: robot ergoCub, 194 links, 193 joints
Joints:
- joint waist_imu_0_fixed_joint: origin xyz=0.0354497 0.00639688 0.060600 rpy=-1.5707322 1.5707963 0 -> xyz=0.0354497 0.00639688 0.060600 rpy=-1.5708 0 1.5708

File: urdf/ergoCub/robots/ergoCubGazeboV1_minContacts/model.urdf (robot description, URDF)
Before this commit: robot ergoCub, 194 links, 193 joints
Joints:
- joint waist_imu_0_fixed_joint: origin xyz=0.0354497 0.00639688 0.060600 rpy=-1.5707322 1.5707963 0 -> xyz=0.0354497 0.00639688 0.060600 rpy=-1.5708 0 1.5708

File: urdf/ergoCub/robots/ergoCubSN000/model.urdf (robot description, URDF)
Before this commit: robot ergoCub, 194 links, 193 joints
Joints:
- joint waist_imu_0_fixed_joint: origin xyz=0.0354497 0.00639688 0.060600 rpy=-1.5707322 1.5707963 0 -> xyz=0.0354497 0.00639688 0.060600 rpy=-1.5708 0 1.5708
