Commit message: Automatic update of urdf

File: urdf/ergoCub/robots/ergoCubGazeboV1/model.urdf (robot description, URDF)
Before this commit: robot ergoCub, 194 links, 193 joints
Joints:
- joint l_index_add: limit lower=0.0 upper=0.3490658503988659 effort=50000 velocity=120.0 -> lower=0.0 upper=0.2617993877991494 effort=50000 velocity=100.0
- joint l_index_dist: limit lower=0.0 upper=2.792526803190927 effort=50000 velocity=120.0 -> lower=0.0 upper=1.7313666179783749 effort=50000 velocity=100.0
- joint l_index_prox: limit lower=0.0 upper=2.792526803190927 effort=50000 velocity=120.0 -> lower=0.0 upper=1.5707963267948966 effort=50000 velocity=100.0
- joint l_middle_dist: limit lower=0.0 upper=2.792526803190927 effort=50000 velocity=120.0 -> lower=0.0 upper=1.7313666179783749 effort=50000 velocity=100.0
- joint l_middle_prox: limit lower=0.0 upper=2.792526803190927 effort=50000 velocity=120.0 -> lower=0.0 upper=1.5707963267948966 effort=50000 velocity=100.0
- joint l_pinkie_dist: limit lower=0.0 upper=2.792526803190927 effort=50000 velocity=120.0 -> lower=0.0 upper=1.6283921921107094 effort=50000 velocity=100.0
- joint l_pinkie_prox: limit lower=0.0 upper=2.792526803190927 effort=50000 velocity=120.0 -> lower=0.0 upper=1.5707963267948966 effort=50000 velocity=100.0
- joint l_ring_dist: limit lower=0.0 upper=2.792526803190927 effort=50000 velocity=120.0 -> lower=0.0 upper=1.7313666179783749 effort=50000 velocity=100.0
- joint l_ring_prox: limit lower=0.0 upper=2.792526803190927 effort=50000 velocity=120.0 -> lower=0.0 upper=1.5707963267948966 effort=50000 velocity=100.0
- joint l_thumb_add: limit lower=0.0 upper=1.0471975511965976 effort=50000 velocity=120.0 -> lower=0.0 upper=1.5707963267948966 effort=50000 velocity=100.0
- joint l_thumb_dist: limit lower=0.0 upper=2.792526803190927 effort=50000 velocity=120.0 -> lower=0.0 upper=0.9354964790689606 effort=50000 velocity=120.0
- joint l_thumb_prox: limit lower=0.0 upper=2.792526803190927 effort=50000 velocity=120.0 -> lower=0.0 upper=1.4329153158873444 effort=50000 velocity=100.0
- joint r_index_add: limit lower=0.0 upper=0.3490658503988659 effort=50000 velocity=120.0 -> lower=0.0 upper=0.2617993877991494 effort=50000 velocity=100.0
- joint r_index_dist: limit lower=0.0 upper=2.792526803190927 effort=50000 velocity=120.0 -> lower=0.0 upper=1.7313666179783749 effort=50000 velocity=100.0
- joint r_index_prox: limit lower=0.0 upper=2.792526803190927 effort=50000 velocity=120.0 -> lower=0.0 upper=1.5707963267948966 effort=50000 velocity=100.0
- joint r_middle_dist: limit lower=0.0 upper=2.792526803190927 effort=50000 velocity=120.0 -> lower=0.0 upper=1.7313666179783749 effort=50000 velocity=100.0
- joint r_middle_prox: limit lower=0.0 upper=2.792526803190927 effort=50000 velocity=120.0 -> lower=0.0 upper=1.5707963267948966 effort=50000 velocity=100.0
- joint r_pinkie_dist: limit lower=0.0 upper=2.792526803190927 effort=50000 velocity=120.0 -> lower=0.0 upper=1.6283921921107094 effort=50000 velocity=100.0
- joint r_pinkie_prox: limit lower=0.0 upper=2.792526803190927 effort=50000 velocity=120.0 -> lower=0.0 upper=1.5707963267948966 effort=50000 velocity=100.0
- joint r_ring_dist: limit lower=0.0 upper=2.792526803190927 effort=50000 velocity=120.0 -> lower=0.0 upper=1.7313666179783749 effort=50000 velocity=100.0
- joint r_ring_prox: limit lower=0.0 upper=2.792526803190927 effort=50000 velocity=120.0 -> lower=0.0 upper=1.5707963267948966 effort=50000 velocity=100.0
- joint r_thumb_add: limit lower=0.0 upper=1.0471975511965976 effort=50000 velocity=120.0 -> lower=0.0 upper=1.5707963267948966 effort=50000 velocity=100.0
- joint r_thumb_dist: limit lower=0.0 upper=2.792526803190927 effort=50000 velocity=120.0 -> lower=0.0 upper=0.9354964790689606 effort=50000 velocity=120.0
- joint r_thumb_prox: limit lower=0.0 upper=2.792526803190927 effort=50000 velocity=120.0 -> lower=0.0 upper=1.4329153158873444 effort=50000 velocity=100.0

File: urdf/ergoCub/robots/ergoCubGazeboV1_minContacts/model.urdf (robot description, URDF)
Before this commit: robot ergoCub, 194 links, 193 joints
Joints:
- joint l_index_add: limit lower=0.0 upper=0.3490658503988659 effort=50000 velocity=120.0 -> lower=0.0 upper=0.2617993877991494 effort=50000 velocity=100.0
- joint l_index_dist: limit lower=0.0 upper=2.792526803190927 effort=50000 velocity=120.0 -> lower=0.0 upper=1.7313666179783749 effort=50000 velocity=100.0
- joint l_index_prox: limit lower=0.0 upper=2.792526803190927 effort=50000 velocity=120.0 -> lower=0.0 upper=1.5707963267948966 effort=50000 velocity=100.0
- joint l_middle_dist: limit lower=0.0 upper=2.792526803190927 effort=50000 velocity=120.0 -> lower=0.0 upper=1.7313666179783749 effort=50000 velocity=100.0
- joint l_middle_prox: limit lower=0.0 upper=2.792526803190927 effort=50000 velocity=120.0 -> lower=0.0 upper=1.5707963267948966 effort=50000 velocity=100.0
- joint l_pinkie_dist: limit lower=0.0 upper=2.792526803190927 effort=50000 velocity=120.0 -> lower=0.0 upper=1.6283921921107094 effort=50000 velocity=100.0
- joint l_pinkie_prox: limit lower=0.0 upper=2.792526803190927 effort=50000 velocity=120.0 -> lower=0.0 upper=1.5707963267948966 effort=50000 velocity=100.0
- joint l_ring_dist: limit lower=0.0 upper=2.792526803190927 effort=50000 velocity=120.0 -> lower=0.0 upper=1.7313666179783749 effort=50000 velocity=100.0
- joint l_ring_prox: limit lower=0.0 upper=2.792526803190927 effort=50000 velocity=120.0 -> lower=0.0 upper=1.5707963267948966 effort=50000 velocity=100.0
- joint l_thumb_add: limit lower=0.0 upper=1.0471975511965976 effort=50000 velocity=120.0 -> lower=0.0 upper=1.5707963267948966 effort=50000 velocity=100.0
- joint l_thumb_dist: limit lower=0.0 upper=2.792526803190927 effort=50000 velocity=120.0 -> lower=0.0 upper=0.9354964790689606 effort=50000 velocity=120.0
- joint l_thumb_prox: limit lower=0.0 upper=2.792526803190927 effort=50000 velocity=120.0 -> lower=0.0 upper=1.4329153158873444 effort=50000 velocity=100.0
- joint r_index_add: limit lower=0.0 upper=0.3490658503988659 effort=50000 velocity=120.0 -> lower=0.0 upper=0.2617993877991494 effort=50000 velocity=100.0
- joint r_index_dist: limit lower=0.0 upper=2.792526803190927 effort=50000 velocity=120.0 -> lower=0.0 upper=1.7313666179783749 effort=50000 velocity=100.0
- joint r_index_prox: limit lower=0.0 upper=2.792526803190927 effort=50000 velocity=120.0 -> lower=0.0 upper=1.5707963267948966 effort=50000 velocity=100.0
- joint r_middle_dist: limit lower=0.0 upper=2.792526803190927 effort=50000 velocity=120.0 -> lower=0.0 upper=1.7313666179783749 effort=50000 velocity=100.0
- joint r_middle_prox: limit lower=0.0 upper=2.792526803190927 effort=50000 velocity=120.0 -> lower=0.0 upper=1.5707963267948966 effort=50000 velocity=100.0
- joint r_pinkie_dist: limit lower=0.0 upper=2.792526803190927 effort=50000 velocity=120.0 -> lower=0.0 upper=1.6283921921107094 effort=50000 velocity=100.0
- joint r_pinkie_prox: limit lower=0.0 upper=2.792526803190927 effort=50000 velocity=120.0 -> lower=0.0 upper=1.5707963267948966 effort=50000 velocity=100.0
- joint r_ring_dist: limit lower=0.0 upper=2.792526803190927 effort=50000 velocity=120.0 -> lower=0.0 upper=1.7313666179783749 effort=50000 velocity=100.0
- joint r_ring_prox: limit lower=0.0 upper=2.792526803190927 effort=50000 velocity=120.0 -> lower=0.0 upper=1.5707963267948966 effort=50000 velocity=100.0
- joint r_thumb_add: limit lower=0.0 upper=1.0471975511965976 effort=50000 velocity=120.0 -> lower=0.0 upper=1.5707963267948966 effort=50000 velocity=100.0
- joint r_thumb_dist: limit lower=0.0 upper=2.792526803190927 effort=50000 velocity=120.0 -> lower=0.0 upper=0.9354964790689606 effort=50000 velocity=120.0
- joint r_thumb_prox: limit lower=0.0 upper=2.792526803190927 effort=50000 velocity=120.0 -> lower=0.0 upper=1.4329153158873444 effort=50000 velocity=100.0

File: urdf/ergoCub/robots/ergoCubSN000/model.urdf (robot description, URDF)
Before this commit: robot ergoCub, 194 links, 193 joints
Joints:
- joint l_index_add: limit lower=0.0 upper=0.3490658503988659 effort=50000 velocity=120.0 -> lower=0.0 upper=0.2617993877991494 effort=50000 velocity=100.0
- joint l_index_dist: limit lower=0.0 upper=2.792526803190927 effort=50000 velocity=120.0 -> lower=0.0 upper=1.7313666179783749 effort=50000 velocity=100.0
- joint l_index_prox: limit lower=0.0 upper=2.792526803190927 effort=50000 velocity=120.0 -> lower=0.0 upper=1.5707963267948966 effort=50000 velocity=100.0
- joint l_middle_dist: limit lower=0.0 upper=2.792526803190927 effort=50000 velocity=120.0 -> lower=0.0 upper=1.7313666179783749 effort=50000 velocity=100.0
- joint l_middle_prox: limit lower=0.0 upper=2.792526803190927 effort=50000 velocity=120.0 -> lower=0.0 upper=1.5707963267948966 effort=50000 velocity=100.0
- joint l_pinkie_dist: limit lower=0.0 upper=2.792526803190927 effort=50000 velocity=120.0 -> lower=0.0 upper=1.6283921921107094 effort=50000 velocity=100.0
- joint l_pinkie_prox: limit lower=0.0 upper=2.792526803190927 effort=50000 velocity=120.0 -> lower=0.0 upper=1.5707963267948966 effort=50000 velocity=100.0
- joint l_ring_dist: limit lower=0.0 upper=2.792526803190927 effort=50000 velocity=120.0 -> lower=0.0 upper=1.7313666179783749 effort=50000 velocity=100.0
- joint l_ring_prox: limit lower=0.0 upper=2.792526803190927 effort=50000 velocity=120.0 -> lower=0.0 upper=1.5707963267948966 effort=50000 velocity=100.0
- joint l_thumb_add: limit lower=0.0 upper=1.0471975511965976 effort=50000 velocity=120.0 -> lower=0.0 upper=1.5707963267948966 effort=50000 velocity=100.0
- joint l_thumb_dist: limit lower=0.0 upper=2.792526803190927 effort=50000 velocity=120.0 -> lower=0.0 upper=0.9354964790689606 effort=50000 velocity=120.0
- joint l_thumb_prox: limit lower=0.0 upper=2.792526803190927 effort=50000 velocity=120.0 -> lower=0.0 upper=1.4329153158873444 effort=50000 velocity=100.0
- joint r_index_add: limit lower=0.0 upper=0.3490658503988659 effort=50000 velocity=120.0 -> lower=0.0 upper=0.2617993877991494 effort=50000 velocity=100.0
- joint r_index_dist: limit lower=0.0 upper=2.792526803190927 effort=50000 velocity=120.0 -> lower=0.0 upper=1.7313666179783749 effort=50000 velocity=100.0
- joint r_index_prox: limit lower=0.0 upper=2.792526803190927 effort=50000 velocity=120.0 -> lower=0.0 upper=1.5707963267948966 effort=50000 velocity=100.0
- joint r_middle_dist: limit lower=0.0 upper=2.792526803190927 effort=50000 velocity=120.0 -> lower=0.0 upper=1.7313666179783749 effort=50000 velocity=100.0
- joint r_middle_prox: limit lower=0.0 upper=2.792526803190927 effort=50000 velocity=120.0 -> lower=0.0 upper=1.5707963267948966 effort=50000 velocity=100.0
- joint r_pinkie_dist: limit lower=0.0 upper=2.792526803190927 effort=50000 velocity=120.0 -> lower=0.0 upper=1.6283921921107094 effort=50000 velocity=100.0
- joint r_pinkie_prox: limit lower=0.0 upper=2.792526803190927 effort=50000 velocity=120.0 -> lower=0.0 upper=1.5707963267948966 effort=50000 velocity=100.0
- joint r_ring_dist: limit lower=0.0 upper=2.792526803190927 effort=50000 velocity=120.0 -> lower=0.0 upper=1.7313666179783749 effort=50000 velocity=100.0
- joint r_ring_prox: limit lower=0.0 upper=2.792526803190927 effort=50000 velocity=120.0 -> lower=0.0 upper=1.5707963267948966 effort=50000 velocity=100.0
- joint r_thumb_add: limit lower=0.0 upper=1.0471975511965976 effort=50000 velocity=120.0 -> lower=0.0 upper=1.5707963267948966 effort=50000 velocity=100.0
- joint r_thumb_dist: limit lower=0.0 upper=2.792526803190927 effort=50000 velocity=120.0 -> lower=0.0 upper=0.9354964790689606 effort=50000 velocity=120.0
- joint r_thumb_prox: limit lower=0.0 upper=2.792526803190927 effort=50000 velocity=120.0 -> lower=0.0 upper=1.4329153158873444 effort=50000 velocity=100.0

Commit message: Automatic update of urdf

File: urdf/ergoCub/robots/ergoCubGazeboV1/model.urdf (robot description, URDF)
Before this commit: robot ergoCub, 194 links, 193 joints
Joints:
- joint waist_imu_0_fixed_joint: origin xyz=0.0354497 0.00639688 0.060600 rpy=-1.5708 0 1.5708 -> xyz=0.0354497 0.00639688 0.060600 rpy=1.5708 0 -1.5708

File: urdf/ergoCub/robots/ergoCubGazeboV1_minContacts/model.urdf (robot description, URDF)
Before this commit: robot ergoCub, 194 links, 193 joints
Joints:
- joint waist_imu_0_fixed_joint: origin xyz=0.0354497 0.00639688 0.060600 rpy=-1.5708 0 1.5708 -> xyz=0.0354497 0.00639688 0.060600 rpy=1.5708 0 -1.5708

File: urdf/ergoCub/robots/ergoCubSN000/model.urdf (robot description, URDF)
Before this commit: robot ergoCub, 194 links, 193 joints
Joints:
- joint waist_imu_0_fixed_joint: origin xyz=0.0354497 0.00639688 0.060600 rpy=-1.5708 0 1.5708 -> xyz=0.0354497 0.00639688 0.060600 rpy=1.5708 0 -1.5708

Commit message: Automatic update of urdf

File: urdf/ergoCub/robots/ergoCubGazeboV1/model.urdf (robot description, URDF)
Before this commit: robot ergoCub, 194 links, 193 joints
Joints:
- joint head_laser_frame_fixed_joint: origin xyz=4.99999999999997e-05 0 0.13480199999999992 rpy=0 0 1.5707963267948966 -> xyz=4.99999999999997e-05 0 0.13480199999999992 rpy=0 0 -3.6732051038684165e-06

File: urdf/ergoCub/robots/ergoCubGazeboV1_minContacts/model.urdf (robot description, URDF)
Before this commit: robot ergoCub, 194 links, 193 joints
Joints:
- joint head_laser_frame_fixed_joint: origin xyz=4.99999999999997e-05 0 0.13480199999999992 rpy=0 0 1.5707963267948966 -> xyz=4.99999999999997e-05 0 0.13480199999999992 rpy=0 0 -3.6732051038684165e-06

File: urdf/ergoCub/robots/ergoCubSN000/model.urdf (robot description, URDF)
Before this commit: robot ergoCub, 194 links, 193 joints
Joints:
- joint head_laser_frame_fixed_joint: origin xyz=4.99999999999997e-05 0 0.13480199999999992 rpy=0 0 1.5707963267948966 -> xyz=4.99999999999997e-05 0 0.13480199999999992 rpy=0 0 -3.6732051038684165e-06

Commit message: Automatic update of urdf

File: urdf/ergoCub/robots/ergoCubGazeboV1/model.urdf (robot description, URDF)
Before this commit: robot ergoCub, 194 links, 193 joints
Joints:
- joint l_hip_pitch: limit lower=-0.7853981633974483 upper=2.007128639793479 effort=50000 velocity=120.0 -> lower=-0.7504915783575618 upper=1.7976891295541595 effort=50000 velocity=120.0
- joint l_hip_roll: limit lower=-0.6108652381980153 upper=1.9547687622336491 effort=50000 velocity=120.0 -> lower=-0.2792526803190927 upper=1.9024088846738192 effort=50000 velocity=120.0
- joint l_hip_yaw: limit lower=-1.3962634015954636 upper=1.3962634015954636 effort=50000 velocity=120.0 -> lower=-1.3788101090755203 upper=1.3788101090755203 effort=50000 velocity=120.0
- joint l_knee: limit lower=-1.2217304763960306 upper=0.08726646259971647 effort=50000 velocity=120.0 -> lower=-1.8151424220741028 upper=0.10471975511965978 effort=50000 velocity=120.0
- joint r_hip_pitch: limit lower=-0.7853981633974483 upper=2.007128639793479 effort=50000 velocity=120.0 -> lower=-0.7504915783575618 upper=1.7976891295541595 effort=50000 velocity=120.0
- joint r_hip_roll: limit lower=-0.6108652381980153 upper=1.9547687622336491 effort=50000 velocity=120.0 -> lower=-0.2792526803190927 upper=1.9024088846738192 effort=50000 velocity=120.0
- joint r_hip_yaw: limit lower=-1.3962634015954636 upper=1.3962634015954636 effort=50000 velocity=120.0 -> lower=-1.3788101090755203 upper=1.3788101090755203 effort=50000 velocity=120.0
- joint r_knee: limit lower=-1.2217304763960306 upper=0.08726646259971647 effort=50000 velocity=120.0 -> lower=-1.8151424220741028 upper=0.10471975511965978 effort=50000 velocity=120.0

File: urdf/ergoCub/robots/ergoCubGazeboV1_minContacts/model.urdf (robot description, URDF)
Before this commit: robot ergoCub, 194 links, 193 joints
Joints:
- joint l_hip_pitch: limit lower=-0.7853981633974483 upper=2.007128639793479 effort=50000 velocity=120.0 -> lower=-0.7504915783575618 upper=1.7976891295541595 effort=50000 velocity=120.0
- joint l_hip_roll: limit lower=-0.6108652381980153 upper=1.9547687622336491 effort=50000 velocity=120.0 -> lower=-0.2792526803190927 upper=1.9024088846738192 effort=50000 velocity=120.0
- joint l_hip_yaw: limit lower=-1.3962634015954636 upper=1.3962634015954636 effort=50000 velocity=120.0 -> lower=-1.3788101090755203 upper=1.3788101090755203 effort=50000 velocity=120.0
- joint l_knee: limit lower=-1.2217304763960306 upper=0.08726646259971647 effort=50000 velocity=120.0 -> lower=-1.8151424220741028 upper=0.10471975511965978 effort=50000 velocity=120.0
- joint r_hip_pitch: limit lower=-0.7853981633974483 upper=2.007128639793479 effort=50000 velocity=120.0 -> lower=-0.7504915783575618 upper=1.7976891295541595 effort=50000 velocity=120.0
- joint r_hip_roll: limit lower=-0.6108652381980153 upper=1.9547687622336491 effort=50000 velocity=120.0 -> lower=-0.2792526803190927 upper=1.9024088846738192 effort=50000 velocity=120.0
- joint r_hip_yaw: limit lower=-1.3962634015954636 upper=1.3962634015954636 effort=50000 velocity=120.0 -> lower=-1.3788101090755203 upper=1.3788101090755203 effort=50000 velocity=120.0
- joint r_knee: limit lower=-1.2217304763960306 upper=0.08726646259971647 effort=50000 velocity=120.0 -> lower=-1.8151424220741028 upper=0.10471975511965978 effort=50000 velocity=120.0

File: urdf/ergoCub/robots/ergoCubSN000/model.urdf (robot description, URDF)
Before this commit: robot ergoCub, 194 links, 193 joints
Joints:
- joint l_hip_pitch: limit lower=-0.7853981633974483 upper=2.007128639793479 effort=50000 velocity=120.0 -> lower=-0.7504915783575618 upper=1.7976891295541595 effort=50000 velocity=120.0
- joint l_hip_roll: limit lower=-0.6108652381980153 upper=1.9547687622336491 effort=50000 velocity=120.0 -> lower=-0.2792526803190927 upper=1.9024088846738192 effort=50000 velocity=120.0
- joint l_hip_yaw: limit lower=-1.3962634015954636 upper=1.3962634015954636 effort=50000 velocity=120.0 -> lower=-1.3788101090755203 upper=1.3788101090755203 effort=50000 velocity=120.0
- joint l_knee: limit lower=-1.2217304763960306 upper=0.08726646259971647 effort=50000 velocity=120.0 -> lower=-1.8151424220741028 upper=0.10471975511965978 effort=50000 velocity=120.0
- joint r_hip_pitch: limit lower=-0.7853981633974483 upper=2.007128639793479 effort=50000 velocity=120.0 -> lower=-0.7504915783575618 upper=1.7976891295541595 effort=50000 velocity=120.0
- joint r_hip_roll: limit lower=-0.6108652381980153 upper=1.9547687622336491 effort=50000 velocity=120.0 -> lower=-0.2792526803190927 upper=1.9024088846738192 effort=50000 velocity=120.0
- joint r_hip_yaw: limit lower=-1.3962634015954636 upper=1.3962634015954636 effort=50000 velocity=120.0 -> lower=-1.3788101090755203 upper=1.3788101090755203 effort=50000 velocity=120.0
- joint r_knee: limit lower=-1.2217304763960306 upper=0.08726646259971647 effort=50000 velocity=120.0 -> lower=-1.8151424220741028 upper=0.10471975511965978 effort=50000 velocity=120.0

Commit message: Automatic update of urdf

File: urdf/ergoCub/robots/ergoCubGazeboV1/model.urdf (robot description, URDF)
Before this commit: robot ergoCub, 194 links, 193 joints
Joints:
- joint torso_pitch: origin xyz=0 0 0.11800000000000005 rpy=0 0.174533 0 -> xyz=0 0 0.11800000000000005 rpy=0 0 0; type fixed -> revolute

File: urdf/ergoCub/robots/ergoCubGazeboV1_minContacts/model.urdf (robot description, URDF)
Before this commit: robot ergoCub, 194 links, 193 joints
Joints:
- joint torso_pitch: origin xyz=0 0 0.11800000000000005 rpy=0 0.174533 0 -> xyz=0 0 0.11800000000000005 rpy=0 0 0; type fixed -> revolute

File: urdf/ergoCub/robots/ergoCubSN000/model.urdf (robot description, URDF)
Before this commit: robot ergoCub, 194 links, 193 joints
Joints:
- joint torso_pitch: origin xyz=0 0 0.11800000000000005 rpy=0 0.174533 0 -> xyz=0 0 0.11800000000000005 rpy=0 0 0; type fixed -> revolute
