Commit message: Automatic update of urdf

File: urdf/ergoCub/robots/ergoCubGazeboV1/model.urdf (robot description, URDF)
Before this commit: robot ergoCub, 194 links, 193 joints
Links:
- added link l_arm_ft
- added link l_foot_front_ft
- added link l_foot_rear_ft
- added link l_leg_ft
- added link r_arm_ft
- added link r_foot_front_ft
- added link r_foot_rear_ft
- added link r_leg_ft
Joints:
- added joint l_arm_ft_fixed_joint: type fixed, parent l_shoulder_2, child l_arm_ft, origin xyz=-0.004350065786786487 2.435985168580679e-07 -0.054299880148590496 rpy=-3.1415923328972943 0 -1.5707962214346844
- added joint l_foot_front_ft_fixed_joint: type fixed, parent l_ankle_2, child l_foot_front_ft, origin xyz=0.13525 0 -0.04789999999999994 rpy=0 0 -2.0943952105869315
- added joint l_foot_rear_ft_fixed_joint: type fixed, parent l_ankle_2, child l_foot_rear_ft, origin xyz=0.016000000000000004 0 -0.04789999999999994 rpy=0 0 -2.0943952105869315
- added joint l_leg_ft_fixed_joint: type fixed, parent l_hip_2, child l_leg_ft, origin xyz=0.036699999999999997 0 -0.0897 rpy=3.141592653589793 0 2.6179934742070086
- added joint r_arm_ft_fixed_joint: type fixed, parent r_shoulder_2, child r_arm_ft, origin xyz=-0.006849910543190453 3.2679315392636354e-07 -0.05429971877536288 rpy=-3.1415924092528633 0 1.5707964070692688
- added joint r_foot_front_ft_fixed_joint: type fixed, parent r_ankle_2, child r_foot_front_ft, origin xyz=0.13525 0 -0.04789999999999994 rpy=0 0 -2.0943952105869315
- added joint r_foot_rear_ft_fixed_joint: type fixed, parent r_ankle_2, child r_foot_rear_ft, origin xyz=0.016000000000000004 0 -0.04789999999999994 rpy=0 0 -2.0943952105869315
- added joint r_leg_ft_fixed_joint: type fixed, parent r_hip_2, child r_leg_ft, origin xyz=0.036699999999999997 0 -0.0897 rpy=3.141592653589793 0 -2.6179934742070086
- joint l_foot_front_ft_sensor: origin xyz=0.13525 0 -0.07019999999999993 rpy=0 0 0 -> xyz=0.13525 0 -0.04789999999999994 rpy=0 0 0
- joint l_foot_rear_ft_sensor: origin xyz=0.016000000000000004 0 -0.07019999999999993 rpy=0 0 0 -> xyz=0.016000000000000004 0 -0.04789999999999994 rpy=0 0 0
- joint l_sole_fixed_joint: origin xyz=0.05963 0 0 rpy=0 0 0 -> xyz=0.05963 0 -0.022299999999999986 rpy=0 0 0
- joint r_foot_front_ft_sensor: origin xyz=0.13525 0 -0.07019999999999993 rpy=0 0 0 -> xyz=0.13525 0 -0.04789999999999994 rpy=0 0 0
- joint r_foot_rear_ft_sensor: origin xyz=0.016000000000000004 0 -0.07019999999999993 rpy=0 0 0 -> xyz=0.016000000000000004 0 -0.04789999999999994 rpy=0 0 0
- joint r_sole_fixed_joint: origin xyz=0.05963 0 0 rpy=0 0 0 -> xyz=0.05963 0 -0.022299999999999986 rpy=0 0 0

File: urdf/ergoCub/robots/ergoCubGazeboV1_minContacts/model.urdf (robot description, URDF)
Before this commit: robot ergoCub, 194 links, 193 joints
Links:
- added link l_arm_ft
- added link l_foot_front_ft
- added link l_foot_rear_ft
- added link l_leg_ft
- added link r_arm_ft
- added link r_foot_front_ft
- added link r_foot_rear_ft
- added link r_leg_ft
Joints:
- added joint l_arm_ft_fixed_joint: type fixed, parent l_shoulder_2, child l_arm_ft, origin xyz=-0.004350065786786487 2.435985168580679e-07 -0.054299880148590496 rpy=-3.1415923328972943 0 -1.5707962214346844
- added joint l_foot_front_ft_fixed_joint: type fixed, parent l_ankle_2, child l_foot_front_ft, origin xyz=0.13525 0 -0.04789999999999994 rpy=0 0 -2.0943952105869315
- added joint l_foot_rear_ft_fixed_joint: type fixed, parent l_ankle_2, child l_foot_rear_ft, origin xyz=0.016000000000000004 0 -0.04789999999999994 rpy=0 0 -2.0943952105869315
- added joint l_leg_ft_fixed_joint: type fixed, parent l_hip_2, child l_leg_ft, origin xyz=0.036699999999999997 0 -0.0897 rpy=3.141592653589793 0 2.6179934742070086
- added joint r_arm_ft_fixed_joint: type fixed, parent r_shoulder_2, child r_arm_ft, origin xyz=-0.006849910543190453 3.2679315392636354e-07 -0.05429971877536288 rpy=-3.1415924092528633 0 1.5707964070692688
- added joint r_foot_front_ft_fixed_joint: type fixed, parent r_ankle_2, child r_foot_front_ft, origin xyz=0.13525 0 -0.04789999999999994 rpy=0 0 -2.0943952105869315
- added joint r_foot_rear_ft_fixed_joint: type fixed, parent r_ankle_2, child r_foot_rear_ft, origin xyz=0.016000000000000004 0 -0.04789999999999994 rpy=0 0 -2.0943952105869315
- added joint r_leg_ft_fixed_joint: type fixed, parent r_hip_2, child r_leg_ft, origin xyz=0.036699999999999997 0 -0.0897 rpy=3.141592653589793 0 -2.6179934742070086
- joint l_foot_front_ft_sensor: origin xyz=0.13525 0 -0.07019999999999993 rpy=0 0 0 -> xyz=0.13525 0 -0.04789999999999994 rpy=0 0 0
- joint l_foot_rear_ft_sensor: origin xyz=0.016000000000000004 0 -0.07019999999999993 rpy=0 0 0 -> xyz=0.016000000000000004 0 -0.04789999999999994 rpy=0 0 0
- joint l_sole_fixed_joint: origin xyz=0.05963 0 0 rpy=0 0 0 -> xyz=0.05963 0 -0.022299999999999986 rpy=0 0 0
- joint r_foot_front_ft_sensor: origin xyz=0.13525 0 -0.07019999999999993 rpy=0 0 0 -> xyz=0.13525 0 -0.04789999999999994 rpy=0 0 0
- joint r_foot_rear_ft_sensor: origin xyz=0.016000000000000004 0 -0.07019999999999993 rpy=0 0 0 -> xyz=0.016000000000000004 0 -0.04789999999999994 rpy=0 0 0
- joint r_sole_fixed_joint: origin xyz=0.05963 0 0 rpy=0 0 0 -> xyz=0.05963 0 -0.022299999999999986 rpy=0 0 0

File: urdf/ergoCub/robots/ergoCubSN000/model.urdf (robot description, URDF)
Before this commit: robot ergoCub, 194 links, 193 joints
Links:
- added link l_arm_ft
- added link l_foot_front_ft
- added link l_foot_rear_ft
- added link l_leg_ft
- added link r_arm_ft
- added link r_foot_front_ft
- added link r_foot_rear_ft
- added link r_leg_ft
Joints:
- added joint l_arm_ft_fixed_joint: type fixed, parent l_shoulder_2, child l_arm_ft, origin xyz=-0.004350065786786487 2.435985168580679e-07 -0.054299880148590496 rpy=-3.1415923328972943 0 -1.5707962214346844
- added joint l_foot_front_ft_fixed_joint: type fixed, parent l_ankle_2, child l_foot_front_ft, origin xyz=0.13525 0 -0.04789999999999994 rpy=0 0 -2.0943952105869315
- added joint l_foot_rear_ft_fixed_joint: type fixed, parent l_ankle_2, child l_foot_rear_ft, origin xyz=0.016000000000000004 0 -0.04789999999999994 rpy=0 0 -2.0943952105869315
- added joint l_leg_ft_fixed_joint: type fixed, parent l_hip_2, child l_leg_ft, origin xyz=0.036699999999999997 0 -0.0897 rpy=3.141592653589793 0 2.6179934742070086
- added joint r_arm_ft_fixed_joint: type fixed, parent r_shoulder_2, child r_arm_ft, origin xyz=-0.006849910543190453 3.2679315392636354e-07 -0.05429971877536288 rpy=-3.1415924092528633 0 1.5707964070692688
- added joint r_foot_front_ft_fixed_joint: type fixed, parent r_ankle_2, child r_foot_front_ft, origin xyz=0.13525 0 -0.04789999999999994 rpy=0 0 -2.0943952105869315
- added joint r_foot_rear_ft_fixed_joint: type fixed, parent r_ankle_2, child r_foot_rear_ft, origin xyz=0.016000000000000004 0 -0.04789999999999994 rpy=0 0 -2.0943952105869315
- added joint r_leg_ft_fixed_joint: type fixed, parent r_hip_2, child r_leg_ft, origin xyz=0.036699999999999997 0 -0.0897 rpy=3.141592653589793 0 -2.6179934742070086
- joint l_foot_front_ft_sensor: origin xyz=0.13525 0 -0.07019999999999993 rpy=0 0 0 -> xyz=0.13525 0 -0.04789999999999994 rpy=0 0 0
- joint l_foot_rear_ft_sensor: origin xyz=0.016000000000000004 0 -0.07019999999999993 rpy=0 0 0 -> xyz=0.016000000000000004 0 -0.04789999999999994 rpy=0 0 0
- joint l_sole_fixed_joint: origin xyz=0.05963 0 0 rpy=0 0 0 -> xyz=0.05963 0 -0.022299999999999986 rpy=0 0 0
- joint r_foot_front_ft_sensor: origin xyz=0.13525 0 -0.07019999999999993 rpy=0 0 0 -> xyz=0.13525 0 -0.04789999999999994 rpy=0 0 0
- joint r_foot_rear_ft_sensor: origin xyz=0.016000000000000004 0 -0.07019999999999993 rpy=0 0 0 -> xyz=0.016000000000000004 0 -0.04789999999999994 rpy=0 0 0
- joint r_sole_fixed_joint: origin xyz=0.05963 0 0 rpy=0 0 0 -> xyz=0.05963 0 -0.022299999999999986 rpy=0 0 0

Commit message: ergoCubV1: move down l/r_sole frames

File: urdf/ergoCub/robots/ergoCubGazeboV1/model.urdf (robot description, URDF)
Before this commit: robot ergoCub, 202 links, 201 joints
Joints:
- joint l_sole_fixed_joint: origin xyz=0.05963 0 -0.022299999999999986 rpy=0 0 0 -> xyz=0.05963 0 -0.024299999999999877 rpy=0 0 0
- joint r_sole_fixed_joint: origin xyz=0.05963 0 -0.022299999999999986 rpy=0 0 0 -> xyz=0.05963 0 -0.024299999999999877 rpy=0 0 0

File: urdf/ergoCub/robots/ergoCubGazeboV1_minContacts/model.urdf (robot description, URDF)
Before this commit: robot ergoCub, 202 links, 201 joints
Joints:
- joint l_sole_fixed_joint: origin xyz=0.05963 0 -0.022299999999999986 rpy=0 0 0 -> xyz=0.05963 0 -0.024299999999999877 rpy=0 0 0
- joint r_sole_fixed_joint: origin xyz=0.05963 0 -0.022299999999999986 rpy=0 0 0 -> xyz=0.05963 0 -0.024299999999999877 rpy=0 0 0

File: urdf/ergoCub/robots/ergoCubSN000/model.urdf (robot description, URDF)
Before this commit: robot ergoCub, 202 links, 201 joints
Joints:
- joint l_sole_fixed_joint: origin xyz=0.05963 0 -0.022299999999999986 rpy=0 0 0 -> xyz=0.05963 0 -0.024299999999999877 rpy=0 0 0
- joint r_sole_fixed_joint: origin xyz=0.05963 0 -0.022299999999999986 rpy=0 0 0 -> xyz=0.05963 0 -0.024299999999999877 rpy=0 0 0

Commit message: ergoCubV1*: correct names l/r_upperarm w/ r/l_upper_arm
It fixes #197

File: urdf/ergoCub/robots/ergoCubGazeboV1/model.urdf (robot description, URDF)
Before this commit: robot ergoCub, 202 links, 201 joints
Links:
- removed link l_upperarm
- removed link r_upperarm
- added link l_upper_arm, mass 1.77085; collision mesh filename=package://ergoCub/meshes/simmechanics/sim_ecub_l_upperarm_p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 scale=0.001 0.001 0.001; visual mesh filename=package://ergoCub/meshes/simmechanics/sim_ecub_l_upperarm_p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 scale=0.001 0.001 0.001
- added link r_upper_arm, mass 1.77224; collision mesh filename=package://ergoCub/meshes/simmechanics/sim_ecub_r_upperarm_p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 scale=0.001 0.001 0.001; visual mesh filename=package://ergoCub/meshes/simmechanics/sim_ecub_r_upperarm_p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 scale=0.001 0.001 0.001
Joints:
- joint l_elbow: parent l_upperarm -> l_upper_arm
- joint l_shoulder_yaw: child l_upperarm -> l_upper_arm
- joint r_elbow: parent r_upperarm -> r_upper_arm
- joint r_shoulder_yaw: child r_upperarm -> r_upper_arm

File: urdf/ergoCub/robots/ergoCubGazeboV1_minContacts/model.urdf (robot description, URDF)
Before this commit: robot ergoCub, 202 links, 201 joints
Links:
- removed link l_upperarm
- removed link r_upperarm
- added link l_upper_arm, mass 1.77085; collision box size=0.0 0.0 0.0; visual mesh filename=package://ergoCub/meshes/simmechanics/sim_ecub_l_upperarm_p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 scale=0.001 0.001 0.001
- added link r_upper_arm, mass 1.77224; collision box size=0.0 0.0 0.0; visual mesh filename=package://ergoCub/meshes/simmechanics/sim_ecub_r_upperarm_p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 scale=0.001 0.001 0.001
Joints:
- joint l_elbow: parent l_upperarm -> l_upper_arm
- joint l_shoulder_yaw: child l_upperarm -> l_upper_arm
- joint r_elbow: parent r_upperarm -> r_upper_arm
- joint r_shoulder_yaw: child r_upperarm -> r_upper_arm

File: urdf/ergoCub/robots/ergoCubSN000/model.urdf (robot description, URDF)
Before this commit: robot ergoCub, 202 links, 201 joints
Links:
- removed link l_upperarm
- removed link r_upperarm
- added link l_upper_arm, mass 1.77085; collision mesh filename=package://ergoCub/meshes/simmechanics/sim_ecub_l_upperarm_p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 scale=0.001 0.001 0.001; visual mesh filename=package://ergoCub/meshes/simmechanics/sim_ecub_l_upperarm_p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 scale=0.001 0.001 0.001
- added link r_upper_arm, mass 1.77224; collision mesh filename=package://ergoCub/meshes/simmechanics/sim_ecub_r_upperarm_p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 scale=0.001 0.001 0.001; visual mesh filename=package://ergoCub/meshes/simmechanics/sim_ecub_r_upperarm_p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 scale=0.001 0.001 0.001
Joints:
- joint l_elbow: parent l_upperarm -> l_upper_arm
- joint l_shoulder_yaw: child l_upperarm -> l_upper_arm
- joint r_elbow: parent r_upperarm -> r_upper_arm
- joint r_shoulder_yaw: child r_upperarm -> r_upper_arm

Commit message: ergoCub1_0: fix mass and inertia of the head
It has the same head of V1_1 but for some reason it was different, we verified that the V1_1 has the correct values

File: urdf/ergoCub/robots/ergoCubGazeboV1/model.urdf (robot description, URDF)
Before this commit: robot ergoCub, 202 links, 201 joints
Links:
- link head: mass 2.31933 -> 1.972127893184972

File: urdf/ergoCub/robots/ergoCubSN000/model.urdf (robot description, URDF)
Before this commit: robot ergoCub, 202 links, 201 joints
Links:
- link head: mass 2.31933 -> 1.972127893184972
