Commit message: Add .obj meshes + fix collision for the V1 soles

File: urdf/ergoCub/robots/ergoCubGazeboV1/model.urdf (robot description, URDF)
Before this commit: robot ergoCub, 202 links, 201 joints
Links:
- link chest: geometry collision mesh filename=package://ergoCub/meshes/simmechanics/sim_ecub_chest.obj scale=0.001 0.001 0.001; visual mesh filename=package://ergoCub/meshes/simmechanics/sim_ecub_chest.obj scale=0.001 0.001 0.001
- link head: geometry collision mesh filename=package://ergoCub/meshes/simmechanics/sim_ecub_head.obj scale=0.001 0.001 0.001; visual mesh filename=package://ergoCub/meshes/simmechanics/sim_ecub_head.obj scale=0.001 0.001 0.001
- link l_ankle_1: geometry collision mesh filename=package://ergoCub/meshes/simmechanics/sim_ecub_l_ankle_1.obj scale=0.001 0.001 0.001; visual mesh filename=package://ergoCub/meshes/simmechanics/sim_ecub_l_ankle_1.obj scale=0.001 0.001 0.001
- link l_ankle_2: geometry collision mesh filename=package://ergoCub/meshes/simmechanics/sim_ecub_l_ankle_2.obj scale=0.001 0.001 0.001; visual mesh filename=package://ergoCub/meshes/simmechanics/sim_ecub_l_ankle_2.obj scale=0.001 0.001 0.001
- link l_foot_rear: geometry collision box size=0.117 0.1 0.006; visual mesh filename=package://ergoCub/meshes/simmechanics/sim_ecub_l_foot_rear.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 scale=0.001 0.001 0.001
- link l_forearm: geometry collision mesh filename=package://ergoCub/meshes/simmechanics/sim_ecub_l_forearm.obj scale=0.001 0.001 0.001; visual mesh filename=package://ergoCub/meshes/simmechanics/sim_ecub_l_forearm.obj scale=0.001 0.001 0.001
- link l_hand_palm: geometry collision mesh filename=package://ergoCub/meshes/simmechanics/sim_ecub_l_hand_palm.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 scale=0.001 0.001 0.001; visual mesh filename=package://ergoCub/meshes/simmechanics/sim_ecub_l_hand_palm.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 scale=0.001 0.001 0.001
- link l_hip_1: geometry collision mesh filename=package://ergoCub/meshes/simmechanics/sim_ecub_l_hip_1.obj scale=0.001 0.001 0.001; visual mesh filename=package://ergoCub/meshes/simmechanics/sim_ecub_l_hip_1.obj scale=0.001 0.001 0.001
- link l_hip_2: geometry collision mesh filename=package://ergoCub/meshes/simmechanics/sim_ecub_l_hip_2.obj scale=0.001 0.001 0.001; visual mesh filename=package://ergoCub/meshes/simmechanics/sim_ecub_l_hip_2.obj scale=0.001 0.001 0.001
- link l_hip_3: geometry collision mesh filename=package://ergoCub/meshes/simmechanics/sim_ecub_l_hip_3.obj scale=0.001 0.001 0.001; visual mesh filename=package://ergoCub/meshes/simmechanics/sim_ecub_l_hip_3.obj scale=0.001 0.001 0.001
- link l_lower_leg: geometry collision mesh filename=package://ergoCub/meshes/simmechanics/sim_ecub_l_lower_leg.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 scale=0.001 0.001 0.001; visual mesh filename=package://ergoCub/meshes/simmechanics/sim_ecub_l_lower_leg.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 scale=0.001 0.001 0.001
- link l_upper_arm: geometry collision mesh filename=package://ergoCub/meshes/simmechanics/sim_ecub_l_upperarm.o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 scale=0.001 0.001 0.001; visual mesh filename=package://ergoCub/meshes/simmechanics/sim_ecub_l_upperarm.o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 scale=0.001 0.001 0.001
- link l_upper_leg: geometry collision mesh filename=package://ergoCub/meshes/simmechanics/sim_ecub_l_upper_leg.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 scale=0.001 0.001 0.001; visual mesh filename=package://ergoCub/meshes/simmechanics/sim_ecub_l_upper_leg.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 scale=0.001 0.001 0.001
- link l_wrist_1: geometry collision mesh filename=package://ergoCub/meshes/simmechanics/sim_ecub_l_wrist_1.obj scale=0.001 0.001 0.001; visual mesh filename=package://ergoCub/meshes/simmechanics/sim_ecub_l_wrist_1.obj scale=0.001 0.001 0.001
- link l_wrist_2: geometry collision mesh filename=package://ergoCub/meshes/simmechanics/sim_ecub_l_wrist_2.obj scale=0.001 0.001 0.001; visual mesh filename=package://ergoCub/meshes/simmechanics/sim_ecub_l_wrist_2.obj scale=0.001 0.001 0.001
- link neck_2: geometry collision mesh filename=package://ergoCub/meshes/simmechanics/sim_ecub_head_neck_2.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 scale=0.001 0.001 0.001; visual mesh filename=package://ergoCub/meshes/simmechanics/sim_ecub_head_neck_2.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 scale=0.001 0.001 0.001
- link neck_3: geometry collision mesh filename=package://ergoCub/meshes/simmechanics/sim_ecub_head_neck_3.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 scale=0.001 0.001 0.001; visual mesh filename=package://ergoCub/meshes/simmechanics/sim_ecub_head_neck_3.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 scale=0.001 0.001 0.001
- link r_ankle_1: geometry collision mesh filename=package://ergoCub/meshes/simmechanics/sim_ecub_r_ankle_1.obj scale=0.001 0.001 0.001; visual mesh filename=package://ergoCub/meshes/simmechanics/sim_ecub_r_ankle_1.obj scale=0.001 0.001 0.001
- link r_ankle_2: geometry collision mesh filename=package://ergoCub/meshes/simmechanics/sim_ecub_r_ankle_2.obj scale=0.001 0.001 0.001; visual mesh filename=package://ergoCub/meshes/simmechanics/sim_ecub_r_ankle_2.obj scale=0.001 0.001 0.001
- link r_foot_rear: geometry collision box size=0.117 0.1 0.006; visual mesh filename=package://ergoCub/meshes/simmechanics/sim_ecub_r_foot_rear.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 scale=0.001 0.001 0.001
- link r_forearm: geometry collision mesh filename=package://ergoCub/meshes/simmechanics/sim_ecub_r_forearm.obj scale=0.001 0.001 0.001; visual mesh filename=package://ergoCub/meshes/simmechanics/sim_ecub_r_forearm.obj scale=0.001 0.001 0.001
- link r_hand_palm: geometry collision mesh filename=package://ergoCub/meshes/simmechanics/sim_ecub_r_hand_palm.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 scale=0.001 0.001 0.001; visual mesh filename=package://ergoCub/meshes/simmechanics/sim_ecub_r_hand_palm.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 scale=0.001 0.001 0.001
- link r_hip_1: geometry collision mesh filename=package://ergoCub/meshes/simmechanics/sim_ecub_r_hip_1.obj scale=0.001 0.001 0.001; visual mesh filename=package://ergoCub/meshes/simmechanics/sim_ecub_r_hip_1.obj scale=0.001 0.001 0.001
- link r_hip_2: geometry collision mesh filename=package://ergoCub/meshes/simmechanics/sim_ecub_r_hip_2.obj scale=0.001 0.001 0.001; visual mesh filename=package://ergoCub/meshes/simmechanics/sim_ecub_r_hip_2.obj scale=0.001 0.001 0.001
- link r_hip_3: geometry collision mesh filename=package://ergoCub/meshes/simmechanics/sim_ecub_r_hip_3.obj scale=0.001 0.001 0.001; visual mesh filename=package://ergoCub/meshes/simmechanics/sim_ecub_r_hip_3.obj scale=0.001 0.001 0.001
- link r_lower_leg: geometry collision mesh filename=package://ergoCub/meshes/simmechanics/sim_ecub_r_lower_leg.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 scale=0.001 0.001 0.001; visual mesh filename=package://ergoCub/meshes/simmechanics/sim_ecub_r_lower_leg.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 scale=0.001 0.001 0.001
- link r_upper_arm: geometry collision mesh filename=package://ergoCub/meshes/simmechanics/sim_ecub_r_upperarm.o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 scale=0.001 0.001 0.001; visual mesh filename=package://ergoCub/meshes/simmechanics/sim_ecub_r_upperarm.o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 scale=0.001 0.001 0.001
- link r_upper_leg: geometry collision mesh filename=package://ergoCub/meshes/simmechanics/sim_ecub_r_upper_leg.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 scale=0.001 0.001 0.001; visual mesh filename=package://ergoCub/meshes/simmechanics/sim_ecub_r_upper_leg.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 scale=0.001 0.001 0.001
- link r_wrist_1: geometry collision mesh filename=package://ergoCub/meshes/simmechanics/sim_ecub_r_wrist_1.obj scale=0.001 0.001 0.001; visual mesh filename=package://ergoCub/meshes/simmechanics/sim_ecub_r_wrist_1.obj scale=0.001 0.001 0.001
- link r_wrist_2: geometry collision mesh filename=package://ergoCub/meshes/simmechanics/sim_ecub_r_wrist_2.obj scale=0.001 0.001 0.001; visual mesh filename=package://ergoCub/meshes/simmechanics/sim_ecub_r_wrist_2.obj scale=0.001 0.001 0.001
- link realsense: geometry collision mesh filename=package://ergoCub/meshes/simmechanics/sim_ecub_realsense.obj scale=0.001 0.001 0.001; visual mesh filename=package://ergoCub/meshes/simmechanics/sim_ecub_realsense.obj scale=0.001 0.001 0.001
- link root_link: geometry collision mesh filename=package://ergoCub/meshes/simmechanics/sim_ecub_root_link.obj scale=0.001 0.001 0.001; visual mesh filename=package://ergoCub/meshes/simmechanics/sim_ecub_root_link.obj scale=0.001 0.001 0.001
- link torso_1: geometry collision mesh filename=package://ergoCub/meshes/simmechanics/sim_ecub_torso_1.obj scale=0.001 0.001 0.001; visual mesh filename=package://ergoCub/meshes/simmechanics/sim_ecub_torso_1.obj scale=0.001 0.001 0.001
- link torso_2: geometry collision mesh filename=package://ergoCub/meshes/simmechanics/sim_ecub_torso_2.obj scale=0.001 0.001 0.001; visual mesh filename=package://ergoCub/meshes/simmechanics/sim_ecub_torso_2.obj scale=0.001 0.001 0.001

File: urdf/ergoCub/robots/ergoCubGazeboV1_1/model.urdf (robot description, URDF)
Before this commit: robot ergoCub, 204 links, 203 joints
Links:
- link chest: geometry collision mesh filename=package://ergoCub/meshes/simmechanics/sim_ecub_1-1_chest.obj scale=0.001 0.001 0.001; visual mesh filename=package://ergoCub/meshes/simmechanics/sim_ecub_1-1_chest.obj scale=0.001 0.001 0.001
- link head: geometry collision mesh filename=package://ergoCub/meshes/simmechanics/sim_ecub_1-1_head.obj scale=0.001 0.001 0.001; visual mesh filename=package://ergoCub/meshes/simmechanics/sim_ecub_1-1_head.obj scale=0.001 0.001 0.001

File: urdf/ergoCub/robots/ergoCubGazeboV1_1_minContacts/model.urdf (robot description, URDF)
Before this commit: robot ergoCub, 204 links, 203 joints
Links:
- link chest: geometry collision box size=0 0 0; visual mesh filename=package://ergoCub/meshes/simmechanics/sim_ecub_1-1_chest.obj scale=0.001 0.001 0.001
- link head: geometry collision box size=0 0 0; visual mesh filename=package://ergoCub/meshes/simmechanics/sim_ecub_1-1_head.obj scale=0.001 0.001 0.001

File: urdf/ergoCub/robots/ergoCubGazeboV1_2/model.urdf (robot description, URDF)
Before this commit: robot ergoCub, 204 links, 203 joints
Links:
- link chest: geometry collision mesh filename=package://ergoCub/meshes/simmechanics/sim_ecub_1-1_chest.obj scale=0.001 0.001 0.001; visual mesh filename=package://ergoCub/meshes/simmechanics/sim_ecub_1-1_chest.obj scale=0.001 0.001 0.001
- link head: geometry collision mesh filename=package://ergoCub/meshes/simmechanics/sim_ecub_1-1_head.obj scale=0.001 0.001 0.001; visual mesh filename=package://ergoCub/meshes/simmechanics/sim_ecub_1-1_head.obj scale=0.001 0.001 0.001

File: urdf/ergoCub/robots/ergoCubGazeboV1_2_minContacts/model.urdf (robot description, URDF)
Before this commit: robot ergoCub, 204 links, 203 joints
Links:
- link chest: geometry collision box size=0 0 0; visual mesh filename=package://ergoCub/meshes/simmechanics/sim_ecub_1-1_chest.obj scale=0.001 0.001 0.001
- link head: geometry collision box size=0 0 0; visual mesh filename=package://ergoCub/meshes/simmechanics/sim_ecub_1-1_head.obj scale=0.001 0.001 0.001

File: urdf/ergoCub/robots/ergoCubGazeboV1_minContacts/model.urdf (robot description, URDF)
Before this commit: robot ergoCub, 202 links, 201 joints
Links:
- link chest: geometry collision box size=0.0 0.0 0.0; visual mesh filename=package://ergoCub/meshes/simmechanics/sim_ecub_chest.obj scale=0.001 0.001 0.001
- link head: geometry collision box size=0.0 0.0 0.0; visual mesh filename=package://ergoCub/meshes/simmechanics/sim_ecub_head.obj scale=0.001 0.001 0.001
- link l_ankle_1: geometry collision box size=0.0 0.0 0.0; visual mesh filename=package://ergoCub/meshes/simmechanics/sim_ecub_l_ankle_1.obj scale=0.001 0.001 0.001
- link l_ankle_2: geometry collision box size=0.0 0.0 0.0; visual mesh filename=package://ergoCub/meshes/simmechanics/sim_ecub_l_ankle_2.obj scale=0.001 0.001 0.001
- link l_foot_rear: geometry collision box size=0.117 0.1 0.006; visual mesh filename=package://ergoCub/meshes/simmechanics/sim_ecub_l_foot_rear.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 scale=0.001 0.001 0.001
- link l_forearm: geometry collision box size=0.0 0.0 0.0; visual mesh filename=package://ergoCub/meshes/simmechanics/sim_ecub_l_forearm.obj scale=0.001 0.001 0.001
- link l_hand_palm: geometry collision box size=0.0 0.0 0.0; visual mesh filename=package://ergoCub/meshes/simmechanics/sim_ecub_l_hand_palm.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 scale=0.001 0.001 0.001
- link l_hip_1: geometry collision box size=0.0 0.0 0.0; visual mesh filename=package://ergoCub/meshes/simmechanics/sim_ecub_l_hip_1.obj scale=0.001 0.001 0.001
- link l_hip_2: geometry collision box size=0.0 0.0 0.0; visual mesh filename=package://ergoCub/meshes/simmechanics/sim_ecub_l_hip_2.obj scale=0.001 0.001 0.001
- link l_hip_3: geometry collision box size=0.0 0.0 0.0; visual mesh filename=package://ergoCub/meshes/simmechanics/sim_ecub_l_hip_3.obj scale=0.001 0.001 0.001
- link l_lower_leg: geometry collision box size=0.0 0.0 0.0; visual mesh filename=package://ergoCub/meshes/simmechanics/sim_ecub_l_lower_leg.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 scale=0.001 0.001 0.001
- link l_upper_arm: geometry collision box size=0.0 0.0 0.0; visual mesh filename=package://ergoCub/meshes/simmechanics/sim_ecub_l_upperarm.o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 scale=0.001 0.001 0.001
- link l_upper_leg: geometry collision box size=0.0 0.0 0.0; visual mesh filename=package://ergoCub/meshes/simmechanics/sim_ecub_l_upper_leg.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 scale=0.001 0.001 0.001
- link l_wrist_1: geometry collision box size=0.0 0.0 0.0; visual mesh filename=package://ergoCub/meshes/simmechanics/sim_ecub_l_wrist_1.obj scale=0.001 0.001 0.001
- link l_wrist_2: geometry collision box size=0.0 0.0 0.0; visual mesh filename=package://ergoCub/meshes/simmechanics/sim_ecub_l_wrist_2.obj scale=0.001 0.001 0.001
- link neck_2: geometry collision box size=0.0 0.0 0.0; visual mesh filename=package://ergoCub/meshes/simmechanics/sim_ecub_head_neck_2.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 scale=0.001 0.001 0.001
- link neck_3: geometry collision box size=0.0 0.0 0.0; visual mesh filename=package://ergoCub/meshes/simmechanics/sim_ecub_head_neck_3.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 scale=0.001 0.001 0.001
- link r_ankle_1: geometry collision box size=0.0 0.0 0.0; visual mesh filename=package://ergoCub/meshes/simmechanics/sim_ecub_r_ankle_1.obj scale=0.001 0.001 0.001
- link r_ankle_2: geometry collision box size=0.0 0.0 0.0; visual mesh filename=package://ergoCub/meshes/simmechanics/sim_ecub_r_ankle_2.obj scale=0.001 0.001 0.001
- link r_foot_rear: geometry collision box size=0.117 0.1 0.006; visual mesh filename=package://ergoCub/meshes/simmechanics/sim_ecub_r_foot_rear.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 scale=0.001 0.001 0.001
- link r_forearm: geometry collision box size=0.0 0.0 0.0; visual mesh filename=package://ergoCub/meshes/simmechanics/sim_ecub_r_forearm.obj scale=0.001 0.001 0.001
- link r_hand_palm: geometry collision box size=0.0 0.0 0.0; visual mesh filename=package://ergoCub/meshes/simmechanics/sim_ecub_r_hand_palm.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 scale=0.001 0.001 0.001
- link r_hip_1: geometry collision box size=0.0 0.0 0.0; visual mesh filename=package://ergoCub/meshes/simmechanics/sim_ecub_r_hip_1.obj scale=0.001 0.001 0.001
- link r_hip_2: geometry collision box size=0.0 0.0 0.0; visual mesh filename=package://ergoCub/meshes/simmechanics/sim_ecub_r_hip_2.obj scale=0.001 0.001 0.001
- link r_hip_3: geometry collision box size=0.0 0.0 0.0; visual mesh filename=package://ergoCub/meshes/simmechanics/sim_ecub_r_hip_3.obj scale=0.001 0.001 0.001
- link r_lower_leg: geometry collision box size=0.0 0.0 0.0; visual mesh filename=package://ergoCub/meshes/simmechanics/sim_ecub_r_lower_leg.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 scale=0.001 0.001 0.001
- link r_upper_arm: geometry collision box size=0.0 0.0 0.0; visual mesh filename=package://ergoCub/meshes/simmechanics/sim_ecub_r_upperarm.o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 scale=0.001 0.001 0.001
- link r_upper_leg: geometry collision box size=0.0 0.0 0.0; visual mesh filename=package://ergoCub/meshes/simmechanics/sim_ecub_r_upper_leg.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 scale=0.001 0.001 0.001
- link r_wrist_1: geometry collision box size=0.0 0.0 0.0; visual mesh filename=package://ergoCub/meshes/simmechanics/sim_ecub_r_wrist_1.obj scale=0.001 0.001 0.001
- link r_wrist_2: geometry collision box size=0.0 0.0 0.0; visual mesh filename=package://ergoCub/meshes/simmechanics/sim_ecub_r_wrist_2.obj scale=0.001 0.001 0.001
- link realsense: geometry collision box size=0.0 0.0 0.0; visual mesh filename=package://ergoCub/meshes/simmechanics/sim_ecub_realsense.obj scale=0.001 0.001 0.001
- link root_link: geometry collision box size=0.0 0.0 0.0; visual mesh filename=package://ergoCub/meshes/simmechanics/sim_ecub_root_link.obj scale=0.001 0.001 0.001
- link torso_1: geometry collision box size=0.0 0.0 0.0; visual mesh filename=package://ergoCub/meshes/simmechanics/sim_ecub_torso_1.obj scale=0.001 0.001 0.001
- link torso_2: geometry collision box size=0.0 0.0 0.0; visual mesh filename=package://ergoCub/meshes/simmechanics/sim_ecub_torso_2.obj scale=0.001 0.001 0.001
