Commit message: Add .obj meshes + fix collision for the V1 soles

File: urdf/ergoCub/robots/ergoCubSN000/model.urdf (robot description, URDF)
Before this commit: robot ergoCub, 202 links, 201 joints
Links:
- link chest: geometry collision mesh filename=package://ergoCub/meshes/simmechanics/sim_ecub_chest.obj scale=0.001 0.001 0.001; visual mesh filename=package://ergoCub/meshes/simmechanics/sim_ecub_chest.obj scale=0.001 0.001 0.001
- link head: geometry collision mesh filename=package://ergoCub/meshes/simmechanics/sim_ecub_head.obj scale=0.001 0.001 0.001; visual mesh filename=package://ergoCub/meshes/simmechanics/sim_ecub_head.obj scale=0.001 0.001 0.001
- link l_ankle_1: geometry collision mesh filename=package://ergoCub/meshes/simmechanics/sim_ecub_l_ankle_1.obj scale=0.001 0.001 0.001; visual mesh filename=package://ergoCub/meshes/simmechanics/sim_ecub_l_ankle_1.obj scale=0.001 0.001 0.001
- link l_ankle_2: geometry collision mesh filename=package://ergoCub/meshes/simmechanics/sim_ecub_l_ankle_2.obj scale=0.001 0.001 0.001; visual mesh filename=package://ergoCub/meshes/simmechanics/sim_ecub_l_ankle_2.obj scale=0.001 0.001 0.001
- link l_foot_rear: geometry collision mesh filename=package://ergoCub/meshes/simmechanics/sim_ecub_l_foot_rear.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 scale=0.001 0.001 0.001; visual mesh filename=package://ergoCub/meshes/simmechanics/sim_ecub_l_foot_rear.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 scale=0.001 0.001 0.001
- link l_forearm: geometry collision mesh filename=package://ergoCub/meshes/simmechanics/sim_ecub_l_forearm.obj scale=0.001 0.001 0.001; visual mesh filename=package://ergoCub/meshes/simmechanics/sim_ecub_l_forearm.obj scale=0.001 0.001 0.001
- link l_hand_palm: geometry collision mesh filename=package://ergoCub/meshes/simmechanics/sim_ecub_l_hand_palm.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 scale=0.001 0.001 0.001; visual mesh filename=package://ergoCub/meshes/simmechanics/sim_ecub_l_hand_palm.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 scale=0.001 0.001 0.001
- link l_hip_1: geometry collision mesh filename=package://ergoCub/meshes/simmechanics/sim_ecub_l_hip_1.obj scale=0.001 0.001 0.001; visual mesh filename=package://ergoCub/meshes/simmechanics/sim_ecub_l_hip_1.obj scale=0.001 0.001 0.001
- link l_hip_2: geometry collision mesh filename=package://ergoCub/meshes/simmechanics/sim_ecub_l_hip_2.obj scale=0.001 0.001 0.001; visual mesh filename=package://ergoCub/meshes/simmechanics/sim_ecub_l_hip_2.obj scale=0.001 0.001 0.001
- link l_hip_3: geometry collision mesh filename=package://ergoCub/meshes/simmechanics/sim_ecub_l_hip_3.obj scale=0.001 0.001 0.001; visual mesh filename=package://ergoCub/meshes/simmechanics/sim_ecub_l_hip_3.obj scale=0.001 0.001 0.001
- link l_lower_leg: geometry collision mesh filename=package://ergoCub/meshes/simmechanics/sim_ecub_l_lower_leg.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 scale=0.001 0.001 0.001; visual mesh filename=package://ergoCub/meshes/simmechanics/sim_ecub_l_lower_leg.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 scale=0.001 0.001 0.001
- link l_upper_arm: geometry collision mesh filename=package://ergoCub/meshes/simmechanics/sim_ecub_l_upperarm.o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 scale=0.001 0.001 0.001; visual mesh filename=package://ergoCub/meshes/simmechanics/sim_ecub_l_upperarm.o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 scale=0.001 0.001 0.001
- link l_upper_leg: geometry collision mesh filename=package://ergoCub/meshes/simmechanics/sim_ecub_l_upper_leg.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 scale=0.001 0.001 0.001; visual mesh filename=package://ergoCub/meshes/simmechanics/sim_ecub_l_upper_leg.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 scale=0.001 0.001 0.001
- link l_wrist_1: geometry collision mesh filename=package://ergoCub/meshes/simmechanics/sim_ecub_l_wrist_1.obj scale=0.001 0.001 0.001; visual mesh filename=package://ergoCub/meshes/simmechanics/sim_ecub_l_wrist_1.obj scale=0.001 0.001 0.001
- link l_wrist_2: geometry collision mesh filename=package://ergoCub/meshes/simmechanics/sim_ecub_l_wrist_2.obj scale=0.001 0.001 0.001; visual mesh filename=package://ergoCub/meshes/simmechanics/sim_ecub_l_wrist_2.obj scale=0.001 0.001 0.001
- link neck_2: geometry collision mesh filename=package://ergoCub/meshes/simmechanics/sim_ecub_head_neck_2.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 scale=0.001 0.001 0.001; visual mesh filename=package://ergoCub/meshes/simmechanics/sim_ecub_head_neck_2.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 scale=0.001 0.001 0.001
- link neck_3: geometry collision mesh filename=package://ergoCub/meshes/simmechanics/sim_ecub_head_neck_3.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 scale=0.001 0.001 0.001; visual mesh filename=package://ergoCub/meshes/simmechanics/sim_ecub_head_neck_3.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 scale=0.001 0.001 0.001
- link r_ankle_1: geometry collision mesh filename=package://ergoCub/meshes/simmechanics/sim_ecub_r_ankle_1.obj scale=0.001 0.001 0.001; visual mesh filename=package://ergoCub/meshes/simmechanics/sim_ecub_r_ankle_1.obj scale=0.001 0.001 0.001
- link r_ankle_2: geometry collision mesh filename=package://ergoCub/meshes/simmechanics/sim_ecub_r_ankle_2.obj scale=0.001 0.001 0.001; visual mesh filename=package://ergoCub/meshes/simmechanics/sim_ecub_r_ankle_2.obj scale=0.001 0.001 0.001
- link r_foot_rear: geometry collision mesh filename=package://ergoCub/meshes/simmechanics/sim_ecub_r_foot_rear.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 scale=0.001 0.001 0.001; visual mesh filename=package://ergoCub/meshes/simmechanics/sim_ecub_r_foot_rear.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 scale=0.001 0.001 0.001
- link r_forearm: geometry collision mesh filename=package://ergoCub/meshes/simmechanics/sim_ecub_r_forearm.obj scale=0.001 0.001 0.001; visual mesh filename=package://ergoCub/meshes/simmechanics/sim_ecub_r_forearm.obj scale=0.001 0.001 0.001
- link r_hand_palm: geometry collision mesh filename=package://ergoCub/meshes/simmechanics/sim_ecub_r_hand_palm.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 scale=0.001 0.001 0.001; visual mesh filename=package://ergoCub/meshes/simmechanics/sim_ecub_r_hand_palm.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 scale=0.001 0.001 0.001
- link r_hip_1: geometry collision mesh filename=package://ergoCub/meshes/simmechanics/sim_ecub_r_hip_1.obj scale=0.001 0.001 0.001; visual mesh filename=package://ergoCub/meshes/simmechanics/sim_ecub_r_hip_1.obj scale=0.001 0.001 0.001
- link r_hip_2: geometry collision mesh filename=package://ergoCub/meshes/simmechanics/sim_ecub_r_hip_2.obj scale=0.001 0.001 0.001; visual mesh filename=package://ergoCub/meshes/simmechanics/sim_ecub_r_hip_2.obj scale=0.001 0.001 0.001
- link r_hip_3: geometry collision mesh filename=package://ergoCub/meshes/simmechanics/sim_ecub_r_hip_3.obj scale=0.001 0.001 0.001; visual mesh filename=package://ergoCub/meshes/simmechanics/sim_ecub_r_hip_3.obj scale=0.001 0.001 0.001
- link r_lower_leg: geometry collision mesh filename=package://ergoCub/meshes/simmechanics/sim_ecub_r_lower_leg.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 scale=0.001 0.001 0.001; visual mesh filename=package://ergoCub/meshes/simmechanics/sim_ecub_r_lower_leg.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 scale=0.001 0.001 0.001
- link r_upper_arm: geometry collision mesh filename=package://ergoCub/meshes/simmechanics/sim_ecub_r_upperarm.o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 scale=0.001 0.001 0.001; visual mesh filename=package://ergoCub/meshes/simmechanics/sim_ecub_r_upperarm.o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 scale=0.001 0.001 0.001
- link r_upper_leg: geometry collision mesh filename=package://ergoCub/meshes/simmechanics/sim_ecub_r_upper_leg.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 scale=0.001 0.001 0.001; visual mesh filename=package://ergoCub/meshes/simmechanics/sim_ecub_r_upper_leg.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 scale=0.001 0.001 0.001
- link r_wrist_1: geometry collision mesh filename=package://ergoCub/meshes/simmechanics/sim_ecub_r_wrist_1.obj scale=0.001 0.001 0.001; visual mesh filename=package://ergoCub/meshes/simmechanics/sim_ecub_r_wrist_1.obj scale=0.001 0.001 0.001
- link r_wrist_2: geometry collision mesh filename=package://ergoCub/meshes/simmechanics/sim_ecub_r_wrist_2.obj scale=0.001 0.001 0.001; visual mesh filename=package://ergoCub/meshes/simmechanics/sim_ecub_r_wrist_2.obj scale=0.001 0.001 0.001
- link realsense: geometry collision mesh filename=package://ergoCub/meshes/simmechanics/sim_ecub_realsense.obj scale=0.001 0.001 0.001; visual mesh filename=package://ergoCub/meshes/simmechanics/sim_ecub_realsense.obj scale=0.001 0.001 0.001
- link root_link: geometry collision mesh filename=package://ergoCub/meshes/simmechanics/sim_ecub_root_link.obj scale=0.001 0.001 0.001; visual mesh filename=package://ergoCub/meshes/simmechanics/sim_ecub_root_link.obj scale=0.001 0.001 0.001
- link torso_1: geometry collision mesh filename=package://ergoCub/meshes/simmechanics/sim_ecub_torso_1.obj scale=0.001 0.001 0.001; visual mesh filename=package://ergoCub/meshes/simmechanics/sim_ecub_torso_1.obj scale=0.001 0.001 0.001
- link torso_2: geometry collision mesh filename=package://ergoCub/meshes/simmechanics/sim_ecub_torso_2.obj scale=0.001 0.001 0.001; visual mesh filename=package://ergoCub/meshes/simmechanics/sim_ecub_torso_2.obj scale=0.001 0.001 0.001

File: urdf/ergoCub/robots/ergoCubSN002/model.urdf (robot description, URDF)
Before this commit: robot ergoCub, 204 links, 203 joints
Links:
- link chest: geometry collision mesh filename=package://ergoCub/meshes/simmechanics/sim_ecub_1-1_chest.obj scale=0.001 0.001 0.001; visual mesh filename=package://ergoCub/meshes/simmechanics/sim_ecub_1-1_chest.obj scale=0.001 0.001 0.001
- link head: geometry collision mesh filename=package://ergoCub/meshes/simmechanics/sim_ecub_1-1_head.obj scale=0.001 0.001 0.001; visual mesh filename=package://ergoCub/meshes/simmechanics/sim_ecub_1-1_head.obj scale=0.001 0.001 0.001

Commit message: ergoCubGazeboV1: fix imu waist by hand

File: urdf/ergoCub/robots/ergoCubGazeboV1/model.urdf (robot description, URDF)
Before this commit: robot ergoCub, 202 links, 201 joints
Joints:
- joint waist_imu_0_fixed_joint: origin xyz=0.0354497 0.00639688 0.060600 rpy=1.5708 0 -1.5708 -> xyz=0.0606 -0.00639428 0.01745 rpy=1.5708 -0.000105208 -1.5708

File: urdf/ergoCub/robots/ergoCubGazeboV1_minContacts/model.urdf (robot description, URDF)
Before this commit: robot ergoCub, 202 links, 201 joints
Joints:
- joint waist_imu_0_fixed_joint: origin xyz=0.0354497 0.00639688 0.060600 rpy=1.5708 0 -1.5708 -> xyz=0.0606 -0.00639428 0.01745 rpy=1.5708 -0.000105208 -1.5708

File: urdf/ergoCub/robots/ergoCubSN000/model.urdf (robot description, URDF)
Before this commit: robot ergoCub, 202 links, 201 joints
Joints:
- joint waist_imu_0_fixed_joint: origin xyz=0.0354497 0.00639688 0.060600 rpy=1.5708 0 -1.5708 -> xyz=0.0606 -0.00639428 0.01745 rpy=1.5708 -0.000105208 -1.5708

Commit message: ergoCubV1: fix limits
See #295. #296

File: urdf/ergoCub/robots/ergoCubGazeboV1/model.urdf (robot description, URDF)
Before this commit: robot ergoCub, 202 links, 201 joints
Joints:
- joint l_elbow: limit lower=-0.05235987755982989 upper=1.3089969389957472 effort=50000 velocity=120.0 -> lower=-0.08726646259971647 upper=2.0943951023931953 effort=50000 velocity=120.0
- joint l_hip_pitch: limit lower=-0.7504915783575618 upper=1.7976891295541595 effort=50000 velocity=120.0 -> lower=-0.767944870877505 upper=1.9198621771937625 effort=50000 velocity=120.0
- joint l_hip_roll: limit lower=-0.2792526803190927 upper=1.9024088846738192 effort=50000 velocity=120.0 -> lower=-0.3490658503988659 upper=1.9373154697137058 effort=50000 velocity=120.0
- joint l_hip_yaw: limit lower=-1.3788101090755203 upper=1.3788101090755203 effort=50000 velocity=120.0 -> lower=-1.413716694115407 upper=1.413716694115407 effort=50000 velocity=120.0
- joint l_knee: limit lower=-1.8151424220741028 upper=0.10471975511965978 effort=50000 velocity=120.0 -> lower=-1.8325957145940461 upper=0.12217304763960307 effort=50000 velocity=120.0
- joint l_shoulder_yaw: limit lower=-0.8726646259971648 upper=1.3962634015954636 effort=50000 velocity=120.0 -> lower=-0.9075712110370514 upper=1.4311699866353502 effort=50000 velocity=120.0
- joint l_wrist_pitch: limit lower=-0.5585053606381855 upper=0.5585053606381855 effort=50000 velocity=120.0 -> lower=-0.3490658503988659 upper=0.3490658503988659 effort=50000 velocity=120.0
- joint l_wrist_roll: limit lower=-1.0821041362364843 upper=0.9075712110370514 effort=50000 velocity=120.0 -> lower=-0.3490658503988659 upper=0.5235987755982988 effort=50000 velocity=120.0
- joint neck_pitch: limit lower=-0.5235987755982988 upper=0.3839724354387525 effort=50000 velocity=120.0 -> lower=-0.7853981633974483 upper=0.3839724354387525 effort=50000 velocity=120.0
- joint r_elbow: limit lower=-0.05235987755982989 upper=1.3089969389957472 effort=50000 velocity=120.0 -> lower=-0.08726646259971647 upper=2.0943951023931953 effort=50000 velocity=120.0
- joint r_hip_pitch: limit lower=-0.7504915783575618 upper=1.7976891295541595 effort=50000 velocity=120.0 -> lower=-0.767944870877505 upper=1.9198621771937625 effort=50000 velocity=120.0
- joint r_hip_roll: limit lower=-0.2792526803190927 upper=1.9024088846738192 effort=50000 velocity=120.0 -> lower=-0.3490658503988659 upper=1.9373154697137058 effort=50000 velocity=120.0
- joint r_hip_yaw: limit lower=-1.3788101090755203 upper=1.3788101090755203 effort=50000 velocity=120.0 -> lower=-1.413716694115407 upper=1.413716694115407 effort=50000 velocity=120.0
- joint r_knee: limit lower=-1.8151424220741028 upper=0.10471975511965978 effort=50000 velocity=120.0 -> lower=-1.8325957145940461 upper=0.12217304763960307 effort=50000 velocity=120.0
- joint r_shoulder_yaw: limit lower=-0.8726646259971648 upper=1.3962634015954636 effort=50000 velocity=120.0 -> lower=-0.9075712110370514 upper=1.4311699866353502 effort=50000 velocity=120.0
- joint r_wrist_pitch: limit lower=-0.5585053606381855 upper=0.5585053606381855 effort=50000 velocity=120.0 -> lower=-0.3490658503988659 upper=0.3490658503988659 effort=50000 velocity=120.0
- joint r_wrist_roll: limit lower=-1.0821041362364843 upper=0.9075712110370514 effort=50000 velocity=120.0 -> lower=-0.3490658503988659 upper=0.5235987755982988 effort=50000 velocity=120.0
- joint torso_pitch: limit lower=-0.3141592653589793 upper=0.7853981633974483 effort=50000 velocity=120.0 -> lower=-0.3490658503988659 upper=1.1344640137963142 effort=50000 velocity=120.0
- joint torso_roll: limit lower=-0.4014257279586958 upper=0.4014257279586958 effort=50000 velocity=120.0 -> lower=-0.4363323129985824 upper=0.4363323129985824 effort=50000 velocity=120.0
- joint torso_yaw: limit lower=-0.7504915783575618 upper=0.7504915783575618 effort=50000 velocity=120.0 -> lower=-0.7853981633974483 upper=0.7853981633974483 effort=50000 velocity=120.0

File: urdf/ergoCub/robots/ergoCubGazeboV1_minContacts/model.urdf (robot description, URDF)
Before this commit: robot ergoCub, 202 links, 201 joints
Joints:
- joint l_elbow: limit lower=-0.05235987755982989 upper=1.3089969389957472 effort=50000 velocity=120.0 -> lower=-0.08726646259971647 upper=2.0943951023931953 effort=50000 velocity=120.0
- joint l_hip_pitch: limit lower=-0.7504915783575618 upper=1.7976891295541595 effort=50000 velocity=120.0 -> lower=-0.767944870877505 upper=1.9198621771937625 effort=50000 velocity=120.0
- joint l_hip_roll: limit lower=-0.2792526803190927 upper=1.9024088846738192 effort=50000 velocity=120.0 -> lower=-0.3490658503988659 upper=1.9373154697137058 effort=50000 velocity=120.0
- joint l_hip_yaw: limit lower=-1.3788101090755203 upper=1.3788101090755203 effort=50000 velocity=120.0 -> lower=-1.413716694115407 upper=1.413716694115407 effort=50000 velocity=120.0
- joint l_knee: limit lower=-1.8151424220741028 upper=0.10471975511965978 effort=50000 velocity=120.0 -> lower=-1.8325957145940461 upper=0.12217304763960307 effort=50000 velocity=120.0
- joint l_shoulder_yaw: limit lower=-0.8726646259971648 upper=1.3962634015954636 effort=50000 velocity=120.0 -> lower=-0.9075712110370514 upper=1.4311699866353502 effort=50000 velocity=120.0
- joint l_wrist_pitch: limit lower=-0.5585053606381855 upper=0.5585053606381855 effort=50000 velocity=120.0 -> lower=-0.3490658503988659 upper=0.3490658503988659 effort=50000 velocity=120.0
- joint l_wrist_roll: limit lower=-1.0821041362364843 upper=0.9075712110370514 effort=50000 velocity=120.0 -> lower=-0.3490658503988659 upper=0.5235987755982988 effort=50000 velocity=120.0
- joint neck_pitch: limit lower=-0.5235987755982988 upper=0.3839724354387525 effort=50000 velocity=120.0 -> lower=-0.7853981633974483 upper=0.3839724354387525 effort=50000 velocity=120.0
- joint r_elbow: limit lower=-0.05235987755982989 upper=1.3089969389957472 effort=50000 velocity=120.0 -> lower=-0.08726646259971647 upper=2.0943951023931953 effort=50000 velocity=120.0
- joint r_hip_pitch: limit lower=-0.7504915783575618 upper=1.7976891295541595 effort=50000 velocity=120.0 -> lower=-0.767944870877505 upper=1.9198621771937625 effort=50000 velocity=120.0
- joint r_hip_roll: limit lower=-0.2792526803190927 upper=1.9024088846738192 effort=50000 velocity=120.0 -> lower=-0.3490658503988659 upper=1.9373154697137058 effort=50000 velocity=120.0
- joint r_hip_yaw: limit lower=-1.3788101090755203 upper=1.3788101090755203 effort=50000 velocity=120.0 -> lower=-1.413716694115407 upper=1.413716694115407 effort=50000 velocity=120.0
- joint r_knee: limit lower=-1.8151424220741028 upper=0.10471975511965978 effort=50000 velocity=120.0 -> lower=-1.8325957145940461 upper=0.12217304763960307 effort=50000 velocity=120.0
- joint r_shoulder_yaw: limit lower=-0.8726646259971648 upper=1.3962634015954636 effort=50000 velocity=120.0 -> lower=-0.9075712110370514 upper=1.4311699866353502 effort=50000 velocity=120.0
- joint r_wrist_pitch: limit lower=-0.5585053606381855 upper=0.5585053606381855 effort=50000 velocity=120.0 -> lower=-0.3490658503988659 upper=0.3490658503988659 effort=50000 velocity=120.0
- joint r_wrist_roll: limit lower=-1.0821041362364843 upper=0.9075712110370514 effort=50000 velocity=120.0 -> lower=-0.3490658503988659 upper=0.5235987755982988 effort=50000 velocity=120.0
- joint torso_pitch: limit lower=-0.3141592653589793 upper=0.7853981633974483 effort=50000 velocity=120.0 -> lower=-0.3490658503988659 upper=1.1344640137963142 effort=50000 velocity=120.0
- joint torso_roll: limit lower=-0.4014257279586958 upper=0.4014257279586958 effort=50000 velocity=120.0 -> lower=-0.4363323129985824 upper=0.4363323129985824 effort=50000 velocity=120.0
- joint torso_yaw: limit lower=-0.7504915783575618 upper=0.7504915783575618 effort=50000 velocity=120.0 -> lower=-0.7853981633974483 upper=0.7853981633974483 effort=50000 velocity=120.0

File: urdf/ergoCub/robots/ergoCubSN000/model.urdf (robot description, URDF)
Before this commit: robot ergoCub, 202 links, 201 joints
Joints:
- joint l_elbow: limit lower=-0.05235987755982989 upper=1.3089969389957472 effort=50000 velocity=120.0 -> lower=-0.08726646259971647 upper=2.0943951023931953 effort=50000 velocity=120.0
- joint l_hip_pitch: limit lower=-0.7504915783575618 upper=1.7976891295541595 effort=50000 velocity=120.0 -> lower=-0.767944870877505 upper=1.9198621771937625 effort=50000 velocity=120.0
- joint l_hip_roll: limit lower=-0.2792526803190927 upper=1.9024088846738192 effort=50000 velocity=120.0 -> lower=-0.3490658503988659 upper=1.9373154697137058 effort=50000 velocity=120.0
- joint l_hip_yaw: limit lower=-1.3788101090755203 upper=1.3788101090755203 effort=50000 velocity=120.0 -> lower=-1.413716694115407 upper=1.413716694115407 effort=50000 velocity=120.0
- joint l_knee: limit lower=-1.8151424220741028 upper=0.10471975511965978 effort=50000 velocity=120.0 -> lower=-1.8325957145940461 upper=0.12217304763960307 effort=50000 velocity=120.0
- joint l_shoulder_yaw: limit lower=-0.8726646259971648 upper=1.3962634015954636 effort=50000 velocity=120.0 -> lower=-0.9075712110370514 upper=1.4311699866353502 effort=50000 velocity=120.0
- joint l_wrist_pitch: limit lower=-0.5585053606381855 upper=0.5585053606381855 effort=50000 velocity=120.0 -> lower=-0.3490658503988659 upper=0.3490658503988659 effort=50000 velocity=120.0
- joint l_wrist_roll: limit lower=-1.0821041362364843 upper=0.9075712110370514 effort=50000 velocity=120.0 -> lower=-0.3490658503988659 upper=0.5235987755982988 effort=50000 velocity=120.0
- joint neck_pitch: limit lower=-0.5235987755982988 upper=0.3839724354387525 effort=50000 velocity=120.0 -> lower=-0.7853981633974483 upper=0.3839724354387525 effort=50000 velocity=120.0
- joint r_elbow: limit lower=-0.05235987755982989 upper=1.3089969389957472 effort=50000 velocity=120.0 -> lower=-0.08726646259971647 upper=2.0943951023931953 effort=50000 velocity=120.0
- joint r_hip_pitch: limit lower=-0.7504915783575618 upper=1.7976891295541595 effort=50000 velocity=120.0 -> lower=-0.767944870877505 upper=1.9198621771937625 effort=50000 velocity=120.0
- joint r_hip_roll: limit lower=-0.2792526803190927 upper=1.9024088846738192 effort=50000 velocity=120.0 -> lower=-0.3490658503988659 upper=1.9373154697137058 effort=50000 velocity=120.0
- joint r_hip_yaw: limit lower=-1.3788101090755203 upper=1.3788101090755203 effort=50000 velocity=120.0 -> lower=-1.413716694115407 upper=1.413716694115407 effort=50000 velocity=120.0
- joint r_knee: limit lower=-1.8151424220741028 upper=0.10471975511965978 effort=50000 velocity=120.0 -> lower=-1.8325957145940461 upper=0.12217304763960307 effort=50000 velocity=120.0
- joint r_shoulder_yaw: limit lower=-0.8726646259971648 upper=1.3962634015954636 effort=50000 velocity=120.0 -> lower=-0.9075712110370514 upper=1.4311699866353502 effort=50000 velocity=120.0
- joint r_wrist_pitch: limit lower=-0.5585053606381855 upper=0.5585053606381855 effort=50000 velocity=120.0 -> lower=-0.3490658503988659 upper=0.3490658503988659 effort=50000 velocity=120.0
- joint r_wrist_roll: limit lower=-1.0821041362364843 upper=0.9075712110370514 effort=50000 velocity=120.0 -> lower=-0.3490658503988659 upper=0.5235987755982988 effort=50000 velocity=120.0
- joint torso_pitch: limit lower=-0.3141592653589793 upper=0.7853981633974483 effort=50000 velocity=120.0 -> lower=-0.3490658503988659 upper=1.1344640137963142 effort=50000 velocity=120.0
- joint torso_roll: limit lower=-0.4014257279586958 upper=0.4014257279586958 effort=50000 velocity=120.0 -> lower=-0.4363323129985824 upper=0.4363323129985824 effort=50000 velocity=120.0
- joint torso_yaw: limit lower=-0.7504915783575618 upper=0.7504915783575618 effort=50000 velocity=120.0 -> lower=-0.7853981633974483 upper=0.7853981633974483 effort=50000 velocity=120.0
