Commit message: Add assigned geometricshapes

File: urdf/ergoCub/robots/ergoCubGazeboV1_1_minContacts/model.urdf (robot description, URDF)
Before this commit: robot ergoCub, 204 links, 203 joints
Links:
- link chest: geometry collision box size=0 0 0; visual mesh filename=package://ergoCub/meshes/simmechanics/sim_ecub_1-1_chest.stl scale=0.001 0.001 0.001
- link head: geometry collision box size=0 0 0; visual mesh filename=package://ergoCub/meshes/simmechanics/sim_ecub_1-1_head.stl scale=0.001 0.001 0.001
- link l_ankle_1: geometry collision box size=0 0 0; visual mesh filename=package://ergoCub/meshes/simmechanics/sim_ecub_1-1_l_ankle_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 scale=0.001 0.001 0.001
- link l_ankle_2: geometry collision box size=0 0 0; visual mesh filename=package://ergoCub/meshes/simmechanics/sim_ecub_1-1_l_ankle_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 scale=0.001 0.001 0.001
- link l_foot_front: geometry collision box size=0.117 0.1 0.006; visual mesh filename=package://ergoCub/meshes/simmechanics/sim_ecub_1-1_l_foot_f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 scale=0.001 0.001 0.001
- link l_foot_rear: geometry collision box size=0.117 0.1 0.006; visual mesh filename=package://ergoCub/meshes/simmechanics/sim_ecub_1-1_l_foot_r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 scale=0.001 0.001 0.001
- link l_forearm: geometry collision box size=0 0 0; visual mesh filename=package://ergoCub/meshes/simmechanics/sim_ecub_1-1_l_forear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 scale=0.001 0.001 0.001
- link l_hand_index_1: geometry collision box size=0 0 0; visual mesh filename=package://ergoCub/meshes/simmechanics/sim_ecub_1-1_l_hand_i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 scale=0.001 0.001 0.001
- link l_hand_index_2: geometry collision box size=0 0 0; visual mesh filename=package://ergoCub/meshes/simmechanics/sim_ecub_1-1_l_hand_i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 scale=0.001 0.001 0.001
- link l_hand_index_3: geometry collision box size=0 0 0; visual mesh filename=package://ergoCub/meshes/simmechanics/sim_ecub_1-1_l_hand_i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 scale=0.001 0.001 0.001
- link l_hand_middle_1: geometry collision box size=0 0 0; visual mesh filename=package://ergoCub/meshes/simmechanics/sim_ecub_1-1_l_hand_m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 scale=0.001 0.001 0.001
- link l_hand_middle_2: geometry collision box size=0 0 0; visual mesh filename=package://ergoCub/meshes/simmechanics/sim_ecub_1-1_l_hand_m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 scale=0.001 0.001 0.001
- link l_hand_palm: geometry collision box size=0 0 0; visual mesh filename=package://ergoCub/meshes/simmechanics/sim_ecub_1-1_l_hand_p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 scale=0.001 0.001 0.001
- link l_hand_pinkie_1: geometry collision box size=0 0 0; visual mesh filename=package://ergoCub/meshes/simmechanics/sim_ecub_1-1_l_hand_p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 scale=0.001 0.001 0.001
- link l_hand_pinkie_2: geometry collision box size=0 0 0; visual mesh filename=package://ergoCub/meshes/simmechanics/sim_ecub_1-1_l_hand_p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 scale=0.001 0.001 0.001
- link l_hand_ring_1: geometry collision box size=0 0 0; visual mesh filename=package://ergoCub/meshes/simmechanics/sim_ecub_1-1_l_hand_r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 scale=0.001 0.001 0.001
- link l_hand_ring_2: geometry collision box size=0 0 0; visual mesh filename=package://ergoCub/meshes/simmechanics/sim_ecub_1-1_l_hand_r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 scale=0.001 0.001 0.001
- link l_hand_thumb_1: geometry collision box size=0 0 0; visual mesh filename=package://ergoCub/meshes/simmechanics/sim_ecub_1-1_l_hand_t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 scale=0.001 0.001 0.001
- link l_hand_thumb_2: geometry collision box size=0 0 0; visual mesh filename=package://ergoCub/meshes/simmechanics/sim_ecub_1-1_l_hand_t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 scale=0.001 0.001 0.001
- link l_hand_thumb_3: geometry collision box size=0 0 0; visual mesh filename=package://ergoCub/meshes/simmechanics/sim_ecub_1-1_l_hand_t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 scale=0.001 0.001 0.001
- link l_hip_1: geometry collision box size=0 0 0; visual mesh filename=package://ergoCub/meshes/simmechanics/sim_ecub_1-1_l_hip_1.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 scale=0.001 0.001 0.001
- link l_hip_2: geometry collision box size=0 0 0; visual mesh filename=package://ergoCub/meshes/simmechanics/sim_ecub_1-1_l_hip_2.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 scale=0.001 0.001 0.001
- link l_hip_3: geometry collision box size=0 0 0; visual mesh filename=package://ergoCub/meshes/simmechanics/sim_ecub_1-1_l_hip_3.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 scale=0.001 0.001 0.001
- link l_lower_leg: geometry collision box size=0 0 0; visual mesh filename=package://ergoCub/meshes/simmechanics/sim_ecub_1-1_l_lower_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 scale=0.001 0.001 0.001
- link l_shoulder_1: geometry collision box size=0 0 0; visual mesh filename=package://ergoCub/meshes/simmechanics/sim_ecub_1-1_l_should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 scale=0.001 0.001 0.001
- link l_shoulder_2: geometry collision box size=0 0 0; visual mesh filename=package://ergoCub/meshes/simmechanics/sim_ecub_1-1_l_should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 scale=0.001 0.001 0.001
- link l_shoulder_3: geometry collision box size=0 0 0; visual mesh filename=package://ergoCub/meshes/simmechanics/sim_ecub_1-1_l_should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 scale=0.001 0.001 0.001
- link l_upper_leg: geometry collision box size=0 0 0; visual mesh filename=package://ergoCub/meshes/simmechanics/sim_ecub_1-1_l_upper_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 scale=0.001 0.001 0.001
- link l_wrist_1: geometry collision box size=0 0 0; visual mesh filename=package://ergoCub/meshes/simmechanics/sim_ecub_1-1_l_wrist_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 scale=0.001 0.001 0.001
- link l_wrist_2: geometry collision box size=0 0 0; visual mesh filename=package://ergoCub/meshes/simmechanics/sim_ecub_1-1_l_wrist_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 scale=0.001 0.001 0.001
- link neck_2: geometry collision box size=0 0 0; visual mesh filename=package://ergoCub/meshes/simmechanics/sim_ecub_1-1_head_nec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 scale=0.001 0.001 0.001
- link neck_3: geometry collision box size=0 0 0; visual mesh filename=package://ergoCub/meshes/simmechanics/sim_ecub_1-1_head_nec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 scale=0.001 0.001 0.001
- link r_ankle_1: geometry collision box size=0 0 0; visual mesh filename=package://ergoCub/meshes/simmechanics/sim_ecub_1-1_r_ankle_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 scale=0.001 0.001 0.001
- link r_ankle_2: geometry collision box size=0 0 0; visual mesh filename=package://ergoCub/meshes/simmechanics/sim_ecub_1-1_r_ankle_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 scale=0.001 0.001 0.001
- link r_foot_front: geometry collision box size=0.117 0.1 0.006; visual mesh filename=package://ergoCub/meshes/simmechanics/sim_ecub_1-1_r_foot_f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 scale=0.001 0.001 0.001
- link r_foot_rear: geometry collision box size=0.117 0.1 0.006; visual mesh filename=package://ergoCub/meshes/simmechanics/sim_ecub_1-1_r_foot_r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 scale=0.001 0.001 0.001
- link r_forearm: geometry collision box size=0 0 0; visual mesh filename=package://ergoCub/meshes/simmechanics/sim_ecub_1-1_r_forear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 scale=0.001 0.001 0.001
- link r_hand_index_1: geometry collision box size=0 0 0; visual mesh filename=package://ergoCub/meshes/simmechanics/sim_ecub_1-1_r_hand_i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 scale=0.001 0.001 0.001
- link r_hand_index_2: geometry collision box size=0 0 0; visual mesh filename=package://ergoCub/meshes/simmechanics/sim_ecub_1-1_r_hand_i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 scale=0.001 0.001 0.001
- link r_hand_index_3: geometry collision box size=0 0 0; visual mesh filename=package://ergoCub/meshes/simmechanics/sim_ecub_1-1_r_hand_i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 scale=0.001 0.001 0.001
- link r_hand_middle_1: geometry collision box size=0 0 0; visual mesh filename=package://ergoCub/meshes/simmechanics/sim_ecub_1-1_r_hand_m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 scale=0.001 0.001 0.001
- link r_hand_middle_2: geometry collision box size=0 0 0; visual mesh filename=package://ergoCub/meshes/simmechanics/sim_ecub_1-1_r_hand_m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 scale=0.001 0.001 0.001
- link r_hand_palm: geometry collision box size=0 0 0; visual mesh filename=package://ergoCub/meshes/simmechanics/sim_ecub_1-1_r_hand_p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 scale=0.001 0.001 0.001
- link r_hand_pinkie_1: geometry collision box size=0 0 0; visual mesh filename=package://ergoCub/meshes/simmechanics/sim_ecub_1-1_r_hand_p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 scale=0.001 0.001 0.001
- link r_hand_pinkie_2: geometry collision box size=0 0 0; visual mesh filename=package://ergoCub/meshes/simmechanics/sim_ecub_1-1_r_hand_p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 scale=0.001 0.001 0.001
- link r_hand_ring_1: geometry collision box size=0 0 0; visual mesh filename=package://ergoCub/meshes/simmechanics/sim_ecub_1-1_r_hand_r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 scale=0.001 0.001 0.001
- link r_hand_ring_2: geometry collision box size=0 0 0; visual mesh filename=package://ergoCub/meshes/simmechanics/sim_ecub_1-1_r_hand_r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 scale=0.001 0.001 0.001
- link r_hand_thumb_1: geometry collision box size=0 0 0; visual mesh filename=package://ergoCub/meshes/simmechanics/sim_ecub_1-1_r_hand_t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 scale=0.001 0.001 0.001
- link r_hand_thumb_2: geometry collision box size=0 0 0; visual mesh filename=package://ergoCub/meshes/simmechanics/sim_ecub_1-1_r_hand_t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 scale=0.001 0.001 0.001
- link r_hand_thumb_3: geometry collision box size=0 0 0; visual mesh filename=package://ergoCub/meshes/simmechanics/sim_ecub_1-1_r_hand_t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 scale=0.001 0.001 0.001
- link r_hip_1: geometry collision box size=0 0 0; visual mesh filename=package://ergoCub/meshes/simmechanics/sim_ecub_1-1_r_hip_1.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 scale=0.001 0.001 0.001
- link r_hip_2: geometry collision box size=0 0 0; visual mesh filename=package://ergoCub/meshes/simmechanics/sim_ecub_1-1_r_hip_2.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 scale=0.001 0.001 0.001
- link r_hip_3: geometry collision box size=0 0 0; visual mesh filename=package://ergoCub/meshes/simmechanics/sim_ecub_1-1_r_hip_3.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 scale=0.001 0.001 0.001
- link r_lower_leg: geometry collision box size=0 0 0; visual mesh filename=package://ergoCub/meshes/simmechanics/sim_ecub_1-1_r_lower_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 scale=0.001 0.001 0.001
- link r_shoulder_1: geometry collision box size=0 0 0; visual mesh filename=package://ergoCub/meshes/simmechanics/sim_ecub_1-1_r_should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 scale=0.001 0.001 0.001
- link r_shoulder_2: geometry collision box size=0 0 0; visual mesh filename=package://ergoCub/meshes/simmechanics/sim_ecub_1-1_r_should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 scale=0.001 0.001 0.001
- link r_shoulder_3: geometry collision box size=0 0 0; visual mesh filename=package://ergoCub/meshes/simmechanics/sim_ecub_1-1_r_should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 scale=0.001 0.001 0.001
- link r_upper_leg: geometry collision box size=0 0 0; visual mesh filename=package://ergoCub/meshes/simmechanics/sim_ecub_1-1_r_upper_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 scale=0.001 0.001 0.001
- link r_wrist_1: geometry collision box size=0 0 0; visual mesh filename=package://ergoCub/meshes/simmechanics/sim_ecub_1-1_r_wrist_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 scale=0.001 0.001 0.001
- link r_wrist_2: geometry collision box size=0 0 0; visual mesh filename=package://ergoCub/meshes/simmechanics/sim_ecub_1-1_r_wrist_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 scale=0.001 0.001 0.001
- link realsense: geometry collision box size=0 0 0; visual mesh filename=package://ergoCub/meshes/simmechanics/sim_ecub_1-1_realsens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 scale=0.001 0.001 0.001
- link root_link: geometry collision box size=0 0 0; visual mesh filename=package://ergoCub/meshes/simmechanics/sim_ecub_1-1_root_lin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 scale=0.001 0.001 0.001
- link torso_1: geometry collision box size=0 0 0; visual mesh filename=package://ergoCub/meshes/simmechanics/sim_ecub_1-1_torso_1.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 scale=0.001 0.001 0.001
- link torso_2: geometry collision box size=0 0 0; visual mesh filename=package://ergoCub/meshes/simmechanics/sim_ecub_1-1_torso_2.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 scale=0.001 0.001 0.001

Commit message: ergoCubV1_1_minContacts: fix the collision after the fix of upperarm links

File: urdf/ergoCub/robots/ergoCubGazeboV1_1_minContacts/model.urdf (robot description, URDF)
Before this commit: robot ergoCub, 204 links, 203 joints
Links:
- link l_upper_arm: geometry collision box size=0 0 0; visual mesh filename=package://ergoCub/meshes/simmechanics/sim_ecub_1-1_l_uppera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 scale=0.001 0.001 0.001
- link r_upper_arm: geometry collision box size=0 0 0; visual mesh filename=package://ergoCub/meshes/simmechanics/sim_ecub_1-1_r_uppera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 scale=0.001 0.001 0.001

Commit message: ergoCubGazeboV1_1_minContacts: fix regression after #222

File: urdf/ergoCub/robots/ergoCubGazeboV1_1_minContacts/model.urdf (robot description, URDF)
Before this commit: robot ergoCub, 204 links, 203 joints
Joints:
- joint l_index_add: axis 1.3005559878087045e-15 1.0000000000000002 -1.953448495705706e-15 -> 1.1895336853461886e-15 0.9999999999999999 -1.9812040713213337e-15; origin xyz=0.022500000000000034 -0.0015000000000006397 -0.06859999999999966 rpy=-8.126657451512497e-16 -0.2967059722446555 1.7414265967526777e-16 -> xyz=0.022500000000000023 -0.0015000000000006952 -0.0685999999999996 rpy=-8.416895217637947e-16 -0.29670597224465534 5.804755322508926e-17
- joint l_index_dist: axis -1 -1.804112664227406e-16 9.020562801946248e-17 -> -1 -2.359224176539984e-16 4.163337069211178e-17; origin xyz=-2.7755575615628914e-17 -0.0014999999999999736 -0.039999999999999925 rpy=-7.482326169760975e-8 1.734723475976807e-16 -6.106226635438361e-16 -> xyz=-1.3877787807814457e-17 -0.001500000000000029 -0.03999999999999987 rpy=-7.482326172536535e-8 1.8041124150158794e-16 -6.106226635438361e-16
- joint l_index_prox: axis -1.0000000000000002 2.7755575615627613e-17 7.023654366444809e-10 -> -1 8.326672684688522e-17 7.023654435833748e-10; origin xyz=0.009192533346793416 -2.7755575615628914e-17 -0.030713451309624162 rpy=-2.7755575615628914e-16 -7.023611553469422e-10 -7.771561172376094e-16 -> xyz=0.00919253334679343 0 -0.030713451309624218 rpy=-3.0531133177191815e-16 -7.023611484080483e-10 -7.771561172376096e-16

Commit message: ergoCubSN001/ergoCubGazeboV1_1*: fix orientation of inertias
It fixes #224. Model regenerated after https://github.com/icub-tech-iit/creo2urdf/pull/83

File: urdf/ergoCub/robots/ergoCubGazeboV1_1_minContacts/model.urdf (robot description, URDF)
Before this commit: robot ergoCub, 204 links, 203 joints
Joints:
- joint l_index_add: axis 1.1895336853461886e-15 0.9999999999999999 -1.9812040713213337e-15 -> 1.3005559878087045e-15 1.0000000000000002 -1.953448495705706e-15; origin xyz=0.022500000000000023 -0.0015000000000006952 -0.0685999999999996 rpy=-8.416895217637947e-16 -0.29670597224465534 5.804755322508926e-17 -> xyz=0.022500000000000034 -0.0015000000000006397 -0.06859999999999966 rpy=-8.126657451512497e-16 -0.2967059722446555 1.7414265967526777e-16
- joint l_index_dist: axis -1 -2.359224176539984e-16 4.163337069211178e-17 -> -1 -1.804112664227406e-16 9.020562801946248e-17; origin xyz=-1.3877787807814457e-17 -0.001500000000000029 -0.03999999999999987 rpy=-7.482326172536535e-8 1.8041124150158794e-16 -6.106226635438361e-16 -> xyz=-2.7755575615628914e-17 -0.0014999999999999736 -0.039999999999999925 rpy=-7.482326169760975e-8 1.734723475976807e-16 -6.106226635438361e-16
- joint l_index_prox: axis -1 8.326672684688522e-17 7.023654435833748e-10 -> -1.0000000000000002 2.7755575615627613e-17 7.023654366444809e-10; origin xyz=0.00919253334679343 0 -0.030713451309624218 rpy=-3.0531133177191815e-16 -7.023611484080483e-10 -7.771561172376096e-16 -> xyz=0.009192533346793416 -2.7755575615628914e-17 -0.030713451309624162 rpy=-2.7755575615628914e-16 -7.023611553469422e-10 -7.771561172376094e-16
