Commit message: Automatic update of urdf triggered by GitHub Action
ergocub-software = 5b657faa8a3a180de7a4c1ffbfdb4935380d4e4a
cad-libraries    = https://github.com/icub-tech-iit/cad-libraries/commit/f5522204eb73c981c8722c15328c65abaf0c1f7f
cad-mechanics    = https://github.com/icub-tech-iit/cad-mechanics/commit/7221fbdf8a6d1332bf47bfb82cc037e8c1ac252e
creo2urdf        = https://github.com/icub-tech-iit/creo2urdf/releases/tag/v0.5.11

File: urdf/ergoCub/robots/ergoCubGazeboV1_1_minContacts/model.urdf (robot description, URDF)
Before this commit: robot ergoCub, 204 links, 203 joints
Links:
- link chest: geometry collision mesh filename=package://ergoCub/meshes/simmechanics/sim_ecub_1-1_chest.obj scale=0.001 0.001 0.001; visual mesh filename=package://ergoCub/meshes/simmechanics/sim_ecub_1-1_chest.obj scale=0.001 0.001 0.001
- link head: geometry collision mesh filename=package://ergoCub/meshes/simmechanics/sim_ecub_1-1_head.obj scale=0.001 0.001 0.001; visual mesh filename=package://ergoCub/meshes/simmechanics/sim_ecub_1-1_head.obj scale=0.001 0.001 0.001
- link l_ankle_1: geometry collision mesh filename=package://ergoCub/meshes/simmechanics/sim_ecub_1-1_l_ankle_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 scale=0.001 0.001 0.001; visual mesh filename=package://ergoCub/meshes/simmechanics/sim_ecub_1-1_l_ankle_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 scale=0.001 0.001 0.001
- link l_ankle_2: geometry collision mesh filename=package://ergoCub/meshes/simmechanics/sim_ecub_1-1_l_ankle_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 scale=0.001 0.001 0.001; visual mesh filename=package://ergoCub/meshes/simmechanics/sim_ecub_1-1_l_ankle_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 scale=0.001 0.001 0.001
- link l_forearm: geometry collision mesh filename=package://ergoCub/meshes/simmechanics/sim_ecub_1-1_l_forear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 scale=0.001 0.001 0.001; visual mesh filename=package://ergoCub/meshes/simmechanics/sim_ecub_1-1_l_forear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 scale=0.001 0.001 0.001
- link l_hand_index_1: geometry collision mesh filename=package://ergoCub/meshes/simmechanics/sim_ecub_1-1_l_hand_i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 scale=0.001 0.001 0.001; visual mesh filename=package://ergoCub/meshes/simmechanics/sim_ecub_1-1_l_hand_i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 scale=0.001 0.001 0.001
- link l_hand_index_2: geometry collision mesh filename=package://ergoCub/meshes/simmechanics/sim_ecub_1-1_l_hand_i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 scale=0.001 0.001 0.001; visual mesh filename=package://ergoCub/meshes/simmechanics/sim_ecub_1-1_l_hand_i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 scale=0.001 0.001 0.001
- link l_hand_index_3: geometry collision mesh filename=package://ergoCub/meshes/simmechanics/sim_ecub_1-1_l_hand_i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 scale=0.001 0.001 0.001; visual mesh filename=package://ergoCub/meshes/simmechanics/sim_ecub_1-1_l_hand_i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 scale=0.001 0.001 0.001
- link l_hand_middle_1: geometry collision mesh filename=package://ergoCub/meshes/simmechanics/sim_ecub_1-1_l_hand_m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 scale=0.001 0.001 0.001; visual mesh filename=package://ergoCub/meshes/simmechanics/sim_ecub_1-1_l_hand_m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 scale=0.001 0.001 0.001
- link l_hand_middle_2: geometry collision mesh filename=package://ergoCub/meshes/simmechanics/sim_ecub_1-1_l_hand_m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 scale=0.001 0.001 0.001; visual mesh filename=package://ergoCub/meshes/simmechanics/sim_ecub_1-1_l_hand_m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 scale=0.001 0.001 0.001
- link l_hand_palm: geometry collision mesh filename=package://ergoCub/meshes/simmechanics/sim_ecub_1-1_l_hand_p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 scale=0.001 0.001 0.001; visual mesh filename=package://ergoCub/meshes/simmechanics/sim_ecub_1-1_l_hand_p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 scale=0.001 0.001 0.001
- link l_hand_pinkie_1: geometry collision mesh filename=package://ergoCub/meshes/simmechanics/sim_ecub_1-1_l_hand_p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 scale=0.001 0.001 0.001; visual mesh filename=package://ergoCub/meshes/simmechanics/sim_ecub_1-1_l_hand_p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 scale=0.001 0.001 0.001
- link l_hand_pinkie_2: geometry collision mesh filename=package://ergoCub/meshes/simmechanics/sim_ecub_1-1_l_hand_p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 scale=0.001 0.001 0.001; visual mesh filename=package://ergoCub/meshes/simmechanics/sim_ecub_1-1_l_hand_p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 scale=0.001 0.001 0.001
- link l_hand_ring_1: geometry collision mesh filename=package://ergoCub/meshes/simmechanics/sim_ecub_1-1_l_hand_r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 scale=0.001 0.001 0.001; visual mesh filename=package://ergoCub/meshes/simmechanics/sim_ecub_1-1_l_hand_r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 scale=0.001 0.001 0.001
- link l_hand_ring_2: geometry collision mesh filename=package://ergoCub/meshes/simmechanics/sim_ecub_1-1_l_hand_r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 scale=0.001 0.001 0.001; visual mesh filename=package://ergoCub/meshes/simmechanics/sim_ecub_1-1_l_hand_r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 scale=0.001 0.001 0.001
- link l_hand_thumb_1: geometry collision mesh filename=package://ergoCub/meshes/simmechanics/sim_ecub_1-1_l_hand_t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 scale=0.001 0.001 0.001; visual mesh filename=package://ergoCub/meshes/simmechanics/sim_ecub_1-1_l_hand_t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 scale=0.001 0.001 0.001
- link l_hand_thumb_2: geometry collision mesh filename=package://ergoCub/meshes/simmechanics/sim_ecub_1-1_l_hand_t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 scale=0.001 0.001 0.001; visual mesh filename=package://ergoCub/meshes/simmechanics/sim_ecub_1-1_l_hand_t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 scale=0.001 0.001 0.001
- link l_hand_thumb_3: geometry collision mesh filename=package://ergoCub/meshes/simmechanics/sim_ecub_1-1_l_hand_t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 scale=0.001 0.001 0.001; visual mesh filename=package://ergoCub/meshes/simmechanics/sim_ecub_1-1_l_hand_t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 scale=0.001 0.001 0.001
- link l_hip_1: geometry collision mesh filename=package://ergoCub/meshes/simmechanics/sim_ecub_1-1_l_hip_1.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 scale=0.001 0.001 0.001; visual mesh filename=package://ergoCub/meshes/simmechanics/sim_ecub_1-1_l_hip_1.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 scale=0.001 0.001 0.001
- link l_hip_2: geometry collision mesh filename=package://ergoCub/meshes/simmechanics/sim_ecub_1-1_l_hip_2.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 scale=0.001 0.001 0.001; visual mesh filename=package://ergoCub/meshes/simmechanics/sim_ecub_1-1_l_hip_2.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 scale=0.001 0.001 0.001
- link l_hip_3: geometry collision mesh filename=package://ergoCub/meshes/simmechanics/sim_ecub_1-1_l_hip_3.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 scale=0.001 0.001 0.001; visual mesh filename=package://ergoCub/meshes/simmechanics/sim_ecub_1-1_l_hip_3.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 scale=0.001 0.001 0.001
- link l_lower_leg: geometry collision mesh filename=package://ergoCub/meshes/simmechanics/sim_ecub_1-1_l_lower_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 scale=0.001 0.001 0.001; visual mesh filename=package://ergoCub/meshes/simmechanics/sim_ecub_1-1_l_lower_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 scale=0.001 0.001 0.001
- link l_shoulder_1: geometry collision mesh filename=package://ergoCub/meshes/simmechanics/sim_ecub_1-1_l_should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 scale=0.001 0.001 0.001; visual mesh filename=package://ergoCub/meshes/simmechanics/sim_ecub_1-1_l_should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 scale=0.001 0.001 0.001
- link l_shoulder_2: geometry collision mesh filename=package://ergoCub/meshes/simmechanics/sim_ecub_1-1_l_should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 scale=0.001 0.001 0.001; visual mesh filename=package://ergoCub/meshes/simmechanics/sim_ecub_1-1_l_should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 scale=0.001 0.001 0.001
- link l_shoulder_3: geometry collision mesh filename=package://ergoCub/meshes/simmechanics/sim_ecub_1-1_l_should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 scale=0.001 0.001 0.001; visual mesh filename=package://ergoCub/meshes/simmechanics/sim_ecub_1-1_l_should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 scale=0.001 0.001 0.001
- link l_upper_arm: geometry collision mesh filename=package://ergoCub/meshes/simmechanics/sim_ecub_1-1_l_uppera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 scale=0.001 0.001 0.001; visual mesh filename=package://ergoCub/meshes/simmechanics/sim_ecub_1-1_l_uppera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 scale=0.001 0.001 0.001
- link l_upper_leg: geometry collision mesh filename=package://ergoCub/meshes/simmechanics/sim_ecub_1-1_l_upper_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 scale=0.001 0.001 0.001; visual mesh filename=package://ergoCub/meshes/simmechanics/sim_ecub_1-1_l_upper_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 scale=0.001 0.001 0.001
- link l_wrist_1: geometry collision mesh filename=package://ergoCub/meshes/simmechanics/sim_ecub_1-1_l_wrist_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 scale=0.001 0.001 0.001; visual mesh filename=package://ergoCub/meshes/simmechanics/sim_ecub_1-1_l_wrist_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 scale=0.001 0.001 0.001
- link l_wrist_2: geometry collision mesh filename=package://ergoCub/meshes/simmechanics/sim_ecub_1-1_l_wrist_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 scale=0.001 0.001 0.001; visual mesh filename=package://ergoCub/meshes/simmechanics/sim_ecub_1-1_l_wrist_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 scale=0.001 0.001 0.001
- link neck_2: geometry collision mesh filename=package://ergoCub/meshes/simmechanics/sim_ecub_1-1_head_nec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 scale=0.001 0.001 0.001; visual mesh filename=package://ergoCub/meshes/simmechanics/sim_ecub_1-1_head_nec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 scale=0.001 0.001 0.001
- link neck_3: geometry collision mesh filename=package://ergoCub/meshes/simmechanics/sim_ecub_1-1_head_nec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 scale=0.001 0.001 0.001; visual mesh filename=package://ergoCub/meshes/simmechanics/sim_ecub_1-1_head_nec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 scale=0.001 0.001 0.001
- link r_ankle_1: geometry collision mesh filename=package://ergoCub/meshes/simmechanics/sim_ecub_1-1_r_ankle_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 scale=0.001 0.001 0.001; visual mesh filename=package://ergoCub/meshes/simmechanics/sim_ecub_1-1_r_ankle_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 scale=0.001 0.001 0.001
- link r_ankle_2: geometry collision mesh filename=package://ergoCub/meshes/simmechanics/sim_ecub_1-1_r_ankle_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 scale=0.001 0.001 0.001; visual mesh filename=package://ergoCub/meshes/simmechanics/sim_ecub_1-1_r_ankle_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 scale=0.001 0.001 0.001
- link r_forearm: geometry collision mesh filename=package://ergoCub/meshes/simmechanics/sim_ecub_1-1_r_forear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 scale=0.001 0.001 0.001; visual mesh filename=package://ergoCub/meshes/simmechanics/sim_ecub_1-1_r_forear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 scale=0.001 0.001 0.001
- link r_hand_index_1: geometry collision mesh filename=package://ergoCub/meshes/simmechanics/sim_ecub_1-1_r_hand_i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 scale=0.001 0.001 0.001; visual mesh filename=package://ergoCub/meshes/simmechanics/sim_ecub_1-1_r_hand_i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 scale=0.001 0.001 0.001
- link r_hand_index_2: geometry collision mesh filename=package://ergoCub/meshes/simmechanics/sim_ecub_1-1_r_hand_i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 scale=0.001 0.001 0.001; visual mesh filename=package://ergoCub/meshes/simmechanics/sim_ecub_1-1_r_hand_i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 scale=0.001 0.001 0.001
- link r_hand_index_3: geometry collision mesh filename=package://ergoCub/meshes/simmechanics/sim_ecub_1-1_r_hand_i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 scale=0.001 0.001 0.001; visual mesh filename=package://ergoCub/meshes/simmechanics/sim_ecub_1-1_r_hand_i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 scale=0.001 0.001 0.001
- link r_hand_middle_1: geometry collision mesh filename=package://ergoCub/meshes/simmechanics/sim_ecub_1-1_r_hand_m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 scale=0.001 0.001 0.001; visual mesh filename=package://ergoCub/meshes/simmechanics/sim_ecub_1-1_r_hand_m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 scale=0.001 0.001 0.001
- link r_hand_middle_2: geometry collision mesh filename=package://ergoCub/meshes/simmechanics/sim_ecub_1-1_r_hand_m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 scale=0.001 0.001 0.001; visual mesh filename=package://ergoCub/meshes/simmechanics/sim_ecub_1-1_r_hand_m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 scale=0.001 0.001 0.001
- link r_hand_palm: geometry collision mesh filename=package://ergoCub/meshes/simmechanics/sim_ecub_1-1_r_hand_p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 scale=0.001 0.001 0.001; visual mesh filename=package://ergoCub/meshes/simmechanics/sim_ecub_1-1_r_hand_p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 scale=0.001 0.001 0.001
- link r_hand_pinkie_1: geometry collision mesh filename=package://ergoCub/meshes/simmechanics/sim_ecub_1-1_r_hand_p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 scale=0.001 0.001 0.001; visual mesh filename=package://ergoCub/meshes/simmechanics/sim_ecub_1-1_r_hand_p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 scale=0.001 0.001 0.001
- link r_hand_pinkie_2: geometry collision mesh filename=package://ergoCub/meshes/simmechanics/sim_ecub_1-1_r_hand_p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 scale=0.001 0.001 0.001; visual mesh filename=package://ergoCub/meshes/simmechanics/sim_ecub_1-1_r_hand_p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 scale=0.001 0.001 0.001
- link r_hand_ring_1: geometry collision mesh filename=package://ergoCub/meshes/simmechanics/sim_ecub_1-1_r_hand_r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 scale=0.001 0.001 0.001; visual mesh filename=package://ergoCub/meshes/simmechanics/sim_ecub_1-1_r_hand_r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 scale=0.001 0.001 0.001
- link r_hand_ring_2: geometry collision mesh filename=package://ergoCub/meshes/simmechanics/sim_ecub_1-1_r_hand_r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 scale=0.001 0.001 0.001; visual mesh filename=package://ergoCub/meshes/simmechanics/sim_ecub_1-1_r_hand_r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 scale=0.001 0.001 0.001
- link r_hand_thumb_1: geometry collision mesh filename=package://ergoCub/meshes/simmechanics/sim_ecub_1-1_r_hand_t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 scale=0.001 0.001 0.001; visual mesh filename=package://ergoCub/meshes/simmechanics/sim_ecub_1-1_r_hand_t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 scale=0.001 0.001 0.001
- link r_hand_thumb_2: geometry collision mesh filename=package://ergoCub/meshes/simmechanics/sim_ecub_1-1_r_hand_t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 scale=0.001 0.001 0.001; visual mesh filename=package://ergoCub/meshes/simmechanics/sim_ecub_1-1_r_hand_t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 scale=0.001 0.001 0.001
- link r_hand_thumb_3: geometry collision mesh filename=package://ergoCub/meshes/simmechanics/sim_ecub_1-1_r_hand_t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 scale=0.001 0.001 0.001; visual mesh filename=package://ergoCub/meshes/simmechanics/sim_ecub_1-1_r_hand_t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 scale=0.001 0.001 0.001
- link r_hip_1: geometry collision mesh filename=package://ergoCub/meshes/simmechanics/sim_ecub_1-1_r_hip_1.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 scale=0.001 0.001 0.001; visual mesh filename=package://ergoCub/meshes/simmechanics/sim_ecub_1-1_r_hip_1.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 scale=0.001 0.001 0.001
- link r_hip_2: geometry collision mesh filename=package://ergoCub/meshes/simmechanics/sim_ecub_1-1_r_hip_2.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 scale=0.001 0.001 0.001; visual mesh filename=package://ergoCub/meshes/simmechanics/sim_ecub_1-1_r_hip_2.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 scale=0.001 0.001 0.001
- link r_hip_3: geometry collision mesh filename=package://ergoCub/meshes/simmechanics/sim_ecub_1-1_r_hip_3.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 scale=0.001 0.001 0.001; visual mesh filename=package://ergoCub/meshes/simmechanics/sim_ecub_1-1_r_hip_3.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 scale=0.001 0.001 0.001
- link r_lower_leg: geometry collision mesh filename=package://ergoCub/meshes/simmechanics/sim_ecub_1-1_r_lower_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 scale=0.001 0.001 0.001; visual mesh filename=package://ergoCub/meshes/simmechanics/sim_ecub_1-1_r_lower_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 scale=0.001 0.001 0.001
- link r_shoulder_1: geometry collision mesh filename=package://ergoCub/meshes/simmechanics/sim_ecub_1-1_r_should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 scale=0.001 0.001 0.001; visual mesh filename=package://ergoCub/meshes/simmechanics/sim_ecub_1-1_r_should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 scale=0.001 0.001 0.001
- link r_shoulder_2: geometry collision mesh filename=package://ergoCub/meshes/simmechanics/sim_ecub_1-1_r_should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 scale=0.001 0.001 0.001; visual mesh filename=package://ergoCub/meshes/simmechanics/sim_ecub_1-1_r_should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 scale=0.001 0.001 0.001
- link r_shoulder_3: geometry collision mesh filename=package://ergoCub/meshes/simmechanics/sim_ecub_1-1_r_should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 scale=0.001 0.001 0.001; visual mesh filename=package://ergoCub/meshes/simmechanics/sim_ecub_1-1_r_should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 scale=0.001 0.001 0.001
- link r_upper_arm: geometry collision mesh filename=package://ergoCub/meshes/simmechanics/sim_ecub_1-1_r_uppera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 scale=0.001 0.001 0.001; visual mesh filename=package://ergoCub/meshes/simmechanics/sim_ecub_1-1_r_uppera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 scale=0.001 0.001 0.001
- link r_upper_leg: geometry collision mesh filename=package://ergoCub/meshes/simmechanics/sim_ecub_1-1_r_upper_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 scale=0.001 0.001 0.001; visual mesh filename=package://ergoCub/meshes/simmechanics/sim_ecub_1-1_r_upper_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 scale=0.001 0.001 0.001
- link r_wrist_1: geometry collision mesh filename=package://ergoCub/meshes/simmechanics/sim_ecub_1-1_r_wrist_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 scale=0.001 0.001 0.001; visual mesh filename=package://ergoCub/meshes/simmechanics/sim_ecub_1-1_r_wrist_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 scale=0.001 0.001 0.001
- link r_wrist_2: geometry collision mesh filename=package://ergoCub/meshes/simmechanics/sim_ecub_1-1_r_wrist_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 scale=0.001 0.001 0.001; visual mesh filename=package://ergoCub/meshes/simmechanics/sim_ecub_1-1_r_wrist_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 scale=0.001 0.001 0.001
- link realsense: geometry collision mesh filename=package://ergoCub/meshes/simmechanics/sim_ecub_1-1_realsens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 scale=0.001 0.001 0.001; visual mesh filename=package://ergoCub/meshes/simmechanics/sim_ecub_1-1_realsens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 scale=0.001 0.001 0.001
- link root_link: geometry collision mesh filename=package://ergoCub/meshes/simmechanics/sim_ecub_1-1_root_lin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 scale=0.001 0.001 0.001; visual mesh filename=package://ergoCub/meshes/simmechanics/sim_ecub_1-1_root_lin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 scale=0.001 0.001 0.001
- link torso_1: geometry collision mesh filename=package://ergoCub/meshes/simmechanics/sim_ecub_1-1_torso_1.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 scale=0.001 0.001 0.001; visual mesh filename=package://ergoCub/meshes/simmechanics/sim_ecub_1-1_torso_1.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 scale=0.001 0.001 0.001
- link torso_2: geometry collision mesh filename=package://ergoCub/meshes/simmechanics/sim_ecub_1-1_torso_2.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 scale=0.001 0.001 0.001; visual mesh filename=package://ergoCub/meshes/simmechanics/sim_ecub_1-1_torso_2.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 scale=0.001 0.001 0.001
