Commit message: urdf-test: adjust for ergoCub 1.1

File: urdf/ergoCub/robots/ergoCubGazeboV1_1/model.urdf (robot description, URDF)
Before this commit: robot ergoCub, 194 links, 193 joints
Links:
- added link head_imu_0
- added link l_arm_ft
- added link l_foot_front_ft
- added link l_foot_rear_ft
- added link l_leg_ft
- added link r_arm_ft
- added link r_foot_front_ft
- added link r_foot_rear_ft
- added link r_leg_ft
- added link realsense_imu_0
Joints:
- added joint head_imu_0_fixed_joint: type fixed, parent head, child head_imu_0, origin xyz=-0.004299999999999899 -0.005500000000001061 0.03823450000000106 rpy=-3.141592653589788 -9.688477917552238e-15 1.5707963267948986
- added joint l_arm_ft_fixed_joint: type fixed, parent l_shoulder_2, child l_arm_ft, origin xyz=-0.004349999999999996 -2.7755575615628914e-17 -0.054300000000000015 rpy=3.141592653589793 2.498001805406602e-16 -1.5707963267948952
- added joint l_foot_front_ft_fixed_joint: type fixed, parent l_ankle_2, child l_foot_front_ft, origin xyz=0.13525 -4.163336342344337e-17 -0.047899999999999054 rpy=-4.259189482954547e-17 -7.513330770412076e-17 -2.0943951023931966
- added joint l_foot_rear_ft_fixed_joint: type fixed, parent l_ankle_2, child l_foot_rear_ft, origin xyz=0.015999999999999993 -2.7755575615628914e-17 -0.04789999999999983 rpy=-4.259189482954531e-17 -7.513330770412153e-17 -2.0943951023931957
- added joint l_leg_ft_fixed_joint: type fixed, parent l_hip_2, child l_leg_ft, origin xyz=0.03669999999999986 -1.3877787807814457e-17 -0.08969999999999997 rpy=-3.1415926535897927 -1.4675346083959194e-15 2.617993877991494
- added joint r_arm_ft_fixed_joint: type fixed, parent r_shoulder_2, child r_arm_ft, origin xyz=-0.006849999999999986 -2.7755575615628914e-17 -0.05429999999999999 rpy=3.141592653589793 1.6653345369377348e-16 1.5707963267948981
- added joint r_foot_front_ft_fixed_joint: type fixed, parent r_ankle_2, child r_foot_front_ft, origin xyz=0.13525 1.3877787807814457e-17 -0.04789999999999983 rpy=-4.2591894829555776e-17 -7.513330770412949e-17 -2.094395102393197
- added joint r_foot_rear_ft_fixed_joint: type fixed, parent r_ankle_2, child r_foot_rear_ft, origin xyz=0.016 1.3877787807814457e-17 -0.04789999999999994 rpy=-4.2591894829543154e-17 -7.513330770412949e-17 -2.0943951023931966
- added joint r_leg_ft_fixed_joint: type fixed, parent r_hip_2, child r_leg_ft, origin xyz=0.03669999999999999 0 -0.08969999999999997 rpy=-3.1415926535897927 -8.654368135774127e-16 -2.6179938779914935
- added joint realsense_imu_0_fixed_joint: type fixed, parent realsense, child realsense_imu_0, origin xyz=0.007515481871156526 0.010000000000000002 1.7352099479506222e-8 rpy=-1.5707963267948966 3.7596758519972983e-16 -1.5707963267948966
- joint camera_tilt: axis -3.9202157447443984e-15 -1 6.441144250374745e-15 -> -3.611636085008543e-15 -1 -1.9429477071513935e-15
- joint head_laser_frame_fixed_joint: origin xyz=5.000000000061726e-5 -1.938549701738834e-15 0.13480249990363524 rpy=-5.331605011312536e-15 9.721935097880831e-15 -1.5707999999999969 -> xyz=5.000000000061726e-5 -1.938549701738834e-15 0.13480249990363524 rpy=9.721954681893984e-15 5.33156930061495e-15 3.167605067133685e-15
- joint l_ankle_pitch: axis -2.4058767102531433e-16 1 6.181058845623604e-17 -> 2.405876710253171e-16 1 6.181058845623607e-17
- joint l_ankle_roll: axis 1 -5.715619358951494e-16 9.923542537202003e-15 -> 1 -5.715619358951517e-16 -1.2940468202020292e-15
- joint l_elbow: axis 7.615436059538283e-15 -0.9999999999999953 6.60582699651967e-15 -> -6.9388939037918944e-18 -0.9999999999999953 6.4392935428256776e-15
- joint l_hip_pitch: axis -1.9810138796730044e-16 -1 3.944692124145837e-15 -> -5.772831379991284e-17 -1 -1.3843833381666392e-17
- joint l_hip_roll: axis 1 -3.3878809611365558e-16 5.765028837511044e-16 -> 1 -2.277657936511405e-16 5.765028837511023e-16
- joint l_hip_yaw: axis -1.1393662311292266e-14 3.784611153925698e-16 1 -> -8.067476499456731e-16 -6.18105884562747e-17 1
- joint l_index_add: axis 2.0450056094659772e-11 1 -3.544797195260885e-11 -> -2.3462306050979376e-11 -1 3.353175760248158e-11
- joint l_index_dist: axis -0.9999999999999999 2.3460773848806167e-11 2.1596168778964057e-10 -> -0.9999999999999999 2.3461101117417404e-11 1.0798067476965604e-10
- joint l_index_prox: axis -0.9999999999999999 2.3462037868071655e-11 3.184952301871927e-15 -> -0.9999999999999999 2.3461982356920424e-11 3.573530360490732e-15
- joint l_knee: axis -2.432856785186233e-15 1 6.181058845620829e-17 -> -2.4058767102531225e-16 1 6.181058845623608e-17
- joint l_middle_dist: axis -1 3.207539530165494e-11 2.149340264851616e-10 -> -1 2.824224757752587e-11 1.074840171400902e-10
- joint l_middle_prox: axis -1.0000000000000004 2.6293685263269454e-11 -2.6114387043662774e-14 -> -1.0000000000000004 2.629437932314885e-11 -9.97489772601784e-15
- joint l_pinkie_dist: axis -0.9999999998538324 7.646158528658914e-6 -1.529286228865057e-5 -> -0.9999999998538307 7.645479968428705e-6 -1.529330960500596e-5
- joint l_pinkie_prox: axis -0.9958502615677921 0.026193998942269946 -0.087155785549627 -> -0.9999999998538291 7.644801389928454e-6 -1.529375688869017e-5
- joint l_ring_dist: axis -1 2.838757093914722e-11 2.167147637103091e-10 -> -1 2.8664399475776237e-11 1.0876850894396261e-10
- joint l_ring_prox: axis -0.9958533270485439 0.026180434936035543 -0.0871248290265561 -> -1.0000000000000004 2.8926232503452798e-11 8.259087858064618e-13
- joint l_shoulder_pitch: axis -0.2714473275142867 0.9351131265310296 -0.22777135240129398 -> -3.452099717193846e-16 1.0000000000000002 3.0531133177191805e-16
- joint l_shoulder_roll: axis 1 3.1450536619460376e-15 5.002942504717091e-15 -> 1 7.615436059538576e-16 3.2196467714129958e-15
- joint l_shoulder_yaw: axis 5.979938766387244e-14 -6.8001160258292716e-15 0.9999999999999977 -> -2.982336599899327e-14 3.2196467714129528e-15 -0.9999999999999977
- joint l_thumb_add: axis 0.22146760053702236 0.039434487008100656 -0.9743700647837975 -> -6.391803752947567e-12 3.5905271811298434e-11 -1
- joint l_thumb_dist: axis -1.2816985320219744e-11 -7.052246286941839e-11 -0.9999999999999996 -> 5.648245760041583e-12 -5.177168416189185e-11 -0.9999999999999996
- joint l_thumb_prox: axis 0.13705874871064627 -0.9710270891801924 -0.195758247540464 -> 2.4115921065659407e-11 -3.3017838463322846e-11 -0.9999999999999997
- joint l_wrist_pitch: axis 2.6294398953241403e-11 1.0000000000000002 -3.135580683704409e-11 -> -2.6293939251520427e-11 -1.0000000000000002 3.1357194615824926e-11
- joint l_wrist_roll: axis -1.0000000000000004 2.6293798735532767e-11 1.0798209548745775e-10 -> -1.0000000000000004 2.6294445787389307e-11 1.0798215793750289e-10
- joint l_wrist_yaw: axis 1.0805985967143856e-10 3.135858239744487e-11 0.9999999999999981 -> -3.1939728639684985e-14 2.7755575615628937e-15 -0.9999999999999981
- joint neck_pitch: axis 1.3900353108727565e-15 -1 -2.3071799250996495e-15 -> 2.6474328740344387e-18 -1 -7.807082888609213e-16
- joint neck_roll: axis 1 -3.264103040198241e-15 -4.068108956268403e-15 -> 1 -1.6832426434147407e-15 -3.770068640066623e-15
- joint neck_yaw: axis 1.1543337812533589e-10 8.494511599802698e-16 0.9999999999999998 -> 3.4240774521066226e-15 -2.686540855695209e-16 0.9999999999999998
- joint r_ankle_pitch: axis -2.0458189416623182e-17 1 -4.187064692186876e-16 -> 1.8699102912341645e-16 1 -1.9666186429286112e-16
- joint r_ankle_roll: axis -1 5.921959240260381e-17 -3.6278999431864895e-14 -> -1 5.921958056855112e-17 2.5592852998214428e-15
- joint r_elbow: axis 8.401265794155823e-15 -1.0000000000000027 3.760880495917715e-14 -> 4.163336342349831e-17 -1.0000000000000027 2.5673907444456773e-14
- joint r_hip_pitch: axis -1.3496551942062083e-16 -1 4.000067457672489e-15 -> -1.0880513989386065e-16 -1 1.384383338166008e-17
- joint r_hip_roll: axis -1 -3.4417706449949065e-15 -8.557927305479742e-14 -> -1 -3.3813287685014083e-16 -8.532880891569492e-14
- joint r_hip_yaw: axis 8.603002509777097e-14 5.354644403999342e-15 -1 -> 8.528600225431674e-14 1.503215654809462e-15 -1
- joint r_index_add: axis 2.629933689451614e-11 -0.9999999999999998 -3.132698178918718e-11 -> -2.3468226053640166e-11 0.9999999999999998 -3.349943223875093e-11
- joint r_index_dist: axis -0.9999999999999997 -2.3468990639763418e-11 -2.158693918064003e-10 -> -0.9999999999999997 -2.3468990639763373e-11 -1.0793547999821127e-10
- joint r_index_prox: axis -0.9999999999999996 -2.3465354659357726e-11 -3.094746681145229e-15 -> -0.9999999999999996 -2.3465285270418687e-11 -2.8727020762201978e-15
- joint r_knee: axis 1.2193157699107697e-6 0.9999999999992566 -6.563010759392968e-14 -> -2.0458175022504648e-17 1 2.5382740632965355e-17
- joint r_middle_dist: axis -0.9999999999999998 -2.6300765925370995e-11 -2.15864696157152e-10 -> -0.9999999999999998 -2.630088161156088e-11 -1.079318529386326e-10
- joint r_middle_prox: axis -0.9999999999999997 -2.6304106462426976e-11 1.0793264892949847e-10 -> -0.9999999999999997 -2.6303362266055585e-11 -1.6375789613479553e-15
- joint r_pinkie_dist: axis -0.9999999999999999 -2.844378743174392e-11 -1.0878290583060967e-10 -> -0.9999999999999999 -2.8584519595543556e-11 -1.0874608649338082e-10
- joint r_pinkie_prox: axis -0.9958533270390026 -0.02614114144842622 0.08713662690925286 -> -0.9999999999999998 -2.8722006374562025e-11 -1.0870657152217689e-10
- joint r_ring_dist: axis -0.9999999999999999 -2.8434902002438743e-11 -2.1661359858593516e-10 -> -0.9999999999999999 -2.8681237072836204e-11 -1.0871797212486101e-10
- joint r_ring_prox: axis -0.9958533270389924 -0.026176948337041112 0.0871258767596002 -> -0.9999999999999999 -2.893151623156253e-11 -8.271161533457416e-13
- joint r_shoulder_pitch: axis 0.27144732751428424 0.9351131265310277 0.22777135240130472 -> -2.445960101127298e-16 1 3.552713678800501e-15
- joint r_shoulder_roll: axis -1.0000000000000007 -3.700165174258527e-15 -9.783840404509184e-15 -> -1.0000000000000007 1.0148132334463434e-15 -2.567390744445154e-16
- joint r_shoulder_yaw: axis -3.7470027081098055e-15 1.2934098236883104e-14 1.0000000000000004 -> 3.122502256758238e-16 -2.498001805406602e-16 1.0000000000000004
- joint r_thumb_add: axis 0.2249510542387036 -3.643432777700184e-11 0.9743700648095136 -> 3.164135620181696e-15 -3.643548754324866e-11 0.9999999999999999
- joint r_thumb_dist: axis 2.4120195424380822e-11 -3.298984696530608e-11 -0.9999999999999999 -> -5.6626925371494566e-12 5.173264594478845e-11 -0.9999999999999999
- joint r_thumb_prox: axis 0.13705874875237367 -0.9710270891738038 -0.19575824754294113 -> 2.4122360359202233e-11 -3.299033268788776e-11 -0.9999999999999999
- joint r_wrist_pitch: axis 2.6299299543675044e-11 -0.9999999999999998 -3.1325692040340414e-11 -> 2.6298942190638996e-11 -0.9999999999999998 -3.132558101803795e-11
- joint r_wrist_roll: axis 0.9999999999999997 2.6298437386107445e-11 -1.0793524407581856e-10 -> 0.9999999999999997 2.6298196259544278e-11 -1.0793549387599907e-10
- joint r_wrist_yaw: axis 1.0794686672310797e-10 -3.1326607974335516e-11 1.000000000000002 -> 6.057654378111005e-15 -5.273559366969643e-16 1.000000000000002
- joint torso_pitch: axis 2.1175823115833007e-22 1 -3.97151242917118e-15 -> 1.058791184074231e-22 1 4.336808689942018e-19
- joint torso_roll: axis -1 5.656623812198896e-30 1.4239886692466155e-15 -> -1 0 1.4239886692466155e-15
- joint torso_yaw: axis 2.0848912754007678e-15 1.8581752484505413e-15 -1 -> 2.084891490280543e-15 -2.11369334484512e-15 -1

File: urdf/ergoCub/robots/ergoCubGazeboV1_1_minContacts/model.urdf (robot description, URDF)
Before this commit: robot ergoCub, 194 links, 193 joints
Links:
- added link head_imu_0
- added link l_arm_ft
- added link l_foot_front_ft
- added link l_foot_rear_ft
- added link l_leg_ft
- added link r_arm_ft
- added link r_foot_front_ft
- added link r_foot_rear_ft
- added link r_leg_ft
- added link realsense_imu_0
Joints:
- added joint head_imu_0_fixed_joint: type fixed, parent head, child head_imu_0, origin xyz=-0.004299999999999899 -0.005500000000001061 0.03823450000000106 rpy=-3.141592653589788 -9.688477917552238e-15 1.5707963267948986
- added joint l_arm_ft_fixed_joint: type fixed, parent l_shoulder_2, child l_arm_ft, origin xyz=-0.004349999999999996 -2.7755575615628914e-17 -0.054300000000000015 rpy=3.141592653589793 2.498001805406602e-16 -1.5707963267948952
- added joint l_foot_front_ft_fixed_joint: type fixed, parent l_ankle_2, child l_foot_front_ft, origin xyz=0.13525 -4.163336342344337e-17 -0.047899999999999054 rpy=-4.259189482954547e-17 -7.513330770412076e-17 -2.0943951023931966
- added joint l_foot_rear_ft_fixed_joint: type fixed, parent l_ankle_2, child l_foot_rear_ft, origin xyz=0.015999999999999993 -2.7755575615628914e-17 -0.04789999999999983 rpy=-4.259189482954531e-17 -7.513330770412153e-17 -2.0943951023931957
- added joint l_leg_ft_fixed_joint: type fixed, parent l_hip_2, child l_leg_ft, origin xyz=0.03669999999999986 -1.3877787807814457e-17 -0.08969999999999997 rpy=-3.1415926535897927 -1.4675346083959194e-15 2.617993877991494
- added joint r_arm_ft_fixed_joint: type fixed, parent r_shoulder_2, child r_arm_ft, origin xyz=-0.006849999999999986 -2.7755575615628914e-17 -0.05429999999999999 rpy=3.141592653589793 1.6653345369377348e-16 1.5707963267948981
- added joint r_foot_front_ft_fixed_joint: type fixed, parent r_ankle_2, child r_foot_front_ft, origin xyz=0.13525 1.3877787807814457e-17 -0.04789999999999983 rpy=-4.2591894829555776e-17 -7.513330770412949e-17 -2.094395102393197
- added joint r_foot_rear_ft_fixed_joint: type fixed, parent r_ankle_2, child r_foot_rear_ft, origin xyz=0.016 1.3877787807814457e-17 -0.04789999999999994 rpy=-4.2591894829543154e-17 -7.513330770412949e-17 -2.0943951023931966
- added joint r_leg_ft_fixed_joint: type fixed, parent r_hip_2, child r_leg_ft, origin xyz=0.03669999999999999 0 -0.08969999999999997 rpy=-3.1415926535897927 -8.654368135774127e-16 -2.6179938779914935
- added joint realsense_imu_0_fixed_joint: type fixed, parent realsense, child realsense_imu_0, origin xyz=0.007515481871156526 0.010000000000000002 1.7352099479506222e-8 rpy=-1.5707963267948966 3.7596758519972983e-16 -1.5707963267948966
- joint camera_tilt: axis 3.9202157447443984e-15 1 -6.441144250374745e-15 -> -3.611636085008543e-15 -1 -1.9429477071513935e-15
- joint head_laser_frame_fixed_joint: origin xyz=5.000000000061726e-5 -1.938549701738834e-15 0.13480249990363524 rpy=-5.331605011312536e-15 9.721935097880831e-15 -1.5707999999999969 -> xyz=5.000000000061726e-5 -1.938549701738834e-15 0.13480249990363524 rpy=9.721954681893984e-15 5.33156930061495e-15 3.167605067133685e-15
- joint l_ankle_pitch: axis -2.4058767102531433e-16 1 6.181058845623604e-17 -> 2.405876710253171e-16 1 6.181058845623607e-17
- joint l_ankle_roll: axis -1 5.715619358951494e-16 -9.923542537202003e-15 -> 1 -5.715619358951517e-16 -1.2940468202020292e-15
- joint l_elbow: axis 7.615436059538283e-15 -0.9999999999999953 6.60582699651967e-15 -> -6.9388939037918944e-18 -0.9999999999999953 6.4392935428256776e-15
- joint l_hip_pitch: axis 1.9810138796730044e-16 1 -3.944692124145837e-15 -> -5.772831379991284e-17 -1 -1.3843833381666392e-17
- joint l_hip_roll: axis -1 3.3878809611365558e-16 -5.765028837511044e-16 -> 1 -2.277657936511405e-16 5.765028837511023e-16
- joint l_hip_yaw: axis 1.1393662311292266e-14 -3.784611153925698e-16 -1 -> -8.067476499456731e-16 -6.18105884562747e-17 1
- joint l_index_add: axis 2.0450056094659772e-11 1 -3.544797195260885e-11 -> -2.3462306050979376e-11 -1 3.353175760248158e-11
- joint l_index_dist: axis -0.9999999999999999 2.3460773848806167e-11 2.1596168778964057e-10 -> -0.9999999999999999 2.3461101117417404e-11 1.0798067476965604e-10
- joint l_index_prox: axis -0.9999999999999999 2.3462037868071655e-11 3.184952301871927e-15 -> -0.9999999999999999 2.3461982356920424e-11 3.573530360490732e-15
- joint l_knee: axis -2.432856785186233e-15 1 6.181058845620829e-17 -> -2.4058767102531225e-16 1 6.181058845623608e-17
- joint l_middle_dist: axis -1 3.207539530165494e-11 2.149340264851616e-10 -> -1 2.824224757752587e-11 1.074840171400902e-10
- joint l_middle_prox: axis -1.0000000000000004 2.6293685263269454e-11 -2.6114387043662774e-14 -> -1.0000000000000004 2.629437932314885e-11 -9.97489772601784e-15
- joint l_pinkie_dist: axis -0.9999999998538324 7.646158528658914e-6 -1.529286228865057e-5 -> -0.9999999998538307 7.645479968428705e-6 -1.529330960500596e-5
- joint l_pinkie_prox: axis -0.9958502615677921 0.026193998942269946 -0.087155785549627 -> -0.9999999998538291 7.644801389928454e-6 -1.529375688869017e-5
- joint l_ring_dist: axis -1 2.838757093914722e-11 2.167147637103091e-10 -> -1 2.8664399475776237e-11 1.0876850894396261e-10
- joint l_ring_prox: axis -0.9958533270485439 0.026180434936035543 -0.0871248290265561 -> -1.0000000000000004 2.8926232503452798e-11 8.259087858064618e-13
- joint l_shoulder_pitch: axis 0.2714473275142867 -0.9351131265310296 0.22777135240129398 -> -3.452099717193846e-16 1.0000000000000002 3.0531133177191805e-16
- joint l_shoulder_roll: axis 1 3.1450536619460376e-15 5.002942504717091e-15 -> 1 7.615436059538576e-16 3.2196467714129958e-15
- joint l_shoulder_yaw: axis 5.979938766387244e-14 -6.8001160258292716e-15 0.9999999999999977 -> -2.982336599899327e-14 3.2196467714129528e-15 -0.9999999999999977
- joint l_thumb_add: axis 0.22146760053702236 0.039434487008100656 -0.9743700647837975 -> -6.391803752947567e-12 3.5905271811298434e-11 -1
- joint l_thumb_dist: axis -1.2816985320219744e-11 -7.052246286941839e-11 -0.9999999999999996 -> 5.648245760041583e-12 -5.177168416189185e-11 -0.9999999999999996
- joint l_thumb_prox: axis 0.13705874871064627 -0.9710270891801924 -0.195758247540464 -> 2.4115921065659407e-11 -3.3017838463322846e-11 -0.9999999999999997
- joint l_wrist_pitch: axis 2.6294398953241403e-11 1.0000000000000002 -3.135580683704409e-11 -> -2.6293939251520427e-11 -1.0000000000000002 3.1357194615824926e-11
- joint l_wrist_roll: axis 1.0000000000000004 -2.6293798735532767e-11 -1.0798209548745775e-10 -> -1.0000000000000004 2.6294445787389307e-11 1.0798215793750289e-10
- joint l_wrist_yaw: axis 1.0805985967143856e-10 3.135858239744487e-11 0.9999999999999981 -> -3.1939728639684985e-14 2.7755575615628937e-15 -0.9999999999999981
- joint neck_pitch: axis -1.3900353108727565e-15 1 2.3071799250996495e-15 -> 2.6474328740344387e-18 -1 -7.807082888609213e-16
- joint neck_roll: axis -1 3.264103040198241e-15 4.068108956268403e-15 -> 1 -1.6832426434147407e-15 -3.770068640066623e-15
- joint neck_yaw: axis -1.1543337812533589e-10 -8.494511599802698e-16 -0.9999999999999998 -> 3.4240774521066226e-15 -2.686540855695209e-16 0.9999999999999998
- joint r_ankle_pitch: axis -2.0458189416623182e-17 1 -4.187064692186876e-16 -> 1.8699102912341645e-16 1 -1.9666186429286112e-16
- joint r_ankle_roll: axis 1 -5.921959240260381e-17 3.6278999431864895e-14 -> -1 5.921958056855112e-17 2.5592852998214428e-15
- joint r_elbow: axis 8.401265794155823e-15 -1.0000000000000027 3.760880495917715e-14 -> 4.163336342349831e-17 -1.0000000000000027 2.5673907444456773e-14
- joint r_hip_pitch: axis 1.3496551942062083e-16 1 -4.000067457672489e-15 -> -1.0880513989386065e-16 -1 1.384383338166008e-17
- joint r_hip_roll: axis 1 3.4417706449949065e-15 8.557927305479742e-14 -> -1 -3.3813287685014083e-16 -8.532880891569492e-14
- joint r_hip_yaw: axis -8.603002509777097e-14 -5.354644403999342e-15 1 -> 8.528600225431674e-14 1.503215654809462e-15 -1
- joint r_index_add: axis 2.629933689451614e-11 -0.9999999999999998 -3.132698178918718e-11 -> -2.3468226053640166e-11 0.9999999999999998 -3.349943223875093e-11
- joint r_index_dist: axis -0.9999999999999997 -2.3468990639763418e-11 -2.158693918064003e-10 -> -0.9999999999999997 -2.3468990639763373e-11 -1.0793547999821127e-10
- joint r_index_prox: axis -0.9999999999999996 -2.3465354659357726e-11 -3.094746681145229e-15 -> -0.9999999999999996 -2.3465285270418687e-11 -2.8727020762201978e-15
- joint r_knee: axis 1.2193157699107697e-6 0.9999999999992566 -6.563010759392968e-14 -> -2.0458175022504648e-17 1 2.5382740632965355e-17
- joint r_middle_dist: axis -0.9999999999999998 -2.6300765925370995e-11 -2.15864696157152e-10 -> -0.9999999999999998 -2.630088161156088e-11 -1.079318529386326e-10
- joint r_middle_prox: axis -0.9999999999999997 -2.6304106462426976e-11 1.0793264892949847e-10 -> -0.9999999999999997 -2.6303362266055585e-11 -1.6375789613479553e-15
- joint r_pinkie_dist: axis -0.9999999999999999 -2.844378743174392e-11 -1.0878290583060967e-10 -> -0.9999999999999999 -2.8584519595543556e-11 -1.0874608649338082e-10
- joint r_pinkie_prox: axis -0.9958533270390026 -0.02614114144842622 0.08713662690925286 -> -0.9999999999999998 -2.8722006374562025e-11 -1.0870657152217689e-10
- joint r_ring_dist: axis -0.9999999999999999 -2.8434902002438743e-11 -2.1661359858593516e-10 -> -0.9999999999999999 -2.8681237072836204e-11 -1.0871797212486101e-10
- joint r_ring_prox: axis -0.9958533270389924 -0.026176948337041112 0.0871258767596002 -> -0.9999999999999999 -2.893151623156253e-11 -8.271161533457416e-13
- joint r_shoulder_pitch: axis -0.27144732751428424 -0.9351131265310277 -0.22777135240130472 -> -2.445960101127298e-16 1 3.552713678800501e-15
- joint r_shoulder_roll: axis -1.0000000000000007 -3.700165174258527e-15 -9.783840404509184e-15 -> -1.0000000000000007 1.0148132334463434e-15 -2.567390744445154e-16
- joint r_shoulder_yaw: axis 3.7470027081098055e-15 -1.2934098236883104e-14 -1.0000000000000004 -> 3.122502256758238e-16 -2.498001805406602e-16 1.0000000000000004
- joint r_thumb_add: axis 0.2249510542387036 -3.643432777700184e-11 0.9743700648095136 -> 3.164135620181696e-15 -3.643548754324866e-11 0.9999999999999999
- joint r_thumb_dist: axis 2.4120195424380822e-11 -3.298984696530608e-11 -0.9999999999999999 -> -5.6626925371494566e-12 5.173264594478845e-11 -0.9999999999999999
- joint r_thumb_prox: axis 0.13705874875237367 -0.9710270891738038 -0.19575824754294113 -> 2.4122360359202233e-11 -3.299033268788776e-11 -0.9999999999999999
- joint r_wrist_pitch: axis -2.6299299543675044e-11 0.9999999999999998 3.1325692040340414e-11 -> 2.6298942190638996e-11 -0.9999999999999998 -3.132558101803795e-11
- joint r_wrist_roll: axis -0.9999999999999997 -2.6298437386107445e-11 1.0793524407581856e-10 -> 0.9999999999999997 2.6298196259544278e-11 -1.0793549387599907e-10
- joint r_wrist_yaw: axis -1.0794686672310797e-10 3.1326607974335516e-11 -1.000000000000002 -> 6.057654378111005e-15 -5.273559366969643e-16 1.000000000000002
- joint torso_pitch: axis -2.1175823115833007e-22 -1 3.97151242917118e-15 -> 1.058791184074231e-22 1 4.336808689942018e-19
- joint torso_roll: axis 1 -5.656623812198896e-30 -1.4239886692466155e-15 -> -1 0 1.4239886692466155e-15
- joint torso_yaw: axis -2.0848912754007678e-15 -1.8581752484505413e-15 1 -> 2.084891490280543e-15 -2.11369334484512e-15 -1
