Commit message: Final version of gazebo model

File: urdf/ergoCub/robots/ergoCubGazeboV1_1/model.urdf (robot description, URDF)
Before this commit: robot ergoCub, 204 links, 203 joints
Links:
- link l_foot_front: geometry collision box size=0.117 0.1 0.006; visual mesh filename=package://ergoCub/meshes/simmechanics/sim_ecub_1-1_l_foot_f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 scale=0.001 0.001 0.001
- link l_foot_rear: geometry collision box size=0.117 0.1 0.006; visual mesh filename=package://ergoCub/meshes/simmechanics/sim_ecub_1-1_l_foot_r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 scale=0.001 0.001 0.001
- link r_foot_front: geometry collision box size=0.117 0.1 0.006; visual mesh filename=package://ergoCub/meshes/simmechanics/sim_ecub_1-1_r_foot_f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 scale=0.001 0.001 0.001
- link r_foot_rear: geometry collision box size=0.117 0.1 0.006; visual mesh filename=package://ergoCub/meshes/simmechanics/sim_ecub_1-1_r_foot_r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 scale=0.001 0.001 0.001

Commit message: ergoCubV1_1: update urdf

File: urdf/ergoCub/robots/ergoCubGazeboV1_1/model.urdf (robot description, URDF)
Before this commit: robot ergoCub, 204 links, 203 joints
Joints:
- joint l_index_dist: limit lower=0 upper=1.7313666179783749 effort=1e+9 velocity=1e+9 -> lower=0 upper=1.7994344588061537 effort=1e+9 velocity=1e+9
- joint l_middle_dist: limit lower=0 upper=1.7313666179783749 effort=1e+9 velocity=1e+9 -> lower=0 upper=1.7994344588061537 effort=1e+9 velocity=1e+9
- joint l_pinkie_dist: limit lower=0 upper=1.6283921921107094 effort=1e+9 velocity=1e+9 -> lower=0 upper=1.7226399717184033 effort=1e+9 velocity=1e+9
- joint l_ring_dist: limit lower=0 upper=1.7313666179783749 effort=1e+9 velocity=1e+9 -> lower=0 upper=1.7994344588061537 effort=1e+9 velocity=1e+9
- joint l_thumb_add: limit lower=0 upper=1.5707963267948966 effort=1e+9 velocity=1e+9 -> lower=0 upper=1.7453292519943295 effort=1e+9 velocity=1e+9
- joint l_thumb_dist: limit lower=0 upper=0.9354964790689606 effort=1e+9 velocity=1e+9 -> lower=0 upper=1.7697638615222502 effort=1e+9 velocity=1e+9
- joint l_thumb_prox: limit lower=0 upper=1.4329153158873444 effort=1e+9 velocity=1e+9 -> lower=0 upper=1.5707963267948966 effort=1e+9 velocity=1e+9
- joint r_index_dist: limit lower=0 upper=1.7313666179783749 effort=1e+9 velocity=1e+9 -> lower=0 upper=1.7994344588061537 effort=1e+9 velocity=1e+9
- joint r_middle_dist: limit lower=0 upper=1.7313666179783749 effort=1e+9 velocity=1e+9 -> lower=0 upper=1.7994344588061537 effort=1e+9 velocity=1e+9
- joint r_pinkie_dist: limit lower=0 upper=1.6283921921107094 effort=1e+9 velocity=1e+9 -> lower=0 upper=1.7226399717184033 effort=1e+9 velocity=1e+9
- joint r_ring_dist: limit lower=0 upper=1.7313666179783749 effort=1e+9 velocity=1e+9 -> lower=0 upper=1.7994344588061537 effort=1e+9 velocity=1e+9
- joint r_thumb_add: limit lower=0 upper=1.5707963267948966 effort=1e+9 velocity=1e+9 -> lower=0 upper=1.7453292519943295 effort=1e+9 velocity=1e+9
- joint r_thumb_dist: limit lower=0 upper=0.9354964790689606 effort=1e+9 velocity=1e+9 -> lower=0 upper=1.7697638615222502 effort=1e+9 velocity=1e+9
- joint r_thumb_prox: limit lower=0 upper=1.4329153158873444 effort=1e+9 velocity=1e+9 -> lower=0 upper=1.5707963267948966 effort=1e+9 velocity=1e+9

File: urdf/ergoCub/robots/ergoCubGazeboV1_1_minContacts/model.urdf (robot description, URDF)
Before this commit: robot ergoCub, 204 links, 203 joints
Joints:
- joint l_index_dist: limit lower=0 upper=1.7313666179783749 effort=1e+9 velocity=1e+9 -> lower=0 upper=1.7994344588061537 effort=1e+9 velocity=1e+9
- joint l_middle_dist: limit lower=0 upper=1.7313666179783749 effort=1e+9 velocity=1e+9 -> lower=0 upper=1.7994344588061537 effort=1e+9 velocity=1e+9
- joint l_pinkie_dist: limit lower=0 upper=1.6283921921107094 effort=1e+9 velocity=1e+9 -> lower=0 upper=1.7226399717184033 effort=1e+9 velocity=1e+9
- joint l_ring_dist: limit lower=0 upper=1.7313666179783749 effort=1e+9 velocity=1e+9 -> lower=0 upper=1.7994344588061537 effort=1e+9 velocity=1e+9
- joint l_thumb_add: limit lower=0 upper=1.5707963267948966 effort=1e+9 velocity=1e+9 -> lower=0 upper=1.7453292519943295 effort=1e+9 velocity=1e+9
- joint l_thumb_dist: limit lower=0 upper=0.9354964790689606 effort=1e+9 velocity=1e+9 -> lower=0 upper=1.7697638615222502 effort=1e+9 velocity=1e+9
- joint l_thumb_prox: limit lower=0 upper=1.4329153158873444 effort=1e+9 velocity=1e+9 -> lower=0 upper=1.5707963267948966 effort=1e+9 velocity=1e+9
- joint r_index_dist: limit lower=0 upper=1.7313666179783749 effort=1e+9 velocity=1e+9 -> lower=0 upper=1.7994344588061537 effort=1e+9 velocity=1e+9
- joint r_middle_dist: limit lower=0 upper=1.7313666179783749 effort=1e+9 velocity=1e+9 -> lower=0 upper=1.7994344588061537 effort=1e+9 velocity=1e+9
- joint r_pinkie_dist: limit lower=0 upper=1.6283921921107094 effort=1e+9 velocity=1e+9 -> lower=0 upper=1.7226399717184033 effort=1e+9 velocity=1e+9
- joint r_ring_dist: limit lower=0 upper=1.7313666179783749 effort=1e+9 velocity=1e+9 -> lower=0 upper=1.7994344588061537 effort=1e+9 velocity=1e+9
- joint r_thumb_add: limit lower=0 upper=1.5707963267948966 effort=1e+9 velocity=1e+9 -> lower=0 upper=1.7453292519943295 effort=1e+9 velocity=1e+9
- joint r_thumb_dist: limit lower=0 upper=0.9354964790689606 effort=1e+9 velocity=1e+9 -> lower=0 upper=1.7697638615222502 effort=1e+9 velocity=1e+9
- joint r_thumb_prox: limit lower=0 upper=1.4329153158873444 effort=1e+9 velocity=1e+9 -> lower=0 upper=1.5707963267948966 effort=1e+9 velocity=1e+9

File: urdf/ergoCub/robots/ergoCubSN001/model.urdf (robot description, URDF)
Before this commit: robot ergoCub, 204 links, 203 joints
Joints:
- joint l_index_dist: limit lower=0 upper=1.7313666179783749 effort=1e+9 velocity=1e+9 -> lower=0 upper=1.7994344588061537 effort=1e+9 velocity=1e+9
- joint l_middle_dist: limit lower=0 upper=1.7313666179783749 effort=1e+9 velocity=1e+9 -> lower=0 upper=1.7994344588061537 effort=1e+9 velocity=1e+9
- joint l_pinkie_dist: limit lower=0 upper=1.6283921921107094 effort=1e+9 velocity=1e+9 -> lower=0 upper=1.7226399717184033 effort=1e+9 velocity=1e+9
- joint l_ring_dist: limit lower=0 upper=1.7313666179783749 effort=1e+9 velocity=1e+9 -> lower=0 upper=1.7994344588061537 effort=1e+9 velocity=1e+9
- joint l_thumb_add: limit lower=0 upper=1.5707963267948966 effort=1e+9 velocity=1e+9 -> lower=0 upper=1.7453292519943295 effort=1e+9 velocity=1e+9
- joint l_thumb_dist: limit lower=0 upper=0.9354964790689606 effort=1e+9 velocity=1e+9 -> lower=0 upper=1.7697638615222502 effort=1e+9 velocity=1e+9
- joint l_thumb_prox: limit lower=0 upper=1.4329153158873444 effort=1e+9 velocity=1e+9 -> lower=0 upper=1.5707963267948966 effort=1e+9 velocity=1e+9
- joint r_index_dist: limit lower=0 upper=1.7313666179783749 effort=1e+9 velocity=1e+9 -> lower=0 upper=1.7994344588061537 effort=1e+9 velocity=1e+9
- joint r_middle_dist: limit lower=0 upper=1.7313666179783749 effort=1e+9 velocity=1e+9 -> lower=0 upper=1.7994344588061537 effort=1e+9 velocity=1e+9
- joint r_pinkie_dist: limit lower=0 upper=1.6283921921107094 effort=1e+9 velocity=1e+9 -> lower=0 upper=1.7226399717184033 effort=1e+9 velocity=1e+9
- joint r_ring_dist: limit lower=0 upper=1.7313666179783749 effort=1e+9 velocity=1e+9 -> lower=0 upper=1.7994344588061537 effort=1e+9 velocity=1e+9
- joint r_thumb_add: limit lower=0 upper=1.5707963267948966 effort=1e+9 velocity=1e+9 -> lower=0 upper=1.7453292519943295 effort=1e+9 velocity=1e+9
- joint r_thumb_dist: limit lower=0 upper=0.9354964790689606 effort=1e+9 velocity=1e+9 -> lower=0 upper=1.7697638615222502 effort=1e+9 velocity=1e+9
- joint r_thumb_prox: limit lower=0 upper=1.4329153158873444 effort=1e+9 velocity=1e+9 -> lower=0 upper=1.5707963267948966 effort=1e+9 velocity=1e+9
