Commit message: ergoCubV1_1: correct index_add joint

File: urdf/ergoCub/robots/ergoCubGazeboV1_1/model.urdf (robot description, URDF)
Before this commit: robot ergoCub, 204 links, 203 joints
Joints:
- joint l_index_add: axis -2.3462306050979376e-11 -1 3.353175760248158e-11 -> 1.5978340464762954e-11 0.9999999999999999 -3.7677226824487294e-11; origin xyz=0.022500000000000103 -0.0015000000000006675 -0.06859999999999955 rpy=-7.244015325404705e-16 -0.08726646259971596 -6.686783377296649e-16 -> xyz=0.022500000000000023 -0.0015000000000006952 -0.0685999999999996 rpy=-8.416895217637947e-16 -0.29670597224465534 5.804755322508926e-17
- joint l_index_dist: axis -0.9999999999999999 2.3461101117417404e-11 1.0798067476965604e-10 -> -0.9781476007113552 -1.553317034713362e-8 0.20791169092337955; origin xyz=1.5226389593614442e-11 -0.0015000000000001679 -0.03999999999723247 rpy=-7.4823262335988e-8 -1.0798106159226606e-10 -4.996003610813205e-16 -> xyz=-1.3877787807814457e-17 -0.001500000000000029 -0.03999999999999987 rpy=-7.482326172536535e-8 1.8041124150158794e-16 -6.106226635438361e-16
- joint l_index_prox: axis -0.9999999999999999 2.3461982356920424e-11 3.573530360490732e-15 -> -0.9781476007113543 2.3461557522424743e-11 0.2079116909233844; origin xyz=0.009192533317427871 -1.6653345369377348e-16 -0.030713451316238316 rpy=1.5543122344752197e-15 3.5388358909926865e-16 -1.1102230246251568e-16 -> xyz=0.00919253334679343 0 -0.030713451309624218 rpy=-3.0531133177191815e-16 -7.023611484080483e-10 -7.771561172376096e-16
- joint l_middle_prox: axis -1.0000000000000004 2.629437932314885e-11 -9.97489772601784e-15 -> -1.0000000000000004 2.629437917485816e-11 -9.988775473196015e-15; origin xyz=0.009600000000000143 -0.0015000000000005842 -0.10299999999999959 rpy=5.479728916549446e-4 1.6930901125533637e-15 -8.32667268468867e-16 -> xyz=0.00960000000000016 -0.0015000000000005842 -0.10299999999999959 rpy=5.479728916549446e-4 1.4363510381087963e-15 -8.32667268468867e-16
- joint l_pinkie_prox: axis -0.9999999998538291 7.644801389928454e-6 -1.529375688869017e-5 -> -0.9999999998538291 7.64480138992604e-6 -1.5293756888704046e-5; origin xyz=-0.03598232224952729 -0.0023883158589564635 -0.09206560929209856 rpy=-1.993459149294906e-5 0.08728175651239253 0.026187612448127052 -> xyz=-0.035982322249527285 -0.0023883158589564635 -0.09206560929209856 rpy=-1.9934591492976922e-5 0.08728175651239228 0.02618761244812705
- joint l_ring_prox: axis -1.0000000000000004 2.8926232503452798e-11 8.259087858064618e-13 -> -1.0000000000000002 2.8926226625044144e-11 8.259226635942696e-13; origin xyz=-0.015417755558120048 -0.0018498137284707894 -0.09788067183884419 rpy=-4.001819369801849e-5 0.0872664625997324 0.026179938779914452 -> xyz=-0.015417755558120038 -0.0018498137284707894 -0.09788067183884419 rpy=-4.001819369804634e-5 0.08726646259973214 0.026179938779914452
- joint l_thumb_add: axis -6.391803752947567e-12 3.5905271811298434e-11 -1 -> -6.391803752947567e-12 3.590529956687405e-11 -1.0000000000000002; origin xyz=0.02337486325639077 -0.0030000000000002525 -0.03452383847355461 rpy=-0.040449700618590975 0.2233191863655349 2.9608435412698353 -> xyz=0.02337486325639077 -0.0030000000000002525 -0.03452383847355461 rpy=-0.04044970061859103 0.22331918636553513 2.9608435412698353
- joint l_wrist_pitch: axis -2.6293939251520427e-11 -1.0000000000000002 3.1357194615824926e-11 -> -2.6293939251520434e-11 -1.0000000000000002 3.135719461582492e-11; origin xyz=-1.2836953722228372e-16 -1.6653345369377348e-16 0 rpy=-4.163336342344336e-16 1.079816722149296e-10 3.330669073875468e-16 -> xyz=-1.214306433183765e-16 -1.6653345369377348e-16 0 rpy=-4.163336342344336e-16 1.0798191507621624e-10 3.330669073875468e-16
- joint r_index_add: axis -2.3468226053640166e-11 0.9999999999999998 -3.349943223875093e-11 -> 1.5990673923572052e-11 -0.9999999999999999 3.764672729074698e-11; origin xyz=0.02249999999259583 0.0015000000000003066 -0.06860000000242839 rpy=-1.5881110520929587e-15 0.08726646249178613 3.1415926535897922 -> xyz=0.022499999999999992 0.0015000000000002234 -0.06859999999999983 rpy=-1.6833790438334957e-15 0.29670597283904 3.141592653589792
- joint r_index_dist: axis -0.9999999999999997 -2.3468990639763373e-11 -1.0793547999821127e-10 -> -0.9781476007113639 -2.3469068155297194e-11 -0.2079116909233363; origin xyz=-1.521995723896552e-11 -0.001500000000000029 -0.03999999999723369 rpy=4.1633363423443375e-16 1.0793393956376462e-10 -5.551115123125785e-17 -> xyz=4.163336342344337e-17 -0.0014999999999998903 -0.040000000000000036 rpy=1.942890293094024e-16 3.469446951953614e-17 1.665334536937736e-16
- joint r_index_prox: axis -0.9999999999999996 -2.3465285270418687e-11 -2.8727020762201978e-15 -> -0.9781476007113635 -2.3465277303774676e-11 -0.20791169092333764; origin xyz=-0.009192533317427698 8.326672684688674e-17 -0.030713451316238427 rpy=-8.881784197001254e-16 2.3592239273284576e-16 -1.6653345369377356e-16 -> xyz=-0.009192533317427393 5.551115123125783e-17 -0.030713451316238316 rpy=-3.0531133177191805e-16 -2.0816681711721685e-17 0
- joint r_middle_prox: axis -0.9999999999999997 -2.6303362266055585e-11 -1.6375789613479553e-15 -> -0.9999999999999996 -2.6303416042483343e-11 -1.6098233857581758e-15; origin xyz=0.009599999988883008 0.0015000000000004454 -0.10300000000103599 rpy=-1.8596235662471376e-15 -1.0793112237283964e-10 3.1415926535897927 -> xyz=0.009599999988882939 0.00150000000000039 -0.1030000000010361 rpy=-1.8596235662471376e-15 -1.0793124727292991e-10 3.1415926535897927
- joint r_pinkie_prox: axis -0.9999999999999998 -2.8722006374562025e-11 -1.0870657152217689e-10 -> -0.9999999999999998 -2.8722034177571486e-11 -1.0870652988881346e-10; origin xyz=-0.035982680943166104 0.002377759579109656 -0.0920682813194636 rpy=4.1095343980510334e-4 -0.0872664625997285 3.1154127148098776 -> xyz=-0.035982680943166166 0.002377759579109573 -0.09206828131946371 rpy=4.1095343980510334e-4 -0.08726646259972864 3.1154127148098776
- joint r_ring_prox: axis -0.9999999999999999 -2.893151623156253e-11 -8.271161533457416e-13 -> -0.9999999999999999 -2.893157069232462e-11 -8.271022755579338e-13; origin xyz=-0.015417755568684362 0.0018498137284712335 -0.09788067183717974 rpy=2.0171796521702004e-14 -0.08726646270762457 3.11541271480963 -> xyz=-0.015417755568684424 0.001849813728471178 -0.09788067183717986 rpy=2.019965811910767e-14 -0.08726646270762471 3.11541271480963
- joint r_thumb_add: axis 3.164135620181696e-15 -3.643548754324866e-11 0.9999999999999999 -> 3.219646771412954e-15 -3.6435554830318275e-11 0.9999999999999998; origin xyz=0.023374863252664378 0.0030000000000001414 -0.03452383847607732 rpy=1.595197030995694e-15 -0.22689280265133213 -5.127419028200447e-16 -> xyz=0.023374863252664337 0.003000000000000058 -0.03452383847607743 rpy=1.566711369727914e-15 -0.226892802651332 -5.127419028200447e-16
- joint r_wrist_pitch: axis 2.6298942190638996e-11 -0.9999999999999998 -3.132558101803795e-11 -> 2.6298942190638987e-11 -0.9999999999999998 -3.1325553262462336e-11; origin xyz=-9.367506770274758e-17 -8.326672684688674e-17 -8.326672684688674e-17 rpy=2.775557561562892e-16 1.0408340855860843e-16 -3.8857805861880494e-16 -> xyz=-4.85722573273506e-17 0 2.7755575615628914e-17 rpy=2.2204460492503136e-16 -5.551115123125783e-17 -3.88578058618805e-16

File: urdf/ergoCub/robots/ergoCubGazeboV1_1_minContacts/model.urdf (robot description, URDF)
Before this commit: robot ergoCub, 204 links, 203 joints
Joints:
- joint l_index_add: axis -2.3462306050979376e-11 -1 3.353175760248158e-11 -> 1.5978340464762954e-11 0.9999999999999999 -3.7677226824487294e-11; origin xyz=0.022500000000000103 -0.0015000000000006675 -0.06859999999999955 rpy=-7.244015325404705e-16 -0.08726646259971596 -6.686783377296649e-16 -> xyz=0.022500000000000023 -0.0015000000000006952 -0.0685999999999996 rpy=-8.416895217637947e-16 -0.29670597224465534 5.804755322508926e-17
- joint l_index_dist: axis -0.9999999999999999 2.3461101117417404e-11 1.0798067476965604e-10 -> -0.9781476007113552 -1.553317034713362e-8 0.20791169092337955; origin xyz=1.5226389593614442e-11 -0.0015000000000001679 -0.03999999999723247 rpy=-7.4823262335988e-8 -1.0798106159226606e-10 -4.996003610813205e-16 -> xyz=-1.3877787807814457e-17 -0.001500000000000029 -0.03999999999999987 rpy=-7.482326172536535e-8 1.8041124150158794e-16 -6.106226635438361e-16
- joint l_index_prox: axis -0.9999999999999999 2.3461982356920424e-11 3.573530360490732e-15 -> -0.9781476007113543 2.3461557522424743e-11 0.2079116909233844; origin xyz=0.009192533317427871 -1.6653345369377348e-16 -0.030713451316238316 rpy=1.5543122344752197e-15 3.5388358909926865e-16 -1.1102230246251568e-16 -> xyz=0.00919253334679343 0 -0.030713451309624218 rpy=-3.0531133177191815e-16 -7.023611484080483e-10 -7.771561172376096e-16
- joint l_middle_prox: axis -1.0000000000000004 2.629437932314885e-11 -9.97489772601784e-15 -> -1.0000000000000004 2.629437917485816e-11 -9.988775473196015e-15; origin xyz=0.009600000000000143 -0.0015000000000005842 -0.10299999999999959 rpy=5.479728916549446e-4 1.6930901125533637e-15 -8.32667268468867e-16 -> xyz=0.00960000000000016 -0.0015000000000005842 -0.10299999999999959 rpy=5.479728916549446e-4 1.4363510381087963e-15 -8.32667268468867e-16
- joint l_pinkie_prox: axis -0.9999999998538291 7.644801389928454e-6 -1.529375688869017e-5 -> -0.9999999998538291 7.64480138992604e-6 -1.5293756888704046e-5; origin xyz=-0.03598232224952729 -0.0023883158589564635 -0.09206560929209856 rpy=-1.993459149294906e-5 0.08728175651239253 0.026187612448127052 -> xyz=-0.035982322249527285 -0.0023883158589564635 -0.09206560929209856 rpy=-1.9934591492976922e-5 0.08728175651239228 0.02618761244812705
- joint l_ring_prox: axis -1.0000000000000004 2.8926232503452798e-11 8.259087858064618e-13 -> -1.0000000000000002 2.8926226625044144e-11 8.259226635942696e-13; origin xyz=-0.015417755558120048 -0.0018498137284707894 -0.09788067183884419 rpy=-4.001819369801849e-5 0.0872664625997324 0.026179938779914452 -> xyz=-0.015417755558120038 -0.0018498137284707894 -0.09788067183884419 rpy=-4.001819369804634e-5 0.08726646259973214 0.026179938779914452
- joint l_thumb_add: axis -6.391803752947567e-12 3.5905271811298434e-11 -1 -> -6.391803752947567e-12 3.590529956687405e-11 -1.0000000000000002; origin xyz=0.02337486325639077 -0.0030000000000002525 -0.03452383847355461 rpy=-0.040449700618590975 0.2233191863655349 2.9608435412698353 -> xyz=0.02337486325639077 -0.0030000000000002525 -0.03452383847355461 rpy=-0.04044970061859103 0.22331918636553513 2.9608435412698353
- joint l_wrist_pitch: axis -2.6293939251520427e-11 -1.0000000000000002 3.1357194615824926e-11 -> -2.6293939251520434e-11 -1.0000000000000002 3.135719461582492e-11; origin xyz=-1.2836953722228372e-16 -1.6653345369377348e-16 0 rpy=-4.163336342344336e-16 1.079816722149296e-10 3.330669073875468e-16 -> xyz=-1.214306433183765e-16 -1.6653345369377348e-16 0 rpy=-4.163336342344336e-16 1.0798191507621624e-10 3.330669073875468e-16
- joint r_index_add: axis -2.3468226053640166e-11 0.9999999999999998 -3.349943223875093e-11 -> 1.5990673923572052e-11 -0.9999999999999999 3.764672729074698e-11; origin xyz=0.02249999999259583 0.0015000000000003066 -0.06860000000242839 rpy=-1.5881110520929587e-15 0.08726646249178613 3.1415926535897922 -> xyz=0.022499999999999992 0.0015000000000002234 -0.06859999999999983 rpy=-1.6833790438334957e-15 0.29670597283904 3.141592653589792
- joint r_index_dist: axis -0.9999999999999997 -2.3468990639763373e-11 -1.0793547999821127e-10 -> -0.9781476007113639 -2.3469068155297194e-11 -0.2079116909233363; origin xyz=-1.521995723896552e-11 -0.001500000000000029 -0.03999999999723369 rpy=4.1633363423443375e-16 1.0793393956376462e-10 -5.551115123125785e-17 -> xyz=4.163336342344337e-17 -0.0014999999999998903 -0.040000000000000036 rpy=1.942890293094024e-16 3.469446951953614e-17 1.665334536937736e-16
- joint r_index_prox: axis -0.9999999999999996 -2.3465285270418687e-11 -2.8727020762201978e-15 -> -0.9781476007113635 -2.3465277303774676e-11 -0.20791169092333764; origin xyz=-0.009192533317427698 8.326672684688674e-17 -0.030713451316238427 rpy=-8.881784197001254e-16 2.3592239273284576e-16 -1.6653345369377356e-16 -> xyz=-0.009192533317427393 5.551115123125783e-17 -0.030713451316238316 rpy=-3.0531133177191805e-16 -2.0816681711721685e-17 0
- joint r_middle_prox: axis -0.9999999999999997 -2.6303362266055585e-11 -1.6375789613479553e-15 -> -0.9999999999999996 -2.6303416042483343e-11 -1.6098233857581758e-15; origin xyz=0.009599999988883008 0.0015000000000004454 -0.10300000000103599 rpy=-1.8596235662471376e-15 -1.0793112237283964e-10 3.1415926535897927 -> xyz=0.009599999988882939 0.00150000000000039 -0.1030000000010361 rpy=-1.8596235662471376e-15 -1.0793124727292991e-10 3.1415926535897927
- joint r_pinkie_prox: axis -0.9999999999999998 -2.8722006374562025e-11 -1.0870657152217689e-10 -> -0.9999999999999998 -2.8722034177571486e-11 -1.0870652988881346e-10; origin xyz=-0.035982680943166104 0.002377759579109656 -0.0920682813194636 rpy=4.1095343980510334e-4 -0.0872664625997285 3.1154127148098776 -> xyz=-0.035982680943166166 0.002377759579109573 -0.09206828131946371 rpy=4.1095343980510334e-4 -0.08726646259972864 3.1154127148098776
- joint r_ring_prox: axis -0.9999999999999999 -2.893151623156253e-11 -8.271161533457416e-13 -> -0.9999999999999999 -2.893157069232462e-11 -8.271022755579338e-13; origin xyz=-0.015417755568684362 0.0018498137284712335 -0.09788067183717974 rpy=2.0171796521702004e-14 -0.08726646270762457 3.11541271480963 -> xyz=-0.015417755568684424 0.001849813728471178 -0.09788067183717986 rpy=2.019965811910767e-14 -0.08726646270762471 3.11541271480963
- joint r_thumb_add: axis 3.164135620181696e-15 -3.643548754324866e-11 0.9999999999999999 -> 3.219646771412954e-15 -3.6435554830318275e-11 0.9999999999999998; origin xyz=0.023374863252664378 0.0030000000000001414 -0.03452383847607732 rpy=1.595197030995694e-15 -0.22689280265133213 -5.127419028200447e-16 -> xyz=0.023374863252664337 0.003000000000000058 -0.03452383847607743 rpy=1.566711369727914e-15 -0.226892802651332 -5.127419028200447e-16
- joint r_wrist_pitch: axis 2.6298942190638996e-11 -0.9999999999999998 -3.132558101803795e-11 -> 2.6298942190638987e-11 -0.9999999999999998 -3.1325553262462336e-11; origin xyz=-9.367506770274758e-17 -8.326672684688674e-17 -8.326672684688674e-17 rpy=2.775557561562892e-16 1.0408340855860843e-16 -3.8857805861880494e-16 -> xyz=-4.85722573273506e-17 0 2.7755575615628914e-17 rpy=2.2204460492503136e-16 -5.551115123125783e-17 -3.88578058618805e-16

File: urdf/ergoCub/robots/ergoCubSN001/model.urdf (robot description, URDF)
Before this commit: robot ergoCub, 204 links, 203 joints
Joints:
- joint l_index_add: axis -2.3462306050979376e-11 -1 3.353175760248158e-11 -> 1.5978340464762954e-11 0.9999999999999999 -3.7677226824487294e-11; origin xyz=0.022500000000000103 -0.0015000000000006675 -0.06859999999999955 rpy=-7.244015325404705e-16 -0.08726646259971596 -6.686783377296649e-16 -> xyz=0.022500000000000023 -0.0015000000000006952 -0.0685999999999996 rpy=-8.416895217637947e-16 -0.29670597224465534 5.804755322508926e-17
- joint l_index_dist: axis -0.9999999999999999 2.3461101117417404e-11 1.0798067476965604e-10 -> -0.9781476007113552 -1.553317034713362e-8 0.20791169092337955; origin xyz=1.5226389593614442e-11 -0.0015000000000001679 -0.03999999999723247 rpy=-7.4823262335988e-8 -1.0798106159226606e-10 -4.996003610813205e-16 -> xyz=-1.3877787807814457e-17 -0.001500000000000029 -0.03999999999999987 rpy=-7.482326172536535e-8 1.8041124150158794e-16 -6.106226635438361e-16
- joint l_index_prox: axis -0.9999999999999999 2.3461982356920424e-11 3.573530360490732e-15 -> -0.9781476007113543 2.3461557522424743e-11 0.2079116909233844; origin xyz=0.009192533317427871 -1.6653345369377348e-16 -0.030713451316238316 rpy=1.5543122344752197e-15 3.5388358909926865e-16 -1.1102230246251568e-16 -> xyz=0.00919253334679343 0 -0.030713451309624218 rpy=-3.0531133177191815e-16 -7.023611484080483e-10 -7.771561172376096e-16
- joint l_middle_prox: axis -1.0000000000000004 2.629437932314885e-11 -9.97489772601784e-15 -> -1.0000000000000004 2.629437917485816e-11 -9.988775473196015e-15; origin xyz=0.009600000000000143 -0.0015000000000005842 -0.10299999999999959 rpy=5.479728916549446e-4 1.6930901125533637e-15 -8.32667268468867e-16 -> xyz=0.00960000000000016 -0.0015000000000005842 -0.10299999999999959 rpy=5.479728916549446e-4 1.4363510381087963e-15 -8.32667268468867e-16
- joint l_pinkie_prox: axis -0.9999999998538291 7.644801389928454e-6 -1.529375688869017e-5 -> -0.9999999998538291 7.64480138992604e-6 -1.5293756888704046e-5; origin xyz=-0.03598232224952729 -0.0023883158589564635 -0.09206560929209856 rpy=-1.993459149294906e-5 0.08728175651239253 0.026187612448127052 -> xyz=-0.035982322249527285 -0.0023883158589564635 -0.09206560929209856 rpy=-1.9934591492976922e-5 0.08728175651239228 0.02618761244812705
- joint l_ring_prox: axis -1.0000000000000004 2.8926232503452798e-11 8.259087858064618e-13 -> -1.0000000000000002 2.8926226625044144e-11 8.259226635942696e-13; origin xyz=-0.015417755558120048 -0.0018498137284707894 -0.09788067183884419 rpy=-4.001819369801849e-5 0.0872664625997324 0.026179938779914452 -> xyz=-0.015417755558120038 -0.0018498137284707894 -0.09788067183884419 rpy=-4.001819369804634e-5 0.08726646259973214 0.026179938779914452
- joint l_thumb_add: axis -6.391803752947567e-12 3.5905271811298434e-11 -1 -> -6.391803752947567e-12 3.590529956687405e-11 -1.0000000000000002; origin xyz=0.02337486325639077 -0.0030000000000002525 -0.03452383847355461 rpy=-0.040449700618590975 0.2233191863655349 2.9608435412698353 -> xyz=0.02337486325639077 -0.0030000000000002525 -0.03452383847355461 rpy=-0.04044970061859103 0.22331918636553513 2.9608435412698353
- joint l_wrist_pitch: axis -2.6293939251520427e-11 -1.0000000000000002 3.1357194615824926e-11 -> -2.6293939251520434e-11 -1.0000000000000002 3.135719461582492e-11; origin xyz=-1.2836953722228372e-16 -1.6653345369377348e-16 0 rpy=-4.163336342344336e-16 1.079816722149296e-10 3.330669073875468e-16 -> xyz=-1.214306433183765e-16 -1.6653345369377348e-16 0 rpy=-4.163336342344336e-16 1.0798191507621624e-10 3.330669073875468e-16
- joint r_index_add: axis -2.3468226053640166e-11 0.9999999999999998 -3.349943223875093e-11 -> 1.5990673923572052e-11 -0.9999999999999999 3.764672729074698e-11; origin xyz=0.02249999999259583 0.0015000000000003066 -0.06860000000242839 rpy=-1.5881110520929587e-15 0.08726646249178613 3.1415926535897922 -> xyz=0.022499999999999992 0.0015000000000002234 -0.06859999999999983 rpy=-1.6833790438334957e-15 0.29670597283904 3.141592653589792
- joint r_index_dist: axis -0.9999999999999997 -2.3468990639763373e-11 -1.0793547999821127e-10 -> -0.9781476007113639 -2.3469068155297194e-11 -0.2079116909233363; origin xyz=-1.521995723896552e-11 -0.001500000000000029 -0.03999999999723369 rpy=4.1633363423443375e-16 1.0793393956376462e-10 -5.551115123125785e-17 -> xyz=4.163336342344337e-17 -0.0014999999999998903 -0.040000000000000036 rpy=1.942890293094024e-16 3.469446951953614e-17 1.665334536937736e-16
- joint r_index_prox: axis -0.9999999999999996 -2.3465285270418687e-11 -2.8727020762201978e-15 -> -0.9781476007113635 -2.3465277303774676e-11 -0.20791169092333764; origin xyz=-0.009192533317427698 8.326672684688674e-17 -0.030713451316238427 rpy=-8.881784197001254e-16 2.3592239273284576e-16 -1.6653345369377356e-16 -> xyz=-0.009192533317427393 5.551115123125783e-17 -0.030713451316238316 rpy=-3.0531133177191805e-16 -2.0816681711721685e-17 0
- joint r_middle_prox: axis -0.9999999999999997 -2.6303362266055585e-11 -1.6375789613479553e-15 -> -0.9999999999999996 -2.6303416042483343e-11 -1.6098233857581758e-15; origin xyz=0.009599999988883008 0.0015000000000004454 -0.10300000000103599 rpy=-1.8596235662471376e-15 -1.0793112237283964e-10 3.1415926535897927 -> xyz=0.009599999988882939 0.00150000000000039 -0.1030000000010361 rpy=-1.8596235662471376e-15 -1.0793124727292991e-10 3.1415926535897927
- joint r_pinkie_prox: axis -0.9999999999999998 -2.8722006374562025e-11 -1.0870657152217689e-10 -> -0.9999999999999998 -2.8722034177571486e-11 -1.0870652988881346e-10; origin xyz=-0.035982680943166104 0.002377759579109656 -0.0920682813194636 rpy=4.1095343980510334e-4 -0.0872664625997285 3.1154127148098776 -> xyz=-0.035982680943166166 0.002377759579109573 -0.09206828131946371 rpy=4.1095343980510334e-4 -0.08726646259972864 3.1154127148098776
- joint r_ring_prox: axis -0.9999999999999999 -2.893151623156253e-11 -8.271161533457416e-13 -> -0.9999999999999999 -2.893157069232462e-11 -8.271022755579338e-13; origin xyz=-0.015417755568684362 0.0018498137284712335 -0.09788067183717974 rpy=2.0171796521702004e-14 -0.08726646270762457 3.11541271480963 -> xyz=-0.015417755568684424 0.001849813728471178 -0.09788067183717986 rpy=2.019965811910767e-14 -0.08726646270762471 3.11541271480963
- joint r_thumb_add: axis 3.164135620181696e-15 -3.643548754324866e-11 0.9999999999999999 -> 3.219646771412954e-15 -3.6435554830318275e-11 0.9999999999999998; origin xyz=0.023374863252664378 0.0030000000000001414 -0.03452383847607732 rpy=1.595197030995694e-15 -0.22689280265133213 -5.127419028200447e-16 -> xyz=0.023374863252664337 0.003000000000000058 -0.03452383847607743 rpy=1.566711369727914e-15 -0.226892802651332 -5.127419028200447e-16
- joint r_wrist_pitch: axis 2.6298942190638996e-11 -0.9999999999999998 -3.132558101803795e-11 -> 2.6298942190638987e-11 -0.9999999999999998 -3.1325553262462336e-11; origin xyz=-9.367506770274758e-17 -8.326672684688674e-17 -8.326672684688674e-17 rpy=2.775557561562892e-16 1.0408340855860843e-16 -3.8857805861880494e-16 -> xyz=-4.85722573273506e-17 0 2.7755575615628914e-17 rpy=2.2204460492503136e-16 -5.551115123125783e-17 -3.88578058618805e-16
