Commit message: ergoCubV1_1: Fix reference frame in the lower legs
It fixes #74. Note that ergoCubV1 model will be not fixed since the the simulation model has not been changed since a while

File: urdf/ergoCub/robots/ergoCubGazeboV1_1/model.urdf (robot description, URDF)
Before this commit: robot ergoCub, 204 links, 203 joints
Links:
- link l_lower_leg: mass 3.741614150537795 -> 3.767581145212888
- link r_lower_leg: mass 3.7416141515311727 -> 3.7621532589747924
Joints:
- joint l_ankle_pitch: axis 2.405876710253171e-16 1 6.181058845623607e-17 -> -7.24267500143743e-17 1 6.181058845623533e-17; origin xyz=-3.701899897734506e-15 -0.03189999999999994 0.3209999999999994 rpy=-3.141592653589793 8.673617379885829e-19 -3.1554436208840472e-30 -> xyz=-4.468647674116255e-15 0.03189999999999981 -0.3209999999999995 rpy=-1.9704864186927032e-16 -8.673617379880112e-19 -1.8683953730959558e-16
- joint l_index_add: axis 1.5978340464762954e-11 0.9999999999999999 -3.7677226824487294e-11 -> 1.5978451487065422e-11 1.0000000000000002 -3.767719906891169e-11; origin xyz=0.022500000000000023 -0.0015000000000006952 -0.0685999999999996 rpy=-8.416895217637947e-16 -0.29670597224465534 5.804755322508926e-17 -> xyz=0.022500000000000034 -0.0015000000000006397 -0.06859999999999966 rpy=-8.126657451512497e-16 -0.2967059722446555 1.7414265967526777e-16
- joint l_index_dist: axis -0.9781476007113552 -1.553317034713362e-8 0.20791169092337955 -> -0.9781476007113552 -1.5533170287064815e-8 0.2079116909233797; origin xyz=-1.3877787807814457e-17 -0.001500000000000029 -0.03999999999999987 rpy=-7.482326172536535e-8 1.8041124150158794e-16 -6.106226635438361e-16 -> xyz=-2.7755575615628914e-17 -0.0014999999999999736 -0.039999999999999925 rpy=-7.482326169760975e-8 1.734723475976807e-16 -6.106226635438361e-16
- joint l_index_prox: axis -0.9781476007113543 2.3461557522424743e-11 0.2079116909233844 -> -0.9781476007113546 2.346155062839741e-11 0.20791169092338443; origin xyz=0.00919253334679343 0 -0.030713451309624218 rpy=-3.0531133177191815e-16 -7.023611484080483e-10 -7.771561172376096e-16 -> xyz=0.009192533346793416 -2.7755575615628914e-17 -0.030713451309624162 rpy=-2.7755575615628914e-16 -7.023611553469422e-10 -7.771561172376094e-16
- joint l_knee: axis -2.4058767102531225e-16 1 6.181058845623608e-17 -> -4.27427208334911e-16 -1 1.3523805341303425e-16; origin xyz=0.010600000000000049 -0.00790000000000024 -0.17969999999999958 rpy=-3.141592653589793 -1.1419428146632273e-14 2.6734444562115447e-15 -> xyz=0.010600000000000822 -0.007900000000000185 -0.17969999999999958 rpy=1.970486418692682e-16 -1.1419428146632273e-14 2.8602839935211434e-15
- joint r_ankle_pitch: axis 1.8699102912341645e-16 1 -1.9666186429286112e-16 -> -1.342621999194175e-15 1 -3.530978817196621e-14; origin xyz=-1.2462253451417382e-14 0.031899999999999984 0.3210000000000002 rpy=-3.141592653589793 1.2923622733154212e-30 -1.6653283970679406e-16 -> xyz=-5.936223734792634e-15 -0.03190000000000005 -0.3210000000000002 rpy=-2.9932805576414174e-15 -2.0242047360524565e-14 8.880636788937802e-17
- joint r_ankle_roll: axis -1 5.921958056855112e-17 2.5592852998214428e-15 -> -1 -2.1833586821066654e-16 2.39275322255624e-15; origin xyz=-0.05275000000000156 0.018200000000000008 -0.03499999999999759 rpy=1.1129880739582211e-25 3.883828473168634e-14 1.1834052693462316e-23 -> xyz=-0.052750000000001546 0.018200000000000008 -0.0349999999999977 rpy=-1.0176053241861382e-24 3.8838282931741325e-14 -9.278622199115707e-23
- joint r_foot_front_ft_sensor: origin xyz=0.13524999999999998 4.163336342344337e-17 -0.04789999999999983 rpy=2.6613913647137395e-17 -9.208113692419518e-17 -1.4551885312033586e-15 -> xyz=0.13525000000000004 0 -0.04789999999999994 rpy=2.66139136471374e-17 -9.20811369242055e-17 -1.4551888385804406e-15
- joint r_foot_rear_ft_sensor: origin xyz=0.016 2.7755575615628914e-17 -0.04789999999999983 rpy=2.6613913647112164e-17 -9.20811369242145e-17 -1.5662108336658734e-15 -> xyz=0.016 0 -0.04789999999999983 rpy=2.661391364712478e-17 -9.208113692419957e-17 -1.566211141042955e-15
- joint r_knee: axis -2.0458175022504648e-17 1 2.5382740632965355e-17 -> 1.7937066152151813e-16 -1 3.2454535731621664e-15; origin xyz=0.01060000963260986 0.007899987075259199 -0.17970000000000103 rpy=-3.1415926535897274 -8.69101748565412e-14 -1.2193157698906137e-6 -> xyz=0.01060000963260985 0.007899987075259289 -0.17970000000000058 rpy=6.892643261935339e-14 -6.650159361880639e-14 -1.2193157700904425e-6

File: urdf/ergoCub/robots/ergoCubGazeboV1_1_minContacts/model.urdf (robot description, URDF)
Before this commit: robot ergoCub, 204 links, 203 joints
Links:
- link l_lower_leg: mass 3.741614150537795 -> 3.767581145212888
- link r_lower_leg: mass 3.7416141515311727 -> 3.7621532589747924
Joints:
- joint l_ankle_pitch: axis 2.405876710253171e-16 1 6.181058845623607e-17 -> -7.24267500143743e-17 1 6.181058845623533e-17; origin xyz=-3.701899897734506e-15 -0.03189999999999994 0.3209999999999994 rpy=-3.141592653589793 8.673617379885829e-19 -3.1554436208840472e-30 -> xyz=-4.468647674116255e-15 0.03189999999999981 -0.3209999999999995 rpy=-1.9704864186927032e-16 -8.673617379880112e-19 -1.8683953730959558e-16
- joint l_index_add: axis 1.5978340464762954e-11 0.9999999999999999 -3.7677226824487294e-11 -> 1.5978451487065422e-11 1.0000000000000002 -3.767719906891169e-11; origin xyz=0.022500000000000023 -0.0015000000000006952 -0.0685999999999996 rpy=-8.416895217637947e-16 -0.29670597224465534 5.804755322508926e-17 -> xyz=0.022500000000000034 -0.0015000000000006397 -0.06859999999999966 rpy=-8.126657451512497e-16 -0.2967059722446555 1.7414265967526777e-16
- joint l_index_dist: axis -0.9781476007113552 -1.553317034713362e-8 0.20791169092337955 -> -0.9781476007113552 -1.5533170287064815e-8 0.2079116909233797; origin xyz=-1.3877787807814457e-17 -0.001500000000000029 -0.03999999999999987 rpy=-7.482326172536535e-8 1.8041124150158794e-16 -6.106226635438361e-16 -> xyz=-2.7755575615628914e-17 -0.0014999999999999736 -0.039999999999999925 rpy=-7.482326169760975e-8 1.734723475976807e-16 -6.106226635438361e-16
- joint l_index_prox: axis -0.9781476007113543 2.3461557522424743e-11 0.2079116909233844 -> -0.9781476007113546 2.346155062839741e-11 0.20791169092338443; origin xyz=0.00919253334679343 0 -0.030713451309624218 rpy=-3.0531133177191815e-16 -7.023611484080483e-10 -7.771561172376096e-16 -> xyz=0.009192533346793416 -2.7755575615628914e-17 -0.030713451309624162 rpy=-2.7755575615628914e-16 -7.023611553469422e-10 -7.771561172376094e-16
- joint l_knee: axis -2.4058767102531225e-16 1 6.181058845623608e-17 -> -4.27427208334911e-16 -1 1.3523805341303425e-16; origin xyz=0.010600000000000049 -0.00790000000000024 -0.17969999999999958 rpy=-3.141592653589793 -1.1419428146632273e-14 2.6734444562115447e-15 -> xyz=0.010600000000000822 -0.007900000000000185 -0.17969999999999958 rpy=1.970486418692682e-16 -1.1419428146632273e-14 2.8602839935211434e-15
- joint r_ankle_pitch: axis 1.8699102912341645e-16 1 -1.9666186429286112e-16 -> -1.342621999194175e-15 1 -3.530978817196621e-14; origin xyz=-1.2462253451417382e-14 0.031899999999999984 0.3210000000000002 rpy=-3.141592653589793 1.2923622733154212e-30 -1.6653283970679406e-16 -> xyz=-5.936223734792634e-15 -0.03190000000000005 -0.3210000000000002 rpy=-2.9932805576414174e-15 -2.0242047360524565e-14 8.880636788937802e-17
- joint r_ankle_roll: axis -1 5.921958056855112e-17 2.5592852998214428e-15 -> -1 -2.1833586821066654e-16 2.39275322255624e-15; origin xyz=-0.05275000000000156 0.018200000000000008 -0.03499999999999759 rpy=1.1129880739582211e-25 3.883828473168634e-14 1.1834052693462316e-23 -> xyz=-0.052750000000001546 0.018200000000000008 -0.0349999999999977 rpy=-1.0176053241861382e-24 3.8838282931741325e-14 -9.278622199115707e-23
- joint r_foot_front_ft_sensor: origin xyz=0.13524999999999998 4.163336342344337e-17 -0.04789999999999983 rpy=2.6613913647137395e-17 -9.208113692419518e-17 -1.4551885312033586e-15 -> xyz=0.13525000000000004 0 -0.04789999999999994 rpy=2.66139136471374e-17 -9.20811369242055e-17 -1.4551888385804406e-15
- joint r_foot_rear_ft_sensor: origin xyz=0.016 2.7755575615628914e-17 -0.04789999999999983 rpy=2.6613913647112164e-17 -9.20811369242145e-17 -1.5662108336658734e-15 -> xyz=0.016 0 -0.04789999999999983 rpy=2.661391364712478e-17 -9.208113692419957e-17 -1.566211141042955e-15
- joint r_knee: axis -2.0458175022504648e-17 1 2.5382740632965355e-17 -> 1.7937066152151813e-16 -1 3.2454535731621664e-15; origin xyz=0.01060000963260986 0.007899987075259199 -0.17970000000000103 rpy=-3.1415926535897274 -8.69101748565412e-14 -1.2193157698906137e-6 -> xyz=0.01060000963260985 0.007899987075259289 -0.17970000000000058 rpy=6.892643261935339e-14 -6.650159361880639e-14 -1.2193157700904425e-6

File: urdf/ergoCub/robots/ergoCubSN001/model.urdf (robot description, URDF)
Before this commit: robot ergoCub, 204 links, 203 joints
Links:
- link l_lower_leg: mass 3.741614150537795 -> 3.767581145212888
- link r_lower_leg: mass 3.7416141515311727 -> 3.7621532589747924
Joints:
- joint l_ankle_pitch: axis 2.405876710253171e-16 1 6.181058845623607e-17 -> -7.24267500143743e-17 1 6.181058845623533e-17; origin xyz=-3.701899897734506e-15 -0.03189999999999994 0.3209999999999994 rpy=-3.141592653589793 8.673617379885829e-19 -3.1554436208840472e-30 -> xyz=-4.468647674116255e-15 0.03189999999999981 -0.3209999999999995 rpy=-1.9704864186927032e-16 -8.673617379880112e-19 -1.8683953730959558e-16
- joint l_knee: axis -2.4058767102531225e-16 1 6.181058845623608e-17 -> -4.27427208334911e-16 -1 1.3523805341303425e-16; origin xyz=0.010600000000000049 -0.00790000000000024 -0.17969999999999958 rpy=-3.141592653589793 -1.1419428146632273e-14 2.6734444562115447e-15 -> xyz=0.010600000000000822 -0.007900000000000185 -0.17969999999999958 rpy=1.970486418692682e-16 -1.1419428146632273e-14 2.8602839935211434e-15
- joint r_ankle_pitch: axis 1.8699102912341645e-16 1 -1.9666186429286112e-16 -> -1.342621999194175e-15 1 -3.530978817196621e-14; origin xyz=-1.2462253451417382e-14 0.031899999999999984 0.3210000000000002 rpy=-3.141592653589793 1.2923622733154212e-30 -1.6653283970679406e-16 -> xyz=-5.936223734792634e-15 -0.03190000000000005 -0.3210000000000002 rpy=-2.9932805576414174e-15 -2.0242047360524565e-14 8.880636788937802e-17
- joint r_ankle_roll: axis -1 5.921958056855112e-17 2.5592852998214428e-15 -> -1 -2.1833586821066654e-16 2.39275322255624e-15; origin xyz=-0.05275000000000156 0.018200000000000008 -0.03499999999999759 rpy=1.1129880739582211e-25 3.883828473168634e-14 1.1834052693462316e-23 -> xyz=-0.052750000000001546 0.018200000000000008 -0.0349999999999977 rpy=-1.0176053241861382e-24 3.8838282931741325e-14 -9.278622199115707e-23
- joint r_foot_front_ft_sensor: origin xyz=0.13524999999999998 4.163336342344337e-17 -0.04789999999999983 rpy=2.6613913647137395e-17 -9.208113692419518e-17 -1.4551885312033586e-15 -> xyz=0.13525000000000004 0 -0.04789999999999994 rpy=2.66139136471374e-17 -9.20811369242055e-17 -1.4551888385804406e-15
- joint r_foot_rear_ft_sensor: origin xyz=0.016 2.7755575615628914e-17 -0.04789999999999983 rpy=2.6613913647112164e-17 -9.20811369242145e-17 -1.5662108336658734e-15 -> xyz=0.016 0 -0.04789999999999983 rpy=2.661391364712478e-17 -9.208113692419957e-17 -1.566211141042955e-15
- joint r_knee: axis -2.0458175022504648e-17 1 2.5382740632965355e-17 -> 1.7937066152151813e-16 -1 3.2454535731621664e-15; origin xyz=0.01060000963260986 0.007899987075259199 -0.17970000000000103 rpy=-3.1415926535897274 -8.69101748565412e-14 -1.2193157698906137e-6 -> xyz=0.01060000963260985 0.007899987075259289 -0.17970000000000058 rpy=6.892643261935339e-14 -6.650159361880639e-14 -1.2193157700904425e-6
