Commit message: ergoCubV1_1: regenerate urdf after creo2urdf axis bugfix

File: urdf/ergoCub/robots/ergoCubSN001/model.urdf (robot description, URDF)
Before this commit: robot ergoCub, 204 links, 203 joints
Joints:
- joint camera_tilt: axis -3.611636085008543e-15 -1 -1.9429477071513935e-15 -> -3.1332662159460226e-17 -1 -1.3036401662462866e-15
- joint l_ankle_pitch: axis -7.24267500143743e-17 1 6.181058845623533e-17 -> -2.389602037081462e-16 1 1.4538275231733847e-16
- joint l_ankle_roll: axis 1 -5.715619358951517e-16 -1.2940468202020292e-15 -> 1 -4.05028482201375e-16 -1.2496691978128869e-15
- joint l_elbow: axis -6.9388939037918944e-18 -0.9999999999999953 6.4392935428256776e-15 -> -4.215378046622413e-16 -0.9999999999999953 6.5780714209038095e-15
- joint l_hip_roll: axis 1 -2.277657936511405e-16 5.765028837511023e-16 -> 1 -6.123233995736708e-17 6.3201403498236e-16
- joint l_hip_yaw: axis -8.067476499456731e-16 -6.18105884562747e-17 1 -> -8.622588011769357e-16 1.593666547307703e-16 1
- joint l_index_add: axis 1.5978451487065422e-11 1.0000000000000002 -3.767719906891169e-11 -> 1.3005559878087045e-15 1.0000000000000002 -1.953448495705706e-15
- joint l_index_dist: axis -0.9781476007113552 -1.5533170287064815e-8 0.2079116909233797 -> -1 -1.804112664227406e-16 9.020562801946248e-17
- joint l_index_prox: axis -0.9781476007113546 2.346155062839741e-11 0.20791169092338443 -> -1.0000000000000002 2.7755575615627613e-17 7.023654366444809e-10
- joint l_knee: axis -4.27427208334911e-16 -1 1.3523805341303425e-16 -> -2.608937546411318e-16 -1 5.166588955193111e-17
- joint l_middle_dist: axis -1 2.824224757752587e-11 1.074840171400902e-10 -> -1 1.952334931070572e-12 1.0795870667149422e-10
- joint l_middle_prox: axis -1.0000000000000004 2.629437917485816e-11 -9.988775473196015e-15 -> -1.0000000000000004 1.6098145522958664e-16 4.176883423103147e-15
- joint l_pinkie_dist: axis -0.9999999998538307 7.645479968428705e-6 -1.529330960500596e-5 -> -0.9999999998538309 7.645451042193251e-6 -1.5293310428212298e-5
- joint l_pinkie_prox: axis -0.9999999998538291 7.64480138992604e-6 -1.5293756888704046e-5 -> -0.9999999998538295 7.644772463726695e-6 -1.529375771042174e-5
- joint l_ring_dist: axis -1 2.8664399475776237e-11 1.0876850894396261e-10 -> -1 -2.617159685310911e-13 1.0794249544288393e-10
- joint l_ring_prox: axis -1.0000000000000002 2.8926226625044144e-11 8.259226635942696e-13 -> -1.0000000000000002 4.364549018964596e-17 3.6637359812630166e-15
- joint l_shoulder_roll: axis 1 7.615436059538576e-16 3.2196467714129958e-15 -> 1 4.891920202255013e-16 3.3029134982598896e-15
- joint l_shoulder_yaw: axis -2.982336599899327e-14 3.2196467714129528e-15 -0.9999999999999977 -> -3.0080105073437835e-14 3.191891195797326e-15 -0.9999999999999977
- joint l_thumb_add: axis -6.391803752947567e-12 3.590529956687405e-11 -1.0000000000000002 -> 9.71445146547012e-16 1.0269562977782698e-15 -1.0000000000000002
- joint l_thumb_dist: axis 5.648245760041583e-12 -5.177168416189185e-11 -0.9999999999999996 -> -1.846719305254041e-11 -1.8750709318560158e-11 -0.9999999999999996
- joint l_thumb_prox: axis 2.4115921065659407e-11 -3.3017838463322846e-11 -0.9999999999999997 -> 5.134781488891349e-16 3.1363800445660672e-15 -0.9999999999999996
- joint l_wrist_pitch: axis -2.6293939251520434e-11 -1.0000000000000002 3.135719461582492e-11 -> -2.4459601009774425e-16 -1.0000000000000002 -1.3600232051562635e-15
- joint l_wrist_roll: axis -1.0000000000000004 2.6294445787389307e-11 1.0798215793750289e-10 -> -1.0000000000000004 4.909267437014364e-16 -2.0122792321330943e-16
- joint l_wrist_yaw: axis -3.1939728639684985e-14 2.7755575615628937e-15 -0.9999999999999981 -> -3.1023794644369224e-14 2.9420910152566676e-15 -0.9999999999999981
- joint neck_pitch: axis 2.6474328740344387e-18 -1 -7.807082888609213e-16 -> 2.6472211157644926e-18 -1 -7.807858529815144e-16
- joint neck_roll: axis 1 -1.6832426434147407e-15 -3.770068640066623e-15 -> 1 -1.6820355477448088e-15 -3.806893332301044e-15
- joint neck_yaw: axis 3.4240774521066226e-15 -2.686540855695209e-16 0.9999999999999998 -> 3.1628618281392715e-15 1.6479574685948862e-15 0.9999999999999998
- joint r_ankle_pitch: axis -1.342621999194175e-15 1 -3.530978817196621e-14 -> -3.505264366441263e-17 1 -1.331317022347139e-16
- joint r_ankle_roll: axis -1 -2.1833586821066654e-16 2.39275322255624e-15 -> -1 -1.628246671334752e-16 2.560295622560413e-15
- joint r_elbow: axis 4.163336342349831e-17 -1.0000000000000027 2.5673907444456773e-14 -> 3.001071613439684e-16 -1.0000000000000027 1.2712053631958044e-14
- joint r_hip_roll: axis -1 -3.3813287685014083e-16 -8.532880891569492e-14 -> -1 -3.3813287685016297e-16 -7.120227705451219e-17
- joint r_hip_yaw: axis 8.528600225431674e-14 1.503215654809462e-15 -1 -> -2.3953050207433507e-20 1.4749328491810949e-15 -1
- joint r_index_add: axis 1.5990673923572052e-11 -0.9999999999999999 3.764672729074698e-11 -> -5.389323627044831e-16 -0.9999999999999999 1.6046911875538946e-15
- joint r_index_dist: axis -0.9781476007113639 -2.3469068155297194e-11 -0.2079116909233363 -> -0.9999999999999993 -2.0122792321330975e-16 -4.510281037539697e-16
- joint r_index_prox: axis -0.9781476007113635 -2.3465277303774676e-11 -0.20791169092333764 -> -0.9999999999999993 3.434752482434078e-15 -1.672273430841644e-15
- joint r_knee: axis 1.7937066152151813e-16 -1 3.2454535731621664e-15 -> 1.2193157766326317e-6 -0.9999999999992566 4.719551160658923e-15
- joint r_middle_dist: axis -0.9999999999999998 -2.630088161156088e-11 -1.079318529386326e-10 -> -0.9999999999999998 -2.0695253452753748e-15 -1.0792969296086812e-10
- joint r_middle_prox: axis -0.9999999999999996 -2.6303416042483343e-11 -1.6098233857581758e-15 -> -0.9999999999999996 -4.562322741819007e-15 1.079337105802658e-10
- joint r_pinkie_dist: axis -0.9999999999999999 -2.8584519595543556e-11 -1.0874608649338082e-10 -> -0.9999999999999999 9.036247971209683e-16 -2.4586692098222613e-15
- joint r_pinkie_prox: axis -0.9999999999999998 -2.8722034177571486e-11 -1.0870652988881346e-10 -> -0.9999999999999998 4.364801434782878e-15 0
- joint r_ring_dist: axis -0.9999999999999999 -2.8681237072836204e-11 -1.0871797212486101e-10 -> -0.9999999999999999 2.4672971998818127e-13 -1.0789569585001324e-10
- joint r_ring_prox: axis -0.9999999999999999 -2.893157069232462e-11 -8.271022755579338e-13 -> -0.9999999999999997 -2.498435601042699e-13 1.0789123761067998e-10
- joint r_shoulder_roll: axis -1.0000000000000007 1.0148132334463434e-15 -2.567390744445154e-16 -> -1.0000000000000007 8.760353553682006e-16 -4.510281037539194e-16
- joint r_shoulder_yaw: axis 3.122502256758238e-16 -2.498001805406602e-16 1.0000000000000004 -> 2.567390744445681e-16 2.775557561562927e-17 1.0000000000000004
- joint r_thumb_add: axis 3.219646771412954e-15 -3.6435554830318275e-11 0.9999999999999998 -> -1.0793213545134961e-10 2.4089270891491094e-15 0.9999999999999998
- joint r_thumb_dist: axis -5.6626925371494566e-12 5.173264594478845e-11 -0.9999999999999999 -> 1.8458673825549887e-11 1.8743298579870785e-11 -0.9999999999999999
- joint r_thumb_prox: axis 2.4122360359202233e-11 -3.299033268788776e-11 -0.9999999999999999 -> 9.992007221626409e-16 -1.1102230246251565e-15 -0.9999999999999997
- joint r_wrist_pitch: axis 2.6298942190638987e-11 -0.9999999999999998 -3.1325553262462336e-11 -> 4.128641872824801e-16 -0.9999999999999998 -8.049116928532385e-16
- joint r_wrist_roll: axis 0.9999999999999997 2.6298196259544278e-11 -1.0793549387599907e-10 -> 0.9999999999999997 -2.480654570646835e-16 -1.873501354054953e-16
- joint r_wrist_yaw: axis 6.057654378111005e-15 -5.273559366969643e-16 1.000000000000002 -> 5.5788706987414416e-15 -1.2628786905111175e-14 1.000000000000002
- joint torso_yaw: axis 2.084891490280543e-15 -2.11369334484512e-15 -1 -> 2.084864385226231e-15 -2.114127025714114e-15 -1

Commit message: ergoCubV1_1: move down the l/r_sole frames
It fixes #186

File: urdf/ergoCub/robots/ergoCubGazeboV1_1/model.urdf (robot description, URDF)
Before this commit: robot ergoCub, 204 links, 203 joints
Joints:
- joint l_index_add: axis 1.3005559878087045e-15 1.0000000000000002 -1.953448495705706e-15 -> 1.1895336853461886e-15 0.9999999999999999 -1.9812040713213337e-15; origin xyz=0.022500000000000034 -0.0015000000000006397 -0.06859999999999966 rpy=-8.126657451512497e-16 -0.2967059722446555 1.7414265967526777e-16 -> xyz=0.022500000000000023 -0.0015000000000006952 -0.0685999999999996 rpy=-8.416895217637947e-16 -0.29670597224465534 5.804755322508926e-17
- joint l_index_dist: axis -1 -1.804112664227406e-16 9.020562801946248e-17 -> -1 -2.359224176539984e-16 4.163337069211178e-17; origin xyz=-2.7755575615628914e-17 -0.0014999999999999736 -0.039999999999999925 rpy=-7.482326169760975e-8 1.734723475976807e-16 -6.106226635438361e-16 -> xyz=-1.3877787807814457e-17 -0.001500000000000029 -0.03999999999999987 rpy=-7.482326172536535e-8 1.8041124150158794e-16 -6.106226635438361e-16
- joint l_index_prox: axis -1.0000000000000002 2.7755575615627613e-17 7.023654366444809e-10 -> -1 8.326672684688522e-17 7.023654435833748e-10; origin xyz=0.009192533346793416 -2.7755575615628914e-17 -0.030713451309624162 rpy=-2.7755575615628914e-16 -7.023611553469422e-10 -7.771561172376094e-16 -> xyz=0.00919253334679343 0 -0.030713451309624218 rpy=-3.0531133177191815e-16 -7.023611484080483e-10 -7.771561172376096e-16
- joint l_sole_fixed_joint: origin xyz=0.059629999999999996 0 1.1102230246251565e-16 rpy=0 1.5094274020956558e-31 0 -> xyz=0.059629999999999996 -1.3877787807814457e-17 -0.024299999999999877 rpy=0 1.5094274020956558e-31 0
- joint r_sole_fixed_joint: origin xyz=0.05963 -1.3877787807814457e-17 7.771561172376096e-16 rpy=0 3.1371750050201436e-30 0 -> xyz=0.05963 -1.3877787807814457e-17 -0.02429999999999999 rpy=0 3.1371750050201436e-30 0

File: urdf/ergoCub/robots/ergoCubGazeboV1_1_minContacts/model.urdf (robot description, URDF)
Before this commit: robot ergoCub, 204 links, 203 joints
Joints:
- joint l_index_add: axis 1.3005559878087045e-15 1.0000000000000002 -1.953448495705706e-15 -> 1.1895336853461886e-15 0.9999999999999999 -1.9812040713213337e-15; origin xyz=0.022500000000000034 -0.0015000000000006397 -0.06859999999999966 rpy=-8.126657451512497e-16 -0.2967059722446555 1.7414265967526777e-16 -> xyz=0.022500000000000023 -0.0015000000000006952 -0.0685999999999996 rpy=-8.416895217637947e-16 -0.29670597224465534 5.804755322508926e-17
- joint l_index_dist: axis -1 -1.804112664227406e-16 9.020562801946248e-17 -> -1 -2.359224176539984e-16 4.163337069211178e-17; origin xyz=-2.7755575615628914e-17 -0.0014999999999999736 -0.039999999999999925 rpy=-7.482326169760975e-8 1.734723475976807e-16 -6.106226635438361e-16 -> xyz=-1.3877787807814457e-17 -0.001500000000000029 -0.03999999999999987 rpy=-7.482326172536535e-8 1.8041124150158794e-16 -6.106226635438361e-16
- joint l_index_prox: axis -1.0000000000000002 2.7755575615627613e-17 7.023654366444809e-10 -> -1 8.326672684688522e-17 7.023654435833748e-10; origin xyz=0.009192533346793416 -2.7755575615628914e-17 -0.030713451309624162 rpy=-2.7755575615628914e-16 -7.023611553469422e-10 -7.771561172376094e-16 -> xyz=0.00919253334679343 0 -0.030713451309624218 rpy=-3.0531133177191815e-16 -7.023611484080483e-10 -7.771561172376096e-16
- joint l_sole_fixed_joint: origin xyz=0.059629999999999996 0 1.1102230246251565e-16 rpy=0 1.5094274020956558e-31 0 -> xyz=0.059629999999999996 -1.3877787807814457e-17 -0.024299999999999877 rpy=0 1.5094274020956558e-31 0
- joint r_sole_fixed_joint: origin xyz=0.05963 -1.3877787807814457e-17 7.771561172376096e-16 rpy=0 3.1371750050201436e-30 0 -> xyz=0.05963 -1.3877787807814457e-17 -0.02429999999999999 rpy=0 3.1371750050201436e-30 0

File: urdf/ergoCub/robots/ergoCubSN001/model.urdf (robot description, URDF)
Before this commit: robot ergoCub, 204 links, 203 joints
Joints:
- joint l_index_add: axis 1.3005559878087045e-15 1.0000000000000002 -1.953448495705706e-15 -> 1.1895336853461886e-15 0.9999999999999999 -1.9812040713213337e-15; origin xyz=0.022500000000000034 -0.0015000000000006397 -0.06859999999999966 rpy=-8.126657451512497e-16 -0.2967059722446555 1.7414265967526777e-16 -> xyz=0.022500000000000023 -0.0015000000000006952 -0.0685999999999996 rpy=-8.416895217637947e-16 -0.29670597224465534 5.804755322508926e-17
- joint l_index_dist: axis -1 -1.804112664227406e-16 9.020562801946248e-17 -> -1 -2.359224176539984e-16 4.163337069211178e-17; origin xyz=-2.7755575615628914e-17 -0.0014999999999999736 -0.039999999999999925 rpy=-7.482326169760975e-8 1.734723475976807e-16 -6.106226635438361e-16 -> xyz=-1.3877787807814457e-17 -0.001500000000000029 -0.03999999999999987 rpy=-7.482326172536535e-8 1.8041124150158794e-16 -6.106226635438361e-16
- joint l_index_prox: axis -1.0000000000000002 2.7755575615627613e-17 7.023654366444809e-10 -> -1 8.326672684688522e-17 7.023654435833748e-10; origin xyz=0.009192533346793416 -2.7755575615628914e-17 -0.030713451309624162 rpy=-2.7755575615628914e-16 -7.023611553469422e-10 -7.771561172376094e-16 -> xyz=0.00919253334679343 0 -0.030713451309624218 rpy=-3.0531133177191815e-16 -7.023611484080483e-10 -7.771561172376096e-16
- joint l_sole_fixed_joint: origin xyz=0.059629999999999996 0 1.1102230246251565e-16 rpy=0 1.5094274020956558e-31 0 -> xyz=0.059629999999999996 -1.3877787807814457e-17 -0.024299999999999877 rpy=0 1.5094274020956558e-31 0
- joint r_sole_fixed_joint: origin xyz=0.05963 -1.3877787807814457e-17 7.771561172376096e-16 rpy=0 3.1371750050201436e-30 0 -> xyz=0.05963 -1.3877787807814457e-17 -0.02429999999999999 rpy=0 3.1371750050201436e-30 0

Commit message: ergoCubV1*: fix alignment of the depth.
It is now aligned w/ the RGB frame as on the real robot.
It fixes #183

File: urdf/ergoCub/robots/ergoCubGazeboV1_1/model.urdf (robot description, URDF)
Before this commit: robot ergoCub, 204 links, 203 joints
Joints:
- joint l_index_add: axis 1.1895336853461886e-15 0.9999999999999999 -1.9812040713213337e-15 -> 1.3005559878087045e-15 1.0000000000000002 -1.953448495705706e-15; origin xyz=0.022500000000000023 -0.0015000000000006952 -0.0685999999999996 rpy=-8.416895217637947e-16 -0.29670597224465534 5.804755322508926e-17 -> xyz=0.022500000000000034 -0.0015000000000006397 -0.06859999999999966 rpy=-8.126657451512497e-16 -0.2967059722446555 1.7414265967526777e-16
- joint l_index_dist: axis -1 -2.359224176539984e-16 4.163337069211178e-17 -> -1 -1.804112664227406e-16 9.020562801946248e-17; origin xyz=-1.3877787807814457e-17 -0.001500000000000029 -0.03999999999999987 rpy=-7.482326172536535e-8 1.8041124150158794e-16 -6.106226635438361e-16 -> xyz=-2.7755575615628914e-17 -0.0014999999999999736 -0.039999999999999925 rpy=-7.482326169760975e-8 1.734723475976807e-16 -6.106226635438361e-16
- joint l_index_prox: axis -1 8.326672684688522e-17 7.023654435833748e-10 -> -1.0000000000000002 2.7755575615627613e-17 7.023654366444809e-10; origin xyz=0.00919253334679343 0 -0.030713451309624218 rpy=-3.0531133177191815e-16 -7.023611484080483e-10 -7.771561172376096e-16 -> xyz=0.009192533346793416 -2.7755575615628914e-17 -0.030713451309624162 rpy=-2.7755575615628914e-16 -7.023611553469422e-10 -7.771561172376094e-16

File: urdf/ergoCub/robots/ergoCubGazeboV1_1_minContacts/model.urdf (robot description, URDF)
Before this commit: robot ergoCub, 204 links, 203 joints
Joints:
- joint l_index_add: axis 1.1895336853461886e-15 0.9999999999999999 -1.9812040713213337e-15 -> 1.3005559878087045e-15 1.0000000000000002 -1.953448495705706e-15; origin xyz=0.022500000000000023 -0.0015000000000006952 -0.0685999999999996 rpy=-8.416895217637947e-16 -0.29670597224465534 5.804755322508926e-17 -> xyz=0.022500000000000034 -0.0015000000000006397 -0.06859999999999966 rpy=-8.126657451512497e-16 -0.2967059722446555 1.7414265967526777e-16
- joint l_index_dist: axis -1 -2.359224176539984e-16 4.163337069211178e-17 -> -1 -1.804112664227406e-16 9.020562801946248e-17; origin xyz=-1.3877787807814457e-17 -0.001500000000000029 -0.03999999999999987 rpy=-7.482326172536535e-8 1.8041124150158794e-16 -6.106226635438361e-16 -> xyz=-2.7755575615628914e-17 -0.0014999999999999736 -0.039999999999999925 rpy=-7.482326169760975e-8 1.734723475976807e-16 -6.106226635438361e-16
- joint l_index_prox: axis -1 8.326672684688522e-17 7.023654435833748e-10 -> -1.0000000000000002 2.7755575615627613e-17 7.023654366444809e-10; origin xyz=0.00919253334679343 0 -0.030713451309624218 rpy=-3.0531133177191815e-16 -7.023611484080483e-10 -7.771561172376096e-16 -> xyz=0.009192533346793416 -2.7755575615628914e-17 -0.030713451309624162 rpy=-2.7755575615628914e-16 -7.023611553469422e-10 -7.771561172376094e-16

File: urdf/ergoCub/robots/ergoCubSN001/model.urdf (robot description, URDF)
Before this commit: robot ergoCub, 204 links, 203 joints
Joints:
- joint l_index_add: axis 1.1895336853461886e-15 0.9999999999999999 -1.9812040713213337e-15 -> 1.3005559878087045e-15 1.0000000000000002 -1.953448495705706e-15; origin xyz=0.022500000000000023 -0.0015000000000006952 -0.0685999999999996 rpy=-8.416895217637947e-16 -0.29670597224465534 5.804755322508926e-17 -> xyz=0.022500000000000034 -0.0015000000000006397 -0.06859999999999966 rpy=-8.126657451512497e-16 -0.2967059722446555 1.7414265967526777e-16
- joint l_index_dist: axis -1 -2.359224176539984e-16 4.163337069211178e-17 -> -1 -1.804112664227406e-16 9.020562801946248e-17; origin xyz=-1.3877787807814457e-17 -0.001500000000000029 -0.03999999999999987 rpy=-7.482326172536535e-8 1.8041124150158794e-16 -6.106226635438361e-16 -> xyz=-2.7755575615628914e-17 -0.0014999999999999736 -0.039999999999999925 rpy=-7.482326169760975e-8 1.734723475976807e-16 -6.106226635438361e-16
- joint l_index_prox: axis -1 8.326672684688522e-17 7.023654435833748e-10 -> -1.0000000000000002 2.7755575615627613e-17 7.023654366444809e-10; origin xyz=0.00919253334679343 0 -0.030713451309624218 rpy=-3.0531133177191815e-16 -7.023611484080483e-10 -7.771561172376096e-16 -> xyz=0.009192533346793416 -2.7755575615628914e-17 -0.030713451309624162 rpy=-2.7755575615628914e-16 -7.023611553469422e-10 -7.771561172376094e-16

Commit message: ergoCubGazeboV1_1: simplify collision geometry of the fingers
For augmenting the real time factor we used to simplify the collision geometry of the fingers with cylinders. The measures have been taken roughtly from the CAD. It fixes #199

File: urdf/ergoCub/robots/ergoCubGazeboV1_1/model.urdf (robot description, URDF)
Before this commit: robot ergoCub, 204 links, 203 joints
Links:
- link l_hand_index_2: geometry collision cylinder length=0.045 radius=0.008; visual mesh filename=package://ergoCub/meshes/simmechanics/sim_ecub_1-1_l_hand_i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 scale=0.001 0.001 0.001
- link l_hand_index_3: geometry collision cylinder length=0.055 radius=0.008; visual mesh filename=package://ergoCub/meshes/simmechanics/sim_ecub_1-1_l_hand_i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 scale=0.001 0.001 0.001
- link l_hand_middle_1: geometry collision cylinder length=0.045 radius=0.008; visual mesh filename=package://ergoCub/meshes/simmechanics/sim_ecub_1-1_l_hand_m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 scale=0.001 0.001 0.001
- link l_hand_middle_2: geometry collision cylinder length=0.055 radius=0.008; visual mesh filename=package://ergoCub/meshes/simmechanics/sim_ecub_1-1_l_hand_m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 scale=0.001 0.001 0.001
- link l_hand_pinkie_1: geometry collision cylinder length=0.04 radius=0.008; visual mesh filename=package://ergoCub/meshes/simmechanics/sim_ecub_1-1_l_hand_p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 scale=0.001 0.001 0.001
- link l_hand_pinkie_2: geometry collision cylinder length=0.05 radius=0.008; visual mesh filename=package://ergoCub/meshes/simmechanics/sim_ecub_1-1_l_hand_p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 scale=0.001 0.001 0.001
- link l_hand_ring_1: geometry collision cylinder length=0.045 radius=0.008; visual mesh filename=package://ergoCub/meshes/simmechanics/sim_ecub_1-1_l_hand_r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 scale=0.001 0.001 0.001
- link l_hand_ring_2: geometry collision cylinder length=0.05 radius=0.008; visual mesh filename=package://ergoCub/meshes/simmechanics/sim_ecub_1-1_l_hand_r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 scale=0.001 0.001 0.001
- link l_hand_thumb_2: geometry collision cylinder length=0.04 radius=0.008; visual mesh filename=package://ergoCub/meshes/simmechanics/sim_ecub_1-1_l_hand_t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 scale=0.001 0.001 0.001
- link l_hand_thumb_3: geometry collision cylinder length=0.05 radius=0.008; visual mesh filename=package://ergoCub/meshes/simmechanics/sim_ecub_1-1_l_hand_t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 scale=0.001 0.001 0.001
- link r_hand_index_2: geometry collision cylinder length=0.045 radius=0.008; visual mesh filename=package://ergoCub/meshes/simmechanics/sim_ecub_1-1_r_hand_i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 scale=0.001 0.001 0.001
- link r_hand_index_3: geometry collision cylinder length=0.055 radius=0.008; visual mesh filename=package://ergoCub/meshes/simmechanics/sim_ecub_1-1_r_hand_i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 scale=0.001 0.001 0.001
- link r_hand_middle_1: geometry collision cylinder length=0.045 radius=0.008; visual mesh filename=package://ergoCub/meshes/simmechanics/sim_ecub_1-1_r_hand_m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 scale=0.001 0.001 0.001
- link r_hand_middle_2: geometry collision cylinder length=0.055 radius=0.008; visual mesh filename=package://ergoCub/meshes/simmechanics/sim_ecub_1-1_r_hand_m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 scale=0.001 0.001 0.001
- link r_hand_pinkie_1: geometry collision cylinder length=0.04 radius=0.008; visual mesh filename=package://ergoCub/meshes/simmechanics/sim_ecub_1-1_r_hand_p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 scale=0.001 0.001 0.001
- link r_hand_pinkie_2: geometry collision cylinder length=0.05 radius=0.008; visual mesh filename=package://ergoCub/meshes/simmechanics/sim_ecub_1-1_r_hand_p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 scale=0.001 0.001 0.001
- link r_hand_ring_1: geometry collision cylinder length=0.045 radius=0.008; visual mesh filename=package://ergoCub/meshes/simmechanics/sim_ecub_1-1_r_hand_r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 scale=0.001 0.001 0.001
- link r_hand_ring_2: geometry collision cylinder length=0.05 radius=0.008; visual mesh filename=package://ergoCub/meshes/simmechanics/sim_ecub_1-1_r_hand_r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 scale=0.001 0.001 0.001
- link r_hand_thumb_2: geometry collision cylinder length=0.04 radius=0.008; visual mesh filename=package://ergoCub/meshes/simmechanics/sim_ecub_1-1_r_hand_t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 scale=0.001 0.001 0.001
- link r_hand_thumb_3: geometry collision cylinder length=0.05 radius=0.008; visual mesh filename=package://ergoCub/meshes/simmechanics/sim_ecub_1-1_r_hand_t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 scale=0.001 0.001 0.001

Commit message: ergoCubV1_1: remove ft sensors of the arms
It fixes #200

File: urdf/ergoCub/robots/ergoCubGazeboV1_1/model.urdf (robot description, URDF)
Before this commit: robot ergoCub, 204 links, 203 joints
Links:
- removed link l_arm_ft
- removed link r_arm_ft
Joints:
- removed joint l_arm_ft_fixed_joint
- removed joint r_arm_ft_fixed_joint

File: urdf/ergoCub/robots/ergoCubGazeboV1_1_minContacts/model.urdf (robot description, URDF)
Before this commit: robot ergoCub, 204 links, 203 joints
Links:
- removed link l_arm_ft
- removed link r_arm_ft
Joints:
- removed joint l_arm_ft_fixed_joint
- removed joint r_arm_ft_fixed_joint

File: urdf/ergoCub/robots/ergoCubSN001/model.urdf (robot description, URDF)
Before this commit: robot ergoCub, 204 links, 203 joints
Links:
- removed link l_arm_ft
- removed link r_arm_ft
Joints:
- removed joint l_arm_ft_fixed_joint
- removed joint r_arm_ft_fixed_joint
