Commit message: ergoCubGazeboV1_1: simplify collision for the palms

File: urdf/ergoCub/robots/ergoCubGazeboV1_1/model.urdf (robot description, URDF)
Before this commit: robot ergoCub, 204 links, 203 joints
Links:
- link l_hand_palm: geometry collision box size=0.1 0.025 0.09; visual mesh filename=package://ergoCub/meshes/simmechanics/sim_ecub_1-1_l_hand_p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 scale=0.001 0.001 0.001
- link r_hand_palm: geometry collision box size=0.1 0.025 0.09; visual mesh filename=package://ergoCub/meshes/simmechanics/sim_ecub_1-1_r_hand_p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 scale=0.001 0.001 0.001

Commit message: ergoCubV1_1: remove collisions  for thumb_1/index_1 links

File: urdf/ergoCub/robots/ergoCubGazeboV1_1/model.urdf (robot description, URDF)
Before this commit: robot ergoCub, 204 links, 203 joints
Links:
- link l_hand_index_1: geometry collision box size=0 0 0; visual mesh filename=package://ergoCub/meshes/simmechanics/sim_ecub_1-1_l_hand_i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 scale=0.001 0.001 0.001
- link l_hand_thumb_1: geometry collision box size=0 0 0; visual mesh filename=package://ergoCub/meshes/simmechanics/sim_ecub_1-1_l_hand_t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 scale=0.001 0.001 0.001
- link r_hand_index_1: geometry collision box size=0 0 0; visual mesh filename=package://ergoCub/meshes/simmechanics/sim_ecub_1-1_r_hand_i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 scale=0.001 0.001 0.001
- link r_hand_thumb_1: geometry collision box size=0 0 0; visual mesh filename=package://ergoCub/meshes/simmechanics/sim_ecub_1-1_r_hand_t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 scale=0.001 0.001 0.001

Commit message: Revert "ergoCubV1_1: remove ft sensors of the arms"
This reverts commit 6be5893296bdf465323ab3ca698745d7b74dc3a3.

File: urdf/ergoCub/robots/ergoCubGazeboV1_1/model.urdf (robot description, URDF)
Before this commit: robot ergoCub, 202 links, 201 joints
Links:
- added link l_arm_ft
- added link r_arm_ft
Joints:
- added joint l_arm_ft_fixed_joint: type fixed, parent l_shoulder_2, child l_arm_ft, origin xyz=-0.004349999999999996 -2.7755575615628914e-17 -0.054300000000000015 rpy=3.141592653589793 2.498001805406602e-16 -1.5707963267948952
- added joint r_arm_ft_fixed_joint: type fixed, parent r_shoulder_2, child r_arm_ft, origin xyz=-0.006849999999999986 -2.7755575615628914e-17 -0.05429999999999999 rpy=3.141592653589793 1.6653345369377348e-16 1.5707963267948981

File: urdf/ergoCub/robots/ergoCubGazeboV1_1_minContacts/model.urdf (robot description, URDF)
Before this commit: robot ergoCub, 202 links, 201 joints
Links:
- added link l_arm_ft
- added link r_arm_ft
Joints:
- added joint l_arm_ft_fixed_joint: type fixed, parent l_shoulder_2, child l_arm_ft, origin xyz=-0.004349999999999996 -2.7755575615628914e-17 -0.054300000000000015 rpy=3.141592653589793 2.498001805406602e-16 -1.5707963267948952
- added joint r_arm_ft_fixed_joint: type fixed, parent r_shoulder_2, child r_arm_ft, origin xyz=-0.006849999999999986 -2.7755575615628914e-17 -0.05429999999999999 rpy=3.141592653589793 1.6653345369377348e-16 1.5707963267948981

File: urdf/ergoCub/robots/ergoCubSN001/model.urdf (robot description, URDF)
Before this commit: robot ergoCub, 202 links, 201 joints
Links:
- added link l_arm_ft
- added link r_arm_ft
Joints:
- added joint l_arm_ft_fixed_joint: type fixed, parent l_shoulder_2, child l_arm_ft, origin xyz=-0.004349999999999996 -2.7755575615628914e-17 -0.054300000000000015 rpy=3.141592653589793 2.498001805406602e-16 -1.5707963267948952
- added joint r_arm_ft_fixed_joint: type fixed, parent r_shoulder_2, child r_arm_ft, origin xyz=-0.006849999999999986 -2.7755575615628914e-17 -0.05429999999999999 rpy=3.141592653589793 1.6653345369377348e-16 1.5707963267948981

Commit message: Add Gazebo Sim support (#230)

File: urdf/ergoCub/robots/ergoCubGazeboV1_1/model.urdf (robot description, URDF)
Before this commit: robot ergoCub, 204 links, 203 joints
Joints:
- joint l_index_add: axis 1.3005559878087045e-15 1.0000000000000002 -1.953448495705706e-15 -> 1.1895336853461886e-15 0.9999999999999999 -1.9812040713213337e-15; origin xyz=0.022500000000000034 -0.0015000000000006397 -0.06859999999999966 rpy=-8.126657451512497e-16 -0.2967059722446555 1.7414265967526777e-16 -> xyz=0.022500000000000023 -0.0015000000000006952 -0.0685999999999996 rpy=-8.416895217637947e-16 -0.29670597224465534 5.804755322508926e-17
- joint l_index_dist: axis -1 -1.804112664227406e-16 9.020562801946248e-17 -> -1 -2.359224176539984e-16 4.163337069211178e-17; origin xyz=-2.7755575615628914e-17 -0.0014999999999999736 -0.039999999999999925 rpy=-7.482326169760975e-8 1.734723475976807e-16 -6.106226635438361e-16 -> xyz=-1.3877787807814457e-17 -0.001500000000000029 -0.03999999999999987 rpy=-7.482326172536535e-8 1.8041124150158794e-16 -6.106226635438361e-16
- joint l_index_prox: axis -1.0000000000000002 2.7755575615627613e-17 7.023654366444809e-10 -> -1 8.326672684688522e-17 7.023654435833748e-10; origin xyz=0.009192533346793416 -2.7755575615628914e-17 -0.030713451309624162 rpy=-2.7755575615628914e-16 -7.023611553469422e-10 -7.771561172376094e-16 -> xyz=0.00919253334679343 0 -0.030713451309624218 rpy=-3.0531133177191815e-16 -7.023611484080483e-10 -7.771561172376096e-16

File: urdf/ergoCub/robots/ergoCubGazeboV1_1_minContacts/model.urdf (robot description, URDF)
Before this commit: robot ergoCub, 204 links, 203 joints
Joints:
- joint l_index_add: axis 1.3005559878087045e-15 1.0000000000000002 -1.953448495705706e-15 -> 1.1895336853461886e-15 0.9999999999999999 -1.9812040713213337e-15; origin xyz=0.022500000000000034 -0.0015000000000006397 -0.06859999999999966 rpy=-8.126657451512497e-16 -0.2967059722446555 1.7414265967526777e-16 -> xyz=0.022500000000000023 -0.0015000000000006952 -0.0685999999999996 rpy=-8.416895217637947e-16 -0.29670597224465534 5.804755322508926e-17
- joint l_index_dist: axis -1 -1.804112664227406e-16 9.020562801946248e-17 -> -1 -2.359224176539984e-16 4.163337069211178e-17; origin xyz=-2.7755575615628914e-17 -0.0014999999999999736 -0.039999999999999925 rpy=-7.482326169760975e-8 1.734723475976807e-16 -6.106226635438361e-16 -> xyz=-1.3877787807814457e-17 -0.001500000000000029 -0.03999999999999987 rpy=-7.482326172536535e-8 1.8041124150158794e-16 -6.106226635438361e-16
- joint l_index_prox: axis -1.0000000000000002 2.7755575615627613e-17 7.023654366444809e-10 -> -1 8.326672684688522e-17 7.023654435833748e-10; origin xyz=0.009192533346793416 -2.7755575615628914e-17 -0.030713451309624162 rpy=-2.7755575615628914e-16 -7.023611553469422e-10 -7.771561172376094e-16 -> xyz=0.00919253334679343 0 -0.030713451309624218 rpy=-3.0531133177191815e-16 -7.023611484080483e-10 -7.771561172376096e-16

File: urdf/ergoCub/robots/ergoCubSN001/model.urdf (robot description, URDF)
Before this commit: robot ergoCub, 204 links, 203 joints
Joints:
- joint l_index_add: axis 1.3005559878087045e-15 1.0000000000000002 -1.953448495705706e-15 -> 1.1895336853461886e-15 0.9999999999999999 -1.9812040713213337e-15; origin xyz=0.022500000000000034 -0.0015000000000006397 -0.06859999999999966 rpy=-8.126657451512497e-16 -0.2967059722446555 1.7414265967526777e-16 -> xyz=0.022500000000000023 -0.0015000000000006952 -0.0685999999999996 rpy=-8.416895217637947e-16 -0.29670597224465534 5.804755322508926e-17
- joint l_index_dist: axis -1 -1.804112664227406e-16 9.020562801946248e-17 -> -1 -2.359224176539984e-16 4.163337069211178e-17; origin xyz=-2.7755575615628914e-17 -0.0014999999999999736 -0.039999999999999925 rpy=-7.482326169760975e-8 1.734723475976807e-16 -6.106226635438361e-16 -> xyz=-1.3877787807814457e-17 -0.001500000000000029 -0.03999999999999987 rpy=-7.482326172536535e-8 1.8041124150158794e-16 -6.106226635438361e-16
- joint l_index_prox: axis -1.0000000000000002 2.7755575615627613e-17 7.023654366444809e-10 -> -1 8.326672684688522e-17 7.023654435833748e-10; origin xyz=0.009192533346793416 -2.7755575615628914e-17 -0.030713451309624162 rpy=-2.7755575615628914e-16 -7.023611553469422e-10 -7.771561172376094e-16 -> xyz=0.00919253334679343 0 -0.030713451309624218 rpy=-3.0531133177191815e-16 -7.023611484080483e-10 -7.771561172376096e-16

Commit message: Regenerate V1_1 models

File: urdf/ergoCub/robots/ergoCubGazeboV1_1/model.urdf (robot description, URDF)
Before this commit: robot ergoCub, 204 links, 203 joints
Joints:
- joint l_index_add: axis 1.1895336853461886e-15 0.9999999999999999 -1.9812040713213337e-15 -> 1.3005559878087045e-15 1.0000000000000002 -1.953448495705706e-15; origin xyz=0.022500000000000023 -0.0015000000000006952 -0.0685999999999996 rpy=-8.416895217637947e-16 -0.29670597224465534 5.804755322508926e-17 -> xyz=0.022500000000000034 -0.0015000000000006397 -0.06859999999999966 rpy=-8.126657451512497e-16 -0.2967059722446555 1.7414265967526777e-16
- joint l_index_dist: axis -1 -2.359224176539984e-16 4.163337069211178e-17 -> -1 -1.804112664227406e-16 9.020562801946248e-17; origin xyz=-1.3877787807814457e-17 -0.001500000000000029 -0.03999999999999987 rpy=-7.482326172536535e-8 1.8041124150158794e-16 -6.106226635438361e-16 -> xyz=-2.7755575615628914e-17 -0.0014999999999999736 -0.039999999999999925 rpy=-7.482326169760975e-8 1.734723475976807e-16 -6.106226635438361e-16
- joint l_index_prox: axis -1 8.326672684688522e-17 7.023654435833748e-10 -> -1.0000000000000002 2.7755575615627613e-17 7.023654366444809e-10; origin xyz=0.00919253334679343 0 -0.030713451309624218 rpy=-3.0531133177191815e-16 -7.023611484080483e-10 -7.771561172376096e-16 -> xyz=0.009192533346793416 -2.7755575615628914e-17 -0.030713451309624162 rpy=-2.7755575615628914e-16 -7.023611553469422e-10 -7.771561172376094e-16

File: urdf/ergoCub/robots/ergoCubGazeboV1_1_minContacts/model.urdf (robot description, URDF)
Before this commit: robot ergoCub, 204 links, 203 joints
Joints:
- joint l_index_add: axis 1.1895336853461886e-15 0.9999999999999999 -1.9812040713213337e-15 -> 1.3005559878087045e-15 1.0000000000000002 -1.953448495705706e-15; origin xyz=0.022500000000000023 -0.0015000000000006952 -0.0685999999999996 rpy=-8.416895217637947e-16 -0.29670597224465534 5.804755322508926e-17 -> xyz=0.022500000000000034 -0.0015000000000006397 -0.06859999999999966 rpy=-8.126657451512497e-16 -0.2967059722446555 1.7414265967526777e-16
- joint l_index_dist: axis -1 -2.359224176539984e-16 4.163337069211178e-17 -> -1 -1.804112664227406e-16 9.020562801946248e-17; origin xyz=-1.3877787807814457e-17 -0.001500000000000029 -0.03999999999999987 rpy=-7.482326172536535e-8 1.8041124150158794e-16 -6.106226635438361e-16 -> xyz=-2.7755575615628914e-17 -0.0014999999999999736 -0.039999999999999925 rpy=-7.482326169760975e-8 1.734723475976807e-16 -6.106226635438361e-16
- joint l_index_prox: axis -1 8.326672684688522e-17 7.023654435833748e-10 -> -1.0000000000000002 2.7755575615627613e-17 7.023654366444809e-10; origin xyz=0.00919253334679343 0 -0.030713451309624218 rpy=-3.0531133177191815e-16 -7.023611484080483e-10 -7.771561172376096e-16 -> xyz=0.009192533346793416 -2.7755575615628914e-17 -0.030713451309624162 rpy=-2.7755575615628914e-16 -7.023611553469422e-10 -7.771561172376094e-16

Commit message: Automatic update of urdf triggered by GitHub Action
ergocub-software = 7309b0f18df089f727b8e9b9d91c5530c359fa8b
cad-libraries    = 5555adec3e34bf3d5cb28889c0f66b09d68f810a
cad-mechanics    = 20b289b76a1edebd7cea54f6a372a7baa033a8c1
creo2urdf        = v0.4.7

File: urdf/ergoCub/robots/ergoCubGazeboV1_1/model.urdf (robot description, URDF)
Before this commit: robot ergoCub, 204 links, 203 joints
Joints:
- joint l_index_add: axis 1.3005559878087045e-15 1.0000000000000002 -1.953448495705706e-15 -> 1.1895336853461886e-15 0.9999999999999999 -1.9812040713213337e-15; origin xyz=0.022500000000000034 -0.0015000000000006397 -0.06859999999999966 rpy=-8.126657451512497e-16 -0.2967059722446555 1.7414265967526777e-16 -> xyz=0.022500000000000023 -0.0015000000000006952 -0.0685999999999996 rpy=-8.416895217637947e-16 -0.29670597224465534 5.804755322508926e-17
- joint l_index_dist: axis -1 -1.804112664227406e-16 9.020562801946248e-17 -> -1 -2.359224176539984e-16 4.163337069211178e-17; origin xyz=-2.7755575615628914e-17 -0.0014999999999999736 -0.039999999999999925 rpy=-7.482326169760975e-8 1.734723475976807e-16 -6.106226635438361e-16 -> xyz=-1.3877787807814457e-17 -0.001500000000000029 -0.03999999999999987 rpy=-7.482326172536535e-8 1.8041124150158794e-16 -6.106226635438361e-16
- joint l_index_prox: axis -1.0000000000000002 2.7755575615627613e-17 7.023654366444809e-10 -> -1 8.326672684688522e-17 7.023654435833748e-10; origin xyz=0.009192533346793416 -2.7755575615628914e-17 -0.030713451309624162 rpy=-2.7755575615628914e-16 -7.023611553469422e-10 -7.771561172376094e-16 -> xyz=0.00919253334679343 0 -0.030713451309624218 rpy=-3.0531133177191815e-16 -7.023611484080483e-10 -7.771561172376096e-16

File: urdf/ergoCub/robots/ergoCubGazeboV1_1_minContacts/model.urdf (robot description, URDF)
Before this commit: robot ergoCub, 204 links, 203 joints
Joints:
- joint l_index_add: axis 1.3005559878087045e-15 1.0000000000000002 -1.953448495705706e-15 -> 1.1895336853461886e-15 0.9999999999999999 -1.9812040713213337e-15; origin xyz=0.022500000000000034 -0.0015000000000006397 -0.06859999999999966 rpy=-8.126657451512497e-16 -0.2967059722446555 1.7414265967526777e-16 -> xyz=0.022500000000000023 -0.0015000000000006952 -0.0685999999999996 rpy=-8.416895217637947e-16 -0.29670597224465534 5.804755322508926e-17
- joint l_index_dist: axis -1 -1.804112664227406e-16 9.020562801946248e-17 -> -1 -2.359224176539984e-16 4.163337069211178e-17; origin xyz=-2.7755575615628914e-17 -0.0014999999999999736 -0.039999999999999925 rpy=-7.482326169760975e-8 1.734723475976807e-16 -6.106226635438361e-16 -> xyz=-1.3877787807814457e-17 -0.001500000000000029 -0.03999999999999987 rpy=-7.482326172536535e-8 1.8041124150158794e-16 -6.106226635438361e-16
- joint l_index_prox: axis -1.0000000000000002 2.7755575615627613e-17 7.023654366444809e-10 -> -1 8.326672684688522e-17 7.023654435833748e-10; origin xyz=0.009192533346793416 -2.7755575615628914e-17 -0.030713451309624162 rpy=-2.7755575615628914e-16 -7.023611553469422e-10 -7.771561172376094e-16 -> xyz=0.00919253334679343 0 -0.030713451309624218 rpy=-3.0531133177191815e-16 -7.023611484080483e-10 -7.771561172376096e-16

Commit message: Automatic update of urdf triggered by GitHub Action
ergocub-software = c4a1fb16044530b32d8cb75ad1fc99b883ef8ebe
cad-libraries    = https://github.com/icub-tech-iit/cad-libraries/commit/e23fdf897b1378fb650f88ffe8d938596559d93e
cad-mechanics    = https://github.com/icub-tech-iit/cad-mechanics/commit/d80569866d28b344b8ba6ffa94d468891d95ea18
creo2urdf        = https://github.com/icub-tech-iit/creo2urdf/releases/tag/v0.5.3

File: urdf/ergoCub/robots/ergoCubGazeboV1_1/model.urdf (robot description, URDF)
Before this commit: robot ergoCub, 204 links, 203 joints
Links:
- link chest: geometry collision mesh filename=package://ergoCub/meshes/simmechanics/sim_ecub_1-1_chest.stl scale=0.001 0.001 0.001; visual mesh filename=package://ergoCub/meshes/simmechanics/sim_ecub_1-1_chest.stl scale=0.001 0.001 0.001
- link head: geometry collision mesh filename=package://ergoCub/meshes/simmechanics/sim_ecub_1-1_head.stl scale=0.001 0.001 0.001; visual mesh filename=package://ergoCub/meshes/simmechanics/sim_ecub_1-1_head.stl scale=0.001 0.001 0.001
Joints:
- joint waist_imu_0_fixed_joint: origin xyz=0.0354497 0.00639688 0.060600 rpy=1.5708 0 -1.5708 -> xyz=0.0606 -0.00639428 0.01745 rpy=1.5708 -0.000105208 -1.5708

File: urdf/ergoCub/robots/ergoCubGazeboV1_1_minContacts/model.urdf (robot description, URDF)
Before this commit: robot ergoCub, 204 links, 203 joints
Links:
- link chest: geometry collision box size=0 0 0; visual mesh filename=package://ergoCub/meshes/simmechanics/sim_ecub_1-1_chest.stl scale=0.001 0.001 0.001
- link head: geometry collision box size=0 0 0; visual mesh filename=package://ergoCub/meshes/simmechanics/sim_ecub_1-1_head.stl scale=0.001 0.001 0.001
Joints:
- joint waist_imu_0_fixed_joint: origin xyz=0.0354497 0.00639688 0.060600 rpy=1.5708 0 -1.5708 -> xyz=0.0606 -0.00639428 0.01745 rpy=1.5708 -0.000105208 -1.5708

File: urdf/ergoCub/robots/ergoCubGazeboV1_2/model.urdf (robot description, URDF)
Before this commit: robot ergoCub, 204 links, 203 joints
Links:
- link chest: geometry collision mesh filename=package://ergoCub/meshes/simmechanics/sim_ecub_1-1_chest.stl scale=0.001 0.001 0.001; visual mesh filename=package://ergoCub/meshes/simmechanics/sim_ecub_1-1_chest.stl scale=0.001 0.001 0.001
- link head: geometry collision mesh filename=package://ergoCub/meshes/simmechanics/sim_ecub_1-1_head.stl scale=0.001 0.001 0.001; visual mesh filename=package://ergoCub/meshes/simmechanics/sim_ecub_1-1_head.stl scale=0.001 0.001 0.001
Joints:
- joint waist_imu_0_fixed_joint: origin xyz=0.0354497 0.00639688 0.060600 rpy=1.5708 0 -1.5708 -> xyz=0.0606 -0.00639428 0.01745 rpy=1.5708 -0.000105208 -1.5708

File: urdf/ergoCub/robots/ergoCubGazeboV1_2_minContacts/model.urdf (robot description, URDF)
Before this commit: robot ergoCub, 204 links, 203 joints
Links:
- link chest: geometry collision box size=0 0 0; visual mesh filename=package://ergoCub/meshes/simmechanics/sim_ecub_1-1_chest.stl scale=0.001 0.001 0.001
- link head: geometry collision box size=0 0 0; visual mesh filename=package://ergoCub/meshes/simmechanics/sim_ecub_1-1_head.stl scale=0.001 0.001 0.001
Joints:
- joint waist_imu_0_fixed_joint: origin xyz=0.0354497 0.00639688 0.060600 rpy=1.5708 0 -1.5708 -> xyz=0.0606 -0.00639428 0.01745 rpy=1.5708 -0.000105208 -1.5708

File: urdf/ergoCub/robots/ergoCubSN001/model.urdf (robot description, URDF)
Before this commit: robot ergoCub, 204 links, 203 joints
Links:
- link chest: geometry collision mesh filename=package://ergoCub/meshes/simmechanics/sim_ecub_1-1_chest.stl scale=0.001 0.001 0.001; visual mesh filename=package://ergoCub/meshes/simmechanics/sim_ecub_1-1_chest.stl scale=0.001 0.001 0.001
- link head: geometry collision mesh filename=package://ergoCub/meshes/simmechanics/sim_ecub_1-1_head.stl scale=0.001 0.001 0.001; visual mesh filename=package://ergoCub/meshes/simmechanics/sim_ecub_1-1_head.stl scale=0.001 0.001 0.001
Joints:
- joint waist_imu_0_fixed_joint: origin xyz=0.0354497 0.00639688 0.060600 rpy=1.5708 0 -1.5708 -> xyz=0.0606 -0.00639428 0.01745 rpy=1.5708 -0.000105208 -1.5708

File: urdf/ergoCub/robots/ergoCubSN002/model.urdf (robot description, URDF)
Before this commit: robot ergoCub, 204 links, 203 joints
Links:
- link chest: geometry collision mesh filename=package://ergoCub/meshes/simmechanics/sim_ecub_1-1_chest.stl scale=0.001 0.001 0.001; visual mesh filename=package://ergoCub/meshes/simmechanics/sim_ecub_1-1_chest.stl scale=0.001 0.001 0.001
- link head: geometry collision mesh filename=package://ergoCub/meshes/simmechanics/sim_ecub_1-1_head.stl scale=0.001 0.001 0.001; visual mesh filename=package://ergoCub/meshes/simmechanics/sim_ecub_1-1_head.stl scale=0.001 0.001 0.001
Joints:
- joint waist_imu_0_fixed_joint: origin xyz=0.0354497 0.00639688 0.060600 rpy=1.5708 0 -1.5708 -> xyz=0.0606 -0.00639428 0.01745 rpy=1.5708 -0.000105208 -1.5708

Commit message: Automatic update of urdf triggered by GitHub Action
ergocub-software = c4a1fb16044530b32d8cb75ad1fc99b883ef8ebe
cad-libraries    = https://github.com/icub-tech-iit/cad-libraries/commit/e23fdf897b1378fb650f88ffe8d938596559d93e
cad-mechanics    = https://github.com/icub-tech-iit/cad-mechanics/commit/c759298794116b0470f58898e3819b6db8be9505
creo2urdf        = https://github.com/icub-tech-iit/creo2urdf/releases/tag/v0.5.4

File: urdf/ergoCub/robots/ergoCubGazeboV1_1/model.urdf (robot description, URDF)
Before this commit: robot ergoCub, 204 links, 203 joints
Joints:
- joint waist_imu_0_fixed_joint: origin xyz=0.0354497 0.00639688 0.060600 rpy=1.5708 0 -1.5708 -> xyz=0.0606 -0.00639428 0.01745 rpy=1.5708 -0.000105208 -1.5708

File: urdf/ergoCub/robots/ergoCubGazeboV1_1_minContacts/model.urdf (robot description, URDF)
Before this commit: robot ergoCub, 204 links, 203 joints
Joints:
- joint waist_imu_0_fixed_joint: origin xyz=0.0354497 0.00639688 0.060600 rpy=1.5708 0 -1.5708 -> xyz=0.0606 -0.00639428 0.01745 rpy=1.5708 -0.000105208 -1.5708

File: urdf/ergoCub/robots/ergoCubGazeboV1_2/model.urdf (robot description, URDF)
Before this commit: robot ergoCub, 204 links, 203 joints
Joints:
- joint waist_imu_0_fixed_joint: origin xyz=0.0354497 0.00639688 0.060600 rpy=1.5708 0 -1.5708 -> xyz=0.0606 -0.00639428 0.01745 rpy=1.5708 -0.000105208 -1.5708

File: urdf/ergoCub/robots/ergoCubGazeboV1_2_minContacts/model.urdf (robot description, URDF)
Before this commit: robot ergoCub, 204 links, 203 joints
Joints:
- joint waist_imu_0_fixed_joint: origin xyz=0.0354497 0.00639688 0.060600 rpy=1.5708 0 -1.5708 -> xyz=0.0606 -0.00639428 0.01745 rpy=1.5708 -0.000105208 -1.5708

File: urdf/ergoCub/robots/ergoCubSN001/model.urdf (robot description, URDF)
Before this commit: robot ergoCub, 204 links, 203 joints
Joints:
- joint waist_imu_0_fixed_joint: origin xyz=0.0354497 0.00639688 0.060600 rpy=1.5708 0 -1.5708 -> xyz=0.0606 -0.00639428 0.01745 rpy=1.5708 -0.000105208 -1.5708

File: urdf/ergoCub/robots/ergoCubSN002/model.urdf (robot description, URDF)
Before this commit: robot ergoCub, 204 links, 203 joints
Joints:
- joint waist_imu_0_fixed_joint: origin xyz=0.0354497 0.00639688 0.060600 rpy=1.5708 0 -1.5708 -> xyz=0.0606 -0.00639428 0.01745 rpy=1.5708 -0.000105208 -1.5708
