Commit message: Automatic update of urdf triggered by GitHub Action
ergocub-software = 40466d4f98f588ff5616d18ad1af58793332cd44
cad-libraries    = https://github.com/icub-tech-iit/cad-libraries/commit/9bf0c88d492dac0d6a3eefaa949221d6f6e85a6c
cad-mechanics    = https://github.com/icub-tech-iit/cad-mechanics/commit/02a8f13785a3ef1320a4d4f97012ae967b847b9b
creo2urdf        = https://github.com/icub-tech-iit/creo2urdf/releases/tag/v0.5.6

File: urdf/ergoCub/robots/ergoCubGazeboV1_1/model.urdf (robot description, URDF)
Before this commit: robot ergoCub, 204 links, 203 joints
Joints:
- joint l_elbow: limit lower=-0.05235987755982989 upper=1.3089969389957472 effort=1e+9 velocity=1e+9 -> lower=-0.08726646259971647 upper=2.0943951023931953 effort=1e+9 velocity=1e+9
- joint l_hip_pitch: limit lower=-0.7504915783575618 upper=1.7976891295541595 effort=1e+9 velocity=1e+9 -> lower=-0.767944870877505 upper=1.9198621771937625 effort=1e+9 velocity=1e+9
- joint l_hip_roll: limit lower=-0.2792526803190927 upper=1.9024088846738192 effort=1e+9 velocity=1e+9 -> lower=-0.3490658503988659 upper=1.9373154697137058 effort=1e+9 velocity=1e+9
- joint l_hip_yaw: limit lower=-1.3788101090755203 upper=1.3788101090755203 effort=1e+9 velocity=1e+9 -> lower=-1.413716694115407 upper=1.413716694115407 effort=1e+9 velocity=1e+9
- joint l_knee: limit lower=-1.8151424220741028 upper=0.10471975511965978 effort=1e+9 velocity=1e+9 -> lower=-1.8325957145940461 upper=0.12217304763960307 effort=1e+9 velocity=1e+9
- joint l_shoulder_yaw: limit lower=-0.8726646259971648 upper=1.3962634015954636 effort=1e+9 velocity=1e+9 -> lower=-0.9075712110370514 upper=1.4311699866353502 effort=1e+9 velocity=1e+9
- joint l_wrist_pitch: limit lower=-0.5585053606381855 upper=0.5585053606381855 effort=1e+9 velocity=1e+9 -> lower=-0.3490658503988659 upper=0.3490658503988659 effort=1e+9 velocity=1e+9
- joint l_wrist_roll: limit lower=-1.0821041362364843 upper=0.9075712110370514 effort=1e+9 velocity=1e+9 -> lower=-0.3490658503988659 upper=0.5235987755982988 effort=1e+9 velocity=1e+9
- joint neck_pitch: limit lower=-0.5235987755982988 upper=0.3839724354387525 effort=1e+9 velocity=1e+9 -> lower=-0.7853981633974483 upper=0.3839724354387525 effort=1e+9 velocity=1e+9
- joint r_elbow: limit lower=-0.05235987755982989 upper=1.3089969389957472 effort=1e+9 velocity=1e+9 -> lower=-0.08726646259971647 upper=2.0943951023931953 effort=1e+9 velocity=1e+9
- joint r_hip_pitch: limit lower=-0.7504915783575618 upper=1.7976891295541595 effort=1e+9 velocity=1e+9 -> lower=-0.767944870877505 upper=1.9198621771937625 effort=1e+9 velocity=1e+9
- joint r_hip_roll: limit lower=-0.2792526803190927 upper=1.9024088846738192 effort=1e+9 velocity=1e+9 -> lower=-0.3490658503988659 upper=1.9373154697137058 effort=1e+9 velocity=1e+9
- joint r_hip_yaw: limit lower=-1.3788101090755203 upper=1.3788101090755203 effort=1e+9 velocity=1e+9 -> lower=-1.413716694115407 upper=1.413716694115407 effort=1e+9 velocity=1e+9
- joint r_knee: limit lower=-1.8151424220741028 upper=0.10471975511965978 effort=1e+9 velocity=1e+9 -> lower=-1.8325957145940461 upper=0.12217304763960307 effort=1e+9 velocity=1e+9
- joint r_shoulder_yaw: limit lower=-0.8726646259971648 upper=1.3962634015954636 effort=1e+9 velocity=1e+9 -> lower=-0.9075712110370514 upper=1.4311699866353502 effort=1e+9 velocity=1e+9
- joint r_wrist_pitch: limit lower=-0.5585053606381855 upper=0.5585053606381855 effort=1e+9 velocity=1e+9 -> lower=-0.3490658503988659 upper=0.3490658503988659 effort=1e+9 velocity=1e+9
- joint r_wrist_roll: limit lower=-1.0821041362364843 upper=0.9075712110370514 effort=1e+9 velocity=1e+9 -> lower=-0.3490658503988659 upper=0.5235987755982988 effort=1e+9 velocity=1e+9
- joint torso_pitch: limit lower=-0.3141592653589793 upper=0.7853981633974483 effort=1e+9 velocity=1e+9 -> lower=-0.3490658503988659 upper=1.1344640137963142 effort=1e+9 velocity=1e+9
- joint torso_roll: limit lower=-0.4014257279586958 upper=0.4014257279586958 effort=1e+9 velocity=1e+9 -> lower=-0.4363323129985824 upper=0.4363323129985824 effort=1e+9 velocity=1e+9
- joint torso_yaw: limit lower=-0.7504915783575618 upper=0.7504915783575618 effort=1e+9 velocity=1e+9 -> lower=-0.7853981633974483 upper=0.7853981633974483 effort=1e+9 velocity=1e+9

File: urdf/ergoCub/robots/ergoCubGazeboV1_1_minContacts/model.urdf (robot description, URDF)
Before this commit: robot ergoCub, 204 links, 203 joints
Joints:
- joint l_elbow: limit lower=-0.05235987755982989 upper=1.3089969389957472 effort=1e+9 velocity=1e+9 -> lower=-0.08726646259971647 upper=2.0943951023931953 effort=1e+9 velocity=1e+9
- joint l_hip_pitch: limit lower=-0.7504915783575618 upper=1.7976891295541595 effort=1e+9 velocity=1e+9 -> lower=-0.767944870877505 upper=1.9198621771937625 effort=1e+9 velocity=1e+9
- joint l_hip_roll: limit lower=-0.2792526803190927 upper=1.9024088846738192 effort=1e+9 velocity=1e+9 -> lower=-0.3490658503988659 upper=1.9373154697137058 effort=1e+9 velocity=1e+9
- joint l_hip_yaw: limit lower=-1.3788101090755203 upper=1.3788101090755203 effort=1e+9 velocity=1e+9 -> lower=-1.413716694115407 upper=1.413716694115407 effort=1e+9 velocity=1e+9
- joint l_knee: limit lower=-1.8151424220741028 upper=0.10471975511965978 effort=1e+9 velocity=1e+9 -> lower=-1.8325957145940461 upper=0.12217304763960307 effort=1e+9 velocity=1e+9
- joint l_shoulder_yaw: limit lower=-0.8726646259971648 upper=1.3962634015954636 effort=1e+9 velocity=1e+9 -> lower=-0.9075712110370514 upper=1.4311699866353502 effort=1e+9 velocity=1e+9
- joint l_wrist_pitch: limit lower=-0.5585053606381855 upper=0.5585053606381855 effort=1e+9 velocity=1e+9 -> lower=-0.3490658503988659 upper=0.3490658503988659 effort=1e+9 velocity=1e+9
- joint l_wrist_roll: limit lower=-1.0821041362364843 upper=0.9075712110370514 effort=1e+9 velocity=1e+9 -> lower=-0.3490658503988659 upper=0.5235987755982988 effort=1e+9 velocity=1e+9
- joint neck_pitch: limit lower=-0.5235987755982988 upper=0.3839724354387525 effort=1e+9 velocity=1e+9 -> lower=-0.7853981633974483 upper=0.3839724354387525 effort=1e+9 velocity=1e+9
- joint r_elbow: limit lower=-0.05235987755982989 upper=1.3089969389957472 effort=1e+9 velocity=1e+9 -> lower=-0.08726646259971647 upper=2.0943951023931953 effort=1e+9 velocity=1e+9
- joint r_hip_pitch: limit lower=-0.7504915783575618 upper=1.7976891295541595 effort=1e+9 velocity=1e+9 -> lower=-0.767944870877505 upper=1.9198621771937625 effort=1e+9 velocity=1e+9
- joint r_hip_roll: limit lower=-0.2792526803190927 upper=1.9024088846738192 effort=1e+9 velocity=1e+9 -> lower=-0.3490658503988659 upper=1.9373154697137058 effort=1e+9 velocity=1e+9
- joint r_hip_yaw: limit lower=-1.3788101090755203 upper=1.3788101090755203 effort=1e+9 velocity=1e+9 -> lower=-1.413716694115407 upper=1.413716694115407 effort=1e+9 velocity=1e+9
- joint r_knee: limit lower=-1.8151424220741028 upper=0.10471975511965978 effort=1e+9 velocity=1e+9 -> lower=-1.8325957145940461 upper=0.12217304763960307 effort=1e+9 velocity=1e+9
- joint r_shoulder_yaw: limit lower=-0.8726646259971648 upper=1.3962634015954636 effort=1e+9 velocity=1e+9 -> lower=-0.9075712110370514 upper=1.4311699866353502 effort=1e+9 velocity=1e+9
- joint r_wrist_pitch: limit lower=-0.5585053606381855 upper=0.5585053606381855 effort=1e+9 velocity=1e+9 -> lower=-0.3490658503988659 upper=0.3490658503988659 effort=1e+9 velocity=1e+9
- joint r_wrist_roll: limit lower=-1.0821041362364843 upper=0.9075712110370514 effort=1e+9 velocity=1e+9 -> lower=-0.3490658503988659 upper=0.5235987755982988 effort=1e+9 velocity=1e+9
- joint torso_pitch: limit lower=-0.3141592653589793 upper=0.7853981633974483 effort=1e+9 velocity=1e+9 -> lower=-0.3490658503988659 upper=1.1344640137963142 effort=1e+9 velocity=1e+9
- joint torso_roll: limit lower=-0.4014257279586958 upper=0.4014257279586958 effort=1e+9 velocity=1e+9 -> lower=-0.4363323129985824 upper=0.4363323129985824 effort=1e+9 velocity=1e+9
- joint torso_yaw: limit lower=-0.7504915783575618 upper=0.7504915783575618 effort=1e+9 velocity=1e+9 -> lower=-0.7853981633974483 upper=0.7853981633974483 effort=1e+9 velocity=1e+9

File: urdf/ergoCub/robots/ergoCubGazeboV1_3/model.urdf (robot description, URDF)
Before this commit: robot ergoCub, 204 links, 203 joints
Joints:
- joint l_elbow: limit lower=-0.05235987755982989 upper=1.3089969389957472 effort=1e+9 velocity=1e+9 -> lower=-0.08726646259971647 upper=2.0943951023931953 effort=1e+9 velocity=1e+9
- joint l_hip_pitch: limit lower=-0.7504915783575618 upper=1.7976891295541595 effort=1e+9 velocity=1e+9 -> lower=-0.767944870877505 upper=1.9198621771937625 effort=1e+9 velocity=1e+9
- joint l_hip_roll: limit lower=-0.2792526803190927 upper=1.9024088846738192 effort=1e+9 velocity=1e+9 -> lower=-0.3490658503988659 upper=1.9373154697137058 effort=1e+9 velocity=1e+9
- joint l_hip_yaw: limit lower=-1.3788101090755203 upper=1.3788101090755203 effort=1e+9 velocity=1e+9 -> lower=-1.413716694115407 upper=1.413716694115407 effort=1e+9 velocity=1e+9
- joint l_knee: limit lower=-1.8151424220741028 upper=0.10471975511965978 effort=1e+9 velocity=1e+9 -> lower=-1.8325957145940461 upper=0.12217304763960307 effort=1e+9 velocity=1e+9
- joint l_shoulder_yaw: limit lower=-0.8726646259971648 upper=1.3962634015954636 effort=1e+9 velocity=1e+9 -> lower=-0.9075712110370514 upper=1.4311699866353502 effort=1e+9 velocity=1e+9
- joint l_wrist_pitch: limit lower=-0.5585053606381855 upper=0.5585053606381855 effort=1e+9 velocity=1e+9 -> lower=-0.3490658503988659 upper=0.3490658503988659 effort=1e+9 velocity=1e+9
- joint l_wrist_roll: limit lower=-1.0821041362364843 upper=0.9075712110370514 effort=1e+9 velocity=1e+9 -> lower=-0.3490658503988659 upper=0.5235987755982988 effort=1e+9 velocity=1e+9
- joint neck_pitch: limit lower=-0.5235987755982988 upper=0.3839724354387525 effort=1e+9 velocity=1e+9 -> lower=-0.7853981633974483 upper=0.3839724354387525 effort=1e+9 velocity=1e+9
- joint r_elbow: limit lower=-0.05235987755982989 upper=1.3089969389957472 effort=1e+9 velocity=1e+9 -> lower=-0.08726646259971647 upper=2.0943951023931953 effort=1e+9 velocity=1e+9
- joint r_hip_pitch: limit lower=-0.7504915783575618 upper=1.7976891295541595 effort=1e+9 velocity=1e+9 -> lower=-0.767944870877505 upper=1.9198621771937625 effort=1e+9 velocity=1e+9
- joint r_hip_roll: limit lower=-0.2792526803190927 upper=1.9024088846738192 effort=1e+9 velocity=1e+9 -> lower=-0.3490658503988659 upper=1.9373154697137058 effort=1e+9 velocity=1e+9
- joint r_hip_yaw: limit lower=-1.3788101090755203 upper=1.3788101090755203 effort=1e+9 velocity=1e+9 -> lower=-1.413716694115407 upper=1.413716694115407 effort=1e+9 velocity=1e+9
- joint r_knee: limit lower=-1.8151424220741028 upper=0.10471975511965978 effort=1e+9 velocity=1e+9 -> lower=-1.8325957145940461 upper=0.12217304763960307 effort=1e+9 velocity=1e+9
- joint r_shoulder_yaw: limit lower=-0.8726646259971648 upper=1.3962634015954636 effort=1e+9 velocity=1e+9 -> lower=-0.9075712110370514 upper=1.4311699866353502 effort=1e+9 velocity=1e+9
- joint r_wrist_pitch: limit lower=-0.5585053606381855 upper=0.5585053606381855 effort=1e+9 velocity=1e+9 -> lower=-0.3490658503988659 upper=0.3490658503988659 effort=1e+9 velocity=1e+9
- joint r_wrist_roll: limit lower=-1.0821041362364843 upper=0.9075712110370514 effort=1e+9 velocity=1e+9 -> lower=-0.3490658503988659 upper=0.5235987755982988 effort=1e+9 velocity=1e+9
- joint torso_pitch: limit lower=-0.3141592653589793 upper=0.7853981633974483 effort=1e+9 velocity=1e+9 -> lower=-0.3490658503988659 upper=1.1344640137963142 effort=1e+9 velocity=1e+9
- joint torso_roll: limit lower=-0.4014257279586958 upper=0.4014257279586958 effort=1e+9 velocity=1e+9 -> lower=-0.4363323129985824 upper=0.4363323129985824 effort=1e+9 velocity=1e+9
- joint torso_yaw: limit lower=-0.7504915783575618 upper=0.7504915783575618 effort=1e+9 velocity=1e+9 -> lower=-0.7853981633974483 upper=0.7853981633974483 effort=1e+9 velocity=1e+9

File: urdf/ergoCub/robots/ergoCubGazeboV1_3_minContacts/model.urdf (robot description, URDF)
Before this commit: robot ergoCub, 204 links, 203 joints
Joints:
- joint l_elbow: limit lower=-0.05235987755982989 upper=1.3089969389957472 effort=1e+9 velocity=1e+9 -> lower=-0.08726646259971647 upper=2.0943951023931953 effort=1e+9 velocity=1e+9
- joint l_hip_pitch: limit lower=-0.7504915783575618 upper=1.7976891295541595 effort=1e+9 velocity=1e+9 -> lower=-0.767944870877505 upper=1.9198621771937625 effort=1e+9 velocity=1e+9
- joint l_hip_roll: limit lower=-0.2792526803190927 upper=1.9024088846738192 effort=1e+9 velocity=1e+9 -> lower=-0.3490658503988659 upper=1.9373154697137058 effort=1e+9 velocity=1e+9
- joint l_hip_yaw: limit lower=-1.3788101090755203 upper=1.3788101090755203 effort=1e+9 velocity=1e+9 -> lower=-1.413716694115407 upper=1.413716694115407 effort=1e+9 velocity=1e+9
- joint l_knee: limit lower=-1.8151424220741028 upper=0.10471975511965978 effort=1e+9 velocity=1e+9 -> lower=-1.8325957145940461 upper=0.12217304763960307 effort=1e+9 velocity=1e+9
- joint l_shoulder_yaw: limit lower=-0.8726646259971648 upper=1.3962634015954636 effort=1e+9 velocity=1e+9 -> lower=-0.9075712110370514 upper=1.4311699866353502 effort=1e+9 velocity=1e+9
- joint l_wrist_pitch: limit lower=-0.5585053606381855 upper=0.5585053606381855 effort=1e+9 velocity=1e+9 -> lower=-0.3490658503988659 upper=0.3490658503988659 effort=1e+9 velocity=1e+9
- joint l_wrist_roll: limit lower=-1.0821041362364843 upper=0.9075712110370514 effort=1e+9 velocity=1e+9 -> lower=-0.3490658503988659 upper=0.5235987755982988 effort=1e+9 velocity=1e+9
- joint neck_pitch: limit lower=-0.5235987755982988 upper=0.3839724354387525 effort=1e+9 velocity=1e+9 -> lower=-0.7853981633974483 upper=0.3839724354387525 effort=1e+9 velocity=1e+9
- joint r_elbow: limit lower=-0.05235987755982989 upper=1.3089969389957472 effort=1e+9 velocity=1e+9 -> lower=-0.08726646259971647 upper=2.0943951023931953 effort=1e+9 velocity=1e+9
- joint r_hip_pitch: limit lower=-0.7504915783575618 upper=1.7976891295541595 effort=1e+9 velocity=1e+9 -> lower=-0.767944870877505 upper=1.9198621771937625 effort=1e+9 velocity=1e+9
- joint r_hip_roll: limit lower=-0.2792526803190927 upper=1.9024088846738192 effort=1e+9 velocity=1e+9 -> lower=-0.3490658503988659 upper=1.9373154697137058 effort=1e+9 velocity=1e+9
- joint r_hip_yaw: limit lower=-1.3788101090755203 upper=1.3788101090755203 effort=1e+9 velocity=1e+9 -> lower=-1.413716694115407 upper=1.413716694115407 effort=1e+9 velocity=1e+9
- joint r_knee: limit lower=-1.8151424220741028 upper=0.10471975511965978 effort=1e+9 velocity=1e+9 -> lower=-1.8325957145940461 upper=0.12217304763960307 effort=1e+9 velocity=1e+9
- joint r_shoulder_yaw: limit lower=-0.8726646259971648 upper=1.3962634015954636 effort=1e+9 velocity=1e+9 -> lower=-0.9075712110370514 upper=1.4311699866353502 effort=1e+9 velocity=1e+9
- joint r_wrist_pitch: limit lower=-0.5585053606381855 upper=0.5585053606381855 effort=1e+9 velocity=1e+9 -> lower=-0.3490658503988659 upper=0.3490658503988659 effort=1e+9 velocity=1e+9
- joint r_wrist_roll: limit lower=-1.0821041362364843 upper=0.9075712110370514 effort=1e+9 velocity=1e+9 -> lower=-0.3490658503988659 upper=0.5235987755982988 effort=1e+9 velocity=1e+9
- joint torso_pitch: limit lower=-0.3141592653589793 upper=0.7853981633974483 effort=1e+9 velocity=1e+9 -> lower=-0.3490658503988659 upper=1.1344640137963142 effort=1e+9 velocity=1e+9
- joint torso_roll: limit lower=-0.4014257279586958 upper=0.4014257279586958 effort=1e+9 velocity=1e+9 -> lower=-0.4363323129985824 upper=0.4363323129985824 effort=1e+9 velocity=1e+9
- joint torso_yaw: limit lower=-0.7504915783575618 upper=0.7504915783575618 effort=1e+9 velocity=1e+9 -> lower=-0.7853981633974483 upper=0.7853981633974483 effort=1e+9 velocity=1e+9

File: urdf/ergoCub/robots/ergoCubSN001/model.urdf (robot description, URDF)
Before this commit: robot ergoCub, 204 links, 203 joints
Joints:
- joint l_elbow: limit lower=-0.05235987755982989 upper=1.3089969389957472 effort=1e+9 velocity=1e+9 -> lower=-0.08726646259971647 upper=2.0943951023931953 effort=1e+9 velocity=1e+9
- joint l_hip_pitch: limit lower=-0.7504915783575618 upper=1.7976891295541595 effort=1e+9 velocity=1e+9 -> lower=-0.767944870877505 upper=1.9198621771937625 effort=1e+9 velocity=1e+9
- joint l_hip_roll: limit lower=-0.2792526803190927 upper=1.9024088846738192 effort=1e+9 velocity=1e+9 -> lower=-0.3490658503988659 upper=1.9373154697137058 effort=1e+9 velocity=1e+9
- joint l_hip_yaw: limit lower=-1.3788101090755203 upper=1.3788101090755203 effort=1e+9 velocity=1e+9 -> lower=-1.413716694115407 upper=1.413716694115407 effort=1e+9 velocity=1e+9
- joint l_knee: limit lower=-1.8151424220741028 upper=0.10471975511965978 effort=1e+9 velocity=1e+9 -> lower=-1.8325957145940461 upper=0.12217304763960307 effort=1e+9 velocity=1e+9
- joint l_shoulder_yaw: limit lower=-0.8726646259971648 upper=1.3962634015954636 effort=1e+9 velocity=1e+9 -> lower=-0.9075712110370514 upper=1.4311699866353502 effort=1e+9 velocity=1e+9
- joint l_wrist_pitch: limit lower=-0.5585053606381855 upper=0.5585053606381855 effort=1e+9 velocity=1e+9 -> lower=-0.3490658503988659 upper=0.3490658503988659 effort=1e+9 velocity=1e+9
- joint l_wrist_roll: limit lower=-1.0821041362364843 upper=0.9075712110370514 effort=1e+9 velocity=1e+9 -> lower=-0.3490658503988659 upper=0.5235987755982988 effort=1e+9 velocity=1e+9
- joint neck_pitch: limit lower=-0.5235987755982988 upper=0.3839724354387525 effort=1e+9 velocity=1e+9 -> lower=-0.7853981633974483 upper=0.3839724354387525 effort=1e+9 velocity=1e+9
- joint r_elbow: limit lower=-0.05235987755982989 upper=1.3089969389957472 effort=1e+9 velocity=1e+9 -> lower=-0.08726646259971647 upper=2.0943951023931953 effort=1e+9 velocity=1e+9
- joint r_hip_pitch: limit lower=-0.7504915783575618 upper=1.7976891295541595 effort=1e+9 velocity=1e+9 -> lower=-0.767944870877505 upper=1.9198621771937625 effort=1e+9 velocity=1e+9
- joint r_hip_roll: limit lower=-0.2792526803190927 upper=1.9024088846738192 effort=1e+9 velocity=1e+9 -> lower=-0.3490658503988659 upper=1.9373154697137058 effort=1e+9 velocity=1e+9
- joint r_hip_yaw: limit lower=-1.3788101090755203 upper=1.3788101090755203 effort=1e+9 velocity=1e+9 -> lower=-1.413716694115407 upper=1.413716694115407 effort=1e+9 velocity=1e+9
- joint r_knee: limit lower=-1.8151424220741028 upper=0.10471975511965978 effort=1e+9 velocity=1e+9 -> lower=-1.8325957145940461 upper=0.12217304763960307 effort=1e+9 velocity=1e+9
- joint r_shoulder_yaw: limit lower=-0.8726646259971648 upper=1.3962634015954636 effort=1e+9 velocity=1e+9 -> lower=-0.9075712110370514 upper=1.4311699866353502 effort=1e+9 velocity=1e+9
- joint r_wrist_pitch: limit lower=-0.5585053606381855 upper=0.5585053606381855 effort=1e+9 velocity=1e+9 -> lower=-0.3490658503988659 upper=0.3490658503988659 effort=1e+9 velocity=1e+9
- joint r_wrist_roll: limit lower=-1.0821041362364843 upper=0.9075712110370514 effort=1e+9 velocity=1e+9 -> lower=-0.3490658503988659 upper=0.5235987755982988 effort=1e+9 velocity=1e+9
- joint torso_pitch: limit lower=-0.3141592653589793 upper=0.7853981633974483 effort=1e+9 velocity=1e+9 -> lower=-0.3490658503988659 upper=1.1344640137963142 effort=1e+9 velocity=1e+9
- joint torso_roll: limit lower=-0.4014257279586958 upper=0.4014257279586958 effort=1e+9 velocity=1e+9 -> lower=-0.4363323129985824 upper=0.4363323129985824 effort=1e+9 velocity=1e+9
- joint torso_yaw: limit lower=-0.7504915783575618 upper=0.7504915783575618 effort=1e+9 velocity=1e+9 -> lower=-0.7853981633974483 upper=0.7853981633974483 effort=1e+9 velocity=1e+9
