Commit message: Automatic update of urdf triggered by GitHub Action
ergocub-software = cd757c5de38fb02ff12db2e797780d62a9312718
cad-libraries    = https://github.com/icub-tech-iit/cad-libraries/commit/eae1efd4a46d6f99a8e87ec6aea8a901ba57c31d
cad-mechanics    = https://github.com/icub-tech-iit/cad-mechanics/commit/a106e100d5e0dc56768ae036dde8d05a730e8294
creo2urdf        = https://github.com/icub-tech-iit/creo2urdf/releases/tag/v0.5.13

File: urdf/ergoCub/robots/ergoCubGazeboV1_1/model.urdf (robot description, URDF)
Before this commit: robot ergoCub, 204 links, 203 joints
Joints:
- joint l_hand_thumb_skin_0_fixed_joint: origin xyz=0 0 0 rpy=0 -0 0 -> xyz=-2.2125551391027898e-11 -0.002433587294553452 -0.026405457778888853 rpy=-1.1609482034540493e-11 -1.2225055986691151 1.5707963268683354
- joint l_hand_thumb_skin_10_fixed_joint: origin xyz=0 0 0 rpy=0 -0 0 -> xyz=-0.003300000023277627 -0.004081610224701271 -0.03276668459736391 rpy=3.1415926535743104 -1.5049109712528579 -1.5707963267955443
- joint l_hand_thumb_skin_11_fixed_joint: origin xyz=0 0 0 rpy=0 -0 0 -> xyz=-0.003300000022465971 -0.0031308168506947176 -0.02828041800469284 rpy=-1.1627790682026587e-11 -1.220094902461357 1.5707963268688572
- joint l_hand_thumb_skin_1_fixed_joint: origin xyz=0 0 0 rpy=0 -0 0 -> xyz=0.003299999977533996 -0.0031308168507229173 -0.028280418005880898 rpy=3.141592653571252 -0.6108652381980162 -1.570796327023918
- joint l_hand_thumb_skin_2_fixed_joint: origin xyz=0 0 0 rpy=0 -0 0 -> xyz=-2.2812751687695254e-11 -0.0037579108898968816 -0.030192049408458887 rpy=-1.0975528579504133e-11 -1.305681332851502 1.5707963268508718
- joint l_hand_thumb_skin_3_fixed_joint: origin xyz=0 0 0 rpy=0 -0 0 -> xyz=0.0032999999767223676 -0.004081610224729415 -0.03276668459855195 rpy=3.141592653571252 -0.6108652381980161 -1.570796327023918
- joint l_hand_thumb_skin_4_fixed_joint: origin xyz=0 0 0 rpy=0 -0 0 -> xyz=0.005929525918969086 -0.0011919899250033839 -0.03300000000106727 rpy=1.570796323948815 -1.507507555817487 -1.5707963239587988
- joint l_hand_thumb_skin_5_fixed_joint: origin xyz=0 0 0 rpy=0 -0 0 -> xyz=-2.364491935580304e-11 -0.0034837613996680783 -0.034821366118633304 rpy=3.141592653576766 -1.0887513297983578 -1.57079632687865
- joint l_hand_thumb_skin_6_fixed_joint: origin xyz=0 0 0 rpy=0 -0 0 -> xyz=0.0032999999760114918 -0.0018284709552043588 -0.03676963440474591 rpy=-4.620360040236946e-16 -0.7657426237199224 -1.5707963267949006
- joint l_hand_thumb_skin_7_fixed_joint: origin xyz=0 0 0 rpy=0 -0 0 -> xyz=-2.4250157437677444e-11 -2.898539006957468e-4 -0.038259640911880916 rpy=-3.1415628662062685 -0.620948017682013 -1.5704313693095489
- joint l_hand_thumb_skin_8_fixed_joint: origin xyz=0 0 0 rpy=0 -0 0 -> xyz=-0.0033000000239885308 -0.0018284709551761869 -0.036769634403557905 rpy=3.071469777395219 -0.7763161157147594 -2.432155397543958
- joint l_hand_thumb_skin_9_fixed_joint: origin xyz=0 0 0 rpy=0 -0 0 -> xyz=-0.005929525965583604 -0.0011919899249527854 -0.032999999998932564 rpy=2.9258803345668243 -1.2928372761145006 -2.5531132071417293
- joint r_hand_thumb_skin_0_fixed_joint: origin xyz=0 0 0 rpy=0 -0 0 -> xyz=-5.551115123125783e-17 -0.002433587294553591 -0.026405457778889127 rpy=2.765053092553465e-15 -1.22250559866914 1.5707963267948857
- joint r_hand_thumb_skin_10_fixed_joint: origin xyz=0 0 0 rpy=0 -0 0 -> xyz=-0.003300000000000053 -0.004081610224715565 -0.032766684597958284 rpy=3.141592653589779 -1.5049109712529725 -1.570796326794926
- joint r_hand_thumb_skin_11_fixed_joint: origin xyz=0 0 0 rpy=0 -0 0 -> xyz=-0.003300000000000053 -0.0031308168507090395 -0.02828041800528719 rpy=2.908401871442372e-15 -1.2200949024613812 1.5707963267948855
- joint r_hand_thumb_skin_1_fixed_joint: origin xyz=0 0 0 rpy=0 -0 0 -> xyz=0.0032999999999999696 -0.0031308168507089285 -0.02828041800528714 rpy=3.1415926535897922 -0.6108652381980179 -1.5707963267949114
- joint r_hand_thumb_skin_2_fixed_joint: origin xyz=0 0 0 rpy=0 -0 0 -> xyz=0 -0.0037579108898970204 -0.03019204940845916 rpy=3.389732024708853e-15 -1.3056813328515338 1.5707963267948863
- joint r_hand_thumb_skin_3_fixed_joint: origin xyz=0 0 0 rpy=0 -0 0 -> xyz=0.0032999999999999974 -0.004081610224715454 -0.032766684597958305 rpy=3.1415926535897922 -0.6108652381980177 -1.5707963267949112
- joint r_hand_thumb_skin_4_fixed_joint: origin xyz=0 0 0 rpy=0 -0 0 -> xyz=0.005929525942276387 -0.0011919899249781263 -0.03300000000000026 rpy=1.5707963267948817 -1.507507552842365 -1.5707963267949265
- joint r_hand_thumb_skin_5_fixed_joint: origin xyz=0 0 0 rpy=0 -0 0 -> xyz=-5.551115123125783e-17 -0.003483761399668245 -0.034821366118633644 rpy=3.1415926535897913 -1.088751329798369 -1.5707963267949128
- joint r_hand_thumb_skin_6_fixed_joint: origin xyz=0 0 0 rpy=0 -0 0 -> xyz=0.0032999999999999974 -0.0018284709551903977 -0.036769634404152235 rpy=-1.3861080081060772e-15 -0.7657426207446857 -1.5707963267949117
- joint r_hand_thumb_skin_7_fixed_joint: origin xyz=0 0 0 rpy=0 -0 0 -> xyz=-2.7755575615628914e-17 -2.898539006959133e-4 -0.038259640911881256 rpy=-3.1415628661866624 -0.6209480176820894 -1.570431369087355
- joint r_hand_thumb_skin_8_fixed_joint: origin xyz=0 0 0 rpy=0 -0 0 -> xyz=-0.0032999999999999974 -0.0018284709551905087 -0.03676963440415227 rpy=3.071469774250236 -0.7763161153414891 -2.432155392931655
- joint r_hand_thumb_skin_9_fixed_joint: origin xyz=0 0 0 rpy=0 -0 0 -> xyz=-0.005929525942276387 -0.0011919899249783206 -0.03300000000000024 rpy=2.9258803249384773 -1.2928372753400146 -2.553113197096302

File: urdf/ergoCub/robots/ergoCubGazeboV1_1_minContacts/model.urdf (robot description, URDF)
Before this commit: robot ergoCub, 204 links, 203 joints
Joints:
- joint l_hand_thumb_skin_0_fixed_joint: origin xyz=0 0 0 rpy=0 -0 0 -> xyz=-2.2125551391027898e-11 -0.002433587294553452 -0.026405457778888853 rpy=-1.1609482034540493e-11 -1.2225055986691151 1.5707963268683354
- joint l_hand_thumb_skin_10_fixed_joint: origin xyz=0 0 0 rpy=0 -0 0 -> xyz=-0.003300000023277627 -0.004081610224701271 -0.03276668459736391 rpy=3.1415926535743104 -1.5049109712528579 -1.5707963267955443
- joint l_hand_thumb_skin_11_fixed_joint: origin xyz=0 0 0 rpy=0 -0 0 -> xyz=-0.003300000022465971 -0.0031308168506947176 -0.02828041800469284 rpy=-1.1627790682026587e-11 -1.220094902461357 1.5707963268688572
- joint l_hand_thumb_skin_1_fixed_joint: origin xyz=0 0 0 rpy=0 -0 0 -> xyz=0.003299999977533996 -0.0031308168507229173 -0.028280418005880898 rpy=3.141592653571252 -0.6108652381980162 -1.570796327023918
- joint l_hand_thumb_skin_2_fixed_joint: origin xyz=0 0 0 rpy=0 -0 0 -> xyz=-2.2812751687695254e-11 -0.0037579108898968816 -0.030192049408458887 rpy=-1.0975528579504133e-11 -1.305681332851502 1.5707963268508718
- joint l_hand_thumb_skin_3_fixed_joint: origin xyz=0 0 0 rpy=0 -0 0 -> xyz=0.0032999999767223676 -0.004081610224729415 -0.03276668459855195 rpy=3.141592653571252 -0.6108652381980161 -1.570796327023918
- joint l_hand_thumb_skin_4_fixed_joint: origin xyz=0 0 0 rpy=0 -0 0 -> xyz=0.005929525918969086 -0.0011919899250033839 -0.03300000000106727 rpy=1.570796323948815 -1.507507555817487 -1.5707963239587988
- joint l_hand_thumb_skin_5_fixed_joint: origin xyz=0 0 0 rpy=0 -0 0 -> xyz=-2.364491935580304e-11 -0.0034837613996680783 -0.034821366118633304 rpy=3.141592653576766 -1.0887513297983578 -1.57079632687865
- joint l_hand_thumb_skin_6_fixed_joint: origin xyz=0 0 0 rpy=0 -0 0 -> xyz=0.0032999999760114918 -0.0018284709552043588 -0.03676963440474591 rpy=-4.620360040236946e-16 -0.7657426237199224 -1.5707963267949006
- joint l_hand_thumb_skin_7_fixed_joint: origin xyz=0 0 0 rpy=0 -0 0 -> xyz=-2.4250157437677444e-11 -2.898539006957468e-4 -0.038259640911880916 rpy=-3.1415628662062685 -0.620948017682013 -1.5704313693095489
- joint l_hand_thumb_skin_8_fixed_joint: origin xyz=0 0 0 rpy=0 -0 0 -> xyz=-0.0033000000239885308 -0.0018284709551761869 -0.036769634403557905 rpy=3.071469777395219 -0.7763161157147594 -2.432155397543958
- joint l_hand_thumb_skin_9_fixed_joint: origin xyz=0 0 0 rpy=0 -0 0 -> xyz=-0.005929525965583604 -0.0011919899249527854 -0.032999999998932564 rpy=2.9258803345668243 -1.2928372761145006 -2.5531132071417293
- joint r_hand_thumb_skin_0_fixed_joint: origin xyz=0 0 0 rpy=0 -0 0 -> xyz=-5.551115123125783e-17 -0.002433587294553591 -0.026405457778889127 rpy=2.765053092553465e-15 -1.22250559866914 1.5707963267948857
- joint r_hand_thumb_skin_10_fixed_joint: origin xyz=0 0 0 rpy=0 -0 0 -> xyz=-0.003300000000000053 -0.004081610224715565 -0.032766684597958284 rpy=3.141592653589779 -1.5049109712529725 -1.570796326794926
- joint r_hand_thumb_skin_11_fixed_joint: origin xyz=0 0 0 rpy=0 -0 0 -> xyz=-0.003300000000000053 -0.0031308168507090395 -0.02828041800528719 rpy=2.908401871442372e-15 -1.2200949024613812 1.5707963267948855
- joint r_hand_thumb_skin_1_fixed_joint: origin xyz=0 0 0 rpy=0 -0 0 -> xyz=0.0032999999999999696 -0.0031308168507089285 -0.02828041800528714 rpy=3.1415926535897922 -0.6108652381980179 -1.5707963267949114
- joint r_hand_thumb_skin_2_fixed_joint: origin xyz=0 0 0 rpy=0 -0 0 -> xyz=0 -0.0037579108898970204 -0.03019204940845916 rpy=3.389732024708853e-15 -1.3056813328515338 1.5707963267948863
- joint r_hand_thumb_skin_3_fixed_joint: origin xyz=0 0 0 rpy=0 -0 0 -> xyz=0.0032999999999999974 -0.004081610224715454 -0.032766684597958305 rpy=3.1415926535897922 -0.6108652381980177 -1.5707963267949112
- joint r_hand_thumb_skin_4_fixed_joint: origin xyz=0 0 0 rpy=0 -0 0 -> xyz=0.005929525942276387 -0.0011919899249781263 -0.03300000000000026 rpy=1.5707963267948817 -1.507507552842365 -1.5707963267949265
- joint r_hand_thumb_skin_5_fixed_joint: origin xyz=0 0 0 rpy=0 -0 0 -> xyz=-5.551115123125783e-17 -0.003483761399668245 -0.034821366118633644 rpy=3.1415926535897913 -1.088751329798369 -1.5707963267949128
- joint r_hand_thumb_skin_6_fixed_joint: origin xyz=0 0 0 rpy=0 -0 0 -> xyz=0.0032999999999999974 -0.0018284709551903977 -0.036769634404152235 rpy=-1.3861080081060772e-15 -0.7657426207446857 -1.5707963267949117
- joint r_hand_thumb_skin_7_fixed_joint: origin xyz=0 0 0 rpy=0 -0 0 -> xyz=-2.7755575615628914e-17 -2.898539006959133e-4 -0.038259640911881256 rpy=-3.1415628661866624 -0.6209480176820894 -1.570431369087355
- joint r_hand_thumb_skin_8_fixed_joint: origin xyz=0 0 0 rpy=0 -0 0 -> xyz=-0.0032999999999999974 -0.0018284709551905087 -0.03676963440415227 rpy=3.071469774250236 -0.7763161153414891 -2.432155392931655
- joint r_hand_thumb_skin_9_fixed_joint: origin xyz=0 0 0 rpy=0 -0 0 -> xyz=-0.005929525942276387 -0.0011919899249783206 -0.03300000000000024 rpy=2.9258803249384773 -1.2928372753400146 -2.553113197096302

File: urdf/ergoCub/robots/ergoCubGazeboV1_3/model.urdf (robot description, URDF)
Before this commit: robot ergoCub, 205 links, 204 joints
Joints:
- joint l_hand_thumb_skin_0_fixed_joint: origin xyz=0 0 0 rpy=0 -0 0 -> xyz=-2.2125551391027898e-11 -0.002433587294553452 -0.026405457778888853 rpy=-1.1609482034540493e-11 -1.2225055986691151 1.5707963268683354
- joint l_hand_thumb_skin_10_fixed_joint: origin xyz=0 0 0 rpy=0 -0 0 -> xyz=-0.003300000023277627 -0.004081610224701271 -0.03276668459736391 rpy=3.1415926535743104 -1.5049109712528579 -1.5707963267955443
- joint l_hand_thumb_skin_11_fixed_joint: origin xyz=0 0 0 rpy=0 -0 0 -> xyz=-0.003300000022465971 -0.0031308168506947176 -0.02828041800469284 rpy=-1.1627790682026587e-11 -1.220094902461357 1.5707963268688572
- joint l_hand_thumb_skin_1_fixed_joint: origin xyz=0 0 0 rpy=0 -0 0 -> xyz=0.003299999977533996 -0.0031308168507229173 -0.028280418005880898 rpy=3.141592653571252 -0.6108652381980162 -1.570796327023918
- joint l_hand_thumb_skin_2_fixed_joint: origin xyz=0 0 0 rpy=0 -0 0 -> xyz=-2.2812751687695254e-11 -0.0037579108898968816 -0.030192049408458887 rpy=-1.0975528579504133e-11 -1.305681332851502 1.5707963268508718
- joint l_hand_thumb_skin_3_fixed_joint: origin xyz=0 0 0 rpy=0 -0 0 -> xyz=0.0032999999767223676 -0.004081610224729415 -0.03276668459855195 rpy=3.141592653571252 -0.6108652381980161 -1.570796327023918
- joint l_hand_thumb_skin_4_fixed_joint: origin xyz=0 0 0 rpy=0 -0 0 -> xyz=0.005929525918969086 -0.0011919899250033839 -0.03300000000106727 rpy=1.570796323948815 -1.507507555817487 -1.5707963239587988
- joint l_hand_thumb_skin_5_fixed_joint: origin xyz=0 0 0 rpy=0 -0 0 -> xyz=-2.364491935580304e-11 -0.0034837613996680783 -0.034821366118633304 rpy=3.141592653576766 -1.0887513297983578 -1.57079632687865
- joint l_hand_thumb_skin_6_fixed_joint: origin xyz=0 0 0 rpy=0 -0 0 -> xyz=0.0032999999760114918 -0.0018284709552043588 -0.03676963440474591 rpy=-4.620360040236946e-16 -0.7657426237199224 -1.5707963267949006
- joint l_hand_thumb_skin_7_fixed_joint: origin xyz=0 0 0 rpy=0 -0 0 -> xyz=-2.4250157437677444e-11 -2.898539006957468e-4 -0.038259640911880916 rpy=-3.1415628662062685 -0.620948017682013 -1.5704313693095489
- joint l_hand_thumb_skin_8_fixed_joint: origin xyz=0 0 0 rpy=0 -0 0 -> xyz=-0.0033000000239885308 -0.0018284709551761869 -0.036769634403557905 rpy=3.071469777395219 -0.7763161157147594 -2.432155397543958
- joint l_hand_thumb_skin_9_fixed_joint: origin xyz=0 0 0 rpy=0 -0 0 -> xyz=-0.005929525965583604 -0.0011919899249527854 -0.032999999998932564 rpy=2.9258803345668243 -1.2928372761145006 -2.5531132071417293
- joint r_hand_thumb_skin_0_fixed_joint: origin xyz=0 0 0 rpy=0 -0 0 -> xyz=-5.551115123125783e-17 -0.002433587294553591 -0.026405457778889127 rpy=2.765053092553465e-15 -1.22250559866914 1.5707963267948857
- joint r_hand_thumb_skin_10_fixed_joint: origin xyz=0 0 0 rpy=0 -0 0 -> xyz=-0.003300000000000053 -0.004081610224715565 -0.032766684597958284 rpy=3.141592653589779 -1.5049109712529725 -1.570796326794926
- joint r_hand_thumb_skin_11_fixed_joint: origin xyz=0 0 0 rpy=0 -0 0 -> xyz=-0.003300000000000053 -0.0031308168507090395 -0.02828041800528719 rpy=2.908401871442372e-15 -1.2200949024613812 1.5707963267948855
- joint r_hand_thumb_skin_1_fixed_joint: origin xyz=0 0 0 rpy=0 -0 0 -> xyz=0.0032999999999999696 -0.0031308168507089285 -0.02828041800528714 rpy=3.1415926535897922 -0.6108652381980179 -1.5707963267949114
- joint r_hand_thumb_skin_2_fixed_joint: origin xyz=0 0 0 rpy=0 -0 0 -> xyz=0 -0.0037579108898970204 -0.03019204940845916 rpy=3.389732024708853e-15 -1.3056813328515338 1.5707963267948863
- joint r_hand_thumb_skin_3_fixed_joint: origin xyz=0 0 0 rpy=0 -0 0 -> xyz=0.0032999999999999974 -0.004081610224715454 -0.032766684597958305 rpy=3.1415926535897922 -0.6108652381980177 -1.5707963267949112
- joint r_hand_thumb_skin_4_fixed_joint: origin xyz=0 0 0 rpy=0 -0 0 -> xyz=0.005929525942276387 -0.0011919899249781263 -0.03300000000000026 rpy=1.5707963267948817 -1.507507552842365 -1.5707963267949265
- joint r_hand_thumb_skin_5_fixed_joint: origin xyz=0 0 0 rpy=0 -0 0 -> xyz=-5.551115123125783e-17 -0.003483761399668245 -0.034821366118633644 rpy=3.1415926535897913 -1.088751329798369 -1.5707963267949128
- joint r_hand_thumb_skin_6_fixed_joint: origin xyz=0 0 0 rpy=0 -0 0 -> xyz=0.0032999999999999974 -0.0018284709551903977 -0.036769634404152235 rpy=-1.3861080081060772e-15 -0.7657426207446857 -1.5707963267949117
- joint r_hand_thumb_skin_7_fixed_joint: origin xyz=0 0 0 rpy=0 -0 0 -> xyz=-2.7755575615628914e-17 -2.898539006959133e-4 -0.038259640911881256 rpy=-3.1415628661866624 -0.6209480176820894 -1.570431369087355
- joint r_hand_thumb_skin_8_fixed_joint: origin xyz=0 0 0 rpy=0 -0 0 -> xyz=-0.0032999999999999974 -0.0018284709551905087 -0.03676963440415227 rpy=3.071469774250236 -0.7763161153414891 -2.432155392931655
- joint r_hand_thumb_skin_9_fixed_joint: origin xyz=0 0 0 rpy=0 -0 0 -> xyz=-0.005929525942276387 -0.0011919899249783206 -0.03300000000000024 rpy=2.9258803249384773 -1.2928372753400146 -2.553113197096302

File: urdf/ergoCub/robots/ergoCubGazeboV1_3_minContacts/model.urdf (robot description, URDF)
Before this commit: robot ergoCub, 205 links, 204 joints
Joints:
- joint l_hand_thumb_skin_0_fixed_joint: origin xyz=0 0 0 rpy=0 -0 0 -> xyz=-2.2125551391027898e-11 -0.002433587294553452 -0.026405457778888853 rpy=-1.1609482034540493e-11 -1.2225055986691151 1.5707963268683354
- joint l_hand_thumb_skin_10_fixed_joint: origin xyz=0 0 0 rpy=0 -0 0 -> xyz=-0.003300000023277627 -0.004081610224701271 -0.03276668459736391 rpy=3.1415926535743104 -1.5049109712528579 -1.5707963267955443
- joint l_hand_thumb_skin_11_fixed_joint: origin xyz=0 0 0 rpy=0 -0 0 -> xyz=-0.003300000022465971 -0.0031308168506947176 -0.02828041800469284 rpy=-1.1627790682026587e-11 -1.220094902461357 1.5707963268688572
- joint l_hand_thumb_skin_1_fixed_joint: origin xyz=0 0 0 rpy=0 -0 0 -> xyz=0.003299999977533996 -0.0031308168507229173 -0.028280418005880898 rpy=3.141592653571252 -0.6108652381980162 -1.570796327023918
- joint l_hand_thumb_skin_2_fixed_joint: origin xyz=0 0 0 rpy=0 -0 0 -> xyz=-2.2812751687695254e-11 -0.0037579108898968816 -0.030192049408458887 rpy=-1.0975528579504133e-11 -1.305681332851502 1.5707963268508718
- joint l_hand_thumb_skin_3_fixed_joint: origin xyz=0 0 0 rpy=0 -0 0 -> xyz=0.0032999999767223676 -0.004081610224729415 -0.03276668459855195 rpy=3.141592653571252 -0.6108652381980161 -1.570796327023918
- joint l_hand_thumb_skin_4_fixed_joint: origin xyz=0 0 0 rpy=0 -0 0 -> xyz=0.005929525918969086 -0.0011919899250033839 -0.03300000000106727 rpy=1.570796323948815 -1.507507555817487 -1.5707963239587988
- joint l_hand_thumb_skin_5_fixed_joint: origin xyz=0 0 0 rpy=0 -0 0 -> xyz=-2.364491935580304e-11 -0.0034837613996680783 -0.034821366118633304 rpy=3.141592653576766 -1.0887513297983578 -1.57079632687865
- joint l_hand_thumb_skin_6_fixed_joint: origin xyz=0 0 0 rpy=0 -0 0 -> xyz=0.0032999999760114918 -0.0018284709552043588 -0.03676963440474591 rpy=-4.620360040236946e-16 -0.7657426237199224 -1.5707963267949006
- joint l_hand_thumb_skin_7_fixed_joint: origin xyz=0 0 0 rpy=0 -0 0 -> xyz=-2.4250157437677444e-11 -2.898539006957468e-4 -0.038259640911880916 rpy=-3.1415628662062685 -0.620948017682013 -1.5704313693095489
- joint l_hand_thumb_skin_8_fixed_joint: origin xyz=0 0 0 rpy=0 -0 0 -> xyz=-0.0033000000239885308 -0.0018284709551761869 -0.036769634403557905 rpy=3.071469777395219 -0.7763161157147594 -2.432155397543958
- joint l_hand_thumb_skin_9_fixed_joint: origin xyz=0 0 0 rpy=0 -0 0 -> xyz=-0.005929525965583604 -0.0011919899249527854 -0.032999999998932564 rpy=2.9258803345668243 -1.2928372761145006 -2.5531132071417293
- joint r_hand_thumb_skin_0_fixed_joint: origin xyz=0 0 0 rpy=0 -0 0 -> xyz=-5.551115123125783e-17 -0.002433587294553591 -0.026405457778889127 rpy=2.765053092553465e-15 -1.22250559866914 1.5707963267948857
- joint r_hand_thumb_skin_10_fixed_joint: origin xyz=0 0 0 rpy=0 -0 0 -> xyz=-0.003300000000000053 -0.004081610224715565 -0.032766684597958284 rpy=3.141592653589779 -1.5049109712529725 -1.570796326794926
- joint r_hand_thumb_skin_11_fixed_joint: origin xyz=0 0 0 rpy=0 -0 0 -> xyz=-0.003300000000000053 -0.0031308168507090395 -0.02828041800528719 rpy=2.908401871442372e-15 -1.2200949024613812 1.5707963267948855
- joint r_hand_thumb_skin_1_fixed_joint: origin xyz=0 0 0 rpy=0 -0 0 -> xyz=0.0032999999999999696 -0.0031308168507089285 -0.02828041800528714 rpy=3.1415926535897922 -0.6108652381980179 -1.5707963267949114
- joint r_hand_thumb_skin_2_fixed_joint: origin xyz=0 0 0 rpy=0 -0 0 -> xyz=0 -0.0037579108898970204 -0.03019204940845916 rpy=3.389732024708853e-15 -1.3056813328515338 1.5707963267948863
- joint r_hand_thumb_skin_3_fixed_joint: origin xyz=0 0 0 rpy=0 -0 0 -> xyz=0.0032999999999999974 -0.004081610224715454 -0.032766684597958305 rpy=3.1415926535897922 -0.6108652381980177 -1.5707963267949112
- joint r_hand_thumb_skin_4_fixed_joint: origin xyz=0 0 0 rpy=0 -0 0 -> xyz=0.005929525942276387 -0.0011919899249781263 -0.03300000000000026 rpy=1.5707963267948817 -1.507507552842365 -1.5707963267949265
- joint r_hand_thumb_skin_5_fixed_joint: origin xyz=0 0 0 rpy=0 -0 0 -> xyz=-5.551115123125783e-17 -0.003483761399668245 -0.034821366118633644 rpy=3.1415926535897913 -1.088751329798369 -1.5707963267949128
- joint r_hand_thumb_skin_6_fixed_joint: origin xyz=0 0 0 rpy=0 -0 0 -> xyz=0.0032999999999999974 -0.0018284709551903977 -0.036769634404152235 rpy=-1.3861080081060772e-15 -0.7657426207446857 -1.5707963267949117
- joint r_hand_thumb_skin_7_fixed_joint: origin xyz=0 0 0 rpy=0 -0 0 -> xyz=-2.7755575615628914e-17 -2.898539006959133e-4 -0.038259640911881256 rpy=-3.1415628661866624 -0.6209480176820894 -1.570431369087355
- joint r_hand_thumb_skin_8_fixed_joint: origin xyz=0 0 0 rpy=0 -0 0 -> xyz=-0.0032999999999999974 -0.0018284709551905087 -0.03676963440415227 rpy=3.071469774250236 -0.7763161153414891 -2.432155392931655
- joint r_hand_thumb_skin_9_fixed_joint: origin xyz=0 0 0 rpy=0 -0 0 -> xyz=-0.005929525942276387 -0.0011919899249783206 -0.03300000000000024 rpy=2.9258803249384773 -1.2928372753400146 -2.553113197096302
