Commit message: Automatic update of urdf triggered by GitHub Action
ergocub-software = 86f3feed868b9aedda679c00bdf0b654aee806bb
cad-libraries    = https://github.com/icub-tech-iit/cad-libraries/commit/3642359f93ea7bcc4d7fc24fc771f9ec5235857c
cad-mechanics    = https://github.com/icub-tech-iit/cad-mechanics/commit/7221fbdf8a6d1332bf47bfb82cc037e8c1ac252e
creo2urdf        = https://github.com/icub-tech-iit/creo2urdf/releases/tag/v0.5.10

File: urdf/ergoCub/robots/ergoCubGazeboV1_3/model.urdf (robot description, URDF)
Before this commit: robot ergoCub, 204 links, 203 joints
Links:
- added link neck_1, mass 0.25627387976979793; collision mesh filename=package://ergoCub/meshes/simmechanics/sim_ecub_1-3_head_nec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 scale=0.001 0.001 0.001; visual mesh filename=package://ergoCub/meshes/simmechanics/sim_ecub_1-3_head_nec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 scale=0.001 0.001 0.001
- link chest: mass 8.7013693071296 -> 8.169083432788879; geometry collision mesh filename=package://ergoCub/meshes/simmechanics/sim_ecub_1-3_chest_wo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 scale=0.001 0.001 0.001; visual mesh filename=package://ergoCub/meshes/simmechanics/sim_ecub_1-3_chest_wo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 scale=0.001 0.001 0.001
- link head: geometry collision mesh filename=package://ergoCub/meshes/simmechanics/sim_ecub_1-1_head.stl scale=0.001 0.001 0.001; visual mesh filename=package://ergoCub/meshes/simmechanics/sim_ecub_1-1_head.stl scale=0.001 0.001 0.001
- link neck_2: mass 0.12100314943032965 -> 0.2950466933335733; geometry collision mesh filename=package://ergoCub/meshes/simmechanics/sim_ecub_1-3_head_nec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 scale=0.001 0.001 0.001; visual mesh filename=package://ergoCub/meshes/simmechanics/sim_ecub_1-3_head_nec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 scale=0.001 0.001 0.001
- link neck_3: mass 0.17811376821431446 -> 0.26196252682452986; geometry collision mesh filename=package://ergoCub/meshes/simmechanics/sim_ecub_1-3_head_nec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 scale=0.001 0.001 0.001; visual mesh filename=package://ergoCub/meshes/simmechanics/sim_ecub_1-3_head_nec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 scale=0.001 0.001 0.001
Joints:
- added joint neck_fixed_joint: type fixed, parent chest, child neck_1, origin xyz=-0.0037500000000000176 7.776068354139607e-18 0.18229999999999996 rpy=2.384521650826854e-16 -8.870011704085565e-17 -1.725433700530891e-15
- joint camera_tilt: axis 2.462374947375715e-16 -1 -1.3590792671843662e-15 -> -4.923107306678176e-15 -1 -8.330651815842126e-16; origin xyz=0.06251000000000005 -3.0000000001050474e-5 0.07639250000000047 rpy=9.111439807357182e-15 2.5958199361708845e-4 1.6567881612466022e-15 -> xyz=0.06250999999999984 -3.0000000000784225e-5 0.07639250000000014 rpy=9.638795761816718e-15 2.5958199361637385e-4 6.82613313682484e-15
- joint l_foot_front_ft_sensor: origin xyz=0.13524999999999998 -5.551115123125783e-17 -0.047899999999999165 rpy=-8.751425667295598e-31 1.9428902930939912e-16 -9.788946385468152e-16 -> xyz=0.13524999999999998 -5.551115123125783e-17 -0.04789999999999894 rpy=-8.997944700177166e-31 1.9428902930939596e-16 -9.788946385468152e-16
- joint l_hip_yaw: axis -8.622588011769357e-16 1.593666547307703e-16 1 -> -8.622588011769357e-16 1.5936665473077025e-16 1; origin xyz=-8.448103328007051e-16 -0.014999999999999944 -0.07269999999999993 rpy=3.011883887564833e-16 1.143142903721238e-14 -2.2204460492502608e-16 -> xyz=-8.396061623727746e-16 -0.014999999999999944 -0.07269999999999993 rpy=3.0118838875648327e-16 1.1431429037212378e-14 -2.775557561562751e-16
- joint l_index_add: axis 1.1895336853461886e-15 0.9999999999999999 -1.9812040713213337e-15 -> 1.1895336853461882e-15 1 -1.9534484957057052e-15; origin xyz=0.022500000000000023 -0.0015000000000006952 -0.0685999999999996 rpy=-8.416895217637947e-16 -0.29670597224465534 5.804755322508926e-17 -> xyz=0.02249999999999998 -0.0015000000000006952 -0.06859999999999966 rpy=-8.126657451512499e-16 -0.29670597224465534 5.804755322508928e-17
- joint l_index_dist: axis -1 -2.359224176539984e-16 4.163337069211178e-17 -> -1 -2.359224176539984e-16 -1.3877780539145996e-17; origin xyz=-1.3877787807814457e-17 -0.001500000000000029 -0.03999999999999987 rpy=-7.482326172536535e-8 1.8041124150158794e-16 -6.106226635438361e-16 -> xyz=-5.551115123125783e-17 -0.0014999999999999458 -0.039999999999999813 rpy=-7.482326172536533e-8 1.734723475976807e-16 -6.106226635438361e-16
- joint l_index_prox: axis -1 8.326672684688522e-17 7.023654435833748e-10 -> -1 1.387778780781435e-16 7.023653811333297e-10; origin xyz=0.00919253334679343 0 -0.030713451309624218 rpy=-3.0531133177191815e-16 -7.023611484080483e-10 -7.771561172376096e-16 -> xyz=0.009192533346793458 0 -0.030713451309624218 rpy=-2.220446049250313e-16 -7.023612108580934e-10 -8.326672684688674e-16
- joint l_leg_ft_sensor: origin xyz=0.03669999999999985 -1.3877787807814457e-17 -0.08970000000000003 rpy=-1.1075796462727634e-15 -2.3847605106274887e-30 2.775557561562846e-16 -> xyz=0.036699999999999844 -1.3877787807814457e-17 -0.08970000000000003 rpy=-1.1075796462727634e-15 -1.9903300580169828e-30 2.775557561562846e-16
- joint l_shoulder_pitch: axis 2.629396873843337e-11 1.0000000000000002 -3.132558101803795e-11 -> -3.139849491518021e-16 1 1.3877787807814457e-16; origin xyz=-0.013518676864309373 0.06704761117227485 0.12351981080785726 rpy=0.2536123239046727 -0.0520316056155768 -0.2752787324155064 -> xyz=-0.013518676842609899 0.06704761117227469 0.12351981080941814 rpy=0.2536123238732621 -0.052031605504493116 -0.2752787324138745
- joint l_shoulder_roll: axis 1 4.891920202255013e-16 3.3029134982598896e-15 -> 1 -2.8796409701211803e-16 4.3853809472694054e-15; origin xyz=0.005000000000000011 0.09329999999999987 -3.0531133177191805e-16 rpy=2.6895152771544417e-14 1.790234627208065e-15 -2.3314683517128287e-15 -> xyz=0.0049999999999999 0.09329999999999991 -1.1102230246251565e-15 rpy=2.042810365310288e-14 2.886579864025407e-15 -1.4988010832439613e-15
- joint neck_pitch: axis -2.4626495883381276e-15 -1 3.2706219863955566e-16 -> -2.2204471080416672e-16 -1 -1.0361039135815426e-16; origin xyz=0.004899999966321172 2.016626664826681e-16 0.2273000000005654 rpy=1.2351224860400058e-15 -1.154319564878164e-10 7.461699457715907e-16 -> xyz=0.00865 1.2535963832308504e-17 0.04500000000000015 rpy=-1.0361039135815426e-16 -9.72407665511517e-16 2.2204471080416672e-16; parent chest -> neck_1
- joint neck_roll: axis 1 -1.0117515096130839e-16 -3.5088530160992675e-15 -> 1 -8.88178419700126e-16 1.5308730180195554e-15; origin xyz=-3.469446951953614e-18 -2.0477512739548602e-18 0.009499999999999786 rpy=3.759485374392081e-16 -7.253140465106665e-31 2.9582283945787943e-31 -> xyz=1.0408340855860843e-17 -1.533495552763227e-17 0.009499999999999953 rpy=-1.9428902930943237e-16 1.530873018019556e-15 8.88178419700126e-16
- joint neck_yaw: axis 1.3864777873731602e-15 5.917688058911091e-16 0.9999999999999998 -> 1.3864778836778403e-15 2.1582026845670445e-16 0.9999999999999999; origin xyz=1.734723475976807e-18 3.161610468866502e-17 0.06915000000000004 rpy=2.158203661135612e-16 -1.3923936280326421e-15 3.7154289088816133e-16 -> xyz=-1.734723475976807e-18 1.005727623029929e-23 0.06914999999999993 rpy=2.1582026845670447e-16 -1.3864778836778403e-15 -7.326653381347455e-15
- joint r_foot_front_ft_sensor: origin xyz=0.13525000000000004 0 -0.04789999999999994 rpy=2.66139136471374e-17 -9.20811369242055e-17 -1.4551888385804406e-15 -> xyz=0.13525000000000004 0 -0.04789999999999972 rpy=2.6613913647124785e-17 -9.20811369242055e-17 -1.4551888385804406e-15
- joint r_foot_rear_ft_sensor: origin xyz=0.016 0 -0.04789999999999983 rpy=2.661391364712478e-17 -9.208113692419957e-17 -1.566211141042955e-15 -> xyz=0.016 0 -0.04789999999999961 rpy=2.6613913647112164e-17 -9.208113692420588e-17 -1.566211141042955e-15
- joint r_hip_yaw: axis -2.3953050207433507e-20 1.4749328491810949e-15 -1 -> -2.3953050245594653e-20 1.4749328491810898e-15 -1; origin xyz=-2.8622937353617317e-16 0.014999999999999777 -0.07269999999999871 rpy=-3.94514163379533e-15 7.430123072146451e-16 1.2193157749540276e-6 -> xyz=-2.8275992658421956e-16 0.014999999999999764 -0.07269999999999871 rpy=-3.9451416337953255e-15 7.430123072146073e-16 1.2193157749540274e-6
- joint r_index_add: axis -5.389323627044831e-16 -0.9999999999999999 1.6046911875538946e-15 -> -4.834212114732253e-16 -1 1.6046911875538944e-15; origin xyz=0.022499999999999992 0.0015000000000002234 -0.06859999999999983 rpy=-1.6833790438334957e-15 0.29670597283904 3.141592653589792 -> xyz=0.02250000000000002 0.0015000000000002234 -0.06859999999999983 rpy=-1.625331490597858e-15 0.29670597283904 3.141592653589792
- joint r_index_dist: axis -0.9999999999999993 -2.0122792321330975e-16 -4.510281037539697e-16 -> -0.9999999999999996 -1.4571677198205192e-16 -5.620504062164854e-16; origin xyz=4.163336342344337e-17 -0.0014999999999998903 -0.040000000000000036 rpy=1.942890293094024e-16 3.469446951953614e-17 1.665334536937736e-16 -> xyz=4.163336342344337e-17 -0.0014999999999998348 -0.040000000000000036 rpy=2.220446049250313e-16 9.020562075079397e-17 5.551115123125785e-17
- joint r_index_prox: axis -0.9999999999999993 3.434752482434078e-15 -1.672273430841644e-15 -> -0.9999999999999996 3.490263633665336e-15 -1.6722734308416438e-15; origin xyz=-0.009192533317427393 5.551115123125783e-17 -0.030713451316238316 rpy=-3.0531133177191805e-16 -2.0816681711721685e-17 0 -> xyz=-0.009192533317427379 0 -0.030713451316238316 rpy=-3.0531133177191805e-16 -2.42861286636753e-16 -1.110223024625157e-16
- joint r_knee: axis 1.2193157766326317e-6 -0.9999999999992566 4.719551160658923e-15 -> 1.2193157766326317e-6 -0.9999999999992567 4.719551160658935e-15; origin xyz=0.01060000963260985 0.007899987075259289 -0.17970000000000058 rpy=6.892643261935339e-14 -6.650159361880639e-14 -1.2193157700904425e-6 -> xyz=0.01060000963260985 0.00789998707525931 -0.17970000000000058 rpy=6.892643261935339e-14 -6.650159361880639e-14 -1.219315770090442e-6
- joint r_shoulder_pitch: axis -2.6293323421300308e-11 1.0000000000000002 3.133054926607315e-11 -> -4.718447854656915e-16 1.0000000000000002 3.524958103184872e-15; origin xyz=-0.013518676864309565 -0.06704761117227466 0.12351981080785729 rpy=-0.2536123239046778 -0.05203160561557753 0.2752787324155041 -> xyz=-0.013518676842610013 -0.06704761117227458 0.12351981080941819 rpy=-0.2536123238732659 -0.052031605504493005 0.27527873241387185
- joint r_shoulder_roll: axis -1.0000000000000007 8.760353553682006e-16 -4.510281037539194e-16 -> -1.0000000000000007 -1.955033357425885e-15 -5.967448757360106e-16; origin xyz=0.007499999999999977 -0.09330000000000004 -3.885780586188048e-16 rpy=-9.325873406851307e-15 9.520162436160717e-15 -4.718447854656912e-15 -> xyz=0.007499999999999448 -0.09330000000000005 -1.3877787807814457e-15 rpy=-2.109423746787796e-15 9.672818102046676e-15 -7.605027718682318e-15
- joint torso_pitch: axis 1.058791184074231e-22 1 4.336808689942018e-19 -> 3.821412071901418e-46 1 0; origin xyz=-7.30886630439206e-17 -4.930380657631324e-32 0.11800000000000001 rpy=3.9719461100401744e-15 2.710505431213761e-20 1.0587911275090697e-22 -> xyz=-7.290101862283748e-17 5.551115123142428e-20 0.11799999999999995 rpy=3.972379790909169e-15 2.710505431213761e-20 -5.6565161406289144e-30
- joint torso_yaw: axis 1.1543031726420953e-10 -1.083564369658416e-15 -1 -> 5.720965878596837e-17 -1.0794921642869322e-22 -1; origin xyz=7.441613918977653e-12 2.6928553289098135e-16 0.06446999999999994 rpy=-5.0024312019752794e-15 1.1542823239978046e-10 -3.182148030458047e-22 -> xyz=1.3429321484223738e-16 2.0428995009916363e-16 0.06446999999999985 rpy=-6.085995463684481e-15 -2.027654770291252e-15 1.0592997798766822e-15

File: urdf/ergoCub/robots/ergoCubGazeboV1_3_minContacts/model.urdf (robot description, URDF)
Before this commit: robot ergoCub, 204 links, 203 joints
Links:
- added link neck_1, mass 0.25627387976979793; collision mesh filename=package://ergoCub/meshes/simmechanics/sim_ecub_1-3_head_nec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 scale=0.001 0.001 0.001; visual mesh filename=package://ergoCub/meshes/simmechanics/sim_ecub_1-3_head_nec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 scale=0.001 0.001 0.001
- link chest: mass 8.7013693071296 -> 8.169083432788879; geometry collision box size=0 0 0; visual mesh filename=package://ergoCub/meshes/simmechanics/sim_ecub_1-3_chest_wo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 scale=0.001 0.001 0.001
- link head: geometry collision box size=0 0 0; visual mesh filename=package://ergoCub/meshes/simmechanics/sim_ecub_1-1_head.stl scale=0.001 0.001 0.001
- link neck_2: mass 0.12100314943032965 -> 0.2950466933335733; geometry collision box size=0 0 0; visual mesh filename=package://ergoCub/meshes/simmechanics/sim_ecub_1-3_head_nec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 scale=0.001 0.001 0.001
- link neck_3: mass 0.17811376821431446 -> 0.26196252682452986; geometry collision box size=0 0 0; visual mesh filename=package://ergoCub/meshes/simmechanics/sim_ecub_1-3_head_nec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 scale=0.001 0.001 0.001
Joints:
- added joint neck_fixed_joint: type fixed, parent chest, child neck_1, origin xyz=-0.0037500000000000176 7.776068354139607e-18 0.18229999999999996 rpy=2.384521650826854e-16 -8.870011704085565e-17 -1.725433700530891e-15
- joint camera_tilt: axis 2.462374947375715e-16 -1 -1.3590792671843662e-15 -> -4.923107306678176e-15 -1 -8.330651815842126e-16; origin xyz=0.06251000000000005 -3.0000000001050474e-5 0.07639250000000047 rpy=9.111439807357182e-15 2.5958199361708845e-4 1.6567881612466022e-15 -> xyz=0.06250999999999984 -3.0000000000784225e-5 0.07639250000000014 rpy=9.638795761816718e-15 2.5958199361637385e-4 6.82613313682484e-15
- joint l_foot_front_ft_sensor: origin xyz=0.13524999999999998 -5.551115123125783e-17 -0.047899999999999165 rpy=-8.751425667295598e-31 1.9428902930939912e-16 -9.788946385468152e-16 -> xyz=0.13524999999999998 -5.551115123125783e-17 -0.04789999999999894 rpy=-8.997944700177166e-31 1.9428902930939596e-16 -9.788946385468152e-16
- joint l_hip_yaw: axis -8.622588011769357e-16 1.593666547307703e-16 1 -> -8.622588011769357e-16 1.5936665473077025e-16 1; origin xyz=-8.448103328007051e-16 -0.014999999999999944 -0.07269999999999993 rpy=3.011883887564833e-16 1.143142903721238e-14 -2.2204460492502608e-16 -> xyz=-8.396061623727746e-16 -0.014999999999999944 -0.07269999999999993 rpy=3.0118838875648327e-16 1.1431429037212378e-14 -2.775557561562751e-16
- joint l_index_add: axis 1.1895336853461886e-15 0.9999999999999999 -1.9812040713213337e-15 -> 1.1895336853461882e-15 1 -1.9534484957057052e-15; origin xyz=0.022500000000000023 -0.0015000000000006952 -0.0685999999999996 rpy=-8.416895217637947e-16 -0.29670597224465534 5.804755322508926e-17 -> xyz=0.02249999999999998 -0.0015000000000006952 -0.06859999999999966 rpy=-8.126657451512499e-16 -0.29670597224465534 5.804755322508928e-17
- joint l_index_dist: axis -1 -2.359224176539984e-16 4.163337069211178e-17 -> -1 -2.359224176539984e-16 -1.3877780539145996e-17; origin xyz=-1.3877787807814457e-17 -0.001500000000000029 -0.03999999999999987 rpy=-7.482326172536535e-8 1.8041124150158794e-16 -6.106226635438361e-16 -> xyz=-5.551115123125783e-17 -0.0014999999999999458 -0.039999999999999813 rpy=-7.482326172536533e-8 1.734723475976807e-16 -6.106226635438361e-16
- joint l_index_prox: axis -1 8.326672684688522e-17 7.023654435833748e-10 -> -1 1.387778780781435e-16 7.023653811333297e-10; origin xyz=0.00919253334679343 0 -0.030713451309624218 rpy=-3.0531133177191815e-16 -7.023611484080483e-10 -7.771561172376096e-16 -> xyz=0.009192533346793458 0 -0.030713451309624218 rpy=-2.220446049250313e-16 -7.023612108580934e-10 -8.326672684688674e-16
- joint l_leg_ft_sensor: origin xyz=0.03669999999999985 -1.3877787807814457e-17 -0.08970000000000003 rpy=-1.1075796462727634e-15 -2.3847605106274887e-30 2.775557561562846e-16 -> xyz=0.036699999999999844 -1.3877787807814457e-17 -0.08970000000000003 rpy=-1.1075796462727634e-15 -1.9903300580169828e-30 2.775557561562846e-16
- joint l_shoulder_pitch: axis 2.629396873843337e-11 1.0000000000000002 -3.132558101803795e-11 -> -3.139849491518021e-16 1 1.3877787807814457e-16; origin xyz=-0.013518676864309373 0.06704761117227485 0.12351981080785726 rpy=0.2536123239046727 -0.0520316056155768 -0.2752787324155064 -> xyz=-0.013518676842609899 0.06704761117227469 0.12351981080941814 rpy=0.2536123238732621 -0.052031605504493116 -0.2752787324138745
- joint l_shoulder_roll: axis 1 4.891920202255013e-16 3.3029134982598896e-15 -> 1 -2.8796409701211803e-16 4.3853809472694054e-15; origin xyz=0.005000000000000011 0.09329999999999987 -3.0531133177191805e-16 rpy=2.6895152771544417e-14 1.790234627208065e-15 -2.3314683517128287e-15 -> xyz=0.0049999999999999 0.09329999999999991 -1.1102230246251565e-15 rpy=2.042810365310288e-14 2.886579864025407e-15 -1.4988010832439613e-15
- joint neck_pitch: axis -2.4626495883381276e-15 -1 3.2706219863955566e-16 -> -2.2204471080416672e-16 -1 -1.0361039135815426e-16; origin xyz=0.004899999966321172 2.016626664826681e-16 0.2273000000005654 rpy=1.2351224860400058e-15 -1.154319564878164e-10 7.461699457715907e-16 -> xyz=0.00865 1.2535963832308504e-17 0.04500000000000015 rpy=-1.0361039135815426e-16 -9.72407665511517e-16 2.2204471080416672e-16; parent chest -> neck_1
- joint neck_roll: axis 1 -1.0117515096130839e-16 -3.5088530160992675e-15 -> 1 -8.88178419700126e-16 1.5308730180195554e-15; origin xyz=-3.469446951953614e-18 -2.0477512739548602e-18 0.009499999999999786 rpy=3.759485374392081e-16 -7.253140465106665e-31 2.9582283945787943e-31 -> xyz=1.0408340855860843e-17 -1.533495552763227e-17 0.009499999999999953 rpy=-1.9428902930943237e-16 1.530873018019556e-15 8.88178419700126e-16
- joint neck_yaw: axis 1.3864777873731602e-15 5.917688058911091e-16 0.9999999999999998 -> 1.3864778836778403e-15 2.1582026845670445e-16 0.9999999999999999; origin xyz=1.734723475976807e-18 3.161610468866502e-17 0.06915000000000004 rpy=2.158203661135612e-16 -1.3923936280326421e-15 3.7154289088816133e-16 -> xyz=-1.734723475976807e-18 1.005727623029929e-23 0.06914999999999993 rpy=2.1582026845670447e-16 -1.3864778836778403e-15 -7.326653381347455e-15
- joint r_foot_front_ft_sensor: origin xyz=0.13525000000000004 0 -0.04789999999999994 rpy=2.66139136471374e-17 -9.20811369242055e-17 -1.4551888385804406e-15 -> xyz=0.13525000000000004 0 -0.04789999999999972 rpy=2.6613913647124785e-17 -9.20811369242055e-17 -1.4551888385804406e-15
- joint r_foot_rear_ft_sensor: origin xyz=0.016 0 -0.04789999999999983 rpy=2.661391364712478e-17 -9.208113692419957e-17 -1.566211141042955e-15 -> xyz=0.016 0 -0.04789999999999961 rpy=2.6613913647112164e-17 -9.208113692420588e-17 -1.566211141042955e-15
- joint r_hip_yaw: axis -2.3953050207433507e-20 1.4749328491810949e-15 -1 -> -2.3953050245594653e-20 1.4749328491810898e-15 -1; origin xyz=-2.8622937353617317e-16 0.014999999999999777 -0.07269999999999871 rpy=-3.94514163379533e-15 7.430123072146451e-16 1.2193157749540276e-6 -> xyz=-2.8275992658421956e-16 0.014999999999999764 -0.07269999999999871 rpy=-3.9451416337953255e-15 7.430123072146073e-16 1.2193157749540274e-6
- joint r_index_add: axis -5.389323627044831e-16 -0.9999999999999999 1.6046911875538946e-15 -> -4.834212114732253e-16 -1 1.6046911875538944e-15; origin xyz=0.022499999999999992 0.0015000000000002234 -0.06859999999999983 rpy=-1.6833790438334957e-15 0.29670597283904 3.141592653589792 -> xyz=0.02250000000000002 0.0015000000000002234 -0.06859999999999983 rpy=-1.625331490597858e-15 0.29670597283904 3.141592653589792
- joint r_index_dist: axis -0.9999999999999993 -2.0122792321330975e-16 -4.510281037539697e-16 -> -0.9999999999999996 -1.4571677198205192e-16 -5.620504062164854e-16; origin xyz=4.163336342344337e-17 -0.0014999999999998903 -0.040000000000000036 rpy=1.942890293094024e-16 3.469446951953614e-17 1.665334536937736e-16 -> xyz=4.163336342344337e-17 -0.0014999999999998348 -0.040000000000000036 rpy=2.220446049250313e-16 9.020562075079397e-17 5.551115123125785e-17
- joint r_index_prox: axis -0.9999999999999993 3.434752482434078e-15 -1.672273430841644e-15 -> -0.9999999999999996 3.490263633665336e-15 -1.6722734308416438e-15; origin xyz=-0.009192533317427393 5.551115123125783e-17 -0.030713451316238316 rpy=-3.0531133177191805e-16 -2.0816681711721685e-17 0 -> xyz=-0.009192533317427379 0 -0.030713451316238316 rpy=-3.0531133177191805e-16 -2.42861286636753e-16 -1.110223024625157e-16
- joint r_knee: axis 1.2193157766326317e-6 -0.9999999999992566 4.719551160658923e-15 -> 1.2193157766326317e-6 -0.9999999999992567 4.719551160658935e-15; origin xyz=0.01060000963260985 0.007899987075259289 -0.17970000000000058 rpy=6.892643261935339e-14 -6.650159361880639e-14 -1.2193157700904425e-6 -> xyz=0.01060000963260985 0.00789998707525931 -0.17970000000000058 rpy=6.892643261935339e-14 -6.650159361880639e-14 -1.219315770090442e-6
- joint r_shoulder_pitch: axis -2.6293323421300308e-11 1.0000000000000002 3.133054926607315e-11 -> -4.718447854656915e-16 1.0000000000000002 3.524958103184872e-15; origin xyz=-0.013518676864309565 -0.06704761117227466 0.12351981080785729 rpy=-0.2536123239046778 -0.05203160561557753 0.2752787324155041 -> xyz=-0.013518676842610013 -0.06704761117227458 0.12351981080941819 rpy=-0.2536123238732659 -0.052031605504493005 0.27527873241387185
- joint r_shoulder_roll: axis -1.0000000000000007 8.760353553682006e-16 -4.510281037539194e-16 -> -1.0000000000000007 -1.955033357425885e-15 -5.967448757360106e-16; origin xyz=0.007499999999999977 -0.09330000000000004 -3.885780586188048e-16 rpy=-9.325873406851307e-15 9.520162436160717e-15 -4.718447854656912e-15 -> xyz=0.007499999999999448 -0.09330000000000005 -1.3877787807814457e-15 rpy=-2.109423746787796e-15 9.672818102046676e-15 -7.605027718682318e-15
- joint torso_pitch: axis 1.058791184074231e-22 1 4.336808689942018e-19 -> 3.821412071901418e-46 1 0; origin xyz=-7.30886630439206e-17 -4.930380657631324e-32 0.11800000000000001 rpy=3.9719461100401744e-15 2.710505431213761e-20 1.0587911275090697e-22 -> xyz=-7.290101862283748e-17 5.551115123142428e-20 0.11799999999999995 rpy=3.972379790909169e-15 2.710505431213761e-20 -5.6565161406289144e-30
- joint torso_yaw: axis 1.1543031726420953e-10 -1.083564369658416e-15 -1 -> 5.720965878596837e-17 -1.0794921642869322e-22 -1; origin xyz=7.441613918977653e-12 2.6928553289098135e-16 0.06446999999999994 rpy=-5.0024312019752794e-15 1.1542823239978046e-10 -3.182148030458047e-22 -> xyz=1.3429321484223738e-16 2.0428995009916363e-16 0.06446999999999985 rpy=-6.085995463684481e-15 -2.027654770291252e-15 1.0592997798766822e-15

File: urdf/ergoCub/robots/ergoCubSN002/model.urdf (robot description, URDF)
Before this commit: robot ergoCub, 205 links, 204 joints
Links:
- link head: geometry collision mesh filename=package://ergoCub/meshes/simmechanics/sim_ecub_1-1_head.obj scale=0.001 0.001 0.001; visual mesh filename=package://ergoCub/meshes/simmechanics/sim_ecub_1-1_head.obj scale=0.001 0.001 0.001
Joints:
- joint neck_roll: axis 1 -8.88178419700126e-16 1.5308730180195554e-15 -> -1 8.88178419700126e-16 -1.5308730180195554e-15
