Commit message: Automatic update of urdf triggered by GitHub Action
ergocub-software = 202163491d8f9084ef81d0cd2b4ba6e1108caf70
cad-libraries    = https://github.com/icub-tech-iit/cad-libraries/commit/624dcc59336f46babe02cd3600a838569e4b5e35
cad-mechanics    = https://github.com/icub-tech-iit/cad-mechanics/commit/0cfde9485643d63afeea1019fd3bfdd717589f37
creo2urdf        = https://github.com/icub-tech-iit/creo2urdf/releases/tag/v0.5.14

File: urdf/ergoCub/robots/ergoCubGazeboV1_3/model.urdf (robot description, URDF)
Before this commit: robot ergoCub, 205 links, 204 joints
Links:
- link neck_2: mass 0.2950466933335733 -> 0.2945770397905417
Joints:
- joint camera_tilt: axis -4.923107306678176e-15 -1 -8.330651815842126e-16 -> 2.4623749474468526e-16 -1 -1.3590792672067983e-15; origin xyz=0.06250999999999984 -3.0000000000784225e-5 0.07639250000000014 rpy=9.638795761816718e-15 2.5958199361637385e-4 6.82613313682484e-15 -> xyz=0.06251000000000001 -3.0000000001050477e-5 0.07639250000000047 rpy=9.111439807334751e-15 2.595819936170884e-4 1.6567881612394884e-15
- joint l_thumb_dist: axis -0.9999999999999997 4.26446167181469e-12 1.800055453177012e-10 -> -0.9999999999999997 4.264582097089572e-12 1.8000554279149736e-10; origin xyz=-2.7755575615628914e-17 -0.003710625424652475 -0.034835057900883704 rpy=-0.06328936289091347 7.216449660063518e-16 3.3514857555871925e-15 -> xyz=0 -0.0037106254246526416 -0.03483505790088366 rpy=-0.06328877097738303 6.661338147750939e-16 3.372302437298914e-15
- joint neck_pitch: axis -2.2204471080416672e-16 -1 -1.0361039135815426e-16 -> 2.1777694761997513e-15 -1 -9.967438430278136e-17; origin xyz=0.00865 1.2535963832308504e-17 0.04500000000000015 rpy=-1.0361039135815426e-16 -9.72407665511517e-16 2.2204471080416672e-16 -> xyz=0.008650000000000012 -3.475400653324001e-18 0.045000000000000095 rpy=-9.967438430278062e-17 -5.5151334385361996e-17 -2.1777694761997513e-15
- joint neck_roll: axis 1 -8.88178419700126e-16 1.5308730180195554e-15 -> 1 9.288242243134705e-16 -1.0059216859858537e-16; origin xyz=1.0408340855860843e-17 -1.533495552763227e-17 0.009499999999999953 rpy=-1.9428902930943237e-16 1.530873018019556e-15 8.88178419700126e-16 -> xyz=-8.673617379884035e-18 7.619916604340795e-16 0.010999999999997845 rpy=2.181085978698084e-16 7.048063206293082e-14 1.1565204487256896e-14
- joint neck_yaw: axis 1.3864778836778403e-15 2.1582026845670445e-16 0.9999999999999999 -> 1.4127649560298857e-15 -3.451106961770346e-17 0.9999999999999999; origin xyz=-1.734723475976807e-18 1.005727623029929e-23 0.06914999999999993 rpy=2.1582026845670447e-16 -1.3864778836778403e-15 -7.326653381347455e-15 -> xyz=-7.979727989493313e-17 1.0161561893579613e-17 0.06914999999999977 rpy=-3.4511069617703464e-17 -1.4127649560298857e-15 7.351849132495494e-16
- joint r_thumb_dist: axis -1.0000000000000018 -2.985473546646551e-14 1.7719107462626453e-15 -> -1.0000000000000018 -2.950779077127015e-14 1.7163995950313907e-15; origin xyz=-2.220446049250313e-16 -0.0037106255282951806 -0.0348350578898439 rpy=-0.0632887739526217 1.7208456881689926e-15 1.3836154444390988e-14 -> xyz=-2.7755575615628914e-17 -0.003710625528295458 -0.03483505788984398 rpy=-0.0632887739526215 1.8318679906315083e-15 1.4169221351778535e-14

File: urdf/ergoCub/robots/ergoCubGazeboV1_3_minContacts/model.urdf (robot description, URDF)
Before this commit: robot ergoCub, 205 links, 204 joints
Links:
- link neck_2: mass 0.2950466933335733 -> 0.2945770397905417
Joints:
- joint camera_tilt: axis -4.923107306678176e-15 -1 -8.330651815842126e-16 -> 2.4623749474468526e-16 -1 -1.3590792672067983e-15; origin xyz=0.06250999999999984 -3.0000000000784225e-5 0.07639250000000014 rpy=9.638795761816718e-15 2.5958199361637385e-4 6.82613313682484e-15 -> xyz=0.06251000000000001 -3.0000000001050477e-5 0.07639250000000047 rpy=9.111439807334751e-15 2.595819936170884e-4 1.6567881612394884e-15
- joint l_thumb_dist: axis -0.9999999999999997 4.26446167181469e-12 1.800055453177012e-10 -> -0.9999999999999997 4.264582097089572e-12 1.8000554279149736e-10; origin xyz=-2.7755575615628914e-17 -0.003710625424652475 -0.034835057900883704 rpy=-0.06328936289091347 7.216449660063518e-16 3.3514857555871925e-15 -> xyz=0 -0.0037106254246526416 -0.03483505790088366 rpy=-0.06328877097738303 6.661338147750939e-16 3.372302437298914e-15
- joint neck_pitch: axis -2.2204471080416672e-16 -1 -1.0361039135815426e-16 -> 2.1777694761997513e-15 -1 -9.967438430278136e-17; origin xyz=0.00865 1.2535963832308504e-17 0.04500000000000015 rpy=-1.0361039135815426e-16 -9.72407665511517e-16 2.2204471080416672e-16 -> xyz=0.008650000000000012 -3.475400653324001e-18 0.045000000000000095 rpy=-9.967438430278062e-17 -5.5151334385361996e-17 -2.1777694761997513e-15
- joint neck_roll: axis 1 -8.88178419700126e-16 1.5308730180195554e-15 -> 1 9.288242243134705e-16 -1.0059216859858537e-16; origin xyz=1.0408340855860843e-17 -1.533495552763227e-17 0.009499999999999953 rpy=-1.9428902930943237e-16 1.530873018019556e-15 8.88178419700126e-16 -> xyz=-8.673617379884035e-18 7.619916604340795e-16 0.010999999999997845 rpy=2.181085978698084e-16 7.048063206293082e-14 1.1565204487256896e-14
- joint neck_yaw: axis 1.3864778836778403e-15 2.1582026845670445e-16 0.9999999999999999 -> 1.4127649560298857e-15 -3.451106961770346e-17 0.9999999999999999; origin xyz=-1.734723475976807e-18 1.005727623029929e-23 0.06914999999999993 rpy=2.1582026845670447e-16 -1.3864778836778403e-15 -7.326653381347455e-15 -> xyz=-7.979727989493313e-17 1.0161561893579613e-17 0.06914999999999977 rpy=-3.4511069617703464e-17 -1.4127649560298857e-15 7.351849132495494e-16
- joint r_thumb_dist: axis -1.0000000000000018 -2.985473546646551e-14 1.7719107462626453e-15 -> -1.0000000000000018 -2.950779077127015e-14 1.7163995950313907e-15; origin xyz=-2.220446049250313e-16 -0.0037106255282951806 -0.0348350578898439 rpy=-0.0632887739526217 1.7208456881689926e-15 1.3836154444390988e-14 -> xyz=-2.7755575615628914e-17 -0.003710625528295458 -0.03483505788984398 rpy=-0.0632887739526215 1.8318679906315083e-15 1.4169221351778535e-14

File: urdf/ergoCub/robots/ergoCubSN002/model.urdf (robot description, URDF)
Before this commit: robot ergoCub, 205 links, 204 joints
Links:
- link neck_2: mass 0.2950466933335733 -> 0.2945770397905417
Joints:
- joint camera_tilt: axis -4.923107306678176e-15 -1 -8.330651815842126e-16 -> 2.4623749474468526e-16 -1 -1.3590792672067983e-15; origin xyz=0.06250999999999984 -3.0000000000784225e-5 0.07639250000000014 rpy=9.638795761816718e-15 2.5958199361637385e-4 6.82613313682484e-15 -> xyz=0.06251000000000001 -3.0000000001050477e-5 0.07639250000000047 rpy=9.111439807334751e-15 2.595819936170884e-4 1.6567881612394884e-15
- joint l_thumb_dist: axis -0.9999999999999997 4.26446167181469e-12 1.800055453177012e-10 -> -0.9999999999999997 4.264582097089572e-12 1.8000554279149736e-10; origin xyz=-2.7755575615628914e-17 -0.003710625424652475 -0.034835057900883704 rpy=-0.06328936289091347 7.216449660063518e-16 3.3514857555871925e-15 -> xyz=0 -0.0037106254246526416 -0.03483505790088366 rpy=-0.06328877097738303 6.661338147750939e-16 3.372302437298914e-15
- joint neck_pitch: axis -2.2204471080416672e-16 -1 -1.0361039135815426e-16 -> 2.1777694761997513e-15 -1 -9.967438430278136e-17; origin xyz=0.00865 1.2535963832308504e-17 0.04500000000000015 rpy=-1.0361039135815426e-16 -9.72407665511517e-16 2.2204471080416672e-16 -> xyz=0.008650000000000012 -3.475400653324001e-18 0.045000000000000095 rpy=-9.967438430278062e-17 -5.5151334385361996e-17 -2.1777694761997513e-15
- joint neck_roll: axis 1 -8.88178419700126e-16 1.5308730180195554e-15 -> 1 9.288242243134705e-16 -1.0059216859858537e-16; origin xyz=1.0408340855860843e-17 -1.533495552763227e-17 0.009499999999999953 rpy=-1.9428902930943237e-16 1.530873018019556e-15 8.88178419700126e-16 -> xyz=-8.673617379884035e-18 7.619916604340795e-16 0.010999999999997845 rpy=2.181085978698084e-16 7.048063206293082e-14 1.1565204487256896e-14
- joint neck_yaw: axis 1.3864778836778403e-15 2.1582026845670445e-16 0.9999999999999999 -> 1.4127649560298857e-15 -3.451106961770346e-17 0.9999999999999999; origin xyz=-1.734723475976807e-18 1.005727623029929e-23 0.06914999999999993 rpy=2.1582026845670447e-16 -1.3864778836778403e-15 -7.326653381347455e-15 -> xyz=-7.979727989493313e-17 1.0161561893579613e-17 0.06914999999999977 rpy=-3.4511069617703464e-17 -1.4127649560298857e-15 7.351849132495494e-16
- joint r_thumb_dist: axis -1.0000000000000018 -2.985473546646551e-14 1.7719107462626453e-15 -> -1.0000000000000018 -2.950779077127015e-14 1.7163995950313907e-15; origin xyz=-2.220446049250313e-16 -0.0037106255282951806 -0.0348350578898439 rpy=-0.0632887739526217 1.7208456881689926e-15 1.3836154444390988e-14 -> xyz=-2.7755575615628914e-17 -0.003710625528295458 -0.03483505788984398 rpy=-0.0632887739526215 1.8318679906315083e-15 1.4169221351778535e-14
