Commit message: Automatic update of urdf triggered by GitHub Action
ergocub-software = c856dfee6420c70904d1c26218bc2fdc0f2c0604
cad-libraries    = https://github.com/icub-tech-iit/cad-libraries/commit/a1f673252a066aa54a35b2979daf70657427860f
cad-mechanics    = https://github.com/icub-tech-iit/cad-mechanics/commit/35ae25a4f1e0c58557472ff0c037a663150ca90e
creo2urdf        = https://github.com/icub-tech-iit/creo2urdf/releases/tag/v0.5.15

File: urdf/ergoCub/robots/ergoCubGazeboV1_3/model.urdf (robot description, URDF)
Before this commit: robot ergoCub, 205 links, 204 joints
Joints:
- joint l_index_add: axis 1.1340225320629768e-15 1.0000000000000002 -1.5371148621453145e-15 -> 1.1340225320629764e-15 1 -1.5371148621453133e-15; origin xyz=0.022499999999999958 -0.0015000000000005842 -0.06859999999999963 rpy=-1.2770461711840297e-15 -0.29670597283903727 0 -> xyz=0.022499999999999937 -0.0015000000000005842 -0.06859999999999958 rpy=-1.2480223945662112e-15 -0.2967059728390372 0
- joint l_index_dist: axis -0.9999999999999997 6.397755632781414e-16 -1.9611158761765728e-16 -> -1 -1.387781272582254e-17 5.551115849900924e-17; origin xyz=0 -0.0014999999999999458 -0.039999999999999925 rpy=0.13212134954326843 1.1102230246251565e-16 5.551115123125785e-17 -> xyz=2.7755575615628914e-17 -0.0015000000000000568 -0.039999999999999925 rpy=-7.48138204997862e-8 4.85722573273506e-17 -2.7755575615628914e-16
- joint l_index_prox: axis -1.0000000000000002 9.71445146047228e-16 3.927413949691585e-15 -> -1 8.604228435847113e-16 3.934352843595493e-15; origin xyz=0.009192533317427629 1.1102230246251565e-16 -0.03071345131623826 rpy=-1.1542702904598913e-10 2.2898349882893854e-16 -1.6653345369377346e-16 -> xyz=0.009192533317427642 1.3877787807814457e-16 -0.030713451316238427 rpy=-1.1542722333501844e-10 2.42861286636753e-16 0
- joint l_middle_dist: axis -1 -3.293254239008947e-16 -3.1398716481110165e-15 -> -1 -3.2532464018194217e-16 -3.071734612871575e-15; origin xyz=-3.8163916471489756e-17 -0.0015000000000000846 -0.03999999999999987 rpy=0.1496571307297435 8.326672684688674e-17 2.220446049250313e-16 -> xyz=-3.122502256758253e-17 -0.0015000000000000568 -0.040000000000000036 rpy=0.017535706372654558 -5.551115123125783e-17 -2.220446049250313e-16
- joint l_middle_prox: axis -1.0000000000000002 2.1649260580331098e-16 3.4413606693588236e-15 -> -1.0000000000000002 2.1649260580330972e-16 3.4413606693588236e-15; origin xyz=0.009599999999999859 -0.0015000000000003344 -0.10299999999999979 rpy=5.479727762273431e-4 2.1649348980190553e-15 -7.771561172376094e-16 -> xyz=0.009599999999999831 -0.0015000000000003344 -0.10299999999999979 rpy=5.479727762271211e-4 2.1718737919229625e-15 -7.771561172376094e-16
- joint l_pinkie_dist: axis -0.9999999998538293 7.645451295717487e-6 -1.5293418371029153e-5 -> -0.9999999998538293 7.645451295729698e-6 -1.5293418371143082e-5; origin xyz=3.469446951953614e-18 -0.0014999999959517396 -0.03500000000409331 rpy=0.09891578175998711 -8.301194511368524e-7 1.4736012528836913e-6 -> xyz=3.469446951953614e-18 -0.0014999999959518229 -0.03500000000409326 rpy=-4.438681163529753e-5 4.85722573273506e-17 -1.3877787807814457e-16
- joint l_pinkie_prox: axis -0.9999999998538296 7.644772463656572e-6 -1.5293757710824196e-5 -> -0.9999999998538296 7.644772463701357e-6 -1.529375771086583e-5; origin xyz=-0.03598232224952739 -0.002388315858956269 -0.09206560929209864 rpy=-1.993466145808309e-5 0.08728175651239324 0.026187612448125907 -> xyz=-0.035982322249527375 -0.0023883158589563247 -0.09206560929209864 rpy=-1.9934661458166675e-5 0.08728175651239324 0.026187612448125907
- joint l_ring_dist: axis -1.0000000000000002 2.026753894137631e-15 -3.7346523596398477e-16 -> -1 2.0175109686126877e-15 -2.981495021006039e-16; origin xyz=-1.474514954580286e-17 -0.0015000000000000013 -0.040000000000000036 rpy=0.13200098128016868 -2.5673907444456745e-16 -1.3877787807814454e-16 -> xyz=4.336808689942018e-18 -0.0015000000000000568 -0.03999999999999998 rpy=-1.20443076919931e-4 -9.020562075079397e-17 -1.6653345369377348e-16
- joint l_ring_prox: axis -1.0000000000000004 1.1828815108406304e-18 3.1780134079895106e-15 -> -1.0000000000000004 4.112937881982706e-17 3.1780134079895106e-15; origin xyz=-0.015417755558120055 -0.0018498137284709282 -0.09788067183884427 rpy=-4.001826366278031e-5 0.0872664625997326 0.02617993877991448 -> xyz=-0.015417755558120076 -0.0018498137284708727 -0.09788067183884427 rpy=-4.001826366291962e-5 0.0872664625997326 0.02617993877991448
- joint l_thumb_dist: axis -0.9999999999999993 4.264416100739981e-12 1.8000581661029442e-10 -> -0.9999999999999994 4.264221274732777e-12 1.800057093249481e-10; origin xyz=1.3877787807814457e-16 -0.0037106254245536374 -0.03483505790088739 rpy=0.03567139761069535 -6.677991493120317e-13 -1.779539710033974e-11 -> xyz=-2.7755575615628914e-17 -0.0037106254246525305 -0.03483505790088372 rpy=-0.06328877097668187 3.885780586188048e-16 3.0045410603918315e-15
- joint l_thumb_prox: axis -0.9999999999999997 1.5642293016426834e-11 1.7937440074944355e-10 -> -0.9999999999999996 1.5642265260851218e-11 1.7937444932170088e-10; origin xyz=-0.038093197450346235 -0.003259193858544507 -0.0036017448037204414 rpy=1.430574412172522 -0.19703059799949255 1.5984202269739936 -> xyz=-0.03809319745034625 -0.003259193858544507 -0.0036017448037204414 rpy=1.4305744121725203 -0.19703059799949255 1.5984202269739936
- joint r_index_dist: axis -0.9999999999999993 -2.567390744445674e-16 -5.689893001203927e-16 -> -0.9999999999999997 -2.567390744445675e-16 -5.707240235963695e-16; origin xyz=-1.3877787807814457e-17 -0.0014999999999998903 -0.03999999999999987 rpy=9.020562075079397e-17 4.5102810375396984e-17 -5.551115123125786e-17 -> xyz=-2.7755575615628914e-17 -0.0014999999999999458 -0.039999999999999813 rpy=9.020562075079397e-17 1.0061396160665481e-16 -1.110223024625157e-16
- joint r_index_prox: axis -0.9999999999999992 3.382063620668255e-15 -1.8100180513169683e-15 -> -0.9999999999999994 3.3820636206682556e-15 -1.8100180513169683e-15; origin xyz=-0.009192533317427865 -5.551115123125783e-17 -0.030713451316238316 rpy=-0.17453292519943325 6.38378239159465e-16 -5.551115123125787e-16 -> xyz=-0.009192533317427837 0 -0.03071345131623837 rpy=-0.17453292519943325 6.453171330633722e-16 -5.551115123125786e-16
- joint r_pinkie_dist: axis -1 1.0701582508147453e-15 -2.649488792179709e-15 -> -1.0000000000000004 1.0424026751991168e-15 -2.6494887921797097e-15; origin xyz=2.7755575615628914e-17 -0.0015141933093791582 -0.034999388832118616 rpy=-0.00129569151982278 -3.469446951953614e-17 -2.7755575615628914e-16 -> xyz=1.0408340855860843e-17 -0.0015141933093791582 -0.03499938883211856 rpy=-0.0012956915198227932 -4.163336342344337e-17 -3.053113317719179e-16
- joint r_pinkie_prox: axis -0.9999999999999998 3.946495907847236e-15 -5.273559366969494e-16 -> -1 4.0054765060304476e-15 -5.412337245047638e-16; origin xyz=-0.03598268094316602 0.0023777595791096007 -0.09206828131946321 rpy=-0.16539532549951783 -0.08726646259972756 3.1154127148098767 -> xyz=-0.03598268094316605 0.0023777595791094897 -0.09206828131946332 rpy=-0.16539532549951783 -0.08726646259972758 3.1154127148098767
- joint r_ring_dist: axis -0.9999999999999999 3.712308238590367e-16 1.144917494144691e-16 -> -1.0000000000000002 3.434752482434079e-16 1.179611963664227e-16; origin xyz=-2.0816681711721685e-17 -0.0014999999999998903 -0.039999999999999813 rpy=-1.526556658859591e-16 -2.393918396847994e-16 -1.9428902930940242e-16 -> xyz=-3.642919299551295e-17 -0.0014999999999998903 -0.03999999999999987 rpy=-1.2490009027033016e-16 -2.463307335887066e-16 -2.2204460492503126e-16

File: urdf/ergoCub/robots/ergoCubGazeboV1_3_minContacts/model.urdf (robot description, URDF)
Before this commit: robot ergoCub, 205 links, 204 joints
Joints:
- joint l_index_add: axis 1.1340225320629768e-15 1.0000000000000002 -1.5371148621453145e-15 -> 1.1340225320629764e-15 1 -1.5371148621453133e-15; origin xyz=0.022499999999999958 -0.0015000000000005842 -0.06859999999999963 rpy=-1.2770461711840297e-15 -0.29670597283903727 0 -> xyz=0.022499999999999937 -0.0015000000000005842 -0.06859999999999958 rpy=-1.2480223945662112e-15 -0.2967059728390372 0
- joint l_index_dist: axis -0.9999999999999997 6.397755632781414e-16 -1.9611158761765728e-16 -> -1 -1.387781272582254e-17 5.551115849900924e-17; origin xyz=0 -0.0014999999999999458 -0.039999999999999925 rpy=0.13212134954326843 1.1102230246251565e-16 5.551115123125785e-17 -> xyz=2.7755575615628914e-17 -0.0015000000000000568 -0.039999999999999925 rpy=-7.48138204997862e-8 4.85722573273506e-17 -2.7755575615628914e-16
- joint l_index_prox: axis -1.0000000000000002 9.71445146047228e-16 3.927413949691585e-15 -> -1 8.604228435847113e-16 3.934352843595493e-15; origin xyz=0.009192533317427629 1.1102230246251565e-16 -0.03071345131623826 rpy=-1.1542702904598913e-10 2.2898349882893854e-16 -1.6653345369377346e-16 -> xyz=0.009192533317427642 1.3877787807814457e-16 -0.030713451316238427 rpy=-1.1542722333501844e-10 2.42861286636753e-16 0
- joint l_middle_dist: axis -1 -3.293254239008947e-16 -3.1398716481110165e-15 -> -1 -3.2532464018194217e-16 -3.071734612871575e-15; origin xyz=-3.8163916471489756e-17 -0.0015000000000000846 -0.03999999999999987 rpy=0.1496571307297435 8.326672684688674e-17 2.220446049250313e-16 -> xyz=-3.122502256758253e-17 -0.0015000000000000568 -0.040000000000000036 rpy=0.017535706372654558 -5.551115123125783e-17 -2.220446049250313e-16
- joint l_middle_prox: axis -1.0000000000000002 2.1649260580331098e-16 3.4413606693588236e-15 -> -1.0000000000000002 2.1649260580330972e-16 3.4413606693588236e-15; origin xyz=0.009599999999999859 -0.0015000000000003344 -0.10299999999999979 rpy=5.479727762273431e-4 2.1649348980190553e-15 -7.771561172376094e-16 -> xyz=0.009599999999999831 -0.0015000000000003344 -0.10299999999999979 rpy=5.479727762271211e-4 2.1718737919229625e-15 -7.771561172376094e-16
- joint l_pinkie_dist: axis -0.9999999998538293 7.645451295717487e-6 -1.5293418371029153e-5 -> -0.9999999998538293 7.645451295729698e-6 -1.5293418371143082e-5; origin xyz=3.469446951953614e-18 -0.0014999999959517396 -0.03500000000409331 rpy=0.09891578175998711 -8.301194511368524e-7 1.4736012528836913e-6 -> xyz=3.469446951953614e-18 -0.0014999999959518229 -0.03500000000409326 rpy=-4.438681163529753e-5 4.85722573273506e-17 -1.3877787807814457e-16
- joint l_pinkie_prox: axis -0.9999999998538296 7.644772463656572e-6 -1.5293757710824196e-5 -> -0.9999999998538296 7.644772463701357e-6 -1.529375771086583e-5; origin xyz=-0.03598232224952739 -0.002388315858956269 -0.09206560929209864 rpy=-1.993466145808309e-5 0.08728175651239324 0.026187612448125907 -> xyz=-0.035982322249527375 -0.0023883158589563247 -0.09206560929209864 rpy=-1.9934661458166675e-5 0.08728175651239324 0.026187612448125907
- joint l_ring_dist: axis -1.0000000000000002 2.026753894137631e-15 -3.7346523596398477e-16 -> -1 2.0175109686126877e-15 -2.981495021006039e-16; origin xyz=-1.474514954580286e-17 -0.0015000000000000013 -0.040000000000000036 rpy=0.13200098128016868 -2.5673907444456745e-16 -1.3877787807814454e-16 -> xyz=4.336808689942018e-18 -0.0015000000000000568 -0.03999999999999998 rpy=-1.20443076919931e-4 -9.020562075079397e-17 -1.6653345369377348e-16
- joint l_ring_prox: axis -1.0000000000000004 1.1828815108406304e-18 3.1780134079895106e-15 -> -1.0000000000000004 4.112937881982706e-17 3.1780134079895106e-15; origin xyz=-0.015417755558120055 -0.0018498137284709282 -0.09788067183884427 rpy=-4.001826366278031e-5 0.0872664625997326 0.02617993877991448 -> xyz=-0.015417755558120076 -0.0018498137284708727 -0.09788067183884427 rpy=-4.001826366291962e-5 0.0872664625997326 0.02617993877991448
- joint l_thumb_dist: axis -0.9999999999999993 4.264416100739981e-12 1.8000581661029442e-10 -> -0.9999999999999994 4.264221274732777e-12 1.800057093249481e-10; origin xyz=1.3877787807814457e-16 -0.0037106254245536374 -0.03483505790088739 rpy=0.03567139761069535 -6.677991493120317e-13 -1.779539710033974e-11 -> xyz=-2.7755575615628914e-17 -0.0037106254246525305 -0.03483505790088372 rpy=-0.06328877097668187 3.885780586188048e-16 3.0045410603918315e-15
- joint l_thumb_prox: axis -0.9999999999999997 1.5642293016426834e-11 1.7937440074944355e-10 -> -0.9999999999999996 1.5642265260851218e-11 1.7937444932170088e-10; origin xyz=-0.038093197450346235 -0.003259193858544507 -0.0036017448037204414 rpy=1.430574412172522 -0.19703059799949255 1.5984202269739936 -> xyz=-0.03809319745034625 -0.003259193858544507 -0.0036017448037204414 rpy=1.4305744121725203 -0.19703059799949255 1.5984202269739936
- joint r_index_dist: axis -0.9999999999999993 -2.567390744445674e-16 -5.689893001203927e-16 -> -0.9999999999999997 -2.567390744445675e-16 -5.707240235963695e-16; origin xyz=-1.3877787807814457e-17 -0.0014999999999998903 -0.03999999999999987 rpy=9.020562075079397e-17 4.5102810375396984e-17 -5.551115123125786e-17 -> xyz=-2.7755575615628914e-17 -0.0014999999999999458 -0.039999999999999813 rpy=9.020562075079397e-17 1.0061396160665481e-16 -1.110223024625157e-16
- joint r_index_prox: axis -0.9999999999999992 3.382063620668255e-15 -1.8100180513169683e-15 -> -0.9999999999999994 3.3820636206682556e-15 -1.8100180513169683e-15; origin xyz=-0.009192533317427865 -5.551115123125783e-17 -0.030713451316238316 rpy=-0.17453292519943325 6.38378239159465e-16 -5.551115123125787e-16 -> xyz=-0.009192533317427837 0 -0.03071345131623837 rpy=-0.17453292519943325 6.453171330633722e-16 -5.551115123125786e-16
- joint r_pinkie_dist: axis -1 1.0701582508147453e-15 -2.649488792179709e-15 -> -1.0000000000000004 1.0424026751991168e-15 -2.6494887921797097e-15; origin xyz=2.7755575615628914e-17 -0.0015141933093791582 -0.034999388832118616 rpy=-0.00129569151982278 -3.469446951953614e-17 -2.7755575615628914e-16 -> xyz=1.0408340855860843e-17 -0.0015141933093791582 -0.03499938883211856 rpy=-0.0012956915198227932 -4.163336342344337e-17 -3.053113317719179e-16
- joint r_pinkie_prox: axis -0.9999999999999998 3.946495907847236e-15 -5.273559366969494e-16 -> -1 4.0054765060304476e-15 -5.412337245047638e-16; origin xyz=-0.03598268094316602 0.0023777595791096007 -0.09206828131946321 rpy=-0.16539532549951783 -0.08726646259972756 3.1154127148098767 -> xyz=-0.03598268094316605 0.0023777595791094897 -0.09206828131946332 rpy=-0.16539532549951783 -0.08726646259972758 3.1154127148098767
- joint r_ring_dist: axis -0.9999999999999999 3.712308238590367e-16 1.144917494144691e-16 -> -1.0000000000000002 3.434752482434079e-16 1.179611963664227e-16; origin xyz=-2.0816681711721685e-17 -0.0014999999999998903 -0.039999999999999813 rpy=-1.526556658859591e-16 -2.393918396847994e-16 -1.9428902930940242e-16 -> xyz=-3.642919299551295e-17 -0.0014999999999998903 -0.03999999999999987 rpy=-1.2490009027033016e-16 -2.463307335887066e-16 -2.2204460492503126e-16

File: urdf/ergoCub/robots/ergoCubSN002/model.urdf (robot description, URDF)
Before this commit: robot ergoCub, 205 links, 204 joints
Joints:
- joint l_index_add: axis 1.1340225320629768e-15 1.0000000000000002 -1.5371148621453145e-15 -> 1.1340225320629764e-15 1 -1.5371148621453133e-15; origin xyz=0.022499999999999958 -0.0015000000000005842 -0.06859999999999963 rpy=-1.2770461711840297e-15 -0.29670597283903727 0 -> xyz=0.022499999999999937 -0.0015000000000005842 -0.06859999999999958 rpy=-1.2480223945662112e-15 -0.2967059728390372 0
- joint l_index_dist: axis -0.9999999999999997 6.397755632781414e-16 -1.9611158761765728e-16 -> -1 -1.387781272582254e-17 5.551115849900924e-17; origin xyz=0 -0.0014999999999999458 -0.039999999999999925 rpy=0.13212134954326843 1.1102230246251565e-16 5.551115123125785e-17 -> xyz=2.7755575615628914e-17 -0.0015000000000000568 -0.039999999999999925 rpy=-7.48138204997862e-8 4.85722573273506e-17 -2.7755575615628914e-16
- joint l_index_prox: axis -1.0000000000000002 9.71445146047228e-16 3.927413949691585e-15 -> -1 8.604228435847113e-16 3.934352843595493e-15; origin xyz=0.009192533317427629 1.1102230246251565e-16 -0.03071345131623826 rpy=-1.1542702904598913e-10 2.2898349882893854e-16 -1.6653345369377346e-16 -> xyz=0.009192533317427642 1.3877787807814457e-16 -0.030713451316238427 rpy=-1.1542722333501844e-10 2.42861286636753e-16 0
- joint l_middle_dist: axis -1 -3.293254239008947e-16 -3.1398716481110165e-15 -> -1 -3.2532464018194217e-16 -3.071734612871575e-15; origin xyz=-3.8163916471489756e-17 -0.0015000000000000846 -0.03999999999999987 rpy=0.1496571307297435 8.326672684688674e-17 2.220446049250313e-16 -> xyz=-3.122502256758253e-17 -0.0015000000000000568 -0.040000000000000036 rpy=0.017535706372654558 -5.551115123125783e-17 -2.220446049250313e-16
- joint l_middle_prox: axis -1.0000000000000002 2.1649260580331098e-16 3.4413606693588236e-15 -> -1.0000000000000002 2.1649260580330972e-16 3.4413606693588236e-15; origin xyz=0.009599999999999859 -0.0015000000000003344 -0.10299999999999979 rpy=5.479727762273431e-4 2.1649348980190553e-15 -7.771561172376094e-16 -> xyz=0.009599999999999831 -0.0015000000000003344 -0.10299999999999979 rpy=5.479727762271211e-4 2.1718737919229625e-15 -7.771561172376094e-16
- joint l_pinkie_dist: axis -0.9999999998538293 7.645451295717487e-6 -1.5293418371029153e-5 -> -0.9999999998538293 7.645451295729698e-6 -1.5293418371143082e-5; origin xyz=3.469446951953614e-18 -0.0014999999959517396 -0.03500000000409331 rpy=0.09891578175998711 -8.301194511368524e-7 1.4736012528836913e-6 -> xyz=3.469446951953614e-18 -0.0014999999959518229 -0.03500000000409326 rpy=-4.438681163529753e-5 4.85722573273506e-17 -1.3877787807814457e-16
- joint l_pinkie_prox: axis -0.9999999998538296 7.644772463656572e-6 -1.5293757710824196e-5 -> -0.9999999998538296 7.644772463701357e-6 -1.529375771086583e-5; origin xyz=-0.03598232224952739 -0.002388315858956269 -0.09206560929209864 rpy=-1.993466145808309e-5 0.08728175651239324 0.026187612448125907 -> xyz=-0.035982322249527375 -0.0023883158589563247 -0.09206560929209864 rpy=-1.9934661458166675e-5 0.08728175651239324 0.026187612448125907
- joint l_ring_dist: axis -1.0000000000000002 2.026753894137631e-15 -3.7346523596398477e-16 -> -1 2.0175109686126877e-15 -2.981495021006039e-16; origin xyz=-1.474514954580286e-17 -0.0015000000000000013 -0.040000000000000036 rpy=0.13200098128016868 -2.5673907444456745e-16 -1.3877787807814454e-16 -> xyz=4.336808689942018e-18 -0.0015000000000000568 -0.03999999999999998 rpy=-1.20443076919931e-4 -9.020562075079397e-17 -1.6653345369377348e-16
- joint l_ring_prox: axis -1.0000000000000004 1.1828815108406304e-18 3.1780134079895106e-15 -> -1.0000000000000004 4.112937881982706e-17 3.1780134079895106e-15; origin xyz=-0.015417755558120055 -0.0018498137284709282 -0.09788067183884427 rpy=-4.001826366278031e-5 0.0872664625997326 0.02617993877991448 -> xyz=-0.015417755558120076 -0.0018498137284708727 -0.09788067183884427 rpy=-4.001826366291962e-5 0.0872664625997326 0.02617993877991448
- joint l_thumb_dist: axis -0.9999999999999993 4.264416100739981e-12 1.8000581661029442e-10 -> -0.9999999999999994 4.264221274732777e-12 1.800057093249481e-10; origin xyz=1.3877787807814457e-16 -0.0037106254245536374 -0.03483505790088739 rpy=0.03567139761069535 -6.677991493120317e-13 -1.779539710033974e-11 -> xyz=-2.7755575615628914e-17 -0.0037106254246525305 -0.03483505790088372 rpy=-0.06328877097668187 3.885780586188048e-16 3.0045410603918315e-15
- joint l_thumb_prox: axis -0.9999999999999997 1.5642293016426834e-11 1.7937440074944355e-10 -> -0.9999999999999996 1.5642265260851218e-11 1.7937444932170088e-10; origin xyz=-0.038093197450346235 -0.003259193858544507 -0.0036017448037204414 rpy=1.430574412172522 -0.19703059799949255 1.5984202269739936 -> xyz=-0.03809319745034625 -0.003259193858544507 -0.0036017448037204414 rpy=1.4305744121725203 -0.19703059799949255 1.5984202269739936
- joint r_index_dist: axis -0.9999999999999993 -2.567390744445674e-16 -5.689893001203927e-16 -> -0.9999999999999997 -2.567390744445675e-16 -5.707240235963695e-16; origin xyz=-1.3877787807814457e-17 -0.0014999999999998903 -0.03999999999999987 rpy=9.020562075079397e-17 4.5102810375396984e-17 -5.551115123125786e-17 -> xyz=-2.7755575615628914e-17 -0.0014999999999999458 -0.039999999999999813 rpy=9.020562075079397e-17 1.0061396160665481e-16 -1.110223024625157e-16
- joint r_index_prox: axis -0.9999999999999992 3.382063620668255e-15 -1.8100180513169683e-15 -> -0.9999999999999994 3.3820636206682556e-15 -1.8100180513169683e-15; origin xyz=-0.009192533317427865 -5.551115123125783e-17 -0.030713451316238316 rpy=-0.17453292519943325 6.38378239159465e-16 -5.551115123125787e-16 -> xyz=-0.009192533317427837 0 -0.03071345131623837 rpy=-0.17453292519943325 6.453171330633722e-16 -5.551115123125786e-16
- joint r_pinkie_dist: axis -1 1.0701582508147453e-15 -2.649488792179709e-15 -> -1.0000000000000004 1.0424026751991168e-15 -2.6494887921797097e-15; origin xyz=2.7755575615628914e-17 -0.0015141933093791582 -0.034999388832118616 rpy=-0.00129569151982278 -3.469446951953614e-17 -2.7755575615628914e-16 -> xyz=1.0408340855860843e-17 -0.0015141933093791582 -0.03499938883211856 rpy=-0.0012956915198227932 -4.163336342344337e-17 -3.053113317719179e-16
- joint r_pinkie_prox: axis -0.9999999999999998 3.946495907847236e-15 -5.273559366969494e-16 -> -1 4.0054765060304476e-15 -5.412337245047638e-16; origin xyz=-0.03598268094316602 0.0023777595791096007 -0.09206828131946321 rpy=-0.16539532549951783 -0.08726646259972756 3.1154127148098767 -> xyz=-0.03598268094316605 0.0023777595791094897 -0.09206828131946332 rpy=-0.16539532549951783 -0.08726646259972758 3.1154127148098767
- joint r_ring_dist: axis -0.9999999999999999 3.712308238590367e-16 1.144917494144691e-16 -> -1.0000000000000002 3.434752482434079e-16 1.179611963664227e-16; origin xyz=-2.0816681711721685e-17 -0.0014999999999998903 -0.039999999999999813 rpy=-1.526556658859591e-16 -2.393918396847994e-16 -1.9428902930940242e-16 -> xyz=-3.642919299551295e-17 -0.0014999999999998903 -0.03999999999999987 rpy=-1.2490009027033016e-16 -2.463307335887066e-16 -2.2204460492503126e-16
