Commit message: Automatic update of urdf triggered by GitHub Action
ergocub-software = e2c368f434eb97858fc890cf714cc5e74cd3f3ee
cad-libraries    = https://github.com/icub-tech-iit/cad-libraries/commit/57405711c8fe86af42b33bbc863a2d676a63e76b
cad-mechanics    = https://github.com/icub-tech-iit/cad-mechanics/commit/05cf61a801a964e9a392b5672bd9e44f04f40bbc
creo2urdf        = https://github.com/icub-tech-iit/creo2urdf/releases/tag/v0.5.16

File: urdf/ergoCub/robots/ergoCubGazeboSN001/model.urdf (robot description, URDF)
Before this commit: robot ergoCub, 204 links, 203 joints
Joints:
- joint l_index_dist: limit lower=0 upper=1.7994344588061537 effort=1e+9 velocity=1e+9 -> lower=0 upper=1.7165313193364231 effort=1e+9 velocity=1e+9
- joint l_index_prox: limit lower=0 upper=1.5707963267948966 effort=1e+9 velocity=1e+9 -> lower=0.10035643198967395 upper=1.710422666954443 effort=1e+9 velocity=1e+9
- joint l_middle_dist: limit lower=0 upper=1.7994344588061537 effort=1e+9 velocity=1e+9 -> lower=0 upper=1.7165313193364231 effort=1e+9 velocity=1e+9
- joint l_middle_prox: limit lower=0 upper=1.5707963267948966 effort=1e+9 velocity=1e+9 -> lower=0.10035643198967395 upper=1.710422666954443 effort=1e+9 velocity=1e+9
- joint l_pinkie_dist: limit lower=0 upper=1.7226399717184033 effort=1e+9 velocity=1e+9 -> lower=0.04852015320544236 upper=1.7763961126798287 effort=1e+9 velocity=1e+9
- joint l_pinkie_prox: limit lower=0 upper=1.5707963267948966 effort=1e+9 velocity=1e+9 -> lower=0.10035643198967395 upper=1.710422666954443 effort=1e+9 velocity=1e+9
- joint l_ring_dist: limit lower=0 upper=1.7994344588061537 effort=1e+9 velocity=1e+9 -> lower=0 upper=1.7165313193364231 effort=1e+9 velocity=1e+9
- joint l_ring_prox: limit lower=0 upper=1.5707963267948966 effort=1e+9 velocity=1e+9 -> lower=0.10035643198967395 upper=1.710422666954443 effort=1e+9 velocity=1e+9
- joint l_thumb_dist: limit lower=0 upper=1.7697638615222502 effort=1e+9 velocity=1e+9 -> lower=0 upper=1.7763961126798287 effort=1e+9 velocity=1e+9
- joint l_thumb_prox: limit lower=0 upper=1.5707963267948966 effort=1e+9 velocity=1e+9 -> lower=0.06335545184739416 upper=1.710422666954443 effort=1e+9 velocity=1e+9
- joint r_index_dist: limit lower=0 upper=1.7994344588061537 effort=1e+9 velocity=1e+9 -> lower=0 upper=1.7165313193364231 effort=1e+9 velocity=1e+9
- joint r_index_prox: limit lower=0 upper=1.5707963267948966 effort=1e+9 velocity=1e+9 -> lower=0.10035643198967395 upper=1.710422666954443 effort=1e+9 velocity=1e+9
- joint r_middle_dist: limit lower=0 upper=1.7994344588061537 effort=1e+9 velocity=1e+9 -> lower=0 upper=1.7165313193364231 effort=1e+9 velocity=1e+9
- joint r_middle_prox: limit lower=0 upper=1.5707963267948966 effort=1e+9 velocity=1e+9 -> lower=0.10035643198967395 upper=1.710422666954443 effort=1e+9 velocity=1e+9
- joint r_pinkie_dist: limit lower=0 upper=1.7226399717184033 effort=1e+9 velocity=1e+9 -> lower=0.04852015320544236 upper=1.7763961126798287 effort=1e+9 velocity=1e+9
- joint r_pinkie_prox: limit lower=0 upper=1.5707963267948966 effort=1e+9 velocity=1e+9 -> lower=0.10035643198967395 upper=1.710422666954443 effort=1e+9 velocity=1e+9
- joint r_ring_dist: limit lower=0 upper=1.7994344588061537 effort=1e+9 velocity=1e+9 -> lower=0 upper=1.7165313193364231 effort=1e+9 velocity=1e+9
- joint r_ring_prox: limit lower=0 upper=1.5707963267948966 effort=1e+9 velocity=1e+9 -> lower=0.10035643198967395 upper=1.710422666954443 effort=1e+9 velocity=1e+9
- joint r_thumb_dist: limit lower=0 upper=1.7697638615222502 effort=1e+9 velocity=1e+9 -> lower=0 upper=1.7763961126798287 effort=1e+9 velocity=1e+9
- joint r_thumb_prox: limit lower=0 upper=1.5707963267948966 effort=1e+9 velocity=1e+9 -> lower=0.06335545184739416 upper=1.710422666954443 effort=1e+9 velocity=1e+9

File: urdf/ergoCub/robots/ergoCubGazeboSN001_minContacts/model.urdf (robot description, URDF)
Before this commit: robot ergoCub, 204 links, 203 joints
Joints:
- joint l_index_dist: limit lower=0 upper=1.7994344588061537 effort=1e+9 velocity=1e+9 -> lower=0 upper=1.7165313193364231 effort=1e+9 velocity=1e+9
- joint l_index_prox: limit lower=0 upper=1.5707963267948966 effort=1e+9 velocity=1e+9 -> lower=0.10035643198967395 upper=1.710422666954443 effort=1e+9 velocity=1e+9
- joint l_middle_dist: limit lower=0 upper=1.7994344588061537 effort=1e+9 velocity=1e+9 -> lower=0 upper=1.7165313193364231 effort=1e+9 velocity=1e+9
- joint l_middle_prox: limit lower=0 upper=1.5707963267948966 effort=1e+9 velocity=1e+9 -> lower=0.10035643198967395 upper=1.710422666954443 effort=1e+9 velocity=1e+9
- joint l_pinkie_dist: limit lower=0 upper=1.7226399717184033 effort=1e+9 velocity=1e+9 -> lower=0.04852015320544236 upper=1.7763961126798287 effort=1e+9 velocity=1e+9
- joint l_pinkie_prox: limit lower=0 upper=1.5707963267948966 effort=1e+9 velocity=1e+9 -> lower=0.10035643198967395 upper=1.710422666954443 effort=1e+9 velocity=1e+9
- joint l_ring_dist: limit lower=0 upper=1.7994344588061537 effort=1e+9 velocity=1e+9 -> lower=0 upper=1.7165313193364231 effort=1e+9 velocity=1e+9
- joint l_ring_prox: limit lower=0 upper=1.5707963267948966 effort=1e+9 velocity=1e+9 -> lower=0.10035643198967395 upper=1.710422666954443 effort=1e+9 velocity=1e+9
- joint l_thumb_dist: limit lower=0 upper=1.7697638615222502 effort=1e+9 velocity=1e+9 -> lower=0 upper=1.7763961126798287 effort=1e+9 velocity=1e+9
- joint l_thumb_prox: limit lower=0 upper=1.5707963267948966 effort=1e+9 velocity=1e+9 -> lower=0.06335545184739416 upper=1.710422666954443 effort=1e+9 velocity=1e+9
- joint r_index_dist: limit lower=0 upper=1.7994344588061537 effort=1e+9 velocity=1e+9 -> lower=0 upper=1.7165313193364231 effort=1e+9 velocity=1e+9
- joint r_index_prox: limit lower=0 upper=1.5707963267948966 effort=1e+9 velocity=1e+9 -> lower=0.10035643198967395 upper=1.710422666954443 effort=1e+9 velocity=1e+9
- joint r_middle_dist: limit lower=0 upper=1.7994344588061537 effort=1e+9 velocity=1e+9 -> lower=0 upper=1.7165313193364231 effort=1e+9 velocity=1e+9
- joint r_middle_prox: limit lower=0 upper=1.5707963267948966 effort=1e+9 velocity=1e+9 -> lower=0.10035643198967395 upper=1.710422666954443 effort=1e+9 velocity=1e+9
- joint r_pinkie_dist: limit lower=0 upper=1.7226399717184033 effort=1e+9 velocity=1e+9 -> lower=0.04852015320544236 upper=1.7763961126798287 effort=1e+9 velocity=1e+9
- joint r_pinkie_prox: limit lower=0 upper=1.5707963267948966 effort=1e+9 velocity=1e+9 -> lower=0.10035643198967395 upper=1.710422666954443 effort=1e+9 velocity=1e+9
- joint r_ring_dist: limit lower=0 upper=1.7994344588061537 effort=1e+9 velocity=1e+9 -> lower=0 upper=1.7165313193364231 effort=1e+9 velocity=1e+9
- joint r_ring_prox: limit lower=0 upper=1.5707963267948966 effort=1e+9 velocity=1e+9 -> lower=0.10035643198967395 upper=1.710422666954443 effort=1e+9 velocity=1e+9
- joint r_thumb_dist: limit lower=0 upper=1.7697638615222502 effort=1e+9 velocity=1e+9 -> lower=0 upper=1.7763961126798287 effort=1e+9 velocity=1e+9
- joint r_thumb_prox: limit lower=0 upper=1.5707963267948966 effort=1e+9 velocity=1e+9 -> lower=0.06335545184739416 upper=1.710422666954443 effort=1e+9 velocity=1e+9

File: urdf/ergoCub/robots/ergoCubSN001/model.urdf (robot description, URDF)
Before this commit: robot ergoCub, 204 links, 203 joints
Joints:
- joint l_index_dist: limit lower=0 upper=1.7994344588061537 effort=1e+9 velocity=1e+9 -> lower=0 upper=1.7165313193364231 effort=1e+9 velocity=1e+9
- joint l_index_prox: limit lower=0 upper=1.5707963267948966 effort=1e+9 velocity=1e+9 -> lower=0.10035643198967395 upper=1.710422666954443 effort=1e+9 velocity=1e+9
- joint l_middle_dist: limit lower=0 upper=1.7994344588061537 effort=1e+9 velocity=1e+9 -> lower=0 upper=1.7165313193364231 effort=1e+9 velocity=1e+9
- joint l_middle_prox: limit lower=0 upper=1.5707963267948966 effort=1e+9 velocity=1e+9 -> lower=0.10035643198967395 upper=1.710422666954443 effort=1e+9 velocity=1e+9
- joint l_pinkie_dist: limit lower=0 upper=1.7226399717184033 effort=1e+9 velocity=1e+9 -> lower=0.04852015320544236 upper=1.7763961126798287 effort=1e+9 velocity=1e+9
- joint l_pinkie_prox: limit lower=0 upper=1.5707963267948966 effort=1e+9 velocity=1e+9 -> lower=0.10035643198967395 upper=1.710422666954443 effort=1e+9 velocity=1e+9
- joint l_ring_dist: limit lower=0 upper=1.7994344588061537 effort=1e+9 velocity=1e+9 -> lower=0 upper=1.7165313193364231 effort=1e+9 velocity=1e+9
- joint l_ring_prox: limit lower=0 upper=1.5707963267948966 effort=1e+9 velocity=1e+9 -> lower=0.10035643198967395 upper=1.710422666954443 effort=1e+9 velocity=1e+9
- joint l_thumb_dist: limit lower=0 upper=1.7697638615222502 effort=1e+9 velocity=1e+9 -> lower=0 upper=1.7763961126798287 effort=1e+9 velocity=1e+9
- joint l_thumb_prox: limit lower=0 upper=1.5707963267948966 effort=1e+9 velocity=1e+9 -> lower=0.06335545184739416 upper=1.710422666954443 effort=1e+9 velocity=1e+9
- joint r_index_dist: limit lower=0 upper=1.7994344588061537 effort=1e+9 velocity=1e+9 -> lower=0 upper=1.7165313193364231 effort=1e+9 velocity=1e+9
- joint r_index_prox: limit lower=0 upper=1.5707963267948966 effort=1e+9 velocity=1e+9 -> lower=0.10035643198967395 upper=1.710422666954443 effort=1e+9 velocity=1e+9
- joint r_middle_dist: limit lower=0 upper=1.7994344588061537 effort=1e+9 velocity=1e+9 -> lower=0 upper=1.7165313193364231 effort=1e+9 velocity=1e+9
- joint r_middle_prox: limit lower=0 upper=1.5707963267948966 effort=1e+9 velocity=1e+9 -> lower=0.10035643198967395 upper=1.710422666954443 effort=1e+9 velocity=1e+9
- joint r_pinkie_dist: limit lower=0 upper=1.7226399717184033 effort=1e+9 velocity=1e+9 -> lower=0.04852015320544236 upper=1.7763961126798287 effort=1e+9 velocity=1e+9
- joint r_pinkie_prox: limit lower=0 upper=1.5707963267948966 effort=1e+9 velocity=1e+9 -> lower=0.10035643198967395 upper=1.710422666954443 effort=1e+9 velocity=1e+9
- joint r_ring_dist: limit lower=0 upper=1.7994344588061537 effort=1e+9 velocity=1e+9 -> lower=0 upper=1.7165313193364231 effort=1e+9 velocity=1e+9
- joint r_ring_prox: limit lower=0 upper=1.5707963267948966 effort=1e+9 velocity=1e+9 -> lower=0.10035643198967395 upper=1.710422666954443 effort=1e+9 velocity=1e+9
- joint r_thumb_dist: limit lower=0 upper=1.7697638615222502 effort=1e+9 velocity=1e+9 -> lower=0 upper=1.7763961126798287 effort=1e+9 velocity=1e+9
- joint r_thumb_prox: limit lower=0 upper=1.5707963267948966 effort=1e+9 velocity=1e+9 -> lower=0.06335545184739416 upper=1.710422666954443 effort=1e+9 velocity=1e+9
